Commit message: fixed issue regarding version

File: vizzy_description/urdf/head/head.ros.gazebo.xacro (robot description, xacro)
@@ -34,5 +34,5 @@
 				<joint>version_joint</joint>
 				<mimicJoint>l_eye_version_joint</mimicJoint>
-				<multiplier>1.0</multiplier>
+				<multiplier>-1.0</multiplier>
 			</plugin>
 		</gazebo>
@@ -41,5 +41,5 @@
 				<joint>version_joint</joint>
 				<mimicJoint>r_eye_version_joint</mimicJoint>
-				<multiplier>1.0</multiplier>
+				<multiplier>-1.0</multiplier>
 			</plugin>
 		</gazebo>

File: vizzy_description/urdf/head/head.ros.urdf.xacro (robot description, xacro)
@@ -246,5 +246,5 @@
       effort="1000.0"
       velocity="5.0" />
-    <mimic joint="version_joint" multiplier="1" offset="0"/>
+    <mimic joint="version_joint" multiplier="-1.0" offset="0"/>
   </joint>
   <link name="r_eye_version_link">
@@ -274,5 +274,5 @@
       effort="1000.0"
       velocity="5.0"/>
-    <mimic joint="version_joint" multiplier="1" offset="0"/>
+    <mimic joint="version_joint" multiplier="-1.0" offset="0"/>
   </joint>
   <link name="vergence_link">
