Commit message: fixed xacro files for yarp

File: vizzy_description/urdf/head/head.yarp.gazebo.xacro (robot description, xacro)
@@ -3,23 +3,59 @@
   <xacro:macro name="head_gazebo">
     <gazebo reference="neck_pan_link">
-      <mu1>0.2</mu1>
-      <mu2>0.2</mu2>
     </gazebo>
     <gazebo reference="neck_tilt_link">
-      <mu1>0.2</mu1>
-      <mu2>0.2</mu2>
     </gazebo>
     <gazebo reference="eyes_tilt_link">
-      <mu1>0.2</mu1>
-      <mu2>0.2</mu2>
     </gazebo>
-    <gazebo reference="r_eye_pan_link">
-      <mu1>0.2</mu1>
-      <mu2>0.2</mu2>
+    <gazebo reference="version_link">
     </gazebo>
-    <gazebo reference="l_eye_pan_link">
-      <mu1>0.2</mu1>
-      <mu2>0.2</mu2>
+    <gazebo reference="r_eye_version_link">
     </gazebo>
+    <gazebo reference="l_eye_version_link">
+    </gazebo>
+    <gazebo reference="vergence_link">
+    </gazebo>
+  <gazebo reference="r_eye_vergence_link">
+    </gazebo>
+    <gazebo reference="l_eye_vergence_link">
+    </gazebo>
+ 		<gazebo reference="neck_pan_joint">
+		</gazebo>
+ 		<gazebo reference="neck_tilt_joint">
+		</gazebo>
+ 		<gazebo reference="eyes_tilt_joint">
+		</gazebo>
+ 		<gazebo reference="version_joint">
+		</gazebo>
+ 		<gazebo reference="vergence_joint">
+		</gazebo>
+		<gazebo>
+			<plugin name="mimic_plugin" filename="libgazebo_mimic_plugin.so">
+				<joint>version_joint</joint>
+				<mimicJoint>l_eye_version_joint</mimicJoint>
+				<multiplier>-1.0</multiplier>
+			</plugin>
+		</gazebo>
+		<gazebo>
+			<plugin name="mimic_plugin" filename="libgazebo_mimic_plugin.so">
+				<joint>version_joint</joint>
+				<mimicJoint>r_eye_version_joint</mimicJoint>
+				<multiplier>-1.0</multiplier>
+			</plugin>
+		</gazebo>
+		<gazebo>
+			<plugin name="mimic_plugin" filename="libgazebo_mimic_plugin.so">
+				<joint>vergence_joint</joint>
+				<mimicJoint>l_eye_vergence_joint</mimicJoint>
+				<multiplier>-0.5</multiplier>
+			</plugin>
+		</gazebo>
+		<gazebo>
+			<plugin name="mimic_plugin" filename="libgazebo_mimic_plugin.so">
+				<joint>vergence_joint</joint>
+				<mimicJoint>r_eye_vergence_joint</mimicJoint>
+				<multiplier>0.5</multiplier>
+			</plugin>
+		</gazebo>
   </xacro:macro>
 </robot>

File: vizzy_description/urdf/head/head.yarp.transmission.xacro (robot description, xacro)
@@ -8,5 +8,5 @@
       <type>transmission_interface/SimpleTransmission</type>
       <joint name="neck_pan_joint">
-        <hardwareInterface>EffortJointInterface</hardwareInterface>
+        <hardwareInterface>VelocityJointInterface</hardwareInterface>
       </joint>
       <actuator name="neck_pan_motor">
@@ -17,5 +17,5 @@
       <type>transmission_interface/SimpleTransmission</type>
       <joint name="neck_tilt_joint">
-        <hardwareInterface>EffortJointInterface</hardwareInterface>
+        <hardwareInterface>VelocityJointInterface</hardwareInterface>
       </joint>
       <actuator name="neck_tilt_motor">
@@ -26,5 +26,5 @@
       <type>transmission_interface/SimpleTransmission</type>
       <joint name="eyes_tilt_joint">
-        <hardwareInterface>EffortJointInterface</hardwareInterface>
+        <hardwareInterface>VelocityJointInterface</hardwareInterface>
       </joint>
       <actuator name="eyes_tilt_motor">
@@ -32,19 +32,55 @@
       </actuator>
     </transmission>
-    <transmission name="r_eye_pan_transmission">
+    <transmission name="version_transmission">
       <type>transmission_interface/SimpleTransmission</type>
-      <joint name="r_eye_pan_joint">
-        <hardwareInterface>EffortJointInterface</hardwareInterface>
+      <joint name="version_joint">
+        <hardwareInterface>VelocityJointInterface</hardwareInterface>
       </joint>
-      <actuator name="r_eye_pan_motor">
+      <actuator name="version_motor">
+        <mechanicalReduction>100</mechanicalReduction>
+      </actuator>
+    </transmission>
+    <transmission name="l_eye_version_transmission">
+      <type>transmission_interface/SimpleTransmission</type>
+      <joint name="l_eye_version_joint">
+        <hardwareInterface>VelocityJointInterface</hardwareInterface>
+      </joint>
+      <actuator name="l_eye_version_motor">
         <mechanicalReduction>1</mechanicalReduction>
       </actuator>
     </transmission>
-    <transmission name="l_eye_pan_transmission">
+    <transmission name="r_eye_version_transmission">
       <type>transmission_interface/SimpleTransmission</type>
-      <joint name="l_eye_pan_joint">
-        <hardwareInterface>EffortJointInterface</hardwareInterface>
+      <joint name="r_eye_version_joint">
+        <hardwareInterface>VelocityJointInterface</hardwareInterface>
       </joint>
-      <actuator name="l_eye_pan_motor">
+      <actuator name="r_eye_version_motor">
+        <mechanicalReduction>1</mechanicalReduction>
+      </actuator>
+    </transmission>
+    <transmission name="vergence_transmission">
+      <type>transmission_interface/SimpleTransmission</type>
+      <joint name="vergence_joint">
+        <hardwareInterface>VelocityJointInterface</hardwareInterface>
+      </joint>
+      <actuator name="vergence_motor">
+        <mechanicalReduction>100</mechanicalReduction>
+      </actuator>
+    </transmission>
+    <transmission name="l_eye_vergence_transmission">
+      <type>transmission_interface/SimpleTransmission</type>
+      <joint name="l_eye_vergence_joint">
+        <hardwareInterface>VelocityJointInterface</hardwareInterface>
+      </joint>
+      <actuator name="l_eye_vergence_motor">
+        <mechanicalReduction>1</mechanicalReduction>
+      </actuator>
+    </transmission>
+    <transmission name="r_eye_vergence_transmission">
+      <type>transmission_interface/SimpleTransmission</type>
+      <joint name="r_eye_vergence_joint">
+        <hardwareInterface>VelocityJointInterface</hardwareInterface>
+      </joint>
+      <actuator name="r_eye_vergence_motor">
         <mechanicalReduction>1</mechanicalReduction>
       </actuator>

File: vizzy_description/urdf/head/head.yarp.urdf.xacro (robot description, xacro)
@@ -8,5 +8,5 @@
  <xacro:include filename="$(find vizzy_description)/urdf/head/head.yarp.gazebo.xacro" />
  <xacro:include filename="$(find vizzy_description)/urdf/head/head.yarp.transmission.xacro" />
-  <xacro:macro name="head" params="name">
+ <xacro:macro name="head" params="name">
    <link name="neck_pan_link">
     <inertial>
@@ -247,4 +247,5 @@
       effort="1000.0"
       velocity="5.0" />
+    <mimic joint="version_joint" multiplier="-1.0" offset="0"/>
   </joint>
   <link name="r_eye_version_link">
@@ -274,4 +275,5 @@
       effort="1000.0"
       velocity="5.0"/>
+    <mimic joint="version_joint" multiplier="-1.0" offset="0"/>
   </joint>
   <link name="vergence_link">
@@ -347,4 +349,5 @@
       effort="1000.0"
       velocity="5.0"/>
+    <mimic joint="vergence_joint" multiplier="0.5" offset="0"/>
   </joint>
   <link name="r_camera_link">
@@ -430,4 +433,5 @@
       effort="1000.0"
       velocity="5.0" />
+    <mimic joint="vergence_joint" multiplier="-0.5" offset="0"/>
   </joint>
   <link name="l_camera_link">
@@ -491,4 +495,5 @@
   </joint>
     <!-- gazebo extensions -->
+    <!-- gazebo extensions -->
     <xacro:head_gazebo/>
     <xacro:head_transmissions />

Commit message: added all links to head.yarp.gazebo changed names to transmission items

File: vizzy_description/urdf/head/head.yarp.gazebo.xacro (robot description, xacro)
@@ -8,54 +8,34 @@
     <gazebo reference="eyes_tilt_link">
     </gazebo>
-    <gazebo reference="version_link">
+    <gazebo reference="eyes_center_link">
     </gazebo>
-    <gazebo reference="r_eye_version_link">
+    <gazebo reference="eyes_center_vision_link">
     </gazebo>
-    <gazebo reference="l_eye_version_link">
+   <gazebo reference="l_eye_link">
     </gazebo>
-    <gazebo reference="vergence_link">
+    <gazebo reference="r_eye_link">
     </gazebo>
-  <gazebo reference="r_eye_vergence_link">
+    <gazebo reference="r_camera_link">
     </gazebo>
-    <gazebo reference="l_eye_vergence_link">
+    <gazebo reference="r_camera_vision_link">
     </gazebo>
- 		<gazebo reference="neck_pan_joint">
-		</gazebo>
- 		<gazebo reference="neck_tilt_joint">
-		</gazebo>
- 		<gazebo reference="eyes_tilt_joint">
-		</gazebo>
- 		<gazebo reference="version_joint">
-		</gazebo>
- 		<gazebo reference="vergence_joint">
-		</gazebo>
-		<gazebo>
-			<plugin name="mimic_plugin" filename="libgazebo_mimic_plugin.so">
-				<joint>version_joint</joint>
-				<mimicJoint>l_eye_version_joint</mimicJoint>
-				<multiplier>-1.0</multiplier>
-			</plugin>
-		</gazebo>
-		<gazebo>
-			<plugin name="mimic_plugin" filename="libgazebo_mimic_plugin.so">
-				<joint>version_joint</joint>
-				<mimicJoint>r_eye_version_joint</mimicJoint>
-				<multiplier>-1.0</multiplier>
-			</plugin>
-		</gazebo>
-		<gazebo>
-			<plugin name="mimic_plugin" filename="libgazebo_mimic_plugin.so">
-				<joint>vergence_joint</joint>
-				<mimicJoint>l_eye_vergence_joint</mimicJoint>
-				<multiplier>-0.5</multiplier>
-			</plugin>
-		</gazebo>
-		<gazebo>
-			<plugin name="mimic_plugin" filename="libgazebo_mimic_plugin.so">
-				<joint>vergence_joint</joint>
-				<mimicJoint>r_eye_vergence_joint</mimicJoint>
-				<multiplier>0.5</multiplier>
-			</plugin>
-		</gazebo>
+    <gazebo reference="l_camera_link">
+    </gazebo>
+    <gazebo reference="l_camera_vision_link">
+    </gazebo>
+    <gazebo reference="ego_frame">
+    </gazebo>
+    <gazebo reference="head_origin_frame">
+    </gazebo>
+    <gazebo reference="neck_pan_joint">
+    </gazebo>
+    <gazebo reference="neck_tilt_joint">
+    </gazebo>
+    <gazebo reference="eyes_tilt_joint">
+    </gazebo>
+    <gazebo reference="l_eye_joint">
+    </gazebo>
+    <gazebo reference="r_eye_joint">
+    </gazebo>
   </xacro:macro>
 </robot>

File: vizzy_description/urdf/head/head.yarp.transmission.xacro (robot description, xacro)
@@ -32,55 +32,19 @@
       </actuator>
     </transmission>
-    <transmission name="version_transmission">
+    <transmission name="l_eye_transmission">
       <type>transmission_interface/SimpleTransmission</type>
-      <joint name="version_joint">
+      <joint name="l_eye_joint">
         <hardwareInterface>VelocityJointInterface</hardwareInterface>
       </joint>
-      <actuator name="version_motor">
-        <mechanicalReduction>100</mechanicalReduction>
-      </actuator>
-    </transmission>
-    <transmission name="l_eye_version_transmission">
-      <type>transmission_interface/SimpleTransmission</type>
-      <joint name="l_eye_version_joint">
-        <hardwareInterface>VelocityJointInterface</hardwareInterface>
-      </joint>
-      <actuator name="l_eye_version_motor">
+      <actuator name="l_eye_motor">
         <mechanicalReduction>1</mechanicalReduction>
       </actuator>
     </transmission>
-    <transmission name="r_eye_version_transmission">
+    <transmission name="r_eye_transmission">
       <type>transmission_interface/SimpleTransmission</type>
-      <joint name="r_eye_version_joint">
+      <joint name="r_eye_joint">
         <hardwareInterface>VelocityJointInterface</hardwareInterface>
       </joint>
-      <actuator name="r_eye_version_motor">
-        <mechanicalReduction>1</mechanicalReduction>
-      </actuator>
-    </transmission>
-    <transmission name="vergence_transmission">
-      <type>transmission_interface/SimpleTransmission</type>
-      <joint name="vergence_joint">
-        <hardwareInterface>VelocityJointInterface</hardwareInterface>
-      </joint>
-      <actuator name="vergence_motor">
-        <mechanicalReduction>100</mechanicalReduction>
-      </actuator>
-    </transmission>
-    <transmission name="l_eye_vergence_transmission">
-      <type>transmission_interface/SimpleTransmission</type>
-      <joint name="l_eye_vergence_joint">
-        <hardwareInterface>VelocityJointInterface</hardwareInterface>
-      </joint>
-      <actuator name="l_eye_vergence_motor">
-        <mechanicalReduction>1</mechanicalReduction>
-      </actuator>
-    </transmission>
-    <transmission name="r_eye_vergence_transmission">
-      <type>transmission_interface/SimpleTransmission</type>
-      <joint name="r_eye_vergence_joint">
-        <hardwareInterface>VelocityJointInterface</hardwareInterface>
-      </joint>
-      <actuator name="r_eye_vergence_motor">
+      <actuator name="r_eye_motor">
         <mechanicalReduction>1</mechanicalReduction>
       </actuator>

File: vizzy_description/urdf/head/head.yarp.urdf.xacro (robot description, xacro)
@@ -173,4 +173,19 @@
   </joint>
   <!-- eyes center virtual link and joint -->
+  <!--<link name="eyes_center_link">
+		<inertial>
+			<origin xyz="0 0 0"
+      rpy="0.0 0.0 0" />
+			<mass value="0.1"/>
+			<inertia
+				ixx="0.001" ixy="0.0" ixz="0.0"
+				iyy="0.001" iyz="0.0" izz="0.001"/>
+		</inertial>
+  </link>
+  <joint name="eyes_center_vision_joint" type="fixed">
+    <origin xyz="0 0 0"       rpy="${-M_PI/2} 0.0 ${-M_PI/2}" />
+    <parent link="eyes_center_link" />
+    <child link="eyes_center_vision_link" />
+  </joint>-->
   <link name="eyes_center_link">
 		<inertial>
@@ -188,21 +203,6 @@
     <child link="eyes_center_vision_link" />
   </joint>
+  <!-- version virtual link and joint -->
   <link name="eyes_center_vision_link">
-		<inertial>
-			<origin xyz="0 0 0"
-      rpy="0.0 0.0 0" />
-			<mass value="0.1"/>
-			<inertia
-				ixx="0.001" ixy="0.0" ixz="0.0"
-				iyy="0.001" iyz="0.0" izz="0.001"/>
-		</inertial>
-  </link>
-  <joint name="eyes_center_joint" type="fixed">
-    <origin xyz="0 0 0"       rpy="${M_PI/2.0} 0.0 0.369599135716446" />
-    <parent link="eyes_tilt_link" />
-    <child link="eyes_center_link" />
-  </joint>
-  <!-- version virtual link and joint -->
-  <link name="eyes_link">
 		<inertial>
 			<origin xyz="0 0 0"
@@ -214,13 +214,13 @@
 		</inertial>
   </link>
-  <joint name="center_joint" type="fixed">
+  <joint name="eyes_center_joint" type="fixed">
     <origin xyz="0 0 0"       rpy="0 0 0" />
-    <parent link="eyes_center_link" />
-    <child link="eyes_link" />
+    <parent link="eyes_tilt_link" />
+    <child link="eyes_center_link" />
     <axis  xyz="0 0 1" />
     <limit lower="-0.698131" upper="0.698131" effort="10.0" velocity="5.0" />
   </joint>
   <link name="l_eye_link">
-<inertial>
+  <inertial>
       <origin
         xyz="0 0 -0.0200000000000069"
@@ -279,5 +279,5 @@
   </joint>
   <link name="r_eye_link">
-<inertial>
+  <inertial>
       <origin
         xyz="0.010 0.0 0.003"
