Commit message: yarp plugins are finally working

File: vizzy_description/urdf/head/head.yarp.urdf.xacro (robot description, xacro)
@@ -8,5 +8,5 @@
  <xacro:include filename="$(find vizzy_description)/urdf/head/head.yarp.gazebo.xacro" />
  <xacro:include filename="$(find vizzy_description)/urdf/head/head.yarp.transmission.xacro" />
- <xacro:macro name="head" params="name">
+ <xacro:macro name="head_yarp" params="name">
    <link name="neck_pan_link">
     <inertial>
@@ -247,5 +247,4 @@
       effort="1000.0"
       velocity="5.0" />
-    <mimic joint="version_joint" multiplier="-1.0" offset="0"/>
   </joint>
   <link name="r_eye_version_link">
@@ -275,5 +274,4 @@
       effort="1000.0"
       velocity="5.0"/>
-    <mimic joint="version_joint" multiplier="-1.0" offset="0"/>
   </joint>
   <link name="vergence_link">
@@ -349,5 +347,4 @@
       effort="1000.0"
       velocity="5.0"/>
-    <mimic joint="vergence_joint" multiplier="0.5" offset="0"/>
   </joint>
   <link name="r_camera_link">
@@ -433,5 +430,4 @@
       effort="1000.0"
       velocity="5.0" />
-    <mimic joint="vergence_joint" multiplier="-0.5" offset="0"/>
   </joint>
   <link name="l_camera_link">
@@ -494,5 +490,4 @@
     <child link="head_origin_frame" />
   </joint>
-    <!-- gazebo extensions -->
     <!-- gazebo extensions -->
     <xacro:head_gazebo/>

Commit message: removing unnecessary ros virtual joints from head

File: vizzy_description/urdf/head/head.yarp.urdf.xacro (robot description, xacro)
@@ -204,5 +204,5 @@
   </joint>
   <!-- version virtual link and joint -->
-  <link name="version_link">
+  <link name="eyes_link">
 		<inertial>
 			<origin xyz="0 0 0"
@@ -214,12 +214,126 @@
 		</inertial>
   </link>
-  <joint name="version_joint" type="revolute">
+  <joint name="center_joint" type="fixed">
     <origin xyz="0 0 0"       rpy="0 0 0" />
     <parent link="eyes_center_link" />
-    <child link="version_link" />
+    <child link="eyes_link" />
     <axis  xyz="0 0 1" />
     <limit lower="-0.698131" upper="0.698131" effort="10.0" velocity="5.0" />
   </joint>
-  <link name="l_eye_version_link">
+  <link name="l_eye_link">
+<inertial>
+      <origin
+        xyz="0 0 -0.0200000000000069"
+        rpy="0 0 1.5708" />
+      <mass
+        value="0.158520637460366" />
+      <inertia
+        ixx="0.000147614970454271"
+        ixy="-1.56210652664748E-09"
+        ixz="8.85544640354075E-10"
+        iyy="0.000177840459249179"
+        iyz="8.21234366300574E-06"
+        izz="0.000144884726537935" />
+    </inertial>
+    <visual>
+      <origin
+        xyz="0.010 0.0 0.003"
+        rpy="0.0 ${M_PI} ${-M_PI/2}" />
+      <geometry>
+        <mesh
+          filename="package://vizzy_description/meshes/M4.dae" />
+      </geometry>
+      <material
+        name="">
+        <color
+          rgba="0 0 0 1" />
+      </material>
+    </visual>
+    <collision>
+ 	<origin
+        xyz="0.010 0.0 0.003"
+        rpy="0.0 ${M_PI} ${-M_PI/2}" />
+      <geometry>
+        <mesh
+          filename="package://vizzy_description/meshes/M4.dae" />
+      </geometry>
+    </collision>
+  </link>
+  <joint
+    name="l_eye_joint"
+    type="revolute">
+    <origin
+      xyz="0.0 0.102 0.0"
+      rpy="0 0 0" />
+    <parent
+      link="eyes_center_link" />
+    <child
+      link="l_eye_link" />
+    <axis
+      xyz="0 0 1" />
+    <limit
+			lower="-1.0"
+			upper="1.0"
+      effort="1000.0"
+      velocity="5.0" />
+  </joint>
+  <link name="r_eye_link">
+<inertial>
+      <origin
+        xyz="0.010 0.0 0.003"
+        rpy="0.0 ${M_PI} ${-M_PI/2}" />
+      <mass
+        value="0.158520637460366" />
+      <inertia
+        ixx="0.000147614970454271"
+        ixy="-1.56210652664748E-09"
+        ixz="8.85544640354075E-10"
+        iyy="0.000177840459249179"
+        iyz="8.21234366300574E-06"
+        izz="0.000144884726537935" />
+    </inertial>
+    <visual>
+      <origin
+        xyz="0.010 0.0 0.003"
+        rpy="0.0 ${M_PI} ${-M_PI/2}" />
+      <geometry>
+        <mesh
+          filename="package://vizzy_description/meshes/M4.dae" />
+      </geometry>
+      <material
+        name="">
+        <color
+          rgba="0 0 0 1" />
+      </material>
+    </visual>
+    <collision>
+      <origin
+        xyz="0.010 0.0 0.003"
+        rpy="0.0 ${M_PI} ${-M_PI/2}" />
+      <geometry>
+        <mesh
+          filename="package://vizzy_description/meshes/M4.dae" />
+      </geometry>
+    </collision>
+  </link>
+  <joint
+    name="r_eye_joint"
+    type="revolute">
+    <origin
+      xyz="0.0 -0.102 0.0"
+      rpy="0 0.0 0" />
+    <parent
+      link="eyes_center_link" />
+    <child
+      link="r_eye_link" />
+    <axis
+      xyz="0 0 1" />
+    <limit
+			lower="-1.0"
+			upper="1.0"
+      effort="1000.0"
+      velocity="5.0"/>
+  </joint>
+  <!--<link name="vergence_link">
  		<inertial>
 			<origin xyz="0 0 0" rpy="0 0 0"/>
@@ -230,58 +344,4 @@
 		</inertial>
   </link>
-  <joint
-    name="l_eye_version_joint"
-    type="revolute">
-    <origin
-      xyz="0.0 0.102 0.0"
-      rpy="0 0 0" />
-    <parent
-      link="eyes_center_link" />
-    <child
-      link="l_eye_version_link" />
-    <axis
-      xyz="0 0 1" />
-    <limit
-			lower="-1.0"
-			upper="1.0"
-      effort="1000.0"
-      velocity="5.0" />
-  </joint>
-  <link name="r_eye_version_link">
- 		<inertial>
-			<origin xyz="0 0 0" rpy="0 0 0"/>
-			<mass value="0.01"/>
-			<inertia
-				ixx="0.001" ixy="0.0" ixz="0.0"
-				iyy="0.001" iyz="0.0" izz="0.001"/>
-		</inertial>
-  </link>
-  <joint
-    name="r_eye_version_joint"
-    type="revolute">
-    <origin
-      xyz="0.0 -0.102 0.0"
-      rpy="0 0.0 0" />
-    <parent
-      link="eyes_center_link" />
-    <child
-      link="r_eye_version_link" />
-    <axis
-      xyz="0 0 1" />
-    <limit
-			lower="-1.0"
-			upper="1.0"
-      effort="1000.0"
-      velocity="5.0"/>
-  </joint>
-  <link name="vergence_link">
- 		<inertial>
-			<origin xyz="0 0 0" rpy="0 0 0"/>
-			<mass value="0.01"/>
-			<inertia
-				ixx="0.001" ixy="0.0" ixz="0.0"
-				iyy="0.001" iyz="0.0" izz="0.001"/>
-		</inertial>
-  </link>
   <joint name="vergence_joint" type="revolute">
     <origin xyz="0.0 0.0 0.0" rpy="0 0.0 0" />
@@ -290,6 +350,6 @@
     <axis  xyz="0 0 1" />
     <limit lower="0.0" upper="0.698131" effort="10.0" velocity="5.0" />
-  </joint>
-  <link name="r_eye_vergence_link">
+  </joint>-->
+  <!--<link name="r_eye_vergence_link">
     <inertial>
       <origin
@@ -337,5 +397,5 @@
       rpy="0.0 0.0 0.0" />
     <parent
-      link="r_eye_version_link" />
+      link="r_eye_link" />
     <child
       link="r_eye_vergence_link" />
@@ -347,5 +407,5 @@
       effort="1000.0"
       velocity="5.0"/>
-  </joint>
+  </joint>-->
   <link name="r_camera_link">
    <visual>
@@ -358,5 +418,5 @@
   <joint name="r_camera_joint" type="fixed">
     <origin xyz="0.0575 0.0 0.0" rpy="0.0 0.0 0.0" />
-    <parent link="r_eye_vergence_link"/>
+    <parent link="r_eye_link"/>
     <child link="r_camera_link" />
   </joint>
@@ -374,5 +434,5 @@
     <child link="r_camera_vision_link" />
   </joint>
-  <link name="l_eye_vergence_link">
+  <!--<link name="l_eye_vergence_link">
    <inertial>
       <origin
@@ -420,5 +480,5 @@
       rpy="0 0 0" />
     <parent
-      link="l_eye_version_link" />
+      link="l_eye_link" />
     <child
       link="l_eye_vergence_link" />
@@ -429,6 +489,5 @@
 			upper="1.0"
       effort="1000.0"
-      velocity="5.0" />
-  </joint>
+      velocity="5.0" />-->
   <link name="l_camera_link">
    <visual>
@@ -441,5 +500,5 @@
   <joint name="l_camera_joint" type="fixed">
     <origin xyz="0.0575 0.0 0.0" rpy="0.0 0.0 0.0" />
-    <parent link="l_eye_vergence_link"/>
+    <parent link="l_eye_link"/>
     <child link="l_camera_link" />
   </joint>

Commit message: added yarpmotorgui config file for vizzy simulation eyes rotation added to the new urdf for yarp

File: vizzy_description/urdf/head/head.yarp.urdf.xacro (robot description, xacro)
@@ -215,5 +215,5 @@
   </link>
   <joint name="eyes_center_joint" type="fixed">
-    <origin xyz="0 0 0"       rpy="0 0 0" />
+    <origin xyz="0 0 0"       rpy="${M_PI/2.0} 0.0 0.369599135716446" />
     <parent link="eyes_tilt_link" />
     <child link="eyes_center_link" />

Commit message: fixed eyes transformations

File: vizzy_description/urdf/head/head.yarp.urdf.xacro (robot description, xacro)
@@ -224,6 +224,6 @@
   <inertial>
       <origin
-        xyz="0 0 -0.0200000000000069"
-        rpy="0 0 1.5708" />
+        xyz="0.0 0.0 0.0"
+        rpy="0 0 ${M_PI/2}" />
       <mass
         value="0.158520637460366" />
@@ -238,6 +238,6 @@
     <visual>
       <origin
-        xyz="0.010 0.0 0.003"
-        rpy="0.0 ${M_PI} ${-M_PI/2}" />
+        xyz="0.0 0.0 0.0"
+        rpy="0.0 0.0 ${M_PI/2}" />
       <geometry>
         <mesh
@@ -252,6 +252,6 @@
     <collision>
  	<origin
-        xyz="0.010 0.0 0.003"
-        rpy="0.0 ${M_PI} ${-M_PI/2}" />
+        xyz="0.0 0 0.0"
+        rpy="0 0 ${M_PI/2}" />
       <geometry>
         <mesh
@@ -265,5 +265,5 @@
     <origin
       xyz="0.0 0.102 0.0"
-      rpy="0 0 0" />
+      rpy="0 ${M_PI} 0" />
     <parent
       link="eyes_center_link" />
@@ -281,6 +281,6 @@
   <inertial>
       <origin
-        xyz="0.010 0.0 0.003"
-        rpy="0.0 ${M_PI} ${-M_PI/2}" />
+        xyz="0.0 0.0 0.0"
+        rpy="0.0 0.0 ${M_PI/2}" />
       <mass
         value="0.158520637460366" />
@@ -295,6 +295,6 @@
     <visual>
       <origin
-        xyz="0.010 0.0 0.003"
-        rpy="0.0 ${M_PI} ${-M_PI/2}" />
+        xyz="0.0 0.0 0.0"
+        rpy="0.0 0.0 ${M_PI/2}" />
       <geometry>
         <mesh
@@ -309,6 +309,6 @@
     <collision>
       <origin
-        xyz="0.010 0.0 0.003"
-        rpy="0.0 ${M_PI} ${-M_PI/2}" />
+        xyz="0.0 0.0 0.0"
+        rpy="0.0 0.0 ${M_PI/2}" />
       <geometry>
         <mesh
@@ -322,5 +322,5 @@
     <origin
       xyz="0.0 -0.102 0.0"
-      rpy="0 0.0 0" />
+      rpy="0 ${M_PI} 0" />
     <parent
       link="eyes_center_link" />
@@ -335,77 +335,4 @@
       velocity="5.0"/>
   </joint>
-  <!--<link name="vergence_link">
- 		<inertial>
-			<origin xyz="0 0 0" rpy="0 0 0"/>
-			<mass value="0.01"/>
-			<inertia
-				ixx="0.001" ixy="0.0" ixz="0.0"
-				iyy="0.001" iyz="0.0" izz="0.001"/>
-		</inertial>
-  </link>
-  <joint name="vergence_joint" type="revolute">
-    <origin xyz="0.0 0.0 0.0" rpy="0 0.0 0" />
-    <parent link="eyes_center_link" />
-    <child link="vergence_link" />
-    <axis  xyz="0 0 1" />
-    <limit lower="0.0" upper="0.698131" effort="10.0" velocity="5.0" />
-  </joint>-->
-  <!--<link name="r_eye_vergence_link">
-    <inertial>
-      <origin
-        xyz="0.010 0.0 0.003"
-        rpy="0.0 ${M_PI} ${-M_PI/2}" />
-      <mass
-        value="0.158520637460366" />
-      <inertia
-        ixx="0.000147614970454271"
-        ixy="-1.56210652664748E-09"
-        ixz="8.85544640354075E-10"
-        iyy="0.000177840459249179"
-        iyz="8.21234366300574E-06"
-        izz="0.000144884726537935" />
-    </inertial>
-    <visual>
-      <origin
-        xyz="0.010 0.0 0.003"
-        rpy="0.0 ${M_PI} ${-M_PI/2}" />
-      <geometry>
-        <mesh
-          filename="package://vizzy_description/meshes/M4.dae" />
-      </geometry>
-      <material
-        name="">
-        <color
-          rgba="0 0 0 1" />
-      </material>
-    </visual>
-    <collision>
-      <origin
-        xyz="0.010 0.0 0.003"
-        rpy="0.0 ${M_PI} ${-M_PI/2}" />
-      <geometry>
-        <mesh
-          filename="package://vizzy_description/meshes/M4.dae" />
-      </geometry>
-    </collision>
-  </link>
-  <joint
-    name="r_eye_vergence_joint"
-    type="revolute">
-    <origin
-      xyz="0.0 0.0 0.0"
-      rpy="0.0 0.0 0.0" />
-    <parent
-      link="r_eye_link" />
-    <child
-      link="r_eye_vergence_link" />
-    <axis
-      xyz="0 0 1" />
-		<limit
-			lower="-1.0"
-			upper="1.0"
-      effort="1000.0"
-      velocity="5.0"/>
-  </joint>-->
   <link name="r_camera_link">
    <visual>
@@ -417,5 +344,5 @@
   </link>
   <joint name="r_camera_joint" type="fixed">
-    <origin xyz="0.0575 0.0 0.0" rpy="0.0 0.0 0.0" />
+    <origin xyz="-0.0275 0.0 0.0" rpy="${M_PI/2} 0.0 ${-M_PI/2}" />
     <parent link="r_eye_link"/>
     <child link="r_camera_link" />
@@ -430,5 +357,5 @@
   </link>
   <joint name="r_camera_vision_joint" type="fixed">
-    <origin xyz="0.0 0.0 0.0" rpy="${-M_PI/2} 0.0 ${-M_PI/2}" />
+    <origin xyz="0.0 0.0 0.0" rpy="0.0 0.0 0.0" />
     <parent link="r_camera_link"/>
     <child link="r_camera_vision_link" />
@@ -499,5 +426,5 @@
   </link>
   <joint name="l_camera_joint" type="fixed">
-    <origin xyz="0.0575 0.0 0.0" rpy="0.0 0.0 0.0" />
+    <origin xyz="-0.0275 0.0 0.0" rpy="${M_PI/2} 0.0 ${-M_PI/2}" />
     <parent link="l_eye_link"/>
     <child link="l_camera_link" />
@@ -512,5 +439,5 @@
   </link>
   <joint name="l_camera_vision_joint" type="fixed">
-    <origin xyz="0.0 0.0 0.0" rpy="${-M_PI/2} 0.0 ${-M_PI/2}" />
+    <origin xyz="0.0 0.0 0.0" rpy="0.0 0.0 0.0" />
     <parent link="l_camera_link"/>
     <child link="l_camera_vision_link" />
