Commit message: Transmission elements commented out Added dynamic coefficients for addressing the velocity control

File: vizzy_description/urdf/head/head.yarp.transmission.xacro (robot description, xacro)
@@ -5,5 +5,5 @@
        xmlns:xacro="http://ros.org/wiki/xacro">
   <xacro:macro name="head_transmissions">
-    <transmission name="neck_pan_transmission">
+    <!-- <transmission name="neck_pan_transmission">
       <type>transmission_interface/SimpleTransmission</type>
       <joint name="neck_pan_joint">
@@ -49,5 +49,5 @@
         <mechanicalReduction>1</mechanicalReduction>
       </actuator>
-    </transmission>
+    </transmission> -->
   </xacro:macro>
 </robot>

File: vizzy_description/urdf/head/head.yarp.urdf.xacro (robot description, xacro)
@@ -61,5 +61,6 @@
       xyz="0 0 1" />
     <!--<limit lower="-0.925024504" upper="0.925024504" effort="10.0" velocity="5.0" />-->
-    <limit lower="-2.025024504" upper="2.025024504" effort="10.0" velocity="5.0" />
+    <limit lower="-2.025024504" upper="2.025024504" effort="100.0" velocity="5.0" />
+    <dynamics damping="5.0" friction="10.0"/>
   </joint>
   <link
@@ -116,4 +117,5 @@
       xyz="0 0 1" />
     <!--<limit lower="-0.314159265" upper="0.645771823" effort="100.0" velocity="5.0" />-->
+    <dynamics damping="0.0" friction="5.0"/>
     <limit lower="-2.014159265" upper="2.45771823" effort="100.0" velocity="5.0" />
   </joint>
@@ -171,4 +173,5 @@
       xyz="0 0 1" />
     <limit lower="-0.663225116" upper="0.663225116" effort="10.0" velocity="5.0" />
+    <dynamics damping="0.0" friction="5.0"/>
   </joint>
   <!-- eyes center virtual link and joint -->
@@ -277,4 +280,5 @@
       effort="1000.0"
       velocity="5.0" />
+    <dynamics damping="0.0" friction="5.0"/>
   </joint>
   <link name="r_eye_link">
@@ -334,4 +338,5 @@
       effort="1000.0"
       velocity="5.0"/>
+    <dynamics damping="0.0" friction="5.0"/>
   </joint>
   <link name="r_camera_link">
