Commit message: fixed camera_links to allow using the gazebo camera plugins (camera optical axis corresponds to x direction)

File: vizzy_description/urdf/head/head.urdf.xacro (robot description, xacro)
@@ -336,5 +336,5 @@
   </link>
   <joint name="r_camera_joint" type="fixed">
-    <origin xyz="-0.0275 0.0 0.0" rpy="${M_PI/2} 0.0 ${-M_PI/2}" />
+    <origin xyz="-0.0275 0.0 0.0" rpy="0.0 ${M_PI} 0.0" />
     <parent link="r_eye_link"/>
     <child link="r_camera_link" />
@@ -349,6 +349,6 @@
   </link>
   <joint name="r_camera_vision_joint" type="fixed">
-    <origin xyz="0.0 0.0 0.0" rpy="0.0 0.0 0.0" />
-    <parent link="r_camera_link"/>
+    <origin xyz="0.0 0.0 0.0" rpy="${M_PI/2} 0.0 ${-M_PI/2}" />
+    <parent link="r_eye_link"/>
     <child link="r_camera_vision_link" />
   </joint>
@@ -362,5 +362,5 @@
   </link>
   <joint name="l_camera_joint" type="fixed">
-    <origin xyz="-0.0275 0.0 0.0" rpy="${M_PI/2} 0.0 ${-M_PI/2}" />
+    <origin xyz="-0.0275 0.0 0.0" rpy="0 ${M_PI} 0" />
     <parent link="l_eye_link"/>
     <child link="l_camera_link" />
@@ -375,6 +375,6 @@
   </link>
   <joint name="l_camera_vision_joint" type="fixed">
-    <origin xyz="0.0 0.0 0.0" rpy="0.0 0.0 0.0" />
-    <parent link="l_camera_link"/>
+    <origin xyz="0.0 0.0 0.0" rpy="${M_PI/2} 0.0 ${-M_PI/2}" />
+    <parent link="l_eye_link"/>
     <child link="l_camera_vision_link" />
   </joint>

Commit message: add head meshes

File: vizzy_description/urdf/head/head.urdf.xacro (robot description, xacro)
@@ -70,4 +70,72 @@
       <limit lower="-2.014159265" upper="2.45771823" effort="100.0" velocity="5.0"/>
     </joint>
+    <!-- Head Shells -->
+    <!-- TODO: Update inertia and collision -->
+    <link name="head_shell_link">
+      <visual>
+        <origin
+          xyz="0 0.41 0"
+          rpy="${M_PI/2} ${M_PI/2} 0"/>
+        <geometry>
+          <mesh
+            filename="package://vizzy_description/meshes/head/head.dae"/>
+        </geometry>
+        <material name="light_gray_1"/>
+      </visual>
+      <inertial>
+        <origin rpy="0 0 0" xyz="0.0 0.0 0.0"/>
+        <mass value="0.001"/>
+        <inertia ixx="0.01" ixy="0" ixz="0" iyy="0.01" iyz="0" izz="0.01"/>
+      </inertial>
+      <collision>
+        <origin rpy="0 0 0" xyz="0.0 0.0 0.0"/>
+        <geometry>
+          <cylinder length="0.001" radius="0.005"/>
+        </geometry>
+      </collision>
+    </link>
+    <joint name="head_shell_joint"
+      type="fixed">
+      <origin
+        xyz="0 0 0"
+        rpy="0 0 0"/>
+      <parent
+        link="neck_tilt_link"/>
+      <child
+        link="head_shell_link"/>
+    </joint>
+    <link name="face_shell_link">
+      <visual>
+        <origin
+          xyz="-0.394 0.69 0.0995"
+          rpy="0 ${M_PI/2} 0"/>
+        <geometry>
+          <mesh
+            filename="package://vizzy_description/meshes/head/face.dae"/>
+        </geometry>
+        <material name="light_gray_1"/>
+      </visual>
+      <inertial>
+        <origin rpy="0 0 0" xyz="0.0 0.0 0.0"/>
+        <mass value="0.001"/>
+        <inertia ixx="0.01" ixy="0" ixz="0" iyy="0.01" iyz="0" izz="0.01"/>
+      </inertial>
+      <collision>
+        <origin rpy="0 0 0" xyz="0.0 0.0 0.0"/>
+        <geometry>
+          <cylinder length="0.001" radius="0.005"/>
+        </geometry>
+      </collision>
+    </link>
+    <joint name="face_shell_joint"
+      type="fixed">
+      <origin
+        xyz="0 0 0"
+        rpy="0 0 0"/>
+      <parent
+        link="neck_tilt_link"/>
+      <child
+        link="face_shell_link"/>
+    </joint>
     <!-- Eyes tilt -->
     <link name="eyes_tilt_link">
