Commit message: Adapting urdfs to be used with yarp control plugins

File: vizzy_description/robots/vizzy.ros.urdf.xacro (robot description, xacro)
@@ -1,5 +1,4 @@
 <?xml version="1.0"?>
 <robot  name="vizzy" xmlns:xacro="http://ros.org/wiki/xacro" >
-	<xacro:arg name="use_yarp" default="false"/>
   <!-- The following include files set up definitions of parts of the robot body  -->
   <!-- misc common stuff -->
@@ -12,15 +11,10 @@
   <xacro:include filename="$(find vizzy_description)/urdf/torso/torso.urdf.xacro" />
   <!-- head -->
-  <xacro:if value="$(arg use_yarp)">
-  	<xacro:include filename="$(find vizzy_description)/urdf/head/head.yarp.urdf.xacro" />
-  </xacro:if>
-  <xacro:unless value="$(arg use_yarp)">
-  	<xacro:include filename="$(find vizzy_description)/urdf/head/head.ros.urdf.xacro" />
-  </xacro:unless>
+  <xacro:include filename="$(find vizzy_description)/urdf/head/head.ros.urdf.xacro" />
   <!-- left arm -->
   <xacro:include filename="$(find vizzy_description)/urdf/arm/left_arm.urdf.xacro" />
   <!-- right arm -->
   <xacro:include filename="$(find vizzy_description)/urdf/arm/right_arm.urdf.xacro" />
-	<!-- The following include files contain gazebo plugins -->
+  <!-- The following include files contain gazebo plugins -->
   <!-- ROS -->
   <xacro:include filename="$(find vizzy_description)/plugins/ros.gazebo.xacro" />
@@ -49,14 +43,5 @@
   <xacro:camera_plugin name="l_camera" prefix="l"/>
   <xacro:camera_plugin name="r_camera" prefix="r"/>
-  <!-- instantiate Yarp plugins -->
-  <xacro:if value="$(arg use_yarp)">
-		<xacro:torso_gazebo_control/>
-		<xacro:head_gazebo_control/>
-		<xacro:left_arm_gazebo_control/>
-		<xacro:right_arm_gazebo_control/>
-  </xacro:if>
   <!-- instantiate ROS plugins -->
-  <xacro:unless value="$(arg use_yarp)">
-		<xacro:ros_control_gazebo/>
-  </xacro:unless>
+  <xacro:ros_control_gazebo/>
 </robot>

File: vizzy_description/urdf/head/head.yarp.gazebo.xacro (robot description, xacro)
@@ -3,15 +3,27 @@
   <xacro:macro name="head_gazebo">
     <gazebo reference="neck_pan_link">
-      <mu1>0.2</mu1>
-      <mu2>0.2</mu2>
     </gazebo>
     <gazebo reference="neck_tilt_link">
-      <mu1>0.2</mu1>
-      <mu2>0.2</mu2>
     </gazebo>
     <gazebo reference="eyes_tilt_link">
-      <mu1>0.2</mu1>
-      <mu2>0.2</mu2>
     </gazebo>
+    <gazebo reference="version_link">
+    </gazebo>
+    <gazebo reference="r_eye_version_link">
+    </gazebo>
+    <gazebo reference="l_eye_version_link">
+    </gazebo>
+    <gazebo reference="vergence_link">
+    </gazebo>
+  <gazebo reference="r_eye_vergence_link">
+    </gazebo>
+    <gazebo reference="l_eye_vergence_link">
+    </gazebo>
+ 		<gazebo reference="neck_pan_joint">
+		</gazebo>
+ 		<gazebo reference="neck_tilt_joint">
+		</gazebo>
+ 		<gazebo reference="eyes_tilt_joint">
+		</gazebo>
     <gazebo reference="r_eye_pan_link">
       <mu1>0.2</mu1>

File: vizzy_description/urdf/head/head.yarp.urdf.xacro (robot description, xacro)
@@ -237,6 +237,5 @@
     <child link="r_camera_link" />
   </joint>
-  <link
-    name="l_eye_pan_link">
+  <link name="l_eye_pan_link">
     <inertial>
       <origin
@@ -299,8 +298,68 @@
     </visual>
   </link>
+  <!-- Camera (Opencv convention) frames -->
   <joint name="l_camera_joint" type="fixed">
     <origin xyz="0.0575 0.0 0.0" rpy="0.0 0.0 0.0" />
     <parent link="l_eye_pan_link"/>
     <child link="l_camera_link" />
+  </joint>
+  <link name="l_camera_vision_link">
+   <visual>
+      <origin xyz="0 0 0" rpy="0 0 0" />
+      <geometry>
+        <box size="0.001 0.001 0.001" />
+      </geometry>
+    </visual>
+  </link>
+  <joint name="l_camera_vision_joint" type="fixed">
+    <origin xyz="0.0 0.0 0.0" rpy="${-M_PI/2} 0.0 ${-M_PI/2}" />
+    <parent link="l_camera_link"/>
+    <child link="l_camera_vision_link" />
+  </joint>
+  <link name="r_camera_vision_link">
+   <visual>
+      <origin xyz="0 0 0" rpy="0 0 0" />
+      <geometry>
+        <box size="0.001 0.001 0.001" />
+      </geometry>
+    </visual>
+  </link>
+  <joint name="r_camera_vision_joint" type="fixed">
+    <origin xyz="0.0 0.0 0.0" rpy="${-M_PI/2} 0.0 ${-M_PI/2}" />
+    <parent link="r_camera_link"/>
+    <child link="r_camera_vision_link" />
+  </joint>
+  <!-- eyes center and ego virtual link and joint -->
+  <link name="ego_frame">
+    <inertial>
+      <origin xyz="0 0 0" rpy="0.0 0.0 0" />
+      <mass value="0.001"/>
+      <inertia
+        ixx="0.001" ixy="0.0" ixz="0.0"
+        iyy="0.001" iyz="0.0" izz="0.001"/>
+    </inertial>
+  </link>
+  <joint name="ego_joint" type="fixed">
+    <origin
+      xyz="0.0 0.370 0.0"
+      rpy="0.0 ${M_PI/2.0} ${M_PI}" />
+    <parent link="waist_link"/>
+    <child link="ego_frame" />
+  </joint>
+  <link name="head_origin_frame">
+    <inertial>
+      <origin xyz="0 0 0" rpy="0.0 0.0 0" />
+      <mass value="0.001"/>
+      <inertia
+        ixx="0.001" ixy="0.0" ixz="0.0"
+        iyy="0.001" iyz="0.0" izz="0.001"/>
+    </inertial>
+  </link>
+  <joint name="head_origin_joint" type="fixed">
+    <origin
+      xyz="0.0 -0.04755 0.0"
+      rpy="0.0 -${M_PI/2.0} 0.0" />
+    <parent link="neck_tilt_link"/>
+    <child link="head_origin_frame" />
   </joint>
     <!-- gazebo extensions -->
