Commit message: yarp flag is now working. Elbow updated to avoid collisions

File: vizzy_description/robots/vizzy.urdf.xacro (robot description, xacro)
@@ -12,15 +12,11 @@
   <xacro:include filename="$(find vizzy_description)/urdf/torso/torso.urdf.xacro" />
   <!-- head -->
-  <xacro:if value="$(arg use_yarp)">
-  	<xacro:include filename="$(find vizzy_description)/urdf/head/head.yarp.urdf.xacro" />
-  </xacro:if>
-  <xacro:unless value="$(arg use_yarp)">
-  	<xacro:include filename="$(find vizzy_description)/urdf/head/head.ros.urdf.xacro" />
-  </xacro:unless>
+ <xacro:include filename="$(find vizzy_description)/urdf/head/head.yarp.urdf.xacro"/>
+ <xacro:include filename="$(find vizzy_description)/urdf/head/head.ros.urdf.xacro"/>
   <!-- left arm -->
   <xacro:include filename="$(find vizzy_description)/urdf/arm/left_arm.urdf.xacro" />
   <!-- right arm -->
   <xacro:include filename="$(find vizzy_description)/urdf/arm/right_arm.urdf.xacro" />
-	<!-- The following include files contain gazebo plugins -->
+  <!-- The following include files contain gazebo plugins -->
   <!-- ROS -->
   <xacro:include filename="$(find vizzy_description)/plugins/ros.gazebo.xacro" />
@@ -32,5 +28,10 @@
   <xacro:torso name="torso"/>
   <!-- instantiate head -->
-  <xacro:head name="head"/>
+  <xacro:if value="$(arg use_yarp)">
+  	<xacro:head_yarp name="head"/>
+  </xacro:if>
+  <xacro:unless value="$(arg use_yarp)">
+  	<xacro:head name="head"/>
+  </xacro:unless>
   <!-- instantiate left arm -->
   <xacro:left_arm name="left_arm" parent="waist_link" sufix="l" reflect="1">

File: vizzy_description/urdf/head/head.ros.urdf.xacro (robot description, xacro)
@@ -60,5 +60,6 @@
     <axis
       xyz="0 0 1" />
-    <limit lower="-0.925024504" upper="0.925024504" effort="10.0" velocity="5.0" />
+    <!--<limit lower="-0.925024504" upper="0.925024504" effort="10.0" velocity="5.0" />-->
+    <limit lower="-2.025024504" upper="2.025024504" effort="10.0" velocity="5.0" />
   </joint>
   <link
@@ -115,5 +116,5 @@
       xyz="0 0 1" />
     <!--<limit lower="-0.314159265" upper="0.645771823" effort="100.0" velocity="5.0" />-->
-    <limit lower="-0.614159265" upper="0.645771823" effort="100.0" velocity="5.0" />
+    <limit lower="-2.014159265" upper="2.45771823" effort="100.0" velocity="5.0" />
   </joint>
   <link

File: vizzy_description/urdf/head/head.yarp.urdf.xacro (robot description, xacro)
@@ -8,5 +8,5 @@
  <xacro:include filename="$(find vizzy_description)/urdf/head/head.yarp.gazebo.xacro" />
  <xacro:include filename="$(find vizzy_description)/urdf/head/head.yarp.transmission.xacro" />
-  <xacro:macro name="head" params="name">
+  <xacro:macro name="head_yarp" params="name">
    <link name="neck_pan_link">
     <inertial>
@@ -237,6 +237,5 @@
     <child link="r_camera_link" />
   </joint>
-  <link
-    name="l_eye_pan_link">
+  <link name="l_eye_pan_link">
     <inertial>
       <origin
@@ -299,8 +298,68 @@
     </visual>
   </link>
+  <!-- Camera (Opencv convention) frames -->
   <joint name="l_camera_joint" type="fixed">
     <origin xyz="0.0575 0.0 0.0" rpy="0.0 0.0 0.0" />
     <parent link="l_eye_pan_link"/>
     <child link="l_camera_link" />
+  </joint>
+  <link name="l_camera_vision_link">
+   <visual>
+      <origin xyz="0 0 0" rpy="0 0 0" />
+      <geometry>
+        <box size="0.001 0.001 0.001" />
+      </geometry>
+    </visual>
+  </link>
+  <joint name="l_camera_vision_joint" type="fixed">
+    <origin xyz="0.0 0.0 0.0" rpy="${-M_PI/2} 0.0 ${-M_PI/2}" />
+    <parent link="l_camera_link"/>
+    <child link="l_camera_vision_link" />
+  </joint>
+  <link name="r_camera_vision_link">
+   <visual>
+      <origin xyz="0 0 0" rpy="0 0 0" />
+      <geometry>
+        <box size="0.001 0.001 0.001" />
+      </geometry>
+    </visual>
+  </link>
+  <joint name="r_camera_vision_joint" type="fixed">
+    <origin xyz="0.0 0.0 0.0" rpy="${-M_PI/2} 0.0 ${-M_PI/2}" />
+    <parent link="r_camera_link"/>
+    <child link="r_camera_vision_link" />
+  </joint>
+  <!-- eyes center and ego virtual link and joint -->
+  <link name="ego_frame">
+    <inertial>
+      <origin xyz="0 0 0" rpy="0.0 0.0 0" />
+      <mass value="0.001"/>
+      <inertia
+        ixx="0.001" ixy="0.0" ixz="0.0"
+        iyy="0.001" iyz="0.0" izz="0.001"/>
+    </inertial>
+  </link>
+  <joint name="ego_joint" type="fixed">
+    <origin
+      xyz="0.0 0.370 0.0"
+      rpy="0.0 ${M_PI/2.0} ${M_PI}" />
+    <parent link="waist_link"/>
+    <child link="ego_frame" />
+  </joint>
+  <link name="head_origin_frame">
+    <inertial>
+      <origin xyz="0 0 0" rpy="0.0 0.0 0" />
+      <mass value="0.001"/>
+      <inertia
+        ixx="0.001" ixy="0.0" ixz="0.0"
+        iyy="0.001" iyz="0.0" izz="0.001"/>
+    </inertial>
+  </link>
+  <joint name="head_origin_joint" type="fixed">
+    <origin
+      xyz="0.0 -0.04755 0.0"
+      rpy="0.0 -${M_PI/2.0} 0.0" />
+    <parent link="neck_tilt_link"/>
+    <child link="head_origin_frame" />
   </joint>
     <!-- gazebo extensions -->

Commit message: started incorporating asus xtion

File: vizzy_description/robots/vizzy.urdf.xacro (robot description, xacro)
@@ -7,4 +7,6 @@
   <!-- sensors -->
   <xacro:include filename="$(find vizzy_description)/urdf/mounts/hokuyo_mount.urdf.xacro" />
+  <!-- Asus Xiton Live Pro -->
+  <xacro:include filename="$(find vizzy_description)/urdf/sensors/asus_camera.urdf.xacro" />
   <!-- base -->
   <xacro:include filename="$(find vizzy_description)/urdf/base/base.urdf.xacro" />
@@ -46,4 +48,7 @@
     <origin xyz="-0.05 0.14 0.15" rpy="${-M_PI/2} ${-M_PI/2} 3.14" />
   </xacro:hokuyo_mount>
+  <xacro:asus_camera name="camera" parent="waist_link">
+    <origin xyz="-0.08 0.12 0.02" rpy="${-M_PI/2} ${M_PI} 0"/>
+  </xacro:asus_camera>
   <!-- instantiate common ROS and Yarp plugins -->
   <xacro:ros_differential_drive_gazebo/>

Commit message: calibrating kinect pose

File: vizzy_description/robots/vizzy.urdf.xacro (robot description, xacro)
@@ -49,5 +49,5 @@
   </xacro:hokuyo_mount>
   <xacro:asus_camera name="camera" parent="waist_link">
-    <origin xyz="-0.08 0.12 0.02" rpy="${-M_PI/2} ${M_PI} 0"/>
+    <origin xyz="-0.08 0.12 0.02" rpy="${-M_PI/2} ${M_PI} ${-20.0*(M_PI/180)}"/>
   </xacro:asus_camera>
   <!-- instantiate common ROS and Yarp plugins -->

Commit message: Asus xtion location is okay, but still needs to be improved
João calibrated the cameras againfor ROS nodes

File: vizzy_description/robots/vizzy.urdf.xacro (robot description, xacro)
@@ -49,5 +49,5 @@
   </xacro:hokuyo_mount>
   <xacro:asus_camera name="camera" parent="waist_link">
-    <origin xyz="-0.08 0.12 0.02" rpy="${-M_PI/2} ${M_PI} ${-20.0*(M_PI/180)}"/>
+    <origin xyz="-0.08 0.16 0.02" rpy="${-M_PI/2} ${M_PI} ${-21.0*(M_PI/180)}"/>
   </xacro:asus_camera>
   <!-- instantiate common ROS and Yarp plugins -->

Commit message: Extrinsic calibration needs to be done
Current asus position is okay, but has an offset dependent on the distance

Intrinsic calibration of asus done

File: vizzy_description/robots/vizzy.urdf.xacro (robot description, xacro)
@@ -49,5 +49,5 @@
   </xacro:hokuyo_mount>
   <xacro:asus_camera name="camera" parent="waist_link">
-    <origin xyz="-0.08 0.16 0.02" rpy="${-M_PI/2} ${M_PI} ${-21.0*(M_PI/180)}"/>
+    <origin xyz="-0.075 0.15 0.02" rpy="${-M_PI/2} ${M_PI} ${-21.0*(M_PI/180)}"/>
   </xacro:asus_camera>
   <!-- instantiate common ROS and Yarp plugins -->

File: vizzy_description/urdf/sensors/asus_camera.urdf.xacro (robot description, xacro)
@@ -4,28 +4,28 @@
 <xacro:macro name="asus_camera_model" params="name parent *origin">
 <joint name="${name}_joint" type="fixed">
-<xacro:insert_block name="origin" />
-<parent link="${parent}"/>
-<child link="${name}_link"/>
+	<xacro:insert_block name="origin" />
+	<parent link="${parent}"/>
+	<child link="${name}_link"/>
 </joint>
 <link name="${name}_link">
-<inertial>
-<mass value="0.200" />
-<origin xyz="0 0 0" rpy="0 0 0" />
-<inertia ixx="5.8083e-4" ixy="0" ixz="0" iyy="3.0833e-5" iyz="0" izz="5.9083e-4" />
-</inertial>
-<visual>
-<origin xyz="0 0 0" rpy="0 0 0" />
-<geometry>
-<mesh filename="package://vizzy_description/meshes/asus_camera/asus_camera_simple.dae"/>
-</geometry>
-</visual>
-<collision>
-<origin xyz="0 0 0" rpy="0 0 0" />
-<geometry>
-<box size="0.035 0.185 0.025"/>
-</geometry>
-</collision>
+	<inertial>
+	<mass value="0.200" />
+	<origin xyz="0 0 0" rpy="0 0 0" />
+	<inertia ixx="5.8083e-4" ixy="0" ixz="0" iyy="3.0833e-5" iyz="0" izz="5.9083e-4" />
+	</inertial>
+	<visual>
+		<origin xyz="0 0 0" rpy="0 0 0" />
+		<geometry>
+			<mesh filename="package://vizzy_description/meshes/asus_camera/asus_camera_simple.dae"/>
+		</geometry>
+	</visual>
+	<collision>
+		<origin xyz="0 0 0" rpy="0 0 0" />
+		<geometry>
+			<box size="0.035 0.185 0.025"/>
+		</geometry>
+	</collision>
 </link>
-<joint name="${name}_depth_joint" type="fixed">
+<!--<joint name="${name}_depth_joint" type="fixed">
 <origin xyz="0.0 0.049 0.0" rpy="0 0 0" />
 <parent link="${name}_link" />
@@ -50,5 +50,5 @@
 <child link="${name}_rgb_optical_frame"/>
 </joint>
-<link name="${name}_rgb_optical_frame"/>
+<link name="${name}_rgb_optical_frame"/>-->
 </xacro:macro>
 <xacro:macro name="asus_camera" params="name parent *origin">

Commit message: new params

File: vizzy_description/robots/vizzy.urdf.xacro (robot description, xacro)
@@ -49,5 +49,5 @@
   </xacro:hokuyo_mount>
   <xacro:asus_camera name="camera" parent="waist_link">
-    <origin xyz="-0.075 0.15 0.02" rpy="${-M_PI/2} ${M_PI} ${-21.0*(M_PI/180)}"/>
+    <origin xyz="-0.195473  0.129382 0.0418749" rpy="1.61049 -0.0262743 2.58442"/>
   </xacro:asus_camera>
   <!-- instantiate common ROS and Yarp plugins -->

Commit message: Extrinsic calibration of the kinect with respect to the left eye
It works one meter next to the robot

File: vizzy_description/robots/vizzy.urdf.xacro (robot description, xacro)
@@ -49,5 +49,5 @@
   </xacro:hokuyo_mount>
   <xacro:asus_camera name="camera" parent="waist_link">
-    <origin xyz="-0.195473  0.129382 0.0418749" rpy="1.61049 -0.0262743 2.58442"/>
+    <origin xyz="-0.195473 0.129382 0.0418749" rpy="1.61049 -0.0262743 2.58442"/>
   </xacro:asus_camera>
   <!-- instantiate common ROS and Yarp plugins -->

Commit message: fixed laser position for the new ulm30 laser

File: vizzy_description/robots/vizzy.urdf.xacro (robot description, xacro)
@@ -6,5 +6,5 @@
   <xacro:include filename="$(find vizzy_description)/urdf/common.urdf.xacro" />
   <!-- sensors -->
-  <xacro:include filename="$(find vizzy_description)/urdf/mounts/hokuyo_mount.urdf.xacro" />
+  <xacro:include filename="$(find vizzy_description)/urdf/sensors/hokuyo_04lx_laser.urdf.xacro" />
   <!-- Asus Xiton Live Pro -->
   <xacro:include filename="$(find vizzy_description)/urdf/sensors/asus_camera.urdf.xacro" />
@@ -45,7 +45,7 @@
   </xacro:right_arm>
   <!-- instantiate hokuyo -->
-  <xacro:hokuyo_mount name="nav_hokuyo" parent="base" length="${SENSOR_BEAM_LENGTH*INCH_TO_M}" ros_topic="scan" update_rate="10" min_angle="${-(5 * M_PI)/12}" max_angle="${(5 * M_PI)/12}">
-    <origin xyz="-0.05 0.14 0.15" rpy="${-M_PI/2} ${-M_PI/2} 3.14" />
-  </xacro:hokuyo_mount>
+  <xacro:hokuyo_04lx_laser name="nav_hokuyo" parent="b_wheel_base" ros_topic="scan" update_rate="10" min_angle="${-(5 * M_PI)/12}" max_angle="${(5 * M_PI)/12}">
+    <origin xyz="-0.025 0.0 -0.00394" rpy="0 ${M_PI} 0" />
+  </xacro:hokuyo_04lx_laser>
   <xacro:asus_camera name="camera" parent="waist_link">
     <origin xyz="-0.195473 0.129382 0.0418749" rpy="1.61049 -0.0262743 2.58442"/>

File: vizzy_description/urdf/mounts/hokuyo_mount.urdf.xacro (robot description, xacro)
@@ -7,5 +7,5 @@
   <xacro:macro name="hokuyo_mount" params="name parent *origin length ros_topic update_rate min_angle max_angle">
     <xacro:hokuyo_04lx_laser name="${name}" parent="${parent}" ros_topic="${ros_topic}" update_rate="${update_rate}" min_angle="${min_angle}" max_angle="${max_angle}">
-      <origin xyz="0 0 0.25" rpy="0 0 ${-M_PI}" />
+      <origin xyz="0 0 2.25" rpy="0 0 ${-M_PI}" />
     </xacro:hokuyo_04lx_laser>
   </xacro:macro>

File: vizzy_description/urdf/sensors/hokuyo_04lx_laser.urdf.xacro (robot description, xacro)
@@ -7,5 +7,4 @@
   <xacro:macro name="hokuyo_04lx_laser" params="name parent *origin ros_topic update_rate min_angle max_angle">
     <joint name="${name}_joint" type="fixed">
-      <axis xyz="0 1 0" />
       <insert_block name="origin" />
       <parent link="${parent}_link"/>
@@ -15,19 +14,13 @@
       <inertial>
         <mass value="0.001" />
-        <origin xyz="0 0 0" rpy="0 0 0" />
+        <insert_block name="origin" />
         <inertia ixx="0.0001" ixy="0" ixz="0" iyy="0.000001" iyz="0" izz="0.0001" />
       </inertial>
       <visual>
-        <origin xyz="0 0 0" rpy="0 0 0" />
+        <origin xyz="0 0 0.058" rpy="0 0 0" />
         <geometry>
-          <mesh filename="package://vizzy_description/meshes/hokuyo.dae" scale="0.0254 0.0254 0.0254" />
+          <mesh filename="package://vizzy_description/meshes/hokuyo_utm30lx/hokuyo_utm_30lxTEST_SELF_FILTER.dae" />
         </geometry>
       </visual>
-      <!-- <collision> -->
-      <!--   <origin xyz="0 0 0" rpy="0 0 0" /> -->
-      <!--   <geometry> -->
-      <!--     <mesh filename="package://vizzy_description/meshes/hokuyo.dae" scale="0.0254 0.0254 0.0254" /> -->
-      <!--   </geometry> -->
-      <!-- </collision> -->
     </link>
     <!-- go from the base of the laser to the actual sensor location -->

Commit message: fixed shaking wrist behavious in the right hand. Fixed laser max range parameters according to Hokuyo lm30x specs

File: vizzy_description/robots/vizzy.urdf.xacro (robot description, xacro)
@@ -45,6 +45,6 @@
   </xacro:right_arm>
   <!-- instantiate hokuyo -->
-  <xacro:hokuyo_04lx_laser name="nav_hokuyo" parent="b_wheel_base" ros_topic="scan" update_rate="10" min_angle="${-(5 * M_PI)/12}" max_angle="${(5 * M_PI)/12}">
-    <origin xyz="-0.025 0.0 -0.00394" rpy="0 ${M_PI} 0" />
+  <xacro:hokuyo_04lx_laser name="nav_hokuyo" parent="base" ros_topic="scan" update_rate="40" min_angle="${-(5 * M_PI)/12}" max_angle="${(5 * M_PI)/12}" max_range="30">
+    <origin xyz="${-0.025-0.060139} 0.001 ${-0.00394+0.14806}" rpy="0 0 ${M_PI}" />
   </xacro:hokuyo_04lx_laser>
   <xacro:asus_camera name="camera" parent="waist_link">

File: vizzy_description/urdf/arm/left_arm.urdf.xacro (robot description, xacro)
@@ -332,18 +332,4 @@
 		  <limit lower="-1.48352986" upper="1.48352986" effort="10" velocity="3" />
 		</joint>
-		<joint
-		  name="l_wrist_abduction_joint"
-		  type="revolute">
-		  <origin
-		    xyz="0.0 0.0 0.11925"
-		    rpy="${M_PI/2.0} 0.0 0.0" />
-		  <parent
-		    link="l_forearm_pronation_link" />
-		  <child
-		    link="l_wrist_abduction_virtual_link" />
-		  <axis
-		    xyz="0 0 1" />
-		  <limit lower="-0.610865238" upper="0.610865238" effort="10" velocity="3" />
-		</joint>
 		<link
 		  name="l_wrist_abduction_virtual_link">
@@ -386,4 +372,18 @@
 		  </collision>
 		</link>
+		<joint
+		  name="l_wrist_abduction_joint"
+		  type="revolute">
+		  <origin
+		    xyz="0.0 0.0 0.11925"
+		    rpy="${M_PI/2.0} 0.0 0.0" />
+		  <parent
+		    link="l_forearm_pronation_link" />
+		  <child
+		    link="l_wrist_abduction_virtual_link" />
+		  <axis
+		    xyz="0 0 1" />
+		  <limit lower="-0.610865238" upper="0.610865238" effort="10" velocity="3" />
+		</joint>
 		<link
 		  name="l_wrist_abduction_link">

File: vizzy_description/urdf/arm/right_arm.urdf.xacro (robot description, xacro)
@@ -339,4 +339,58 @@
 		      rpy="${-M_PI/2.0} 0 ${M_PI}" />
 		    <mass
+		      value="0.151302636921624" />
+		    <inertia
+		      ixx="0.000116373512947626"
+		      ixy="1.31009871908069E-05"
+		      ixz="6.69703789973942E-05"
+		      iyy="0.00020031628400595"
+		      iyz="1.00268924727662E-05"
+		      izz="0.000162164313365602" />
+		  </inertial>
+		  <visual>
+		    <origin
+		      xyz="0.0 0.0 -0.005"
+		      rpy="${-M_PI/2.0} 0 ${M_PI}" />
+		    <geometry>
+		      <mesh
+		        filename="package://vizzy_description/meshes/M6R_back.dae" />
+		    </geometry>
+		    <material
+		      name="">
+		      <color
+		        rgba="0.898039215686275 0.917647058823529 0.929411764705882 1" />
+		    </material>
+		  </visual>
+		  <collision>
+		    <origin
+		      xyz="0.0 0.0 -0.005"
+		      rpy="${-M_PI/2.0} 0 ${M_PI}" />
+		    <geometry>
+		      <mesh
+		        filename="package://vizzy_description/meshes/M6R_back.dae" />
+		    </geometry>
+		  </collision>
+		</link>
+		<joint
+		  name="r_wrist_abduction_joint"
+		  type="revolute">
+		  <origin
+		    xyz="0.0 0.0 -0.11925"
+		    rpy="${M_PI/2.0} 0.0 0.0" />
+		  <parent
+		    link="r_forearm_pronation_link" />
+		  <child
+		    link="r_wrist_abduction_virtual_link" />
+		  <axis
+		    xyz="0 0 1" />
+		  <limit lower="-0.610865238" upper="0.610865238" effort="10" velocity="3" />
+		</joint>
+		<link
+		  name="r_wrist_abduction_link">
+		  <inertial>
+		    <origin
+		      xyz="0.0047 0.028 -0.003"
+		      rpy="${M_PI} ${M_PI} 0" />
+		    <mass
 		      value="0.15130263687109" />
 		    <inertia
@@ -350,58 +404,4 @@
 		  <visual>
 		    <origin
-		      xyz="0.0 0.0 -0.005"
-		      rpy="${-M_PI/2.0} 0 ${M_PI}" />
-		    <geometry>
-		      <mesh
-		        filename="package://vizzy_description/meshes/M6R_back.dae" />
-		    </geometry>
-		    <material
-		      name="">
-		      <color
-		        rgba="0.898039215686275 0.917647058823529 0.929411764705882 1" />
-		    </material>
-		  </visual>
-		  <collision>
-		    <origin
-		      xyz="0.0 0.0 -0.005"
-		      rpy="${-M_PI/2.0} 0 ${M_PI}" />
-		    <geometry>
-		      <mesh
-		        filename="package://vizzy_description/meshes/M6R_back.dae" />
-		    </geometry>
-		  </collision>
-		</link>
-		<joint
-		  name="r_wrist_abduction_joint"
-		  type="revolute">
-		  <origin
-		    xyz="0.0 0.0 -0.11925"
-		    rpy="${M_PI/2.0} 0.0 0.0" />
-		  <parent
-		    link="r_forearm_pronation_link" />
-		  <child
-		    link="r_wrist_abduction_virtual_link" />
-		  <axis
-		    xyz="0 0 1" />
-		  <limit lower="-0.610865238" upper="0.610865238" effort="10" velocity="3" />
-		</joint>
-		<link
-		  name="r_wrist_abduction_link">
-		  <inertial>
-		    <origin
-		      xyz="0.0047 0.028 -0.003"
-		      rpy="${M_PI} ${M_PI} 0" />
-		    <mass
-		      value="0.15130263687109" />
-		    <inertia
-		      ixx="0.000206280948481805"
-		      ixy="-2.10167871847464E-05"
-		      ixz="-1.95502541303483E-06"
-		      iyy="7.18084114032176E-05"
-		      iyz="1.63557763545568E-05"
-		      izz="0.000199867817507994" />
-		  </inertial>
-		  <visual>
-		    <origin
 		      xyz="0.0047 0.028 -0.003"
 		      rpy="${M_PI} ${M_PI} 0" />

File: vizzy_description/urdf/mounts/hokuyo_mount.urdf.xacro (robot description, xacro)
@@ -5,6 +5,6 @@
       xmlns:xacro="http://ros.org/wiki/xacro">
   <xacro:include filename="$(find vizzy_description)/urdf/sensors/hokuyo_04lx_laser.urdf.xacro" />
-  <xacro:macro name="hokuyo_mount" params="name parent *origin length ros_topic update_rate min_angle max_angle">
-    <xacro:hokuyo_04lx_laser name="${name}" parent="${parent}" ros_topic="${ros_topic}" update_rate="${update_rate}" min_angle="${min_angle}" max_angle="${max_angle}">
+  <xacro:macro name="hokuyo_mount" params="name parent *origin length ros_topic update_rate min_angle max_angle max_range">
+    <xacro:hokuyo_04lx_laser name="${name}" parent="${parent}" ros_topic="${ros_topic}" update_rate="${update_rate}" min_angle="${min_angle}" max_angle="${max_angle}" max_range="${max_range}">
       <origin xyz="0 0 2.25" rpy="0 0 ${-M_PI}" />
     </xacro:hokuyo_04lx_laser>

File: vizzy_description/urdf/sensors/hokuyo_04lx_laser.gazebo.xacro (robot description, xacro)
@@ -1,5 +1,5 @@
 <?xml version="1.0"?>
 <root xmlns:xacro="http://ros.org/wiki/xacro">
-  <xacro:macro name="hokuyo_04lx_laser_gazebo" params="name ros_topic update_rate min_angle max_angle">
+  <xacro:macro name="hokuyo_04lx_laser_gazebo" params="name ros_topic update_rate min_angle max_angle max_range">
     <gazebo reference="${name}_link">
       <sensor type="ray" name="${name}">
@@ -7,5 +7,5 @@
         <update_rate>${update_rate}</update_rate>
         <pose>0 0 0 0 0 0</pose>
-        <visualize>false</visualize>
+        <visualize>true</visualize>
         <ray>
           <scan>
@@ -19,5 +19,5 @@
           <range>
             <min>0.02</min>
-            <max>4.0</max>
+            <max>${max_range}</max>
             <resolution>0.03</resolution>
           </range>

File: vizzy_description/urdf/sensors/hokuyo_04lx_laser.urdf.xacro (robot description, xacro)
@@ -5,5 +5,5 @@
       xmlns:xacro="http://ros.org/wiki/xacro">
   <xacro:include filename="$(find vizzy_description)/urdf/sensors/hokuyo_04lx_laser.gazebo.xacro" />
-  <xacro:macro name="hokuyo_04lx_laser" params="name parent *origin ros_topic update_rate min_angle max_angle">
+  <xacro:macro name="hokuyo_04lx_laser" params="name parent *origin ros_topic update_rate min_angle max_angle max_range">
     <joint name="${name}_joint" type="fixed">
       <insert_block name="origin" />
@@ -20,5 +20,5 @@
         <origin xyz="0 0 0.058" rpy="0 0 0" />
         <geometry>
-          <mesh filename="package://vizzy_description/meshes/hokuyo_utm30lx/hokuyo_utm_30lxTEST_SELF_FILTER.dae" />
+          <mesh filename="package://vizzy_description/meshes/hokuyo_utm30lx/hokuyo_utm_30lx.dae" />
         </geometry>
       </visual>
@@ -38,5 +38,5 @@
     </link>
     <!-- gazebo extensions -->
-    <xacro:hokuyo_04lx_laser_gazebo name="${name}_laser" ros_topic="${ros_topic}" update_rate="${update_rate}" min_angle="${min_angle}" max_angle="${max_angle}" />
+    <xacro:hokuyo_04lx_laser_gazebo name="${name}_laser" ros_topic="${ros_topic}" update_rate="${update_rate}" min_angle="${min_angle}" max_angle="${max_angle}" max_range="${max_range}"/>
   </xacro:macro>
 </root>
