Commit message: added right hand meshes and urdf.xacro files. The correct transformation from the wrist to the r_palm_link is still missing

File: vizzy_description/robots/vizzy.urdf.xacro (robot description, xacro)
@@ -20,4 +20,6 @@
   <!-- right arm -->
   <xacro:include filename="$(find vizzy_description)/urdf/arm/right_arm.urdf.xacro" />
+  <!-- right hand -->
+  <xacro:include filename="$(find vizzy_description)/urdf/hand/right_hand.urdf.xacro" />
   <!-- The following include files contain gazebo plugins -->
   <!-- ROS -->
@@ -44,4 +46,8 @@
     <origin xyz="-0.01707 0.0 0.38145" rpy="0.0 0.0 0.0" />
   </xacro:right_arm>
+  <!-- instantiate right hand -->
+  <xacro:right_hand name="right_hand" parent="r_wrist_flection_link" sufix="r" reflect="1">
+    <origin xyz="-0.01707 0.0 0.38145" rpy="0.0 0.0 0.0" />
+  </xacro:right_hand>
   <!-- instantiate hokuyo -->
   <xacro:hokuyo_04lx_laser name="nav_hokuyo" parent="base" ros_topic="scan" update_rate="40" min_angle="${-(5 * M_PI)/12}" max_angle="${(5 * M_PI)/12}" max_range="30">

File: vizzy_description/urdf/arm/right_arm.urdf.xacro (robot description, xacro)
@@ -443,5 +443,5 @@
 		<link
 		  name="r_wrist_flection_link">
-		  <inertial>
+		  <!--<inertial>
 		    <origin
 		      xyz="0.106 0.0077 0.017"
@@ -479,5 +479,5 @@
 		        filename="package://vizzy_description/meshes/M7R.dae" />
 		    </geometry>
-		  </collision>
+		  </collision>-->
 		</link>
 		<joint
@@ -495,5 +495,5 @@
 		  <limit lower="-0.610865238" upper="0.610865238" effort="10" velocity="3" />
 		</joint>
-		<link name="r_palm_link">
+		<!--<link name="r_palm_link">
 		 <visual>
 		    <origin xyz="0 0 0" rpy="0 0 0" />
@@ -507,5 +507,5 @@
 		  <parent link="r_wrist_flection_link"/>
 		  <child link="r_palm_link" />
-		</joint>
+		</joint>-->
     <!-- gazebo extensions -->
     <xacro:right_arm_gazebo/>

File: vizzy_description/urdf/hand/right_hand.urdf.xacro (robot description, xacro)
@@ -6,23 +6,809 @@
   <!-- Things that are needed only for Gazebo (not the physical robot).  These include
        sensor and controller plugin specifications -->
-  <xacro:include filename="$(find vizzy_description)/urdf/arm/right_arm.gazebo.xacro"/>
+<xacro:include filename="$(find vizzy_description)/urdf/arm/right_arm.gazebo.xacro"/>
   <xacro:include filename="$(find vizzy_description)/urdf/arm/right_arm.transmission.xacro"/>
   <xacro:macro name="right_hand" params="name parent sufix reflect *origin">
-		<link name="r_palm_link">
-		 <visual>
-		    <origin xyz="0 0 0" rpy="0 0 0" />
-		    <geometry>
-		      <box size="0.001 0.001 0.001" />
-		    </geometry>
-		  </visual>
-		</link>
-		<joint name="r_palm_joint" type="fixed">
-		  <origin xyz="0.1 0 0.0" rpy="${M_PI/2.0} 0 ${M_PI}" />
-		  <parent link="${parent}"/>
+    <joint name="r_palm_joint" type="fixed">
+		  <origin xyz="0.1 0 0.0" rpy="0 ${M_PI/2.0} 0" />
+		  <parent link="r_wrist_flection_link"/>
 		  <child link="r_palm_link" />
 		</joint>
+  <link
+    name="r_palm_link">
+    <inertial>
+      <origin
+        xyz="-0.006637 0.0034589 0.0058703"
+        rpy="0 0 0" />
+      <mass
+        value="0.14841" />
+      <inertia
+        ixx="0.00014253"
+        ixy="1.9852E-05"
+        ixz="-1.4353E-06"
+        iyy="9.7254E-05"
+        iyz="-2.6916E-06"
+        izz="0.0002182" />
+    </inertial>
+    <visual>
+      <origin
+        xyz="0 0 0"
+        rpy="0 0 0" />
+      <geometry>
+        <mesh
+          filename="package://vizzy_description/meshes/right_hand/r_palm_link.STL" />
+      </geometry>
+      <material
+        name="">
+        <color
+          rgba="0.79608 0.82353 0.93725 1" />
+      </material>
+    </visual>
+    <collision>
+      <origin
+        xyz="0 0 0"
+        rpy="0 0 0" />
+      <geometry>
+        <mesh
+          filename="package://vizzy_description/meshes/right_hand/r_palm_link.STL" />
+      </geometry>
+    </collision>
+  </link>
+  <link
+    name="min_phal_1_link">
+    <inertial>
+      <origin
+        xyz="-0.0065851 -4.2258E-05 0.019478"
+        rpy="0 0 0" />
+      <mass
+        value="0.014476" />
+      <inertia
+        ixx="1.7219E-06"
+        ixy="3.4428E-10"
+        ixz="3.009E-10"
+        iyy="1.7445E-06"
+        iyz="1.5436E-08"
+        izz="5.3067E-07" />
+    </inertial>
+    <visual>
+      <origin
+        xyz="0 0 0"
+        rpy="0 0 0" />
+      <geometry>
+        <mesh
+          filename="package://vizzy_description/meshes/right_hand/min_phal_1_link.STL" />
+      </geometry>
+      <material
+        name="">
+        <color
+          rgba="0.89804 0.91765 0.92941 1" />
+      </material>
+    </visual>
+    <collision>
+      <origin
+        xyz="0 0 0"
+        rpy="0 0 0" />
+      <geometry>
+        <mesh
+          filename="package://vizzy_description/meshes/right_hand/min_phal_1_link.STL" />
+      </geometry>
+    </collision>
+  </link>
+  <joint
+    name="min_phal_1_joint"
+    type="revolute">
+    <origin
+      xyz="0.020602 -0.005836 0.044434"
+      rpy="6.2175E-17 -0.17453 3.1416" />
+    <parent
+      link="r_palm_link" />
+    <child
+      link="min_phal_1_link" />
+    <axis
+      xyz="1 0 0" />
+    <limit
+      lower="0"
+      upper="1.7453"
+      effort="0"
+      velocity="0" />
+  </joint>
+  <link
+    name="min_phal_2_link">
+    <inertial>
+      <origin
+        xyz="-0.0065912 3.9323E-05 0.016339"
+        rpy="0 0 0" />
+      <mass
+        value="0.011277" />
+      <inertia
+        ixx="1.007E-06"
+        ixy="5.324E-10"
+        ixz="5.414E-10"
+        iyy="1.0456E-06"
+        iyz="1.1256E-08"
+        izz="4.1298E-07" />
+    </inertial>
+    <visual>
+      <origin
+        xyz="0 0 0"
+        rpy="0 0 0" />
+      <geometry>
+        <mesh
+          filename="package://vizzy_description/meshes/right_hand/min_phal_2_link.STL" />
+      </geometry>
+      <material
+        name="">
+        <color
+          rgba="0.89804 0.91765 0.92941 1" />
+      </material>
+    </visual>
+    <collision>
+      <origin
+        xyz="0 0 0"
+        rpy="0 0 0" />
+      <geometry>
+        <mesh
+          filename="package://vizzy_description/meshes/right_hand/min_phal_2_link.STL" />
+      </geometry>
+    </collision>
+  </link>
+  <joint
+    name="min_phal_2_joint"
+    type="revolute">
+    <origin
+      xyz="0 0 0.033"
+      rpy="0 -7.2164E-16 0" />
+    <parent
+      link="min_phal_1_link" />
+    <child
+      link="min_phal_2_link" />
+    <axis
+      xyz="1 0 0" />
+    <limit
+      lower="0"
+      upper="1.5708"
+      effort="0"
+      velocity="0" />
+  </joint>
+  <link
+    name="min_phal_3_link">
+    <inertial>
+      <origin
+        xyz="-0.0065949 -2.2728E-05 0.013411"
+        rpy="0 0 0" />
+      <mass
+        value="0.0093855" />
+      <inertia
+        ixx="5.7614E-07"
+        ixy="5.3191E-10"
+        ixz="-3.8097E-11"
+        iyy="5.3414E-07"
+        iyz="3.9566E-09"
+        izz="3.158E-07" />
+    </inertial>
+    <visual>
+      <origin
+        xyz="0 0 0"
+        rpy="0 0 0" />
+      <geometry>
+        <mesh
+          filename="package://vizzy_description/meshes/right_hand/min_phal_3_link.STL" />
+      </geometry>
+      <material
+        name="">
+        <color
+          rgba="0.89804 0.91765 0.92941 1" />
+      </material>
+    </visual>
+    <collision>
+      <origin
+        xyz="0 0 0"
+        rpy="0 0 0" />
+      <geometry>
+        <mesh
+          filename="package://vizzy_description/meshes/right_hand/min_phal_3_link.STL" />
+      </geometry>
+    </collision>
+  </link>
+  <joint
+    name="min_phal_3_joint"
+    type="revolute">
+    <origin
+      xyz="0 0 0.0265"
+      rpy="0 2.7756E-17 0" />
+    <parent
+      link="min_phal_2_link" />
+    <child
+      link="min_phal_3_link" />
+    <axis
+      xyz="1 0 0" />
+    <limit
+      lower="0"
+      upper="1.5708"
+      effort="0"
+      velocity="0" />
+  </joint>
+  <link
+    name="med_phal_1_link">
+    <inertial>
+      <origin
+        xyz="0.0029095 0.0027577 0.019478"
+        rpy="0 0 0" />
+      <mass
+        value="0.014476" />
+      <inertia
+        ixx="1.7219E-06"
+        ixy="3.4427E-10"
+        ixz="3.008E-10"
+        iyy="1.7445E-06"
+        iyz="1.5436E-08"
+        izz="5.3067E-07" />
+    </inertial>
+    <visual>
+      <origin
+        xyz="0 0 0"
+        rpy="0 0 0" />
+      <geometry>
+        <mesh
+          filename="package://vizzy_description/meshes/right_hand/med_phal_1_link.STL" />
+      </geometry>
+      <material
+        name="">
+        <color
+          rgba="0.89804 0.91765 0.92941 1" />
+      </material>
+    </visual>
+    <collision>
+      <origin
+        xyz="0 0 0"
+        rpy="0 0 0" />
+      <geometry>
+        <mesh
+          filename="package://vizzy_description/meshes/right_hand/med_phal_1_link.STL" />
+      </geometry>
+    </collision>
+  </link>
+  <joint
+    name="med_phal_1_joint"
+    type="revolute">
+    <origin
+      xyz="0 -0.003036 0.050139"
+      rpy="6.123E-17 4.5912E-49 3.1416" />
+    <parent
+      link="r_palm_link" />
+    <child
+      link="med_phal_1_link" />
+    <axis
+      xyz="1 0 0" />
+    <limit
+      lower="0"
+      upper="1.7453"
+      effort="0"
+      velocity="0" />
+  </joint>
+  <link
+    name="med_phal_2_link">
+    <inertial>
+      <origin
+        xyz="0.0029034 3.9323E-05 0.01634"
+        rpy="0 0 0" />
+      <mass
+        value="0.011277" />
+      <inertia
+        ixx="1.007E-06"
+        ixy="5.324E-10"
+        ixz="5.4133E-10"
+        iyy="1.0456E-06"
+        iyz="1.1377E-08"
+        izz="4.13E-07" />
+    </inertial>
+    <visual>
+      <origin
+        xyz="0 0 0"
+        rpy="0 0 0" />
+      <geometry>
+        <mesh
+          filename="package://vizzy_description/meshes/right_hand/med_phal_2_link.STL" />
+      </geometry>
+      <material
+        name="">
+        <color
+          rgba="0.89804 0.91765 0.92941 1" />
+      </material>
+    </visual>
+    <collision>
+      <origin
+        xyz="0 0 0"
+        rpy="0 0 0" />
+      <geometry>
+        <mesh
+          filename="package://vizzy_description/meshes/right_hand/med_phal_2_link.STL" />
+      </geometry>
+    </collision>
+  </link>
+  <joint
+    name="med_phal_2_joint"
+    type="revolute">
+    <origin
+      xyz="0 0.0028 0.033"
+      rpy="0 0 0" />
+    <parent
+      link="med_phal_1_link" />
+    <child
+      link="med_phal_2_link" />
+    <axis
+      xyz="1 0 0" />
+    <limit
+      lower="0"
+      upper="1.5708"
+      effort="0"
+      velocity="0" />
+  </joint>
+  <link
+    name="med_phal_3_link">
+    <inertial>
+      <origin
+        xyz="0.0028997 -2.2727E-05 0.013411"
+        rpy="0 0 0" />
+      <mass
+        value="0.0093855" />
+      <inertia
+        ixx="5.7614E-07"
+        ixy="5.3189E-10"
+        ixz="-3.8133E-11"
+        iyy="5.3439E-07"
+        iyz="3.9566E-09"
+        izz="3.1605E-07" />
+    </inertial>
+    <visual>
+      <origin
+        xyz="0 0 0"
+        rpy="0 0 0" />
+      <geometry>
+        <mesh
+          filename="package://vizzy_description/meshes/right_hand/med_phal_3_link.STL" />
+      </geometry>
+      <material
+        name="">
+        <color
+          rgba="0.89804 0.91765 0.92941 1" />
+      </material>
+    </visual>
+    <collision>
+      <origin
+        xyz="0 0 0"
+        rpy="0 0 0" />
+      <geometry>
+        <mesh
+          filename="package://vizzy_description/meshes/right_hand/med_phal_3_link.STL" />
+      </geometry>
+    </collision>
+  </link>
+  <joint
+    name="med_phal_3_joint"
+    type="revolute">
+    <origin
+      xyz="0 0 0.0265"
+      rpy="0 0 -2.7192E-32" />
+    <parent
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
Commit message: removed mimic joints

File: vizzy_description/robots/vizzy.urdf.xacro (robot description, xacro)
@@ -20,5 +20,5 @@
   <xacro:include filename="$(find vizzy_description)/urdf/arm/right_arm.urdf.xacro" />
   <!-- right hand -->
-  <xacro:include filename="$(find vizzy_description)/urdf/hand/right_hand.urdf.xacro" />
+  <!--<xacro:include filename="$(find vizzy_description)/urdf/hand/right_hand.urdf.xacro" />-->
   <!-- The following include files contain gazebo plugins -->
   <!-- ROS -->

File: vizzy_description/urdf/arm/left_arm.urdf.xacro (robot description, xacro)
@@ -495,5 +495,5 @@
 		  <limit lower="-0.610865238" upper="0.610865238" effort="10" velocity="3" />
 		</joint>
-		<link name="l_palm_link">
+		<!--<link name="l_palm_link">
 		 <visual>
 		    <origin xyz="0.0 0.0 0.0" rpy="0.0 0.0 0.0" />
@@ -507,5 +507,5 @@
 		  <parent link="l_wrist_flection_link"/>
 		  <child link="l_palm_link" />
-		</joint>
+		</joint>-->
 		<!-- gazebo extensions -->
 		<xacro:left_arm_gazebo/>

File: vizzy_description/urdf/arm/right_arm.urdf.xacro (robot description, xacro)
@@ -443,5 +443,5 @@
 		<link
 		  name="r_wrist_flection_link">
-		  <!--<inertial>
+		  <inertial>
 		    <origin
 		      xyz="0.106 0.0077 0.017"
@@ -479,5 +479,5 @@
 		        filename="package://vizzy_description/meshes/M7R.dae" />
 		    </geometry>
-		  </collision>-->
+		  </collision>
 		</link>
 		<joint

File: vizzy_description/urdf/head/head.gazebo.xacro (robot description, xacro)
@@ -8,54 +8,8 @@
     <gazebo reference="eyes_tilt_link">
     </gazebo>
-    <gazebo reference="version_link">
-    </gazebo>
     <gazebo reference="r_eye_version_link">
     </gazebo>
     <gazebo reference="l_eye_version_link">
     </gazebo>
-    <gazebo reference="vergence_link">
-    </gazebo>
-		 <gazebo reference="r_eye_vergence_link">
-    </gazebo>
-    <gazebo reference="l_eye_vergence_link">
-    </gazebo>
- 		<gazebo reference="neck_pan_joint">
-		</gazebo>
- 		<gazebo reference="neck_tilt_joint">
-		</gazebo>
- 		<gazebo reference="eyes_tilt_joint">
-		</gazebo>
- 		<gazebo reference="version_joint">
-		</gazebo>
- 		<gazebo reference="vergence_joint">
-		</gazebo>
-		<gazebo>
-			<plugin name="mimic_plugin" filename="libgazebo_mimic_plugin.so">
-				<joint>version_joint</joint>
-				<mimicJoint>l_eye_version_joint</mimicJoint>
-				<multiplier>1.0</multiplier>
-			</plugin>
-		</gazebo>
-		<gazebo>
-			<plugin name="mimic_plugin" filename="libgazebo_mimic_plugin.so">
-				<joint>version_joint</joint>
-				<mimicJoint>r_eye_version_joint</mimicJoint>
-				<multiplier>1.0</multiplier>
-			</plugin>
-		</gazebo>
-		<gazebo>
-			<plugin name="mimic_plugin" filename="libgazebo_mimic_plugin.so">
-				<joint>vergence_joint</joint>
-				<mimicJoint>l_eye_vergence_joint</mimicJoint>
-				<multiplier>-1.0</multiplier>
-			</plugin>
-		</gazebo>
-		<gazebo>
-			<plugin name="mimic_plugin" filename="libgazebo_mimic_plugin.so">
-				<joint>vergence_joint</joint>
-				<mimicJoint>r_eye_vergence_joint</mimicJoint>
-				<multiplier>1.0</multiplier>
-			</plugin>
-		</gazebo>
   </xacro:macro>
 </robot>
