Commit message: updated right hand model

File: vizzy_description/robots/vizzy.urdf.xacro (robot description, xacro)
@@ -20,5 +20,5 @@
   <xacro:include filename="$(find vizzy_description)/urdf/arm/right_arm.urdf.xacro" />
   <!-- right hand -->
-  <!--<xacro:include filename="$(find vizzy_description)/urdf/hand/right_hand.urdf.xacro" />-->
+  <xacro:include filename="$(find vizzy_description)/urdf/hand/right_hand.urdf.xacro" />
   <!-- The following include files contain gazebo plugins -->
   <!-- ROS -->

File: vizzy_description/urdf/arm/right_arm.gazebo.xacro (robot description, xacro)
@@ -35,6 +35,4 @@
       <mu2>0.2</mu2>-->
     </gazebo>
-    <gazebo reference="r_palm_link">
-    </gazebo>
   </xacro:macro>
 </robot>

File: vizzy_description/urdf/arm/right_arm.transmission.xacro (robot description, xacro)
@@ -11,5 +11,4 @@
       </joint>
       <actuator name="r_shoulder_scapula_motor">
-        <hardwareInterface>EffortJointInterface</hardwareInterface>
         <mechanicalReduction>1</mechanicalReduction>
       </actuator>
@@ -21,5 +20,4 @@
       </joint>
       <actuator name="r_shoulder_flection_motor">
-        <hardwareInterface>EffortJointInterface</hardwareInterface>
         <mechanicalReduction>1</mechanicalReduction>
       </actuator>
@@ -31,5 +29,4 @@
       </joint>
       <actuator name="r_shoulder_abduction_motor">
-        <hardwareInterface>EffortJointInterface</hardwareInterface>
         <mechanicalReduction>1</mechanicalReduction>
       </actuator>
@@ -41,5 +38,4 @@
       </joint>
       <actuator name="r_shoulder_rotation_motor">
-        <hardwareInterface>EffortJointInterface</hardwareInterface>
         <mechanicalReduction>1</mechanicalReduction>
       </actuator>
@@ -51,5 +47,4 @@
       </joint>
       <actuator name="r_elbow_flection_motor">
-        <hardwareInterface>EffortJointInterface</hardwareInterface>
         <mechanicalReduction>1</mechanicalReduction>
       </actuator>
@@ -71,5 +66,4 @@
       </joint>
       <actuator name="r_wrist_abduction_motor">
-        <hardwareInterface>EffortJointInterface</hardwareInterface>
         <mechanicalReduction>1</mechanicalReduction>
       </actuator>
@@ -81,5 +75,4 @@
       </joint>
       <actuator name="r_wrist_flection_motor">
-        <hardwareInterface>EffortJointInterface</hardwareInterface>
         <mechanicalReduction>1</mechanicalReduction>
       </actuator>

File: vizzy_description/urdf/arm/right_arm.urdf.xacro (robot description, xacro)
@@ -409,5 +409,5 @@
 		      izz="0.00103049250587026" />
 		  </inertial>
-		  <visual>
+		  <!--<visual>
 		    <origin
 		      xyz="0.106 0.0077 0.017"
@@ -431,5 +431,5 @@
 		        filename="package://vizzy_description/meshes/M7R.dae" />
 		    </geometry>
-		  </collision>
+		  </collision>-->
 		</link>
 		<joint
@@ -448,5 +448,5 @@
 		  <dynamics damping="0.0" friction="1.0"/>
 		</joint>
-		<link name="r_palm_link">
+		<!--<link name="r_palm_link">
                     <inertial>
                         <origin xyz="0 0 0" rpy="0 0 0" />
@@ -469,7 +469,7 @@
                        </geometry>
                    </collision>
-	        </link>
+	        </link>-->
 		<joint name="r_palm_joint" type="fixed">
-		  <origin xyz="0.1 0 0.0" rpy="${M_PI/2.0} 0.0 ${M_PI}" />
+		  <origin xyz="0.075 0.01 -0.005" rpy="0.0 ${M_PI/2.0} 0.0" />
 		  <parent link="r_wrist_flection_link"/>
 		  <child link="r_palm_link" />

File: vizzy_description/urdf/hand/right_hand.urdf.xacro (robot description, xacro)
@@ -6,180 +6,119 @@
   <!-- Things that are needed only for Gazebo (not the physical robot).  These include
        sensor and controller plugin specifications -->
-<xacro:include filename="$(find vizzy_description)/urdf/arm/right_arm.gazebo.xacro"/>
-  <xacro:include filename="$(find vizzy_description)/urdf/arm/right_arm.transmission.xacro"/>
+<xacro:include filename="$(find vizzy_description)/urdf/hand/right_hand.gazebo.xacro"/>
+  <xacro:include filename="$(find vizzy_description)/urdf/hand/right_hand.transmission.xacro"/>
   <xacro:macro name="right_hand" params="name parent sufix reflect *origin">
   <link
-    name="r_hand_link">
-    <inertial>
-      <origin
-        xyz="0.0038463 -0.25763 0.60534"
-        rpy="0 0 0" />
-      <mass
-        value="0.14447" />
-      <inertia
-        ixx="0.00014079"
-        ixy="1.5176E-05"
-        ixz="1.0157E-05"
-        iyy="0.00013841"
-        iyz="5.8477E-05"
-        izz="0.00016255" />
-    </inertial>
-    <visual>
-      <origin
-        xyz="0 0 0"
-        rpy="0 0 0" />
-      <geometry>
-        <mesh
-          filename="package://vizzy_test/meshes/r_hand_link.STL" />
-      </geometry>
-      <material
-        name="">
-        <color
-          rgba="0.89804 0.91765 0.92941 1" />
-      </material>
-    </visual>
-    <collision>
-      <origin
-        xyz="0 0 0"
-        rpy="0 0 0" />
-      <geometry>
-        <mesh
-          filename="package://vizzy_test/meshes/r_hand_link.STL" />
-      </geometry>
-    </collision>
-  </link>
-  <joint
-    name="r_hand_joint"
-    type="fixed">
-    <origin
-      xyz="0.631985243056887 -0.118428097845849 -0.0023641314603528"
-      rpy="-2.73631640958448 -1.55026793601452 2.02896379866596" />
-    <parent
-      link="r_wrist_flection_link" />
-    <child
-      link="r_hand_link" />
-    <axis
-      xyz="0 0 0" />
-  </joint>
-  <link
-    name="r_thumb_1_link">
-    <inertial>
-      <origin
-        xyz="-0.00032032 0.0070152 0.0070409"
-        rpy="0 0 0" />
-      <mass
-        value="0.0081407" />
-      <inertia
-        ixx="6.5008E-07"
-        ixy="7.3119E-10"
-        ixz="2.5546E-09"
-        iyy="5.6171E-07"
-        iyz="2.5969E-09"
-        izz="2.906E-07" />
-    </inertial>
-    <visual>
-      <origin
-        xyz="0 0 0"
-        rpy="0 0 0" />
-      <geometry>
-        <mesh
-          filename="package://vizzy_test/meshes/r_thumb_1_link.STL" />
-      </geometry>
-      <material
-        name="">
-        <color
-          rgba="0.77647 0.75686 0.73725 1" />
-      </material>
-    </visual>
-    <collision>
-      <origin
-        xyz="0 0 0"
-        rpy="0 0 0" />
-      <geometry>
-        <mesh
-          filename="package://vizzy_test/meshes/r_thumb_1_link.STL" />
-      </geometry>
-    </collision>
-  </link>
-  <joint
-    name="r_thumb_1_joint"
-    type="fixed">
-    <origin
-      xyz="-0.051602659641749 -0.261993975608549 0.585670716685399"
-      rpy="1.58918253820798 -0.658618217290863 1.14526673964582" />
-    <parent
-      link="r_hand_link" />
-    <child
-      link="r_thumb_1_link" />
-    <axis
-      xyz="0 0 0" />
-  </joint>
-  <link
-    name="r_thumb_2_link">
-    <inertial>
-      <origin
-        xyz="4.3028E-05 0.0070072 0.013515"
-        rpy="0 0 0" />
-      <mass
-        value="0.014478" />
-      <inertia
-        ixx="1.7439E-06"
-        ixy="3.4418E-10"
-        ixz="1.4451E-08"
-        iyy="1.7213E-06"
-        iyz="3.0158E-10"
-        izz="5.3077E-07" />
-    </inertial>
-    <visual>
-      <origin
-        xyz="0 0 0"
-        rpy="0 0 0" />
-      <geometry>
-        <mesh
-          filename="package://vizzy_test/meshes/r_thumb_2_link.STL" />
-      </geometry>
-      <material
-        name="">
-        <color
-          rgba="0.77647 0.75686 0.73725 1" />
-      </material>
-    </visual>
-    <collision>
-      <origin
-        xyz="0 0 0"
-        rpy="0 0 0" />
-      <geometry>
-        <mesh
-          filename="package://vizzy_test/meshes/r_thumb_2_link.STL" />
-      </geometry>
-    </collision>
-  </link>
-  <joint
-    name="r_thumb_2_joint"
-    type="fixed">
-    <origin
-      xyz="-0.000155193715695168 0 -0.0329996350723843"
-      rpy="2.77558825516292E-17 0.00470285720488725 -5.55117651032584E-17" />
-    <parent
-      link="r_thumb_1_link" />
-    <child
-      link="r_thumb_2_link" />
-    <axis
-      xyz="0 0 0" />
-  </joint>
-  <link
-    name="r_thumb_3_link">
-    <inertial>
-      <origin
-        xyz="-3.9325E-05 0.0070133 0.01016"
+    name="r_palm_link">
+    <inertial>
+      <origin
+        xyz="-0.006637 0.0034589 0.0058703"
+        rpy="0 0 0" />
+      <mass
+        value="0.14841" />
+      <inertia
+        ixx="0.00014253"
+        ixy="1.9852E-05"
+        ixz="-1.4353E-06"
+        iyy="9.7254E-05"
+        iyz="-2.6916E-06"
+        izz="0.0002182" />
+    </inertial>
+    <visual>
+      <origin
+        xyz="0 0 0"
+        rpy="0 0 0" />
+      <geometry>
+        <mesh
+          filename="package://vizzy_description/meshes/right_hand/r_palm_link.STL" />
+      </geometry>
+      <material
+        name="">
+        <color
+          rgba="0.79608 0.82353 0.93725 1" />
+      </material>
+    </visual>
+    <collision>
+      <origin
+        xyz="0 0 0"
+        rpy="0 0 0" />
+      <geometry>
+        <mesh
+          filename="package://vizzy_description/meshes/right_hand/r_palm_link.STL" />
+      </geometry>
+    </collision>
+  </link>
+  <link
+    name="r_min_phal_1_link">
+    <inertial>
+      <origin
+        xyz="-0.0065851 -4.2258E-05 0.019478"
+        rpy="0 0 0" />
+      <mass
+        value="0.014476" />
+      <inertia
+        ixx="1.7219E-06"
+        ixy="3.4428E-10"
+        ixz="3.009E-10"
+        iyy="1.7445E-06"
+        iyz="1.5436E-08"
+        izz="5.3067E-07" />
+    </inertial>
+    <visual>
+      <origin
+        xyz="0 0 0"
+        rpy="0 0 0" />
+      <geometry>
+        <mesh
+          filename="package://vizzy_description/meshes/right_hand/r_min_phal_1_link.STL" />
+      </geometry>
+      <material
+        name="">
+        <color
+          rgba="0.89804 0.91765 0.92941 1" />
+      </material>
+    </visual>
+    <collision>
+      <origin
+        xyz="0 0 0"
+        rpy="0 0 0" />
+      <geometry>
+        <mesh
+          filename="package://vizzy_description/meshes/right_hand/r_min_phal_1_link.STL" />
+      </geometry>
+    </collision>
+  </link>
+  <joint
+    name="r_min_phal_1_joint"
+    type="revolute">
+    <origin
+      xyz="0.020602 -0.005836 0.044434"
+      rpy="6.2175E-17 -0.17453 3.1416" />
+    <parent
+      link="r_palm_link" />
+    <child
+      link="r_min_phal_1_link" />
+    <axis
+      xyz="1 0 0" />
+    <limit
+      lower="0"
+      upper="1.7453"
+      effort="0"
+      velocity="0" />
+  </joint>
+  <link
+    name="r_min_phal_2_link">
+    <inertial>
+      <origin
+        xyz="-0.0065912 3.9323E-05 0.016339"
         rpy="0 0 0" />
       <mass
         value="0.011277" />
       <inertia
-        ixx="1.0456E-06"
+        ixx="1.007E-06"
         ixy="5.324E-10"
-        ixz="1.1256E-08"
-        iyy="1.007E-06"
-        iyz="5.4133E-10"
+        ixz="5.414E-10"
+        iyy="1.0456E-06"
+        iyz="1.1256E-08"
         izz="4.1298E-07" />
     </inertial>
@@ -190,40 +129,45 @@
       <geometry>
         <mesh
-          filename="package://vizzy_test/meshes/r_thumb_3_link.STL" />
-      </geometry>
-      <material
-        name="">
-        <color
-          rgba="0.77647 0.75686 0.73725 1" />
-      </material>
-    </visual>
-    <collision>
-      <origin
-        xyz="0 0 0"
-        rpy="0 0 0" />
-      <geometry>
-        <mesh
-          filename="package://vizzy_test/meshes/r_thumb_3_link.STL" />
-      </geometry>
-    </collision>
-  </link>
-  <joint
-    name="r_thumb_3_joint"
-    type="fixed">
-    <origin
-      xyz="0 0 -0.0265000000000002"
-      rpy="2.08166817117217E-15 -7.63278329429795E-17 4.94049245958195E-15" />
-    <parent
-      link="r_thumb_2_link" />
-    <child
-      link="r_thumb_3_link" />
-    <axis
-      xyz="0 0 0" />
-  </joint>
-  <link
-    name="r_thumb_4_link">
-    <inertial>
-      <origin
-        xyz="-1.702E-05 -2.2727E-05 0.0049109"
+          filename="package://vizzy_description/meshes/right_hand/r_min_phal_2_link.STL" />
+      </geometry>
+      <material
+        name="">
+        <color
+          rgba="0.89804 0.91765 0.92941 1" />
+      </material>
+    </visual>
+    <collision>
+      <origin
+        xyz="0 0 0"
+        rpy="0 0 0" />
+      <geometry>
+        <mesh
+          filename="package://vizzy_description/meshes/right_hand/r_min_phal_2_link.STL" />
+      </geometry>
+    </collision>
+  </link>
+  <joint
+    name="r_min_phal_2_joint"
+    type="revolute">
+    <origin
+      xyz="0 0 0.033"
+      rpy="0 -7.2164E-16 0" />
+    <parent
+      link="r_min_phal_1_link" />
+    <child
+      link="r_min_phal_2_link" />
+    <axis
+      xyz="1 0 0" />
+    <limit
+      lower="0"
+      upper="1.5708"
+      effort="0"
+      velocity="0" />
+  </joint>
+  <link
+    name="r_min_phal_3_link">
+    <inertial>
+      <origin
+        xyz="-0.0065949 -2.2728E-05 0.013411"
         rpy="0 0 0" />
       <mass
@@ -231,264 +175,115 @@
       <inertia
         ixx="5.7614E-07"
-        ixy="5.3189E-10"
-        ixz="-3.8147E-11"
-        iyy="5.3439E-07"
+        ixy="5.3191E-10"
+        ixz="-3.8097E-11"
+        iyy="5.3414E-07"
         iyz="3.9566E-09"
-        izz="3.1605E-07" />
-    </inertial>
-    <visual>
-      <origin
-        xyz="0 0 0"
-        rpy="0 0 0" />
-      <geometry>
-        <mesh
-          filename="package://vizzy_test/meshes/r_thumb_4_link.STL" />
-      </geometry>
-      <material
-        name="">
-        <color
-          rgba="0.89804 0.91765 0.92941 1" />
-      </material>
-    </visual>
-    <collision>
-      <origin
-        xyz="0 0 0"
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
Commit message: Using the the kinect for obstacle avoidance. Some noisy measurements appear that need to be dealt with.

File: vizzy_description/robots/vizzy.urdf.xacro (robot description, xacro)
@@ -49,5 +49,5 @@
   </xacro:hokuyo_04lx_laser>
   <xacro:asus_camera name="camera" parent="waist_link">
-    <origin xyz="-0.195473 0.129382 0.0418749" rpy="1.61049 -0.0262743 2.58442"/>
+    <origin xyz="-0.08 0.16 0.02" rpy="${-M_PI/2} ${M_PI+3.5*(M_PI/180)} ${-7*(M_PI/180)}"/>
   </xacro:asus_camera>
   <!-- instantiate common ROS and Yarp plugins -->

Commit message: Added rear laser and tested in simulation

File: vizzy_description/robots/vizzy.urdf.xacro (robot description, xacro)
@@ -45,6 +45,9 @@
   </xacro:right_hand>
   <!-- instantiate hokuyo -->
-  <xacro:hokuyo_04lx_laser name="nav_hokuyo" parent="base" ros_topic="scan" update_rate="40" min_angle="${-(5 * M_PI)/12}" max_angle="${(5 * M_PI)/12}" max_range="30">
+  <xacro:hokuyo_04lx_laser name="nav_hokuyo" parent="base" mesh_file="package://vizzy_description/meshes/hokuyo_utm30lx/hokuyo_utm_30lx.dae" scale="1.0 1.0 1.0" ros_topic="scan" update_rate="40" min_angle="${-(5 * M_PI)/12}" max_angle="${(5 * M_PI)/12}" max_range="30">
     <origin xyz="${-0.025-0.060139} 0.001 ${-0.00394+0.14806}" rpy="0 0 ${M_PI}" />
+  </xacro:hokuyo_04lx_laser>
+<xacro:hokuyo_04lx_laser name="nav_hokuyo_urg" parent="base" mesh_file="package://vizzy_description/meshes/hokuyo.dae" ros_topic="scan_rear" scale="0.0254 0.0254 0.0254" update_rate="10" min_angle="${-(5 * M_PI)/12}" max_angle="${(5 * M_PI)/12}" max_range="4">
+    <origin xyz="${-0.025-0.060139+0.555} 0.001 ${-0.00394+0.14806}" rpy="0 0 0" />
   </xacro:hokuyo_04lx_laser>
   <xacro:asus_camera name="camera" parent="waist_link">

File: vizzy_description/urdf/sensors/hokuyo_04lx_laser.urdf.xacro (robot description, xacro)
@@ -5,5 +5,5 @@
       xmlns:xacro="http://ros.org/wiki/xacro">
   <xacro:include filename="$(find vizzy_description)/urdf/sensors/hokuyo_04lx_laser.gazebo.xacro" />
-  <xacro:macro name="hokuyo_04lx_laser" params="name parent *origin ros_topic update_rate min_angle max_angle max_range">
+  <xacro:macro name="hokuyo_04lx_laser" params="name parent *origin mesh_file scale ros_topic update_rate min_angle max_angle max_range">
     <joint name="${name}_joint" type="fixed">
       <insert_block name="origin" />
@@ -20,5 +20,5 @@
         <origin xyz="0 0 0.058" rpy="0 0 0" />
         <geometry>
-          <mesh filename="package://vizzy_description/meshes/hokuyo_utm30lx/hokuyo_utm_30lx.dae" />
+          <mesh filename="${mesh_file}" scale="${scale}" />
         </geometry>
       </visual>
