Commit message: fix torso and head description files
Simplified and structured the urdf of the head and torso
The geometric models are quite crude and can be refined later on
Reorganized meshes and removed redundant file

File: vizzy_description/robots/vizzy.urdf.xacro (robot description, xacro)
@@ -28,8 +28,8 @@
   <!-- instantiate base -->
   <xacro:base name="base"/>
-  <!-- instantiate torso -->
-  <xacro:torso name="torso"/>
-  <!-- instantiate head -->
-  <xacro:head name="head"/>
+  <!-- Instantiate the torso -->
+  <xacro:torso name="torso" parent="base_link"/>
+  <!-- Instantiate head -->
+  <xacro:head name="head" parent="waist_link"/>
   <!-- instantiate left arm -->
   <xacro:left_arm name="left_arm" parent="waist_link" sufix="l" reflect="1">

File: vizzy_description/urdf/head/head.gazebo.xacro (robot description, xacro)
@@ -1,15 +1,160 @@
 <?xml version="1.0"?>
-<robot xmlns:xacro="http://ros.org/wiki/xacro">
-  <xacro:macro name="head_gazebo">
-    <gazebo reference="neck_pan_link">
-    </gazebo>
-    <gazebo reference="neck_tilt_link">
-    </gazebo>
-    <gazebo reference="eyes_tilt_link">
-    </gazebo>
-    <gazebo reference="r_eye_version_link">
-    </gazebo>
-    <gazebo reference="l_eye_version_link">
-    </gazebo>
+<robot xmlns:sensor="http://playerstage.sourceforge.net/gazebo/xmlschema/#sensor"
+       xmlns:controller="http://playerstage.sourceforge.net/gazebo/xmlschema/#controller"
+       xmlns:interface="http://playerstage.sourceforge.net/gazebo/xmlschema/#interface"
+       xmlns:xacro="http://ros.org/wiki/xacro">
+  <!-- Load full inertial and collision model or a simplified model -->
+  <xacro:arg name="use_full_gazebo_model" default="false"/>
+  <!-- Neck pan -->
+  <xacro:macro name="vizzy_neck_pan_link_inertial">
+    <inertial>
+      <origin
+        xyz="0.0 0.0 -0.327"
+        rpy="0.0 0.0 ${-M_PI/2}"/>
+      <mass
+        value="0.223143594366725"/>
+      <inertia
+        ixx="0.000359045077001746"
+        ixy="3.18553746848725E-08"
+        ixz="-1.33740307483815E-05"
+        iyy="0.000368715218013968"
+        iyz="-4.52681716726929E-07"
+        izz="8.59048961267353E-05"/>
+    </inertial>
+  </xacro:macro>
+  <xacro:macro name="vizzy_neck_pan_link_collision">
+    <collision>
+      <xacro:if value="$(arg use_full_gazebo_model)">
+        <origin
+          xyz="0 0 -0.327"
+          rpy="0 0 ${-M_PI/2}"/>
+        <geometry>
+          <mesh
+            filename="package://vizzy_description/meshes/head/neck_pan.dae"/>
+        </geometry>
+      </xacro:if>
+      <xacro:unless value="$(arg use_full_gazebo_model)">
+        <origin
+          xyz="0 0 -0.37"
+          rpy="${-M_PI/2} 0 0"/>
+        <geometry>
+          <cylinder length="0.07" radius="0.02"/>
+        </geometry>
+      </xacro:unless>
+    </collision>
+  </xacro:macro>
+  <!-- Neck tilt -->
+  <xacro:macro name="vizzy_neck_tilt_link_inertial">
+    <inertial>
+      <origin
+        xyz="-0.027 -0.027 0.0"
+        rpy="${M_PI} ${M_PI} 0.0"/>
+      <mass
+        value="0.298440723794245"/>
+      <inertia
+        ixx="0.000294229505972848"
+        ixy="0.000128560854269813"
+        ixz="-4.90947453912942E-05"
+        iyy="0.000820635051594153"
+        iyz="-2.69741258639831E-05"
+        izz="0.000854308458364833"/>
+    </inertial>
+  </xacro:macro>
+  <xacro:macro name="vizzy_neck_tilt_link_collision">
+    <collision>
+      <xacro:if value="$(arg use_full_gazebo_model)">
+        <origin
+          xyz="-0.027 -0.027 0"
+          rpy="${M_PI} ${M_PI} 0"/>
+        <geometry>
+          <mesh
+            filename="package://vizzy_description/meshes/head/neck_tilt.dae"/>
+        </geometry>
+      </xacro:if>
+      <xacro:unless value="$(arg use_full_gazebo_model)">
+        <origin
+          xyz="-0.04 -0.05 0"
+          rpy="0 0 0"/>
+        <geometry>
+          <box size="0.1 0.03 0.05"/>
+        </geometry>
+      </xacro:unless>
+    </collision>
+  </xacro:macro>
+  <!-- Eyes tilt -->
+  <xacro:macro name="vizzy_eyes_tilt_link_inertial">
+    <inertial>
+      <origin
+        xyz="-0.007 -0.002 -0.002"
+        rpy="0 0 -1.2012"/>
+      <mass
+        value="0.229222715932625"/>
+      <inertia
+        ixx="0.00135649319186769"
+        ixy="-9.97604007968145E-07"
+        ixz="-4.83114556833996E-07"
+        iyy="0.0012860948285637"
+        iyz="-2.16886651449361E-06"
+        izz="0.000132176408116226"/>
+    </inertial>
+  </xacro:macro>
+  <xacro:macro name="vizzy_eyes_tilt_link_collision">
+    <collision>
+      <xacro:if value="$(arg use_full_gazebo_model)">
+        <origin
+          xyz="-0.007 -0.002 -0.002"
+          rpy="0 0 -1.2012"/>
+        <geometry>
+          <mesh
+            filename="package://vizzy_description/meshes/head/eyes_tilt.dae"/>
+        </geometry>
+      </xacro:if>
+      <xacro:unless value="$(arg use_full_gazebo_model)">
+        <origin
+          xyz="-0.007 -0.002 -0.002"
+          rpy="0 0 -1.2012"/>
+        <geometry>
+          <cylinder length="0.07" radius="0.02"/>
+        </geometry>
+      </xacro:unless>
+    </collision>
+  </xacro:macro>
+  <!-- Eyes -->
+  <xacro:macro name="vizzy_eye_link_inertial">
+    <inertial>
+      <origin
+        xyz="0 0 0"
+        rpy="0 0 ${M_PI/2}"/>
+      <mass
+        value="0.158520637460366"/>
+      <inertia
+        ixx="0.000147614970454271"
+        ixy="-1.56210652664748E-09"
+        ixz="8.85544640354075E-10"
+        iyy="0.000177840459249179"
+        iyz="8.21234366300574E-06"
+        izz="0.000144884726537935"/>
+      </inertial>
+  </xacro:macro>
+  <xacro:macro name="vizzy_eye_link_collision">
+    <collision>
+      <xacro:if value="$(arg use_full_gazebo_model)">
+        <origin
+          xyz="0 0 0"
+          rpy="0 0 ${M_PI/2}"/>
+        <geometry>
+          <mesh
+            filename="package://vizzy_description/meshes/head/eye.dae"/>
+        </geometry>
+      </xacro:if>
+      <xacro:unless value="$(arg use_full_gazebo_model)">
+        <origin
+          xyz="0 0 0"
+          rpy="0 0 ${M_PI/2}"/>
+        <geometry>
+          <sphere radius="0.055"/>
+        </geometry>
+      </xacro:unless>
+    </collision>
   </xacro:macro>
 </robot>

File: vizzy_description/urdf/head/head.urdf.xacro (robot description, xacro)
@@ -6,412 +6,295 @@
   <!-- Things that are needed only for Gazebo (not the physical robot).  These include
        sensor and controller plugin specifications -->
- <xacro:include filename="$(find vizzy_description)/urdf/head/head.gazebo.xacro" />
- <xacro:include filename="$(find vizzy_description)/urdf/head/head.transmission.xacro" />
-  <xacro:macro name="head" params="name">
-   <link name="neck_pan_link">
-    <inertial>
-      <origin
-        xyz="0.0 0.0 -0.327"
-        rpy="0.0 0.0 ${-M_PI/2}" />
-      <mass
-        value="0.223143594366725" />
-      <inertia
-        ixx="0.000359045077001746"
-        ixy="3.18553746848725E-08"
-        ixz="-1.33740307483815E-05"
-        iyy="0.000368715218013968"
-        iyz="-4.52681716726929E-07"
-        izz="8.59048961267353E-05" />
-    </inertial>
-    <visual>
-      <origin
-        xyz="0.0 0.0 -0.327"
-        rpy="0.0 0.0 ${-M_PI/2}" />
-      <geometry>
-        <mesh
-          filename="package://vizzy_description/meshes/M1.dae" />
-      </geometry>
-      <material
-        name="">
-        <color
-          rgba="0.898039215686275 0.917647058823529 0.929411764705882 1" />
-      </material>
-    </visual>
-    <collision>
-      <origin
-        xyz="0.0 0.0 -0.327"
-        rpy="0.0 0.0 ${-M_PI/2}" />
-      <geometry>
-        <mesh
-          filename="package://vizzy_description/meshes/M1.dae" />
-      </geometry>
-    </collision>
-  </link>
-  <joint
-    name="neck_pan_joint"
-    type="revolute">
-    <origin
-      xyz="0.0 0.0 0.0"
-      rpy="${M_PI/2.0} 0.0 0.0" />
-    <parent
-      link="waist_link" />
-    <child
-      link="neck_pan_link" />
-    <axis
-      xyz="0 0 1" />
-    <!--<limit lower="-0.925024504" upper="0.925024504" effort="10.0" velocity="5.0" />-->
-    <limit lower="-2.025024504" upper="2.025024504" effort="100.0" velocity="5.0" />
-    <dynamics damping="5.0" friction="10.0"/>
-  </joint>
-  <link
-    name="neck_tilt_link">
-    <inertial>
-      <origin
-        xyz="-0.027 -0.027 0.0"
-        rpy="${M_PI} ${M_PI} 0.0" />
-      <mass
-        value="0.298440723794245" />
-      <inertia
-        ixx="0.000294229505972848"
-        ixy="0.000128560854269813"
-        ixz="-4.90947453912942E-05"
-        iyy="0.000820635051594153"
-        iyz="-2.69741258639831E-05"
-        izz="0.000854308458364833" />
-    </inertial>
-    <visual>
-      <origin
-        xyz="-0.027 -0.027 0.0"
-        rpy="${M_PI} ${M_PI} 0.0" />
-      <geometry>
-        <mesh
-          filename="package://vizzy_description/meshes/M2.dae" />
-      </geometry>
-      <material
-        name="">
-        <color
-          rgba="0.752941176470588 0.752941176470588 0.752941176470588 1" />
-      </material>
-    </visual>
-    <collision>
-      <origin
-        xyz="-0.027 -0.027 0.0"
-        rpy="${M_PI} ${M_PI} 0.0" />
-      <geometry>
-        <mesh
-          filename="package://vizzy_description/meshes/M2.dae" />
-      </geometry>
-    </collision>
-  </link>
-  <joint
-    name="neck_tilt_joint"
-    type="revolute">
-    <origin
-      xyz="0.0 0.0 -0.370"
-      rpy="${M_PI/2.0} 0.0 0.0" />
-    <parent
-      link="neck_pan_link" />
-    <child
-      link="neck_tilt_link" />
-    <axis
-      xyz="0 0 1" />
-    <!--<limit lower="-0.314159265" upper="0.645771823" effort="100.0" velocity="5.0" />-->
-    <dynamics damping="0.0" friction="5.0"/>
-    <limit lower="-2.014159265" upper="2.45771823" effort="100.0" velocity="5.0" />
-  </joint>
-  <link
-    name="eyes_tilt_link">
-    <inertial>
-      <origin
-        xyz="-0.007 -0.002 -0.002"
-        rpy="0.0 0.0 -1.2012" />
-      <mass
-        value="0.229222715932625" />
-      <inertia
-        ixx="0.00135649319186769"
-        ixy="-9.97604007968145E-07"
-        ixz="-4.83114556833996E-07"
-        iyy="0.0012860948285637"
-        iyz="-2.16886651449361E-06"
-        izz="0.000132176408116226" />
-    </inertial>
-    <visual>
-      <origin
-        xyz="-0.007 -0.002 -0.002"
-        rpy="0.0 0.0 -1.2012" />
-      <geometry>
-        <mesh
-          filename="package://vizzy_description/meshes/M3.dae" />
-      </geometry>
-      <material
-        name="">
-        <color
-          rgba="0 0 0 1" />
-      </material>
-    </visual>
-    <collision>
-      <origin
-        xyz="-0.007 -0.002 -0.002"
-        rpy="0.0 0.0 -1.2012" />
-      <geometry>
-        <mesh
-          filename="package://vizzy_description/meshes/M3.dae" />
-      </geometry>
-    </collision>
-  </link>
-  <joint
-    name="eyes_tilt_joint"
-    type="revolute">
-    <origin
-      xyz="-0.12379 -0.04755 0.0"
-      rpy="${M_PI} 0.0 -2.77199351787335" />
-    <parent
-      link="neck_tilt_link" />
-    <child
-      link="eyes_tilt_link" />
-    <axis
-      xyz="0 0 1" />
-    <limit lower="-0.663225116" upper="0.663225116" effort="10.0" velocity="5.0" />
-    <dynamics damping="0.0" friction="5.0"/>
-  </joint>
-  <!-- eyes center virtual link and joint -->
-  <link name="eyes_center_link">
-		<inertial>
-			<origin xyz="0 0 0"
-      rpy="0.0 0.0 0" />
-			<mass value="0.1"/>
-			<inertia
-				ixx="0.001" ixy="0.0" ixz="0.0"
-				iyy="0.001" iyz="0.0" izz="0.001"/>
-		</inertial>
-  </link>
-  <joint name="eyes_center_joint" type="fixed">
-    <origin xyz="0 0 0"       rpy="${M_PI/2.0} 0.0 0.369599135716446" />
-    <parent link="eyes_tilt_link" />
-    <child link="eyes_center_link" />
-    <axis  xyz="0 0 1" />
-    <limit lower="-0.698131" upper="0.698131" effort="10.0" velocity="5.0" />
-  </joint>
-  <!-- eyes center visual virtual link and joint -->
-  <link name="eyes_center_vision_link">
-		<inertial>
-			<origin xyz="0 0 0"
-      rpy="0.0 0.0 0" />
-			<mass value="0.1"/>
-			<inertia
-				ixx="0.001" ixy="0.0" ixz="0.0"
-				iyy="0.001" iyz="0.0" izz="0.001"/>
-		</inertial>
-  </link>
-  <joint name="eyes_center_vision_joint" type="fixed">
-    <origin xyz="0 0 0"       rpy="${-M_PI/2} 0.0 ${-M_PI/2}" />
-    <parent link="eyes_center_link" />
-    <child link="eyes_center_vision_link" />
-  </joint>
-  <!-- eyes -->
-  <link name="l_eye_link">
-  <inertial>
-      <origin
-        xyz="0.0 0.0 0.0"
-        rpy="0 0 ${M_PI/2}" />
-      <mass
-        value="0.158520637460366" />
-      <inertia
-        ixx="0.000147614970454271"
-        ixy="-1.56210652664748E-09"
-        ixz="8.85544640354075E-10"
-        iyy="0.000177840459249179"
-        iyz="8.21234366300574E-06"
-        izz="0.000144884726537935" />
-    </inertial>
-    <visual>
-      <origin
-        xyz="0.0 0.0 0.0"
-        rpy="0.0 0.0 ${M_PI/2}" />
-      <geometry>
-        <mesh
-          filename="package://vizzy_description/meshes/M4.dae" />
-      </geometry>
-      <material
-        name="">
-        <color
-          rgba="0 0 0 1" />
-      </material>
-    </visual>
-    <collision>
- 	<origin
-        xyz="0.0 0 0.0"
-        rpy="0 0 ${M_PI/2}" />
-      <geometry>
-        <mesh
-          filename="package://vizzy_description/meshes/M4.dae" />
-      </geometry>
-    </collision>
-  </link>
-  <joint
-    name="l_eye_joint"
-    type="revolute">
-    <origin
-      xyz="0.0 0.102 0.0"
-      rpy="0 ${M_PI} 0" />
-    <parent
-      link="eyes_center_link" />
-    <child
-      link="l_eye_link" />
-    <axis
-      xyz="0 0 1" />
-    <limit
-			lower="-1.0"
-			upper="1.0"
-      effort="1000.0"
-      velocity="5.0" />
-    <dynamics damping="0.0" friction="5.0"/>
-  </joint>
-  <link name="r_eye_link">
-  <inertial>
-      <origin
-        xyz="0.0 0.0 0.0"
-        rpy="0.0 0.0 ${M_PI/2}" />
-      <mass
-        value="0.158520637460366" />
-      <inertia
-        ixx="0.000147614970454271"
-        ixy="-1.56210652664748E-09"
-        ixz="8.85544640354075E-10"
-        iyy="0.000177840459249179"
-        iyz="8.21234366300574E-06"
-        izz="0.000144884726537935" />
-    </inertial>
-    <visual>
-      <origin
-        xyz="0.0 0.0 0.0"
-        rpy="0.0 0.0 ${M_PI/2}" />
-      <geometry>
-        <mesh
-          filename="package://vizzy_description/meshes/M4.dae" />
-      </geometry>
-      <material
-        name="">
-        <color
-          rgba="0 0 0 1" />
-      </material>
-    </visual>
-    <collision>
-      <origin
-        xyz="0.0 0.0 0.0"
-        rpy="0.0 0.0 ${M_PI/2}" />
-      <geometry>
-        <mesh
-          filename="package://vizzy_description/meshes/M4.dae" />
-      </geometry>
-    </collision>
-  </link>
-  <joint
-    name="r_eye_joint"
-    type="revolute">
-    <origin
-      xyz="0.0 -0.102 0.0"
-      rpy="0 ${M_PI} 0" />
-    <parent
-      link="eyes_center_link" />
-    <child
-      link="r_eye_link" />
-    <axis
-      xyz="0 0 1" />
-    <limit
-			lower="-1.0"
-			upper="1.0"
-      effort="1000.0"
-      velocity="5.0"/>
-    <dynamics damping="0.0" friction="5.0"/>
-  </joint>
-  <!-- cameras -->
-  <link name="r_camera_link">
-   <visual>
-      <origin xyz="0 0 0" rpy="0 0 0" />
-      <geometry>
-        <box size="0.001 0.001 0.001" />
-      </geometry>
-    </visual>
-  </link>
-  <joint name="r_camera_joint" type="fixed">
-    <origin xyz="-0.0275 0.0 0.0" rpy="0.0 ${M_PI} 0.0" />
-    <parent link="r_eye_link"/>
-    <child link="r_camera_link" />
-  </joint>
-  <link name="r_camera_vision_link">
-   <visual>
-      <origin xyz="0 0 0" rpy="0 0 0" />
-      <geometry>
-        <box size="0.001 0.001 0.001" />
-      </geometry>
-    </visual>
-  </link>
-  <joint name="r_camera_vision_joint" type="fixed">
-    <origin xyz="0.0 0.0 0.0" rpy="${M_PI/2} 0.0 ${-M_PI/2}" />
-    <parent link="r_eye_link"/>
-    <child link="r_camera_vision_link" />
-  </joint>
-  <link name="l_camera_link">
-   <visual>
-      <origin xyz="0 0 0" rpy="0 0 0" />
-      <geometry>
-        <box size="0.001 0.001 0.001" />
-      </geometry>
-    </visual>
-  </link>
-  <joint name="l_camera_joint" type="fixed">
-    <origin xyz="-0.0275 0.0 0.0" rpy="0 ${M_PI} 0" />
-    <parent link="l_eye_link"/>
-    <child link="l_camera_link" />
-  </joint>
-  <link name="l_camera_vision_link">
-   <visual>
-      <origin xyz="0 0 0" rpy="0 0 0" />
-      <geometry>
-        <box size="0.001 0.001 0.001" />
-      </geometry>
-    </visual>
-  </link>
-  <joint name="l_camera_vision_joint" type="fixed">
-    <origin xyz="0.0 0.0 0.0" rpy="${M_PI/2} 0.0 ${-M_PI/2}" />
-    <parent link="l_eye_link"/>
-    <child link="l_camera_vision_link" />
-  </joint>
-  <!-- ego frame -->
-  <link name="ego_frame">
-    <inertial>
-      <origin xyz="0 0 0" rpy="0.0 0.0 0" />
-      <mass value="0.001"/>
-      <inertia
-        ixx="0.001" ixy="0.0" ixz="0.0"
-        iyy="0.001" iyz="0.0" izz="0.001"/>
-    </inertial>
-  </link>
-  <joint name="ego_joint" type="fixed">
-    <origin
-      xyz="0.0 0.370 0.0"
-      rpy="0.0 ${M_PI/2.0} ${M_PI}" />
-    <parent link="waist_link"/>
-    <child link="ego_frame" />
-  </joint>
-  <link name="head_origin_frame">
-    <inertial>
-      <origin xyz="0 0 0" rpy="0.0 0.0 0" />
-      <mass value="0.001"/>
-      <inertia
-        ixx="0.001" ixy="0.0" ixz="0.0"
-        iyy="0.001" iyz="0.0" izz="0.001"/>
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
File: vizzy_description/urdf/torso/torso.gazebo.xacro (robot description, xacro)
@@ -6,11 +6,11 @@
       <mu2>0.2</mu2>
     </gazebo>
- 		<gazebo reference="waist_joint">
-			<kd value="1.0" />
-			<kp value="1000000.0" />
-			<stopCfm value="1000000.0" />
-			<fudgeFactor value="1.0" />
-			<provideFeedback value="true"/>
-		</gazebo>
+    <gazebo reference="waist_joint">
+      <kd value="1.0" />
+      <kp value="1000000.0" />
+      <stopCfm value="1000000.0" />
+      <fudgeFactor value="1.0" />
+      <provideFeedback value="true"/>
+    </gazebo>
   </xacro:macro>
 </robot>
