Commit message: fix arm controllers and description
Fixes #62
Fixes #60

Changed the arms controllers to EffortJointInterface which fixed buggy behaviour
Collapsed both arms urdf into a single set of files for better readibility and less redundancy
Renamed and reorganised mesh files
Refined camera description and mesh
Fixed incorrect camera gazebo plugin configuration
Added several parameters to make the main simulation launcher more modular and documented them accordingly.
Fixed deprecated syntax in xacro processing
This commit concludes the model simplification process and results in upgraded gazebo performance

File: vizzy_description/robots/vizzy.urdf.xacro (robot description, xacro)
@@ -1,30 +1,35 @@
 <?xml version="1.0"?>
 <robot  name="vizzy" xmlns:xacro="http://ros.org/wiki/xacro" >
+  <!-- Load Yarp plugins for real robot execution -->
   <xacro:arg name="use_yarp" default="false"/>
-  <!-- The following include files set up definitions of parts of the robot body  -->
-  <!-- misc common stuff -->
-  <xacro:include filename="$(find vizzy_description)/urdf/common.urdf.xacro" />
-  <!-- sensors -->
-  <xacro:include filename="$(find vizzy_description)/urdf/sensors/hokuyo_04lx_laser.urdf.xacro" />
-  <!-- Asus Xiton Live Pro -->
+  <!-- Load a fully detailed hand model with properly modeled links and joints -->
+  <xacro:arg name="use_full_hand_model" default="false"/>
+  <!-- Disable laser sensors -->
+  <xacro:arg name="disable_laser" default="false"/>
+  <!-- Disable depth camera -->
+  <xacro:arg name="disable_3d_sensor" default="false"/>
+  <!-- Includes -->
+  <!-- Misc common stuff such as constant definitions -->
+  <xacro:include filename="$(find vizzy_description)/urdf/common.urdf.xacro"/>
+  <!-- Sensors -->
+  <!-- Hokuyo URG-04LX laser scanner -->
+  <xacro:include filename="$(find vizzy_description)/urdf/sensors/hokuyo_04lx_laser.urdf.xacro"/>
+  <!-- TODO: Update Asus Xiton Live Pro -->
   <xacro:include filename="$(find vizzy_description)/urdf/sensors/asus_camera.urdf.xacro" />
-  <!-- base -->
+  <!-- Robot body -->
+  <!-- Base -->
   <xacro:include filename="$(find vizzy_description)/urdf/base/base.urdf.xacro" />
-  <!-- torso -->
+  <!-- Torso -->
   <xacro:include filename="$(find vizzy_description)/urdf/torso/torso.urdf.xacro" />
-  <!-- head -->
+  <!-- Head -->
  <xacro:include filename="$(find vizzy_description)/urdf/head/head.urdf.xacro"/>
-  <!-- left arm -->
-  <xacro:include filename="$(find vizzy_description)/urdf/arm/left_arm.urdf.xacro" />
-  <!-- right arm -->
-  <xacro:include filename="$(find vizzy_description)/urdf/arm/right_arm.urdf.xacro" />
-  <!-- right hand -->
-  <xacro:include filename="$(find vizzy_description)/urdf/hand/right_hand.urdf.xacro" />
-  <!-- The following include files contain gazebo plugins -->
+  <!-- Arms -->
+  <xacro:include filename="$(find vizzy_description)/urdf/arm/arm.urdf.xacro" />
+  <!-- Gazebo plugins -->
   <!-- ROS -->
   <xacro:include filename="$(find vizzy_description)/plugins/ros.gazebo.xacro" />
   <!-- Yarp -->
   <xacro:include filename="$(find vizzy_description)/plugins/yarp.gazebo.xacro" />
-  <!-- instantiate base -->
+  <!-- Instantiate base -->
   <xacro:base name="base"/>
   <!-- Instantiate the torso -->
@@ -32,40 +37,53 @@
   <!-- Instantiate head -->
   <xacro:head name="head" parent="waist_link"/>
-  <!-- instantiate left arm -->
-  <xacro:left_arm name="left_arm" parent="waist_link" sufix="l" reflect="1">
-    <origin xyz="-0.01707 0.0 0.38145" rpy="0.0 0.0 0.0" />
-  </xacro:left_arm>
-  <!-- instantiate right arm -->
-  <xacro:right_arm name="right_arm" parent="waist_link" sufix="r" reflect="1">
-    <origin xyz="-0.01707 0.0 0.38145" rpy="0.0 0.0 0.0" />
-  </xacro:right_arm>
-  <!-- instantiate right hand -->
-  <xacro:right_hand name="right_hand" parent="r_wrist_flection_link" sufix="r" reflect="1">
-    <origin xyz="-0.01707 0.0 0.38145" rpy="0.0 0.0 0.0" />
-  </xacro:right_hand>
-  <!-- instantiate hokuyo -->
-  <xacro:hokuyo_04lx_laser name="nav_hokuyo" parent="base" mesh_file="package://vizzy_description/meshes/hokuyo_utm30lx/hokuyo_utm_30lx.dae" scale="1.0 1.0 1.0" ros_topic="scan" update_rate="40" min_angle="${-(5 * M_PI)/12}" max_angle="${(5 * M_PI)/12}" max_range="30">
-    <origin xyz="${-0.025-0.060139} 0.001 ${-0.00394+0.14806}" rpy="0 0 ${M_PI}" />
-  </xacro:hokuyo_04lx_laser>
-<xacro:hokuyo_04lx_laser name="nav_hokuyo_rear" parent="base" mesh_file="package://vizzy_description/meshes/hokuyo.dae" ros_topic="scan_rear" scale="0.0254 0.0254 0.0254" update_rate="10" min_angle="${-(5 * M_PI)/12}" max_angle="${(5 * M_PI)/12}" max_range="4">
-    <origin xyz="${-0.025-0.060139+0.555} 0.001 ${-0.00394+0.14806}" rpy="0 0 0" />
-  </xacro:hokuyo_04lx_laser>
-  <xacro:asus_camera name="camera" parent="waist_link">
-    <origin xyz="-0.08 0.16 0.02" rpy="${-M_PI/2} ${M_PI+3.5*(M_PI/180)} ${-7*(M_PI/180)}"/>
-  </xacro:asus_camera>
-  <!-- instantiate common ROS and Yarp plugins -->
+  <!-- Instantiate arms -->
+  <xacro:arm name="left_arm" parent="waist_link"/>
+  <xacro:arm name="right_arm" parent="waist_link"/>
+  <!-- Instantiate hokuyo laser sensors -->
+  <xacro:unless value="$(arg disable_laser)">
+    <!-- Front laser sensor -->
+    <xacro:hokuyo_04lx_laser name="nav_hokuyo" parent="base"
+      mesh_file="package://vizzy_description/meshes/hokuyo_utm30lx/hokuyo_utm_30lx.dae"
+      scale="1.0 1.0 1.0"
+      ros_topic="scan"
+      update_rate="40"
+      min_angle="${-(5 * M_PI)/12}"
+      max_angle="${(5 * M_PI)/12}"
+      max_range="30">
+      <origin xyz="${-0.025-0.060139} 0.001 ${-0.00394+0.14806}" rpy="0 0 ${M_PI}"/>
+    </xacro:hokuyo_04lx_laser>
+    <!-- Rear laser sensor -->
+    <xacro:hokuyo_04lx_laser name="nav_hokuyo_rear" parent="base"
+      mesh_file="package://vizzy_description/meshes/hokuyo.dae"
+      scale="0.0254 0.0254 0.0254"
+      ros_topic="scan_rear"
+      update_rate="10"
+      min_angle="${-(5 * M_PI)/12}"
+      max_angle="${(5 * M_PI)/12}"
+      max_range="4">
+      <origin xyz="${-0.025-0.060139+0.555} 0.001 ${-0.00394+0.14806}" rpy="0 0 0"/>
+    </xacro:hokuyo_04lx_laser>
+  </xacro:unless>
+  <!-- Instantiate depth camera -->
+  <xacro:unless value="$(arg disable_3d_sensor)">
+    <xacro:sensor_asus_xtion_pro name="asus_camera" parent="waist_link"
+      ros_topic="asus_camera">
+      <origin xyz="-0.08 0.16 0.02" rpy="${-M_PI/2} ${M_PI} ${-7*(M_PI/180)}"/>
+    </xacro:sensor_asus_xtion_pro>
+  </xacro:unless>
+  <!-- Instantiate plugins common to ROS and Yarp -->
   <xacro:ros_differential_drive_gazebo/>
   <xacro:camera_plugin name="l_camera" prefix="l"/>
   <xacro:camera_plugin name="r_camera" prefix="r"/>
-  <!-- instantiate Yarp plugins -->
-	<xacro:if value="$(arg use_yarp)">
-		<xacro:torso_gazebo_control/>
-		<xacro:head_gazebo_control/>
-		<xacro:left_arm_gazebo_control/>
-		<xacro:right_arm_gazebo_control/>
-	</xacro:if>
-  <!-- instantiate ROS plugins -->
+  <!-- Instantiate Yarp plugins -->
+  <xacro:if value="$(arg use_yarp)">
+    <xacro:torso_gazebo_control/>
+    <xacro:head_gazebo_control/>
+    <xacro:left_arm_gazebo_control/>
+    <xacro:right_arm_gazebo_control/>
+  </xacro:if>
+  <!-- Instantiate ROS plugins -->
   <xacro:unless value="$(arg use_yarp)">
-		<xacro:ros_control_gazebo/>
+    <xacro:ros_control_gazebo/>
   </xacro:unless>
 </robot>

File: vizzy_description/urdf/arm/arm.urdf.xacro (robot description, xacro)
@@ -4,448 +4,324 @@
        xmlns:interface="http://playerstage.sourceforge.net/gazebo/xmlschema/#interface"
        xmlns:xacro="http://ros.org/wiki/xacro">
- <xacro:macro name="arm" params="sufix reflect *origin">
-  <link
-    name="M0${sufix}">
-    <inertial>
-      <origin
-        xyz="0 0 ${-reflect*0.0619999999999821}"
-        rpy="0.0 0.0 ${-reflect*3.1416}" />
-      <mass
-        value="0.328838093974495" />
-      <inertia
-        ixx="0.00123108428695023"
-        ixy="-7.89159441144304E-11"
-        ixz="6.34904994947113E-10"
-        iyy="0.000919898935947314"
-        iyz="7.50425183645029E-05"
-        izz="0.000480033534091429" />
-    </inertial>
-    <visual>
-      <origin
-        xyz="0 0 ${-reflect*0.0619999999999821}"
-        rpy="0.0 0.0 ${-reflect*3.1416}" />
-      <geometry>
-        <mesh
-          filename="package://vizzy_description/meshes/M0${sufix}.dae" />
-      </geometry>
-      <material
-        name="">
-        <color
-          rgba="0.898039215686275 0.917647058823529 0.929411764705882 1" />
-      </material>
-    </visual>
-    <collision>
-      <origin
-        xyz="0 0 ${-reflect*0.0619999999999821}"
-        rpy="0.0 0.0 ${-reflect*3.1416}" />
-      <geometry>
-        <mesh
-          filename="package://vizzy_description/meshes/M0${sufix}.dae" />
-      </geometry>
-    </collision>
-  </link>
-  <joint
-    name="M0${sufix}"
-    type="revolute">
-    <insert_block name="origin" />
-    <parent
-      link="M0" />
-    <child
-      link="M0${sufix}" />
-    <axis
-      xyz="0 0 1" />
-    <limit lower="-0.314159265" upper="0.314159265" effort="10" velocity="3" />
-  </joint>
-  <link
-    name="M1${sufix}">
-    <inertial>
-      <origin
-        xyz="0 0 ${reflect*0.0479999999999997}"
-        rpy="0 0 ${-reflect*1.0547}" />
-      <mass
-        value="0.329707501986262" />
-      <inertia
-        ixx="0.00116793344879787"
-        ixy="0.000134890277431864"
-        ixz="-3.78918978637635E-05"
-        iyy="0.0010123206932222"
-        iyz="-6.56607930808342E-05"
-        izz="0.000480378945367471" />
-    </inertial>
-    <visual>
-      <origin
-        xyz="0 0 0.0479999999999997"
-        rpy="0 0 -1.0547" />
-      <geometry>
-        <mesh
-          filename="package://vizzy_description/meshes/M1${sufix}.dae" />
-      </geometry>
-      <material
-        name="">
-        <color
-          rgba="0.898039215686275 0.917647058823529 0.929411764705882 1" />
-      </material>
-    </visual>
-    <collision>
-      <origin
-        xyz="0 0 0.0479999999999997"
-        rpy="0 0 -1.0547" />
-      <geometry>
-        <mesh
-          filename="package://vizzy_description/meshes/M1${sufix}.dae" />
-      </geometry>
-    </collision>
-  </link>
-  <joint
-    name="M1${sufix}"
-    type="revolute">
-    <origin
-      xyz="0 0.0 ${-reflect*0.212}"
-      rpy="-1.5708 0.0 0.0" />
-    <parent
-      link="M0${sufix}" />
-    <child
-      link="M1${sufix}" />
-    <axis
-      xyz="0 0 1" />
-    <limit lower="-1.30899694" upper="2.35619449" effort="10" velocity="3" />
-  </joint>
-  <link
-    name="M2${sufix}">
-    <inertial>
-      <origin
-        xyz="0 0 0.0479999999999997"
-        rpy="0 0 -4.3633" />
-      <mass
-        value="0.337952134412867" />
-      <inertia
-        ixx="0.000722844157573501"
-        ixy="4.62401523525089E-05"
-        ixz="1.45397456168781E-06"
-        iyy="0.000316566987264746"
-        iyz="1.40155768711965E-05"
-        izz="0.000577759873964217" />
-    </inertial>
-    <visual>
-      <origin
-        xyz="0 0 0.0479999999999997"
-        rpy="0 0 -4.3633" />
-      <geometry>
-        <mesh
-          filename="package://vizzy_description/meshes/M2${sufix}.dae" />
-      </geometry>
-      <material
-        name="">
-        <color
-          rgba="0.898039215686275 0.917647058823529 0.929411764705882 1" />
-      </material>
-    </visual>
-    <collision>
-      <origin
-        xyz="0 0 0.0479999999999997"
-        rpy="0 0 -4.3633" />
-      <geometry>
-        <mesh
-          filename="package://vizzy_description/meshes/M2${sufix}.dae" />
-      </geometry>
-    </collision>
-  </link>
-  <joint
-    name="M2${sufix}"
-    type="revolute">
-    <origin
-      xyz="0.0 0.0 ${-reflect*0.10256}"
-      rpy="1.5708 0.0 1.5708" />
-    <parent
-      link="M1${sufix}" />
-    <child
-      link="M2${sufix}" />
-    <axis
-      xyz="0 0 1" />
-    <limit lower="0" upper="1.30899694" effort="10" velocity="3" />
-  </joint>
-  <link
-    name="M3${sufix}">
-    <inertial>
-      <origin
-        xyz="0 0 -0.0519999999999999"
-        rpy="0 0 -1.5708" />
-      <mass
-        value="0.302328099651438" />
-      <inertia
-        ixx="0.00061524641225989"
-        ixy="4.12484077822449E-06"
-        ixz="6.13276820445825E-05"
-        iyy="0.000574848729857274"
-        iyz="-2.49114687077784E-05"
-        izz="0.000240227009768201" />
-    </inertial>
-    <visual>
-      <origin
-        xyz="0 0 -0.0519999999999999"
-        rpy="0 0 -1.5708" />
-      <geometry>
-        <mesh
-          filename="package://vizzy_description/meshes/M3${sufix}.dae" />
-      </geometry>
-      <material
-        name="">
-        <color
-          rgba="0.898039215686275 0.917647058823529 0.929411764705882 1" />
-      </material>
-    </visual>
-    <collision>
-      <origin
-        xyz="0 0 -0.0519999999999999"
-        rpy="0 0 -1.5708" />
-      <geometry>
-        <mesh
-          filename="package://vizzy_description/meshes/M3${sufix}.dae" />
-      </geometry>
-    </collision>
-  </link>
-  <joint
-    name="M3${sufix}"
-    type="revolute">
-    <origin
-      xyz="0.0 0.0 0.0"
-      rpy="-1.5708 0.0 -1.2217" />
-    <parent
-      link="M2${sufix}" />
-    <child
-      link="M3${sufix}" />
-    <axis
-      xyz="0 0 1" />
-    <limit lower="-1.48352986" upper="1.48352986" effort="10" velocity="3" />
-  </joint>
-  <link
-    name="M4${sufix}">
-    <inertial>
-      <origin
-        xyz="0 0 -0.0229999999999996"
-        rpy="0 3.1416 0" />
-      <mass
-        value="0.224019872188573" />
-      <inertia
-        ixx="0.000224266883987209"
-        ixy="-7.91977708288826E-06"
-        ixz="-2.45971183993369E-07"
-        iyy="9.89759646705347E-05"
-        iyz="9.59757272005961E-06"
-        izz="0.000213841891548227" />
-    </inertial>
-    <visual>
-      <origin
-        xyz="0 0 -0.0229999999999996"
-        rpy="0 3.1416 0" />
-      <geometry>
-        <mesh
-          filename="package://vizzy_description/meshes/M4${sufix}.dae" />
-      </geometry>
-      <material
-        name="">
-        <color
-          rgba="0.898039215686275 0.917647058823529 0.929411764705882 1" />
-      </material>
-    </visual>
-    <collision>
-      <origin
-        xyz="0 0 -0.0229999999999996"
-        rpy="0 3.1416 0" />
-      <geometry>
-        <mesh
-          filename="package://vizzy_description/meshes/M4${sufix}.dae" />
-      </geometry>
-    </collision>
-  </link>
-  <joint
-    name="M4${sufix}"
-    type="revolute">
-    <origin
-      xyz="0.0 0.0 ${-reflect*0.16296}"
-      rpy="-1.5708 0.0 1.5708" />
-    <parent
-      link="M3${sufix}" />
-    <child
-      link="M4${sufix}" />
-    <axis
-      xyz="0 0 1" />
-    <limit lower="0" upper="1.91986218" effort="10" velocity="3" />
-  </joint>
-  <link
-    name="M5${sufix}">
-    <inertial>
-      <origin
-        xyz="0 0 -0.0525000000000014"
-        rpy="0 0 1.5708" />
-      <mass
-        value="0.192525480880953" />
-      <inertia
-        ixx="0.000215803121531384"
-        ixy="6.01824209118801E-08"
-        ixz="-9.78525879865635E-06"
-        iyy="0.000229047941469006"
-        iyz="-3.21836442544262E-07"
-        izz="0.000102658857339667" />
-    </inertial>
-    <visual>
-      <origin
-        xyz="0 0 -0.0525000000000014"
-        rpy="0 0 1.5708" />
-      <geometry>
-        <mesh
-          filename="package://vizzy_description/meshes/M5${sufix}.dae" />
-      </geometry>
-      <material
-        name="">
-        <color
-          rgba="0.898039215686275 0.917647058823529 0.929411764705882 1" />
-      </material>
-    </visual>
-    <collision>
-      <origin
-        xyz="0 0 -0.0525000000000014"
-        rpy="0 0 1.5708" />
-      <geometry>
-        <mesh
-          filename="package://vizzy_description/meshes/M5${sufix}.dae" />
-      </geometry>
-    </collision>
-  </link>
-  <joint
-    name="M5${sufix}"
-    type="revolute">
-    <origin
-      xyz="0.0 0.0 0.0"
-      rpy="1.5708 0.0 0.0" />
-    <parent
-      link="M4${sufix}" />
-    <child
-      link="M5${sufix}" />
-    <axis
-      xyz="0 0 1" />
-    <limit lower="-1.48352986" upper="1.48352986" effort="10" velocity="3" />
-  </joint>
-  <link
-    name="M6${sufix}">
-    <inertial>
-      <origin
-        xyz="0 0.0682999999999999 0.0240000000000001"
-        rpy="1.5708 0 2.3562" />
-      <mass
-        value="0.151302636921624" />
-      <inertia
-        ixx="0.000116373512947626"
-        ixy="1.31009871908069E-05"
-        ixz="6.69703789973942E-05"
-        iyy="0.00020031628400595"
-        iyz="1.00268924727662E-05"
-        izz="0.000162164313365602" />
-    </inertial>
-    <visual>
-      <origin
-        xyz="0 0.0682999999999999 0.0240000000000001"
-        rpy="1.5708 0 2.3562" />
-      <geometry>
-        <mesh
-          filename="package://vizzy_description/meshes/M6${sufix}.dae" />
-      </geometry>
-      <material
-        name="">
-        <color
-          rgba="0.898039215686275 0.917647058823529 0.929411764705882 1" />
-      </material>
-    </visual>
-    <collision>
-      <origin
-        xyz="0 0.0682999999999999 0.0240000000000001"
-        rpy="1.5708 0 2.3562" />
-      <geometry>
-        <mesh
-          filename="package://vizzy_description/meshes/M6${sufix}.dae" />
-      </geometry>
-    </collision>
-  </link>
-  <joint
-    name="M6${sufix}"
-    type="revolute">
-    <origin
-      xyz="0.0 0.0 ${-reflect*0.18925}"
-      rpy="1.5708 0.0 0.0" />
-    <parent
-      link="M5${sufix}" />
-    <child
-      link="M6${sufix}" />
-    <axis
-      xyz="0 0 1" />
-    <limit lower="-0.610865238" upper="0.610865238" effort="10" velocity="3" />
-  </joint>
-  <link
-    name="M7${sufix}">
-    <inertial>
-      <origin
-        xyz="0 0 -0.0075"
-        rpy="0 3.1416 -1.5708" />
-      <mass
-        value="0.263177712190575" />
-      <inertia
-        ixx="0.00141536691437145"
-        ixy="-5.47006881402205E-06"
-        ixz="4.93141952833896E-05"
-        iyy="0.000423837541639676"
-        iyz="0.000132116163317958"
-        izz="0.0010337584021873" />
-    </inertial>
-    <visual>
-      <origin
-        xyz="0 0 -0.0075"
-        rpy="0 3.1416 -1.5708" />
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