Commit message: fix arm controllers and description
Fixes #62
Fixes #60

Changed the arms controllers to EffortJointInterface which fixed buggy behaviour
Collapsed both arms urdf into a single set of files for better readibility and less redundancy
Renamed and reorganised mesh files
Refined camera description and mesh
Fixed incorrect camera gazebo plugin configuration
Added several parameters to make the main simulation launcher more modular and documented them accordingly.
Fixed deprecated syntax in xacro processing
This commit concludes the model simplification process and results in upgraded gazebo performance

File: vizzy_description/urdf/sensors/asus_camera.urdf.xacro (robot description, xacro)
@@ -1,92 +1,74 @@
 <?xml version="1.0"?>
-<robot xmlns:xacro="http://ros.org/wiki/xacro">
-<xacro:property name="M_PI" value="3.1415926535897931" />
-<xacro:macro name="asus_camera_model" params="name parent *origin">
-<joint name="${name}_joint" type="fixed">
-	<xacro:insert_block name="origin" />
-	<parent link="${parent}"/>
-	<child link="${name}_link"/>
-</joint>
-<link name="${name}_link">
-	<inertial>
-	<mass value="0.200" />
-	<origin xyz="0 0 0" rpy="0 0 0" />
-	<inertia ixx="5.8083e-4" ixy="0" ixz="0" iyy="3.0833e-5" iyz="0" izz="5.9083e-4" />
-	</inertial>
-	<visual>
-		<origin xyz="0 0 0" rpy="0 0 0" />
-		<geometry>
-			<mesh filename="package://vizzy_description/meshes/asus_camera/asus_camera_simple.dae"/>
-		</geometry>
-	</visual>
-	<collision>
-		<origin xyz="0 0 0" rpy="0 0 0" />
-		<geometry>
-			<box size="0.035 0.185 0.025"/>
-		</geometry>
-	</collision>
-</link>
-<!--<joint name="${name}_depth_joint" type="fixed">
-<origin xyz="0.0 0.049 0.0" rpy="0 0 0" />
-<parent link="${name}_link" />
-<child link="${name}_depth_frame"/>
-</joint>
-<link name="${name}_depth_frame"/>
-<joint name="${name}_depth_optical_joint" type="fixed">
-<origin xyz="0 0 0" rpy="${-M_PI/2} 0.0 ${-M_PI/2}" />
-<parent link="${name}_depth_frame" />
-<child link="${name}_depth_optical_frame"/>
-</joint>
-<link name="${name}_depth_optical_frame"/>
-<joint name="${name}_rgb_joint" type="fixed">
-<origin xyz="0.0 0.022 0.0" rpy="0 0 0" />
-<parent link="${name}_link" />
-<child link="${name}_rgb_frame"/>
-</joint>
-<link name="${name}_rgb_frame"/>
-<joint name="${name}_rgb_optical_joint" type="fixed">
-<origin xyz="0 0 0" rpy="${-M_PI/2} 0.0 ${-M_PI/2}" />
-<parent link="${name}_rgb_frame" />
-<child link="${name}_rgb_optical_frame"/>
-</joint>
-<link name="${name}_rgb_optical_frame"/>-->
-</xacro:macro>
-<xacro:macro name="asus_camera" params="name parent *origin">
-<xacro:asus_camera_model name="${name}" parent="${parent}">
-<xacro:insert_block name="origin" />
-</xacro:asus_camera_model>
-<!-- ASUS Xtion PRO camera for simulation -->
-<gazebo reference="${name}_depth_frame">
-<sensor type="depth" name="${name}">
-<update_rate>20</update_rate>
-<camera>
-<horizontal_fov>${62.8 * M_PI/180.0}</horizontal_fov>
-<image>
-<format>R8G8B8</format>
-<width>640</width>
-<height>480</height>
-</image>
-<clip>
-<near>0.5</near>
-<far>9</far>
-</clip>
-</camera>
-<plugin name="${name}_camera_controller" filename="libgazebo_ros_openni_kinect.so">
-<alwaysOn>true</alwaysOn>
-<updateRate>20</updateRate>
-<imageTopicName>${name}/rgb/image_raw</imageTopicName>
-<cameraInfoTopicName>${name}/rgb/camera_info</cameraInfoTopicName>
-<depthImageTopicName>${name}/depth/image_raw</depthImageTopicName>
-<depthImageCameraInfoTopicName>${name}/depth/camera_info</depthImageCameraInfoTopicName>
-<pointCloudTopicName>${name}/depth/points</pointCloudTopicName>
-<frameName>${name}_depth_optical_frame</frameName>
-<distortion_k1>0.0</distortion_k1>
-<distortion_k2>0.0</distortion_k2>
-<distortion_k3>0.0</distortion_k3>
-<distortion_t1>0.0</distortion_t1>
-<distortion_t2>0.0</distortion_t2>
-</plugin>
-</sensor>
-</gazebo>
-</xacro:macro>
+<robot name="sensor_asus_xtion_pro" xmlns:xacro="http://ros.org/wiki/xacro">
+  <xacro:include filename="$(find vizzy_description)/urdf/sensors/asus_camera.gazebo.xacro"/>
+  <!-- Xacro properties -->
+  <xacro:property name="M_SCALE" value="0.001"/>
+  <xacro:macro name="sensor_asus_xtion_pro"
+    params="name parent *origin ros_topic">
+    <joint name="${name}_rgb_joint" type="fixed">
+      <xacro:insert_block name="origin"/>
+      <parent link="${parent}"/>
+      <child link="${name}_rgb_frame"/>
+    </joint>
+    <link name="${name}_rgb_frame"/>
+    <joint name="${name}_rgb_optical_joint" type="fixed">
+      <origin
+        xyz="0 0 0"
+        rpy="${-M_PI/2} 0 ${-M_PI/2}"/>
+      <parent link="${name}_rgb_frame"/>
+      <child link="${name}_rgb_optical_frame"/>
+    </joint>
+    <link name="${name}_rgb_optical_frame"/>
+    <joint name="${name}_joint" type="fixed">
+      <origin
+        xyz="0 0 0"
+        rpy="0 0 0"/>
+      <parent link="${name}_rgb_frame"/>
+      <child link="${name}_link"/>
+    </joint>
+    <link name="${name}_link">
+      <visual>
+        <origin
+          xyz="-0.015 0.0035 0.004"
+          rpy="0 0 0"/>
+        <geometry>
+          <mesh filename="package://vizzy_description/meshes/asus_xtion_pro/xtion_pro_camera.dae"/>
+        </geometry>
+      </visual>
+      <collision>
+        <origin
+          xyz="0 0 0"
+          rpy="0 0 0"/>
+        <geometry>
+        <box size="0.0730 0.2760 0.0720"/>
+      </geometry>
+      </collision>
+      <inertial>
+        <mass value="0.170"/>
+        <origin xyz="0 0 0"/>
+        <inertia
+          ixx="0.001152600" ixy="0.0" ixz="0.0"
+          iyy="0.000148934" iyz="0.0"
+          izz="0.001154654"/>
+      </inertial>
+    </link>
+    <joint name="${name}_depth_joint" type="fixed">
+      <origin
+        xyz="0 0 0"
+        rpy="0 0 0"/>
+      <parent link="${name}_rgb_frame"/>
+      <child link="${name}_depth_frame"/>
+    </joint>
+    <link name="${name}_depth_frame"/>
+    <joint name="${name}_depth_optical_joint" type="fixed">
+      <origin
+        xyz="0 0 0"
+        rpy="${-M_PI/2} 0 ${-M_PI/2}"/>
+      <parent link="${name}_depth_frame"/>
+      <child link="${name}_depth_optical_frame"/>
+    </joint>
+    <link name="${name}_depth_optical_frame"/>
+    <!-- Gazebo extension -->
+    <xacro:vizzy_sim_3dsensor name="${name}" ros_topic="${ros_topic}"/>
+  </xacro:macro>
 </robot>

File: vizzy_description/urdf/sensors/hokuyo_04lx_laser.urdf.xacro (robot description, xacro)
@@ -7,5 +7,5 @@
   <xacro:macro name="hokuyo_04lx_laser" params="name parent *origin mesh_file scale ros_topic update_rate min_angle max_angle max_range">
     <joint name="${name}_joint" type="fixed">
-      <insert_block name="origin" />
+      <xacro:insert_block name="origin" />
       <parent link="${parent}_link"/>
       <child link="${name}_link"/>
@@ -14,5 +14,5 @@
       <inertial>
         <mass value="0.001" />
-        <insert_block name="origin" />
+        <xacro:insert_block name="origin" />
         <inertia ixx="0.0001" ixy="0" ixz="0" iyy="0.000001" iyz="0" izz="0.0001" />
       </inertial>
