Commit message: add detailed right hand
Gazebo parameters and joint controllers still missing.

File: vizzy_description/robots/vizzy.urdf.xacro (robot description, xacro)
@@ -6,7 +6,7 @@
   <xacro:arg name="use_full_hand_model" default="false"/>
   <!-- Disable laser sensors -->
-  <xacro:arg name="disable_laser" default="false"/>
+  <xacro:arg name="disable_laser" default="true"/>
   <!-- Disable depth camera -->
-  <xacro:arg name="disable_3d_sensor" default="false"/>
+  <xacro:arg name="disable_3d_sensor" default="true"/>
   <!-- Includes -->
   <!-- Misc common stuff such as constant definitions -->
@@ -16,19 +16,28 @@
   <xacro:include filename="$(find vizzy_description)/urdf/sensors/hokuyo_04lx_laser.urdf.xacro"/>
   <!-- TODO: Update Asus Xiton Live Pro -->
-  <xacro:include filename="$(find vizzy_description)/urdf/sensors/asus_camera.urdf.xacro" />
+  <xacro:include filename="$(find vizzy_description)/urdf/sensors/asus_camera.urdf.xacro"/>
   <!-- Robot body -->
   <!-- Base -->
-  <xacro:include filename="$(find vizzy_description)/urdf/base/base.urdf.xacro" />
+  <xacro:include filename="$(find vizzy_description)/urdf/base/base.urdf.xacro">
+    <xacro:arg name="use_full_gazebo_model" value="$(arg use_full_gazebo_model)"/>
+  </xacro:include>
   <!-- Torso -->
-  <xacro:include filename="$(find vizzy_description)/urdf/torso/torso.urdf.xacro" />
+  <xacro:include filename="$(find vizzy_description)/urdf/torso/torso.urdf.xacro">
+    <xacro:arg name="use_full_gazebo_model" value="$(arg use_full_gazebo_model)"/>
+  </xacro:include>
   <!-- Head -->
- <xacro:include filename="$(find vizzy_description)/urdf/head/head.urdf.xacro"/>
+ <xacro:include filename="$(find vizzy_description)/urdf/head/head.urdf.xacro" >
+    <xacro:arg name="use_full_gazebo_model" value="$(arg use_full_gazebo_model)"/>
+  </xacro:include>
   <!-- Arms -->
-  <xacro:include filename="$(find vizzy_description)/urdf/arm/arm.urdf.xacro" />
+  <xacro:include filename="$(find vizzy_description)/urdf/arm/arm.urdf.xacro" >
+    <xacro:arg name="use_full_gazebo_model" value="$(arg use_full_gazebo_model)"/>
+    <xacro:arg name="use_full_hand_model" value="$(arg use_full_hand_model)"/>
+  </xacro:include>
   <!-- Gazebo plugins -->
   <!-- ROS -->
-  <xacro:include filename="$(find vizzy_description)/plugins/ros.gazebo.xacro" />
+  <xacro:include filename="$(find vizzy_description)/plugins/ros.gazebo.xacro"/>
   <!-- Yarp -->
-  <xacro:include filename="$(find vizzy_description)/plugins/yarp.gazebo.xacro" />
+  <xacro:include filename="$(find vizzy_description)/plugins/yarp.gazebo.xacro"/>
   <!-- Instantiate base -->
   <xacro:base name="base"/>

File: vizzy_description/urdf/arm/arm.gazebo.xacro (robot description, xacro)
@@ -283,6 +283,45 @@
     </collision>
   </xacro:macro>
-  <!-- Wrist Flection -->
-  <xacro:macro name="vizzy_wrist_flection_link_inertial"
+  <!-- Wrist Flection (for detailed right hand) -->
+  <xacro:macro name="vizzy_wrist_flection_link_inertial">
+    <inertial>
+      <origin
+        xyz="-1.1031E-10 0.0010189 -0.018796"
+        rpy="0 0 0" />
+      <mass
+        value="0.11337" />
+      <inertia
+        ixx="1.8801E-05"
+        ixy="-1.2487E-13"
+        ixz="4.3746E-14"
+        iyy="1.7551E-05"
+        iyz="6.7867E-07"
+        izz="1.3766E-05" />
+    </inertial>
+  </xacro:macro>
+  <xacro:macro name="vizzy_wrist_flection_link_collision">
+    <collision>
+      <xacro:if value="$(arg use_full_gazebo_model)">
+        <origin
+          xyz="0 0 0"
+          rpy="0 0 0" />
+        <geometry>
+          <mesh
+            filename="package://vizzy_description/meshes/arm/r_wrist_flection_link.STL" />
+        </geometry>
+      </xacro:if>
+      <xacro:unless value="$(arg use_full_gazebo_model)">
+        <!-- TODO -->
+        <origin
+          xyz="0 0 0"
+          rpy="0 0 0" />
+        <geometry>
+          <cylinder length="0.01" radius="0.001"/>
+        </geometry>
+      </xacro:unless>
+    </collision>
+  </xacro:macro>
+  <!-- Wrist Flection (for simple hand) -->
+  <xacro:macro name="vizzy_wrist_flection_simple_link_inertial"
     params="reflect rpy">
     <inertial>
@@ -301,5 +340,5 @@
     </inertial>
   </xacro:macro>
-  <xacro:macro name="vizzy_wrist_flection_link_collision"
+  <xacro:macro name="vizzy_wrist_flection_simple_link_collision"
     params="reflect rpy prefix">
     <collision>
@@ -323,24 +362,3 @@
     </collision>
   </xacro:macro>
-  <!-- Palm -->
-  <xacro:macro name="vizzy_palm_link_inertial">
-    <inertial>
-      <origin
-        xyz="0 0 0"
-        rpy="0 0 0" />
-      <mass value="0.1"/>
-      <inertia
-        ixx="1.0" ixy="0.0" ixz="0.0"
-        iyy="1.0" iyz="0.0"
-        izz="1.0" />
-    </inertial>
-  </xacro:macro>
-  <xacro:macro name="vizzy_palm_link_collision">
-    <collision>
-      <origin xyz="0 0 0" rpy="0 0 0" />
-      <geometry>
-        <cylinder length="0.001" radius="0.001" />
-      </geometry>
-    </collision>
-  </xacro:macro>
 </robot>

File: vizzy_description/urdf/arm/arm.transmission.xacro (robot description, xacro)
@@ -77,16 +77,14 @@
       </actuator>
     </transmission>
-    <xacro:unless value="$(arg use_full_hand_model)">
-      <transmission name="${prefix}_wrist_flection_transmission">
-        <type>transmission_interface/SimpleTransmission</type>
-        <joint name="${prefix}_wrist_flection_joint">
-          <hardwareInterface>hardware_interface/EffortJointInterface</hardwareInterface>
-        </joint>
-        <actuator name="${prefix}_wrist_flection_motor">
-          <hardwareInterface>hardware_interface/EffortJointInterface</hardwareInterface>
-          <mechanicalReduction>1</mechanicalReduction>
-        </actuator>
-      </transmission>
-    </xacro:unless>
+    <transmission name="${prefix}_wrist_flection_transmission">
+      <type>transmission_interface/SimpleTransmission</type>
+      <joint name="${prefix}_wrist_flection_joint">
+        <hardwareInterface>hardware_interface/EffortJointInterface</hardwareInterface>
+      </joint>
+      <actuator name="${prefix}_wrist_flection_motor">
+        <hardwareInterface>hardware_interface/EffortJointInterface</hardwareInterface>
+        <mechanicalReduction>1</mechanicalReduction>
+      </actuator>
+    </transmission>
   </xacro:macro>
 </robot>

File: vizzy_description/urdf/arm/arm.urdf.xacro (robot description, xacro)
@@ -14,4 +14,8 @@
   </xacro:include>
   <xacro:include filename="$(find vizzy_description)/urdf/arm/arm.transmission.xacro" />
+  <!-- Hands -->
+  <xacro:include filename="$(find vizzy_description)/urdf/hand/right_hand.urdf.xacro">
+    <xacro:arg name="use_full_gazebo_model" value="$(arg use_full_gazebo_model)"/>
+  </xacro:include>
   <xacro:macro name="arm"
     params="name parent">
@@ -19,4 +23,5 @@
     <!-- Left arm -->
     <xacro:if value="${name == 'left_arm'}">
+      <xacro:property name="side" value="left"/>
       <xacro:property name="prefix" value="l"/>
       <xacro:property name="reflect" value="-1"/>
@@ -34,4 +39,5 @@
     <!-- Right arm -->
     <xacro:if value="${name == 'right_arm'}">
+      <xacro:property name="side" value="right"/>
       <xacro:property name="prefix" value="r"/>
       <xacro:property name="reflect" value="1"/>
@@ -47,4 +53,11 @@
       <xacro:property name="palm_j_rpy" value="0 ${M_PI/2} 0"/>
     </xacro:if>
+    <!-- Detailed hand -->
+    <xacro:if value="$(arg use_full_hand_model)">
+      <xacro:property name="detailed_hand" value="true"/>
+    </xacro:if>
+    <xacro:unless value="$(arg use_full_hand_model)">
+      <xacro:property name="detailed_hand" value="true"/>
+    </xacro:unless>
     <!-- Shoulder scapula -->
     <link name="${prefix}_shoulder_scapula_link">
@@ -264,13 +277,47 @@
       <dynamics damping="0.0" friction="0.1"/>
     </joint>
-    <!-- Fully detailed model of the hand -->
-    <xacro:if value="$(arg use_full_hand_model)">
-      <!-- TODO: Add detailed hand -->
+    <!--
+    ////////////////////////////////////////////////////////////////////
+      Hands
+    ////////////////////////////////////////////////////////////////////
+    -->
+    <!-- Detailed right Hand -->
+    <xacro:if value="${(prefix == 'r') and (detailed_hand == 'true')}">
+      <!-- Wrist flection -->
+      <link name="r_wrist_flection_link">
+        <vizzy_wrist_flection_link_inertial/>
+        <visual>
+          <origin
+            xyz="0.007 0 0"
+            rpy="0 ${-M_PI/2} ${M_PI}" />
+          <geometry>
+            <mesh
+              filename="package://vizzy_description/meshes/arm/r_wrist_flection_link.STL" />
+          </geometry>
+          <material name="light_gray_3"/>
+        </visual>
+         <vizzy_wrist_flection_link_collision/>
+      </link>
+      <joint name="${prefix}_wrist_flection_joint"
+        type="revolute">
+        <origin
+          xyz="0 0 0"
+          rpy="0 0 0"/>
+        <parent
+          link="${prefix}_wrist_abduction_link"/>
+        <child
+          link="${prefix}_wrist_flection_link"/>
+        <axis
+          xyz="0 0 1"/>
+        <limit lower="-0.610865238" upper="0.610865238" effort="10" velocity="3" />
+        <dynamics damping="0.0" friction="0.1"/>
+      </joint>
+      <xacro:right_hand parent="r_wrist_flection_link"/>
     </xacro:if>
     <!-- Simplified rigid model of the hand -->
-    <xacro:unless value="$(arg use_full_hand_model)">
+    <xacro:unless value="${(prefix == 'r') and (detailed_hand == 'true')}">
       <!-- Wrist flection -->
       <link name="${prefix}_wrist_flection_link">
-        <vizzy_wrist_flection_link_inertial
+        <vizzy_wrist_flection_simple_link_inertial
           reflect="${reflect}" rpy="${wrist_flection_l_rpy}"/>
         <visual>
@@ -280,9 +327,9 @@
           <geometry>
             <mesh
-              filename="package://vizzy_description/meshes/arm/${prefix}_wrist_flection.dae"/>
+              filename="package://vizzy_description/meshes/arm/${prefix}_wrist_flection_simple.dae"/>
           </geometry>
           <material name="light_gray_3"/>
         </visual>
-        <vizzy_wrist_flection_link_collision
+        <vizzy_wrist_flection_simple_link_collision
           reflect="${reflect}" rpy="${wrist_flection_l_rpy}" prefix="${prefix}"/>
       </link>
@@ -301,24 +348,4 @@
         <dynamics damping="0.0" friction="0.1"/>
       </joint>
-      <!-- Palm (virtual) -->
-      <!-- TODO: add?
-      <link name="${prefix}_palm_link">
-        <vizzy_palm_link_inertial/>
-        <visual>
-          <origin xyz="0 0 0" rpy="0 0 0" />
-          <geometry>
-            <box size="0.001 0.001 0.001" />
-          </geometry>
-        </visual>
-        <vizzy_palm_link_collision/>
-      </link>
-      <joint name="${prefix}_palm_joint" type="fixed">
-        <origin
-          xyz="0 0 0"
-          rpy="${palm_j_rpy}"/>
-        <parent link="${prefix}_wrist_flection_link"/>
-        <child link="${prefix}_palm_link" />
-      </joint>
-      -->
     </xacro:unless>
     <!-- Gazebo extensions -->

File: vizzy_description/urdf/hand/right_hand.gazebo.xacro (robot description, xacro)
@@ -1,89 +1,3 @@
 <?xml version="1.0"?>
 <robot xmlns:xacro="http://ros.org/wiki/xacro">
-  <xacro:macro name="right_hand_gazebo">
-   <gazebo reference="r_palm_link">
-   </gazebo>
-   <gazebo reference="r_min_phal_1_link">
-   </gazebo>
-   <gazebo reference="r_min_phal_2_link">
-   </gazebo>
-   <gazebo reference="r_min_phal_3_link">
-   </gazebo>
-   <gazebo reference="r_med_phal_1_link">
-   </gazebo>
-   <gazebo reference="r_med_phal_2_link">
-   </gazebo>
-   <gazebo reference="r_med_phal_3_link">
-   </gazebo>
-   <gazebo reference="r_ind_phal_1_link">
-   </gazebo>
-   <gazebo reference="r_ind_phal_2_link">
-   </gazebo>
-   <gazebo reference="r_ind_phal_3_link">
-   </gazebo>
-   <gazebo reference="r_thumb_phal_1_link">
-   </gazebo>
-   <gazebo reference="r_thumb_phal_2_link">
-   </gazebo>
-   <gazebo reference="r_thumb_phal_3_link">
-   </gazebo>
-   <gazebo reference="r_thumb_phal_4_link">
-   </gazebo>
-		<gazebo>
-			<plugin name="mimic_plugin" filename="libgazebo_mimic_plugin.so">
-				<joint>r_min_phal_1_joint</joint>
-				<mimicJoint>r_min_phal_2_joint</mimicJoint>
-				<multiplier>0.5</multiplier>
-			</plugin>
-		</gazebo>
-		<gazebo>
-			<plugin name="mimic_plugin" filename="libgazebo_mimic_plugin.so">
-				<joint>r_min_phal_1_joint</joint>
-				<mimicJoint>r_min_phal_3_joint</mimicJoint>
-				<multiplier>0.5</multiplier>
-			</plugin>
-		</gazebo>
-		<gazebo>
-			<plugin name="mimic_plugin" filename="libgazebo_mimic_plugin.so">
-				<joint>r_med_phal_1_joint</joint>
-				<mimicJoint>r_med_phal_2_joint</mimicJoint>
-				<multiplier>0.5</multiplier>
-			</plugin>
-		</gazebo>
-		<gazebo>
-			<plugin name="mimic_plugin" filename="libgazebo_mimic_plugin.so">
-				<joint>r_med_phal_1_joint</joint>
-				<mimicJoint>r_med_phal_3_joint</mimicJoint>
-				<multiplier>0.5</multiplier>
-			</plugin>
-		</gazebo>
-		<gazebo>
-			<plugin name="mimic_plugin" filename="libgazebo_mimic_plugin.so">
-				<joint>r_ind_phal_1_joint</joint>
-				<mimicJoint>r_ind_phal_2_joint</mimicJoint>
-				<multiplier>0.5</multiplier>
-			</plugin>
-		</gazebo>
-		<gazebo>
-			<plugin name="mimic_plugin" filename="libgazebo_mimic_plugin.so">
-				<joint>r_ind_phal_1_joint</joint>
-				<mimicJoint>r_ind_phal_3_joint</mimicJoint>
-				<multiplier>0.5</multiplier>
-			</plugin>
-		</gazebo>
-		<gazebo>
-			<plugin name="mimic_plugin" filename="libgazebo_mimic_plugin.so">
-				<joint>r_thumb_phal_2_joint</joint>
-				<mimicJoint>r_thumb_phal_3_joint</mimicJoint>
-				<multiplier>0.5</multiplier>
-			</plugin>
-		</gazebo>
-		<gazebo>
-			<plugin name="mimic_plugin" filename="libgazebo_mimic_plugin.so">
-				<joint>r_thumb_phal_2_joint</joint>
-				<mimicJoint>r_thumb_phal_4_joint</mimicJoint>
-				<multiplier>0.5</multiplier>
-			</plugin>
-		</gazebo>
-  </xacro:macro>
 </robot>

File: vizzy_description/urdf/hand/right_hand.transmission.xacro (robot description, xacro)
@@ -5,103 +5,4 @@
        xmlns:xacro="http://ros.org/wiki/xacro">
   <xacro:macro name="right_hand_transmissions">
-    <transmission name="r_min_phal_1_transmission">
-      <type>transmission_interface/SimpleTransmission</type>
-      <joint name="r_min_phal_1_joint">
-        <hardwareInterface>hardware_interface/VelocityJointInterface</hardwareInterface>
-      </joint>
-      <actuator name="r_min_phal_1_motor">
-        <mechanicalReduction>1</mechanicalReduction>
-      </actuator>
-    </transmission>
-    <transmission name="r_med_phal_1_transmission">
-      <type>transmission_interface/SimpleTransmission</type>
-      <joint name="r_med_phal_1_joint">
-        <hardwareInterface>hardware_interface/VelocityJointInterface</hardwareInterface>
-      </joint>
-      <actuator name="r_med_phal_1_motor">
-        <mechanicalReduction>1</mechanicalReduction>
-      </actuator>
-    </transmission>
-    <transmission name="r_med_phal_2_transmission">
-      <type>transmission_interface/SimpleTransmission</type>
-      <joint name="r_med_phal_2_joint">
-        <hardwareInterface>hardware_interface/VelocityJointInterface</hardwareInterface>
-      </joint>
-      <actuator name="r_med_phal_2_motor">
-        <mechanicalReduction>1</mechanicalReduction>
-      </actuator>
-    </transmission>
-    <transmission name="r_med_phal_3_transmission">
-      <type>transmission_interface/SimpleTransmission</type>
-      <joint name="r_med_phal_3_joint">
-        <hardwareInterface>hardware_interface/VelocityJointInterface</hardwareInterface>
-      </joint>
-      <actuator name="r_med_phal_3_motor">
-        <mechanicalReduction>1</mechanicalReduction>
-      </actuator>
-    </transmission>
-    <transmission name="r_ind_phal_1_transmission">
-      <type>transmission_interface/SimpleTransmission</type>
-      <joint name="r_ind_phal_1_joint">
-        <hardwareInterface>hardware_interface/VelocityJointInterface</hardwareInterface>
-      </joint>
-      <actuator name="r_ind_phal_1_motor">
-        <mechanicalReduction>1</mechanicalReduction>
-      </actuator>
-    </transmission>
-    <transmission name="r_ind_phal_2_transmission">
-      <type>transmission_interface/SimpleTransmission</type>
-      <joint name="r_ind_phal_2_joint">
-        <hardwareInterface>hardware_interface/VelocityJointInterface</hardwareInterface>
-      </joint>
-      <actuator name="r_ind_phal_2_motor">
-        <mechanicalReduction>1</mechanicalReduction>
-      </actuator>
-    </transmission>
-    <transmission name="r_ind_phal_3_transmission">
-      <type>transmission_interface/SimpleTransmission</type>
-      <joint name="r_ind_phal_3_joint">
-        <hardwareInterface>hardware_interface/VelocityJointInterface</hardwareInterface>
-      </joint>
-      <actuator name="r_ind_phal_3_motor">
-        <mechanicalReduction>1</mechanicalReduction>
-      </actuator>
-    </transmission>
-    <transmission name="r_thumb_phal_1_transmission">
-      <type>transmission_interface/SimpleTransmission</type>
-      <joint name="r_thumb_phal_1_joint">
-        <hardwareInterface>hardware_interface/VelocityJointInterface</hardwareInterface>
-      </joint>
-      <actuator name="r_thumb_phal_1_motor">
-        <mechanicalReduction>1</mechanicalReduction>
-      </actuator>
-    </transmission>
-    <transmission name="r_thumb_phal_2_transmission">
-      <type>transmission_interface/SimpleTransmission</type>
-      <joint name="r_thumb_phal_2_joint">
-        <hardwareInterface>hardware_interface/VelocityJointInterface</hardwareInterface>
-      </joint>
-      <actuator name="r_thumb_phal_2_motor">
-        <mechanicalReduction>1</mechanicalReduction>
-      </actuator>
-    </transmission>
-    <transmission name="r_thumb_phal_3_transmission">
-      <type>transmission_interface/SimpleTransmission</type>
-      <joint name="r_thumb_phal_3_joint">
-        <hardwareInterface>hardware_interface/VelocityJointInterface</hardwareInterface>
-      </joint>
-      <actuator name="r_thumb_phal_3_motor">
-        <mechanicalReduction>1</mechanicalReduction>
-      </actuator>
-    </transmission>
-    <transmission name="r_thumb_phal_4_transmission">
-      <type>transmission_interface/SimpleTransmission</type>
-      <joint name="r_thumb_phal_4_joint">
-        <hardwareInterface>hardware_interface/VelocityJointInterface</hardwareInterface>
-      </joint>
-      <actuator name="r_thumb_phal_4_motor">
-        <mechanicalReduction>1</mechanicalReduction>
-      </actuator>
-    </transmission>
   </xacro:macro>
 </robot>
