Commit message: add detailed right hand
Gazebo parameters and joint controllers still missing.

File: vizzy_description/urdf/hand/right_hand.urdf.xacro (robot description, xacro)
@@ -4,808 +4,1507 @@
        xmlns:interface="http://playerstage.sourceforge.net/gazebo/xmlschema/#interface"
        xmlns:xacro="http://ros.org/wiki/xacro">
+  <!-- Load full inertial and collision model or a simplified model -->
+  <xacro:arg name="use_full_gazebo_model" default="false"/>
   <!-- Things that are needed only for Gazebo (not the physical robot).  These include
        sensor and controller plugin specifications -->
-<xacro:include filename="$(find vizzy_description)/urdf/hand/right_hand.gazebo.xacro"/>
+  <xacro:include filename="$(find vizzy_description)/urdf/hand/right_hand.gazebo.xacro"/>
   <xacro:include filename="$(find vizzy_description)/urdf/hand/right_hand.transmission.xacro"/>
-  <xacro:macro name="right_hand" params="name parent sufix reflect *origin">
-  <link
-    name="r_palm_link">
-    <inertial>
-      <origin
-        xyz="-0.006637 0.0034589 0.0058703"
-        rpy="0 0 0" />
-      <mass
-        value="0.14841" />
-      <inertia
-        ixx="0.00014253"
-        ixy="1.9852E-05"
-        ixz="-1.4353E-06"
-        iyy="9.7254E-05"
-        iyz="-2.6916E-06"
-        izz="0.0002182" />
-    </inertial>
-    <visual>
-      <origin
-        xyz="0 0 0"
-        rpy="0 0 0" />
-      <geometry>
-        <mesh
-          filename="package://vizzy_description/meshes/right_hand/r_palm_link.STL" />
-      </geometry>
-      <material
-        name="">
-        <color
-          rgba="0.79608 0.82353 0.93725 1" />
-      </material>
-    </visual>
-    <collision>
-      <origin
-        xyz="0 0 0"
-        rpy="0 0 0" />
-      <geometry>
-        <mesh
-          filename="package://vizzy_description/meshes/right_hand/r_palm_link.STL" />
-      </geometry>
-    </collision>
-  </link>
-  <link
-    name="r_min_phal_1_link">
-    <inertial>
-      <origin
-        xyz="-0.0065851 -4.2258E-05 0.019478"
-        rpy="0 0 0" />
-      <mass
-        value="0.014476" />
-      <inertia
-        ixx="1.7219E-06"
-        ixy="3.4428E-10"
-        ixz="3.009E-10"
-        iyy="1.7445E-06"
-        iyz="1.5436E-08"
-        izz="5.3067E-07" />
-    </inertial>
-    <visual>
-      <origin
-        xyz="0 0 0"
-        rpy="0 0 0" />
-      <geometry>
-        <mesh
-          filename="package://vizzy_description/meshes/right_hand/r_min_phal_1_link.STL" />
-      </geometry>
-      <material
-        name="">
-        <color
-          rgba="0.89804 0.91765 0.92941 1" />
-      </material>
-    </visual>
-    <collision>
-      <origin
-        xyz="0 0 0"
-        rpy="0 0 0" />
-      <geometry>
-        <mesh
-          filename="package://vizzy_description/meshes/right_hand/r_min_phal_1_link.STL" />
-      </geometry>
-    </collision>
-  </link>
-  <joint
-    name="r_min_phal_1_joint"
-    type="revolute">
-    <origin
-      xyz="0.020602 -0.005836 0.044434"
-      rpy="6.2175E-17 -0.17453 3.1416" />
-    <parent
-      link="r_palm_link" />
-    <child
-      link="r_min_phal_1_link" />
-    <axis
-      xyz="1 0 0" />
-    <limit
-      lower="0"
-      upper="1.7453"
-      effort="10"
-      velocity="10" />
-  </joint>
-  <link
-    name="r_min_phal_2_link">
-    <inertial>
-      <origin
-        xyz="-0.0065912 3.9323E-05 0.016339"
-        rpy="0 0 0" />
-      <mass
-        value="0.011277" />
-      <inertia
-        ixx="1.007E-06"
-        ixy="5.324E-10"
-        ixz="5.414E-10"
-        iyy="1.0456E-06"
-        iyz="1.1256E-08"
-        izz="4.1298E-07" />
-    </inertial>
-    <visual>
-      <origin
-        xyz="0 0 0"
-        rpy="0 0 0" />
-      <geometry>
-        <mesh
-          filename="package://vizzy_description/meshes/right_hand/r_min_phal_2_link.STL" />
-      </geometry>
-      <material
-        name="">
-        <color
-          rgba="0.89804 0.91765 0.92941 1" />
-      </material>
-    </visual>
-    <collision>
-      <origin
-        xyz="0 0 0"
-        rpy="0 0 0" />
-      <geometry>
-        <mesh
-          filename="package://vizzy_description/meshes/right_hand/r_min_phal_2_link.STL" />
-      </geometry>
-    </collision>
-  </link>
-  <joint
-    name="r_min_phal_2_joint"
-    type="revolute">
-    <origin
-      xyz="0 0 0.033"
-      rpy="0 -7.2164E-16 0" />
-    <parent
-      link="r_min_phal_1_link" />
-    <child
-      link="r_min_phal_2_link" />
-    <axis
-      xyz="1 0 0" />
-    <limit
-      lower="0"
-      upper="1.5708"
-      effort="10"
-      velocity="10" />
-    <mimic joint="r_min_phal_1_joint" multiplier="1.0" offset="0.0" />
-  </joint>
-  <link
-    name="r_min_phal_3_link">
-    <inertial>
-      <origin
-        xyz="-0.0065949 -2.2728E-05 0.013411"
-        rpy="0 0 0" />
-      <mass
-        value="0.0093855" />
-      <inertia
-        ixx="5.7614E-07"
-        ixy="5.3191E-10"
-        ixz="-3.8097E-11"
-        iyy="5.3414E-07"
-        iyz="3.9566E-09"
-        izz="3.158E-07" />
-    </inertial>
-    <visual>
-      <origin
-        xyz="0 0 0"
-        rpy="0 0 0" />
-      <geometry>
-        <mesh
-          filename="package://vizzy_description/meshes/right_hand/r_min_phal_3_link.STL" />
-      </geometry>
-      <material
-        name="">
-        <color
-          rgba="0.89804 0.91765 0.92941 1" />
-      </material>
-    </visual>
-    <collision>
-      <origin
-        xyz="0 0 0"
-        rpy="0 0 0" />
-      <geometry>
-        <mesh
-          filename="package://vizzy_description/meshes/right_hand/r_min_phal_3_link.STL" />
-      </geometry>
-    </collision>
-  </link>
-  <joint
-    name="r_min_phal_3_joint"
-    type="revolute">
-    <origin
-      xyz="0 0 0.0265"
-      rpy="0 2.7756E-17 0" />
-    <parent
-      link="r_min_phal_2_link" />
-    <child
-      link="r_min_phal_3_link" />
-    <axis
-      xyz="1 0 0" />
-    <limit
-      lower="0"
-      upper="1.5708"
-      effort="10"
-      velocity="10" />
-    <mimic joint="r_min_phal_1_joint" multiplier="1.0" offset="0.0" />
-  </joint>
-  <link
-    name="r_med_phal_1_link">
-    <inertial>
-      <origin
-        xyz="0.0029095 0.0027577 0.019478"
-        rpy="0 0 0" />
-      <mass
-        value="0.014476" />
-      <inertia
-        ixx="1.7219E-06"
-        ixy="3.4427E-10"
-        ixz="3.008E-10"
-        iyy="1.7445E-06"
-        iyz="1.5436E-08"
-        izz="5.3067E-07" />
-    </inertial>
-    <visual>
-      <origin
-        xyz="0 0 0"
-        rpy="0 0 0" />
-      <geometry>
-        <mesh
-          filename="package://vizzy_description/meshes/right_hand/r_med_phal_1_link.STL" />
-      </geometry>
-      <material
-        name="">
-        <color
-          rgba="0.89804 0.91765 0.92941 1" />
-      </material>
-    </visual>
-    <collision>
-      <origin
-        xyz="0 0 0"
-        rpy="0 0 0" />
-      <geometry>
-        <mesh
-          filename="package://vizzy_description/meshes/right_hand/r_med_phal_1_link.STL" />
-      </geometry>
-    </collision>
-  </link>
-  <joint
-    name="r_med_phal_1_joint"
-    type="revolute">
-    <origin
-      xyz="0 -0.003036 0.050139"
-      rpy="6.123E-17 4.5912E-49 3.1416" />
-    <parent
-      link="r_palm_link" />
-    <child
-      link="r_med_phal_1_link" />
-    <axis
-      xyz="1 0 0" />
-    <limit
-      lower="0"
-      upper="1.7453"
-      effort="10"
-      velocity="10" />
-  </joint>
-  <link
-    name="r_med_phal_2_link">
-    <inertial>
-      <origin
-        xyz="0.0029034 3.9323E-05 0.01634"
-        rpy="0 0 0" />
-      <mass
-        value="0.011277" />
-      <inertia
-        ixx="1.007E-06"
-        ixy="5.324E-10"
-        ixz="5.4133E-10"
-        iyy="1.0456E-06"
-        iyz="1.1377E-08"
-        izz="4.13E-07" />
-    </inertial>
-    <visual>
-      <origin
-        xyz="0 0 0"
-        rpy="0 0 0" />
-      <geometry>
-        <mesh
-          filename="package://vizzy_description/meshes/right_hand/r_med_phal_2_link.STL" />
-      </geometry>
-      <material
-        name="">
-        <color
-          rgba="0.89804 0.91765 0.92941 1" />
-      </material>
-    </visual>
-    <collision>
-      <origin
-        xyz="0 0 0"
-        rpy="0 0 0" />
-      <geometry>
-        <mesh
-          filename="package://vizzy_description/meshes/right_hand/r_med_phal_2_link.STL" />
-      </geometry>
-    </collision>
-  </link>
-  <joint
-    name="r_med_phal_2_joint"
-    type="revolute">
-    <origin
-      xyz="0 0.0028 0.033"
-      rpy="0 0 0" />
-    <parent
-      link="r_med_phal_1_link" />
-    <child
-      link="r_med_phal_2_link" />
-    <axis
-      xyz="1 0 0" />
-    <limit
-      lower="0"
-      upper="1.5708"
-      effort="10"
-      velocity="10" />
-  </joint>
-  <link
-    name="r_med_phal_3_link">
-    <inertial>
-      <origin
-        xyz="0.0028997 -2.2727E-05 0.013411"
-        rpy="0 0 0" />
-      <mass
-        value="0.0093855" />
-      <inertia
-        ixx="5.7614E-07"
-        ixy="5.3189E-10"
-        ixz="-3.8133E-11"
-        iyy="5.3439E-07"
-        iyz="3.9566E-09"
-        izz="3.1605E-07" />
-    </inertial>
-    <visual>
-      <origin
-        xyz="0 0 0"
-        rpy="0 0 0" />
-      <geometry>
-        <mesh
-          filename="package://vizzy_description/meshes/right_hand/r_med_phal_3_link.STL" />
-      </geometry>
-      <material
-        name="">
-        <color
-          rgba="0.89804 0.91765 0.92941 1" />
-      </material>
-    </visual>
-    <collision>
-      <origin
-        xyz="0 0 0"
-        rpy="0 0 0" />
-      <geometry>
-        <mesh
-          filename="package://vizzy_description/meshes/right_hand/r_med_phal_3_link.STL" />
-      </geometry>
-    </collision>
-  </link>
-  <joint
-    name="r_med_phal_3_joint"
-    type="revolute">
-    <origin
-      xyz="0 0 0.0265"
-      rpy="0 0 -2.7192E-32" />
-    <parent
-      link="r_med_phal_2_link" />
-    <child
-      link="r_med_phal_3_link" />
-    <axis
-      xyz="1 0 0" />
-    <limit
-      lower="0"
-      upper="1.5708"
-      effort="10"
-      velocity="10" />
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