Commit message: modified the weights of the wheels

File: vizzy_description/urdf/base/base.gazebo.xacro (robot description, xacro)
@@ -11,4 +11,8 @@
     </gazebo>
     <gazebo reference="b_wheel_base_link">
+      <!-- <mu1 value="100.0" />
+      <mu2 value="100.0" />
+      <kp  value="1000000.0" />
+      <kd  value="1.0" /> -->
       <mu1>10000</mu1>
       <mu2>10000</mu2>
@@ -19,4 +23,8 @@
     </gazebo>
     <gazebo reference="f_wheel_base_link">
+      <!-- <mu1 value="100.0" />
+      <mu2 value="100.0" />
+      <kp  value="1000000.0" />
+      <kd  value="1.0" /> -->
       <mu1>10000</mu1>
       <mu2>10000</mu2>

File: vizzy_description/urdf/base/base.urdf.xacro (robot description, xacro)
@@ -145,6 +145,7 @@
         rpy="0 0 0" />
       <geometry>
-        <mesh
-          filename="package://vizzy_description/meshes/F_W.dae" />
+        <!-- <mesh
+          filename="package://vizzy_description/meshes/F_W.dae" />  -->
+        <cylinder length="0.02" radius="0.05"/>
       </geometry>
     </collision>
@@ -251,6 +252,7 @@
         rpy="0 0 0" />
       <geometry>
-        <mesh
-          filename="package://vizzy_description/meshes/B_W.dae" />
+        <!-- <mesh
+          filename="package://vizzy_description/meshes/B_W.dae" /> -->
+        <cylinder length="0.02" radius="0.05"/>
       </geometry>
     </collision>
@@ -276,5 +278,5 @@
         rpy="0 0 0" />
       <mass
-        value="1.22861917507719" />
+        value="150.22861917507719" />
       <inertia
         ixx="0.0106873251772162"
@@ -304,6 +306,7 @@
         rpy="0 0 0" />
       <geometry>
-        <mesh
-          filename="package://vizzy_description/meshes/Left.dae" />
+        <!-- <mesh
+          filename="package://vizzy_description/meshes/Left.dae" /> -->
+        <cylinder length="0.06" radius="0.198"/>
       </geometry>
     </collision>
@@ -330,5 +333,5 @@
         rpy="3.15 0 0" />
       <mass
-        value="1.22861917507742" />
+        value="150.22861917507742" />
       <inertia
         ixx="0.0106873471854323"
@@ -358,6 +361,7 @@
         rpy="3.15 0 0" />
       <geometry>
-        <mesh
-          filename="package://vizzy_description/meshes/Right.dae" />
+        <!-- <mesh
+          filename="package://vizzy_description/meshes/Right.dae" />  -->
+        <cylinder length="0.06" radius="0.198"/>
       </geometry>
     </collision>
