Commit message: abduction transforms corrected (best commit ever)

File: vizzy_description/urdf/arm/left_arm.urdf.xacro (robot description, xacro)
@@ -332,10 +332,24 @@
 		  <limit lower="-1.48352986" upper="1.48352986" effort="10" velocity="3" />
 		</joint>
-		<link
-		  name="l_wrist_abduction_link">
-		  <inertial>
-		    <origin
-		      xyz="-0.0047 -0.022 0.003"
-		      rpy="${M_PI/2} 0.0 ${-M_PI/4}" />
+		<joint
+		  name="l_wrist_abduction_joint"
+		  type="revolute">
+		  <origin
+		    xyz="0.0 0.0 0.11925"
+		    rpy="${M_PI/2.0} 0.0 0.0" />
+		  <parent
+		    link="l_forearm_pronation_link" />
+		  <child
+		    link="l_wrist_abduction_virtual_link" />
+		  <axis
+		    xyz="0 0 1" />
+		  <limit lower="-0.610865238" upper="0.610865238" effort="10" velocity="3" />
+		</joint>
+		<link
+		  name="l_wrist_abduction_virtual_link">
+		  <inertial>
+		    <origin
+		      xyz="0.0 0.0 0.005"
+		      rpy="${M_PI/2} 0.0 0.0" />
 		    <mass
 		      value="0.151302636921624" />
@@ -350,9 +364,49 @@
 		  <visual>
 		    <origin
+		      xyz="0.0 0.0 0.005"
+		      rpy="${M_PI/2} 0.0 0.0" />
+		    <geometry>
+		      <mesh
+		        filename="package://vizzy_description/meshes/M6L_back.dae" />
+		    </geometry>
+		    <material
+		      name="">
+		      <color
+		        rgba="0.898039215686275 0.917647058823529 0.929411764705882 1" />
+		    </material>
+		  </visual>
+		  <collision>
+		    <origin
+		      xyz="0.0 0.0 0.005"
+		      rpy="${M_PI/2} 0.0 0.0" />
+		    <geometry>
+		      <mesh
+		        filename="package://vizzy_description/meshes/M6L_back.dae" />
+		    </geometry>
+		  </collision>
+		</link>
+		<link
+		  name="l_wrist_abduction_link">
+		  <inertial>
+		    <origin
+		      xyz="-0.0047 -0.022 0.003"
+		      rpy="${M_PI/2} 0.0 ${-M_PI/4}" />
+		    <mass
+		      value="0.151302636921624" />
+		    <inertia
+		      ixx="0.000116373512947626"
+		      ixy="1.31009871908069E-05"
+		      ixz="6.69703789973942E-05"
+		      iyy="0.00020031628400595"
+		      iyz="1.00268924727662E-05"
+		      izz="0.000162164313365602" />
+		  </inertial>
+		  <visual>
+		    <origin
 		      xyz="-0.0047 -0.020 0.003"
 		      rpy="${M_PI/2} 0.0 ${-M_PI/4}" />
 		    <geometry>
 		      <mesh
-		        filename="package://vizzy_description/meshes/M6L.dae" />
+		        filename="package://vizzy_description/meshes/M6L_wrist.dae" />
 		    </geometry>
 		    <material
@@ -368,10 +422,10 @@
 		    <geometry>
 		      <mesh
-		        filename="package://vizzy_description/meshes/M6L.dae" />
-		    </geometry>
-		  </collision>
-		</link>
-		<joint
-		  name="l_wrist_abduction_joint"
+		        filename="package://vizzy_description/meshes/M6L_wrist.dae" />
+		    </geometry>
+		  </collision>
+		</link>
+		<joint
+		  name="l_wrist_abduction_virtual_joint"
 		  type="revolute">
 		  <origin
@@ -385,4 +439,5 @@
 		    xyz="0 0 1" />
 		  <limit lower="-0.610865238" upper="0.610865238" effort="10" velocity="3" />
+    		  <mimic joint="l_wrist_abduction_joint" multiplier="1.0" offset="0"/>
 		</joint>
 		<link

File: vizzy_description/urdf/arm/right_arm.urdf.xacro (robot description, xacro)
@@ -333,9 +333,9 @@
 		</joint>
 		<link
-		  name="r_wrist_abduction_link">
-		  <inertial>
-		    <origin
-		      xyz="0.0047 0.028 -0.003"
-		      rpy="${M_PI} ${M_PI} 0" />
+		  name="r_wrist_abduction_virtual_link">
+		  <inertial>
+		    <origin
+		      xyz="0.0 0.0 0.0"
+		      rpy="${-M_PI/2.0} 0 ${M_PI}" />
 		    <mass
 		      value="0.15130263687109" />
@@ -350,17 +350,57 @@
 		  <visual>
 		    <origin
+		      xyz="0.0 0.0 -0.005"
+		      rpy="${-M_PI/2.0} 0 ${M_PI}" />
+		    <geometry>
+		      <mesh
+		        filename="package://vizzy_description/meshes/M6R_back.dae" />
+		    </geometry>
+		    <material
+		      name="">
+		      <color
+		        rgba="0.898039215686275 0.917647058823529 0.929411764705882 1" />
+		    </material>
+		  </visual>
+		  <collision>
+		    <origin
+		      xyz="0.0 0.0 0.0"
+		      rpy="${-M_PI/2.0} 0 ${M_PI}" />
+		    <geometry>
+		      <mesh
+		        filename="package://vizzy_description/meshes/M6R_back.dae" />
+		    </geometry>
+		  </collision>
+		</link>
+		<joint
+		  name="r_wrist_abduction_joint"
+		  type="revolute">
+		  <origin
+		    xyz="0.0 0.0 -0.11925"
+		    rpy="${M_PI/2.0} 0.0 0.0" />
+		  <parent
+		    link="r_forearm_pronation_link" />
+		  <child
+		    link="r_wrist_abduction_virtual_link" />
+		  <axis
+		    xyz="0 0 1" />
+		  <limit lower="-0.610865238" upper="0.610865238" effort="10" velocity="3" />
+		</joint>
+		<link
+		  name="r_wrist_abduction_link">
+		  <inertial>
+		    <origin
 		      xyz="0.0047 0.028 -0.003"
 		      rpy="${M_PI} ${M_PI} 0" />
-		    <geometry>
-		      <mesh
-		        filename="package://vizzy_description/meshes/M6R.dae" />
-		    </geometry>
-		    <material
-		      name="">
-		      <color
-		        rgba="0.898039215686275 0.917647058823529 0.929411764705882 1" />
-		    </material>
-		  </visual>
-		  <collision>
+		    <mass
+		      value="0.15130263687109" />
+		    <inertia
+		      ixx="0.000206280948481805"
+		      ixy="-2.10167871847464E-05"
+		      ixz="-1.95502541303483E-06"
+		      iyy="7.18084114032176E-05"
+		      iyz="1.63557763545568E-05"
+		      izz="0.000199867817507994" />
+		  </inertial>
+		  <visual>
 		    <origin
 		      xyz="0.0047 0.028 -0.003"
@@ -368,10 +408,24 @@
 		    <geometry>
 		      <mesh
-		        filename="package://vizzy_description/meshes/M6R.dae" />
-		    </geometry>
-		  </collision>
-		</link>
-		<joint
-		  name="r_wrist_abduction_joint"
+		        filename="package://vizzy_description/meshes/M6R_wrist.dae" />
+		    </geometry>
+		    <material
+		      name="">
+		      <color
+		        rgba="0.898039215686275 0.917647058823529 0.929411764705882 1" />
+		    </material>
+		  </visual>
+		  <collision>
+		    <origin
+		      xyz="0.0047 0.028 -0.003"
+		      rpy="${M_PI} ${M_PI} 0" />
+		    <geometry>
+		      <mesh
+		        filename="package://vizzy_description/meshes/M6R_wrist.dae" />
+		    </geometry>
+		  </collision>
+		</link>
+		<joint
+		  name="r_wrist_abduction_virtual_joint"
 		  type="revolute">
 		  <origin
@@ -385,4 +439,5 @@
 		    xyz="0 0 1" />
 		  <limit lower="-0.610865238" upper="0.610865238" effort="10" velocity="3" />
+    		  <mimic joint="r_wrist_abduction_joint" multiplier="1.0" offset="0"/>
 		</joint>
 		<link

Commit message: - Set PID parameters of left arm position controllers - Reduced joint friction in the left arm - FollowJointTrajectory actionlib server for yarp-based control working in simulation - ROS-YARP bridge of left arm's FollowJointTrajectory action working in simulation

File: vizzy_description/urdf/arm/left_arm.urdf.xacro (robot description, xacro)
@@ -61,5 +61,5 @@
 		    xyz="0 0 1" />
 		  <limit lower="-0.314159265" upper="0.314159265" effort="10" velocity="3" />
-		  <dynamics damping="0.0" friction="0.6"/>
+		  <dynamics damping="0.0" friction="1.0"/>
 		</joint>
 		<link
@@ -116,5 +116,5 @@
 		    xyz="0 0 1" />
 		  <limit lower="-1.30899694" upper="2.35619449" effort="10" velocity="3" />
-		  <dynamics damping="0.0" friction="0.6"/>
+		  <dynamics damping="0.0" friction="0.2"/>
 		</joint>
 		<link
@@ -226,5 +226,5 @@
 		    xyz="0 0 1" />
 		  <limit lower="-1.48352986" upper="1.48352986" effort="10" velocity="3" />
-		  <dynamics damping="0.0" friction="0.6"/>
+		  <dynamics damping="0.0" friction="0.1"/>
 		</joint>
 		<link
@@ -281,5 +281,5 @@
 		    xyz="0 0 1" />
 		  <limit lower="0" upper="1.91986218" effort="10" velocity="3" />
-		  <dynamics damping="0.0" friction="0.6"/>
+		  <dynamics damping="0.0" friction="0.1"/>
 		</joint>
 		<link
@@ -336,5 +336,5 @@
 		    xyz="0 0 1" />
 		  <limit lower="-1.48352986" upper="1.48352986" effort="10" velocity="3" />
-		  <dynamics damping="0.0" friction="0.6"/>
+		  <dynamics damping="0.0" friction="0.1"/>
 		</joint>
 		<link
@@ -391,5 +391,5 @@
 		    xyz="0 0 1" />
 		  <limit lower="-0.610865238" upper="0.610865238" effort="10" velocity="3" />
-		  <dynamics damping="0.0" friction="0.6"/>
+		  <dynamics damping="0.0" friction="0.1"/>
 		</joint>
 		<link
@@ -447,5 +447,5 @@
 		  <limit lower="-0.610865238" upper="0.610865238" effort="10" velocity="3" />
     		  <mimic joint="l_wrist_abduction_joint" multiplier="1.0" offset="0"/>
-		  <dynamics damping="0.0" friction="0.6"/>
+		  <dynamics damping="0.0" friction="0.1"/>
 		</joint>
 		<link
@@ -502,5 +502,5 @@
 		    xyz="0 0 1" />
 		  <limit lower="-0.610865238" upper="0.610865238" effort="10" velocity="3" />
-		  <dynamics damping="0.0" friction="0.6"/>
+		  <dynamics damping="0.0" friction="0.1"/>
 		</joint>
 		<!--<link name="l_palm_link">
