Commit message: [vizzy_moveit_config] updated groups for planning in 8dof [vizzy_gazebo] added new world with table and objects [vizzy_control] added a new joint for the end-effector

File: vizzy_description/urdf/arm/right_arm.transmission.xacro (robot description, xacro)
@@ -95,4 +95,14 @@
       </actuator>
     </transmission>
+    <transmission name="r_palm_transmission">
+      <type>transmission_interface/SimpleTransmission</type>
+      <joint name="r_palm_joint">
+        <hardwareInterface>PositionJointInterface</hardwareInterface>
+      </joint>
+      <actuator name="r_palm_motor">
+        <hardwareInterface>EffortJointInterface</hardwareInterface>
+        <mechanicalReduction>1</mechanicalReduction>
+      </actuator>
+    </transmission>
   </xacro:macro>
 </robot>

File: vizzy_description/urdf/arm/right_arm.urdf.xacro (robot description, xacro)
@@ -501,7 +501,15 @@
 		    xyz="0 0 1" />
 		  <limit lower="-0.610865238" upper="0.610865238" effort="10" velocity="3" />
-		  <dynamics damping="0.0" friction="5.0"/>
-		</joint>
-		<!--<link name="r_palm_link">
+		  <dynamics damping="0.0" friction="1.0"/>
+		</joint>
+		<link name="r_palm_link">
+<inertial>
+        <origin xyz="0 0 0" rpy="0 0 0" />
+        <mass value="0.1" />
+        <inertia
+          ixx="1.0" ixy="0.0" ixz="0.0"
+          iyy="1.0" iyz="0.0"
+          izz="1.0" />
+    </inertial>
 		 <visual>
 		    <origin xyz="0 0 0" rpy="0 0 0" />
@@ -510,10 +518,17 @@
 		    </geometry>
 		  </visual>
-		</link>
-		<joint name="r_palm_joint" type="fixed">
+ <collision>
+      <origin xyz="0 0 0" rpy="0 0 0" />
+      <geometry>
+        <cylinder length="0.001" radius="0.001" />
+      </geometry>
+    </collision>
+		</link>
+		<joint name="r_palm_joint" type="revolute">
 		  <origin xyz="0.1 0 0.0" rpy="${M_PI/2.0} 0 ${M_PI}" />
 		  <parent link="r_wrist_flection_link"/>
 		  <child link="r_palm_link" />
-		</joint>-->
+		  <limit lower="0.0" upper="0.0" effort="10" velocity="3" />
+		</joint>
     <!-- gazebo extensions -->
     <xacro:right_arm_gazebo/>
