Commit message: [vizzy_moveit_config] Wrist joint now in the planning group [id_selector] Added directions and points in the map

File: vizzy_description/urdf/arm/right_arm.urdf.xacro (robot description, xacro)
@@ -504,25 +504,25 @@
 		</joint>
 		<link name="r_palm_link">
-<inertial>
-        <origin xyz="0 0 0" rpy="0 0 0" />
-        <mass value="0.1" />
-        <inertia
-          ixx="1.0" ixy="0.0" ixz="0.0"
-          iyy="1.0" iyz="0.0"
-          izz="1.0" />
-    </inertial>
-		 <visual>
-		    <origin xyz="0 0 0" rpy="0 0 0" />
-		    <geometry>
-		      <box size="0.001 0.001 0.001" />
-		    </geometry>
-		  </visual>
- <collision>
-      <origin xyz="0 0 0" rpy="0 0 0" />
-      <geometry>
-        <cylinder length="0.001" radius="0.001" />
-      </geometry>
-    </collision>
-		</link>
+                    <inertial>
+                        <origin xyz="0 0 0" rpy="0 0 0" />
+                        <mass value="0.1" />
+                        <inertia
+                            ixx="1.0" ixy="0.0" ixz="0.0"
+                            iyy="1.0" iyz="0.0"
+                            izz="1.0" />
+                   </inertial>
+		   <visual>
+		       <origin xyz="0 0 0" rpy="0 0 0" />
+		       <geometry>
+		          <box size="0.001 0.001 0.001" />
+		       </geometry>
+		   </visual>
+                   <collision>
+                       <origin xyz="0 0 0" rpy="0 0 0" />
+                       <geometry>
+                           <cylinder length="0.001" radius="0.001" />
+                       </geometry>
+                   </collision>
+	        </link>
 		<joint name="r_palm_joint" type="revolute">
 		  <origin xyz="0.1 0 0.0" rpy="${M_PI/2.0} 0 ${M_PI}" />
