Commit message: fixed some problems with virtual links in gazebo

File: vizzy_description/urdf/arm/right_arm.gazebo.xacro (robot description, xacro)
@@ -31,9 +31,9 @@
       <material>Gazebo/Orange</material>
     </gazebo>
-    <gazebo reference="r_wrist_abduction_virtual_link">
+    <!--<gazebo reference="r_wrist_abduction_virtual_link">
       <mu1>0.2</mu1>
       <mu2>0.2</mu2>
       <material>Gazebo/Orange</material>
-    </gazebo>
+    </gazebo>-->
     <gazebo reference="r_wrist_flection_link">
       <mu1>0.2</mu1>
@@ -44,5 +44,5 @@
       <mu2>0.2</mu2>
     </gazebo>
-    <gazebo>
+    <!--<gazebo>
 			<plugin name="mimic_plugin" filename="libgazebo_mimic_plugin.so">
 				<joint>r_wrist_abduction_joint</joint>
@@ -50,5 +50,5 @@
 				<multiplier>1.0</multiplier>
 			</plugin>
-    </gazebo>
+    </gazebo>-->
   </xacro:macro>
 </robot>

File: vizzy_description/urdf/arm/right_arm.transmission.xacro (robot description, xacro)
@@ -75,5 +75,5 @@
       </actuator>
     </transmission>
-    <transmission name="r_wrist_abduction_virtual_transmission">
+    <!--<transmission name="r_wrist_abduction_virtual_transmission">
       <type>transmission_interface/SimpleTransmission</type>
       <joint name="r_wrist_abduction_virtual_joint">
@@ -84,5 +84,5 @@
         <mechanicalReduction>1</mechanicalReduction>
       </actuator>
-    </transmission>
+    </transmission>-->
     <transmission name="r_wrist_flection_transmission">
       <type>transmission_interface/SimpleTransmission</type>

File: vizzy_description/urdf/arm/right_arm.urdf.xacro (robot description, xacro)
@@ -168,5 +168,5 @@
 		  <axis
 		    xyz="0 0 1" />
-		  <limit lower="0" upper="1.30899694" effort="10" velocity="3" />
+		  <limit lower="-0.1" upper="1.30899694" effort="10" velocity="3" />
 		</joint>
 		<link
@@ -332,5 +332,5 @@
 		  <limit lower="-1.48352986" upper="1.48352986" effort="10" velocity="3" />
 		</joint>
-		<link
+		<!--<link
 		  name="r_wrist_abduction_virtual_link">
 		  <inertial>
@@ -371,15 +371,15 @@
 		    </geometry>
 		  </collision>
-		</link>
+		</link>-->
 		<joint
 		  name="r_wrist_abduction_joint"
 		  type="revolute">
 		  <origin
-		    xyz="0.0 0.0 -0.11925"
+		    xyz="0.0 0.0 -0.18925"
 		    rpy="${M_PI/2.0} 0.0 0.0" />
 		  <parent
 		    link="r_forearm_pronation_link" />
 		  <child
-		    link="r_wrist_abduction_virtual_link" />
+		    link="r_wrist_abduction_link" />
 		  <axis
 		    xyz="0 0 1" />
@@ -426,5 +426,5 @@
 		  </collision>
 		</link>
-		<joint
+		<!--<joint
 		  name="r_wrist_abduction_virtual_joint"
 		  type="revolute">
@@ -440,5 +440,5 @@
 		  <limit lower="-0.610865238" upper="0.610865238" effort="10" velocity="3" />
     		  <mimic joint="r_wrist_abduction_joint" multiplier="1.0" offset="0"/>
-		</joint>
+		</joint>-->
 		<link
 		  name="r_wrist_flection_link">

Commit message: more fixes

File: vizzy_description/urdf/arm/right_arm.gazebo.xacro (robot description, xacro)
@@ -31,13 +31,7 @@
       <material>Gazebo/Orange</material>
     </gazebo>
-<<<<<<< HEAD
     <!--<gazebo reference="r_wrist_abduction_virtual_link">
       <mu1>0.2</mu1>
       <mu2>0.2</mu2>
-=======
-    <gazebo reference="r_wrist_abduction_virtual_link">
-      <!--<mu1>0.2</mu1>
-      <mu2>0.2</mu2>-->
->>>>>>> 6d626c85aa043eb21d0ecfe0d48c72bc15980c9a
       <material>Gazebo/Orange</material>
     </gazebo>-->

File: vizzy_description/urdf/arm/right_arm.urdf.xacro (robot description, xacro)
@@ -170,10 +170,6 @@
 		  <axis
 		    xyz="0 0 1" />
-<<<<<<< HEAD
 		  <limit lower="-0.1" upper="1.30899694" effort="10" velocity="3" />
-=======
-		  <limit lower="0" upper="1.30899694" effort="10" velocity="3" />
-		  <dynamics damping="0.0" friction="5.0"/>
->>>>>>> 6d626c85aa043eb21d0ecfe0d48c72bc15980c9a
+		  <dynamics damping="0.0" friction="5.0"/>
 		</joint>
 		<link

Commit message: fixed moveit right arm issues and created ros based wave demo

File: vizzy_description/urdf/arm/right_arm.gazebo.xacro (robot description, xacro)
@@ -41,6 +41,4 @@
     </gazebo>
     <gazebo reference="r_palm_link">
-      <!--<mu1>0.2</mu1>
-      <mu2>0.2</mu2>-->
     </gazebo>
     <!--<gazebo>

File: vizzy_description/urdf/arm/right_arm.transmission.xacro (robot description, xacro)
@@ -95,5 +95,5 @@
       </actuator>
     </transmission>
-    <transmission name="r_palm_transmission">
+    <!--<transmission name="r_palm_transmission">
       <type>transmission_interface/SimpleTransmission</type>
       <joint name="r_palm_joint">
@@ -104,5 +104,5 @@
         <mechanicalReduction>1</mechanicalReduction>
       </actuator>
-    </transmission>
+    </transmission>-->
   </xacro:macro>
 </robot>

File: vizzy_description/urdf/arm/right_arm.urdf.xacro (robot description, xacro)
@@ -525,9 +525,9 @@
                    </collision>
 	        </link>
-		<joint name="r_palm_joint" type="revolute">
+		<joint name="r_palm_joint" type="fixed">
 		  <origin xyz="0.1 0 0.0" rpy="${M_PI/2.0} 0 ${M_PI}" />
 		  <parent link="r_wrist_flection_link"/>
 		  <child link="r_palm_link" />
-		  <limit lower="0.0" upper="0.0" effort="10" velocity="3" />
+		  <!--<limit lower="0.0" upper="0.0" effort="10" velocity="3" />-->
 		</joint>
     <!-- gazebo extensions -->
