Commit message: corrected transmission issues

File: vizzy_description/urdf/arm/left_arm.gazebo.xacro (robot description, xacro)
@@ -29,4 +29,10 @@
       <mu1>0.2</mu1>
       <mu2>0.2</mu2>
+      <material>Gazebo/Orange</material>
+    </gazebo>
+    <gazebo reference="l_wrist_abduction_virtual_link">
+      <mu1>0.2</mu1>
+      <mu2>0.2</mu2>
+      <material>Gazebo/Orange</material>
     </gazebo>
     <gazebo reference="l_wrist_flection_link">
@@ -38,4 +44,11 @@
       <mu2>0.2</mu2>
     </gazebo>
+		<gazebo>
+			<plugin name="mimic_plugin" filename="libgazebo_mimic_plugin.so">
+				<joint>l_wrist_abduction_joint</joint>
+				<mimicJoint>l_wrist_abduction_virtual_joint</mimicJoint>
+				<multiplier>1.0</multiplier>
+			</plugin>
+		</gazebo>
   </xacro:macro>
 </robot>

File: vizzy_description/urdf/arm/left_arm.transmission.xacro (robot description, xacro)
@@ -68,4 +68,13 @@
       </actuator>
     </transmission>
+    <transmission name="l_wrist_abduction_virtual_transmission">
+      <type>transmission_interface/SimpleTransmission</type>
+      <joint name="l_wrist_abduction_virtual_joint">
+        <hardwareInterface>VelocityJointInterface</hardwareInterface>
+      </joint>
+      <actuator name="l_wrist_abduction_virtual_motor">
+        <mechanicalReduction>1</mechanicalReduction>
+      </actuator>
+    </transmission>
     <transmission name="l_wrist_flection_transmission">
       <type>transmission_interface/SimpleTransmission</type>

File: vizzy_description/urdf/arm/left_arm.urdf.xacro (robot description, xacro)
@@ -390,5 +390,5 @@
 		  <inertial>
 		    <origin
-		      xyz="-0.0047 -0.022 0.003"
+		      xyz="-0.0047 -0.028 0.003"
 		      rpy="${M_PI/2} 0.0 ${-M_PI/4}" />
 		    <mass
@@ -404,5 +404,5 @@
 		  <visual>
 		    <origin
-		      xyz="-0.0047 -0.020 0.003"
+		      xyz="-0.0047 -0.028 0.003"
 		      rpy="${M_PI/2} 0.0 ${-M_PI/4}" />
 		    <geometry>
@@ -418,5 +418,5 @@
 		  <collision>
 		    <origin
-		      xyz="-0.0047 -0.022 0.003"
+		      xyz="-0.0047 -0.028 0.003"
 		      rpy="${M_PI/2} 0.0 ${-M_PI/4}" />
 		    <geometry>

File: vizzy_description/urdf/arm/right_arm.gazebo.xacro (robot description, xacro)
@@ -29,4 +29,10 @@
       <mu1>0.2</mu1>
       <mu2>0.2</mu2>
+      <material>Gazebo/Orange</material>
+    </gazebo>
+    <gazebo reference="r_wrist_abduction_virtual_link">
+      <mu1>0.2</mu1>
+      <mu2>0.2</mu2>
+      <material>Gazebo/Orange</material>
     </gazebo>
     <gazebo reference="r_wrist_flection_link">
@@ -38,4 +44,11 @@
       <mu2>0.2</mu2>
     </gazebo>
+		<gazebo>
+			<plugin name="mimic_plugin" filename="libgazebo_mimic_plugin.so">
+				<joint>r_wrist_abduction_joint</joint>
+				<mimicJoint>r_wrist_abduction_virtual_joint</mimicJoint>
+				<multiplier>1.0</multiplier>
+			</plugin>
+		</gazebo>
   </xacro:macro>
 </robot>

File: vizzy_description/urdf/arm/right_arm.transmission.xacro (robot description, xacro)
@@ -68,4 +68,13 @@
       </actuator>
     </transmission>
+    <transmission name="r_wrist_abduction_virtual_transmission">
+      <type>transmission_interface/SimpleTransmission</type>
+      <joint name="r_wrist_abduction_virtual_joint">
+        <hardwareInterface>VelocityJointInterface</hardwareInterface>
+      </joint>
+      <actuator name="r_wrist_abduction_virtual_motor">
+        <mechanicalReduction>1</mechanicalReduction>
+      </actuator>
+    </transmission>
     <transmission name="r_wrist_flection_transmission">
       <type>transmission_interface/SimpleTransmission</type>

File: vizzy_description/urdf/base/base.urdf.xacro (robot description, xacro)
@@ -55,5 +55,5 @@
     <collision>
       <origin
-        xyz="0.19 0 0.2"
+        xyz="0.188 0.001 0.197"
         rpy="0 0 0" />
       <geometry>

File: vizzy_description/urdf/common.urdf.xacro (robot description, xacro)
@@ -41,3 +41,6 @@
     <color rgba="0.02 0.02 0.02 1" />
   </material>
+  <material name="orange">
+    <color rgba="${255/255} ${108/255} ${10/255} 1.0"/>
+  </material>
 </root>

Commit message: fixed problem with arm trajectory controllers. Seems that gazebo 2.0 control interface only supports position controllers

File: vizzy_description/urdf/arm/left_arm.gazebo.xacro (robot description, xacro)
@@ -44,5 +44,5 @@
       <mu2>0.2</mu2>
     </gazebo>
-		<gazebo>
+    <gazebo>
 			<plugin name="mimic_plugin" filename="libgazebo_mimic_plugin.so">
 				<joint>l_wrist_abduction_joint</joint>
@@ -50,5 +50,5 @@
 				<multiplier>1.0</multiplier>
 			</plugin>
-		</gazebo>
+    </gazebo>
   </xacro:macro>
 </robot>

File: vizzy_description/urdf/arm/left_arm.transmission.xacro (robot description, xacro)
@@ -8,7 +8,8 @@
       <type>transmission_interface/SimpleTransmission</type>
       <joint name="l_shoulder_scapula_joint">
-        <hardwareInterface>VelocityJointInterface</hardwareInterface>
+        <hardwareInterface>PositionJointInterface</hardwareInterface>
       </joint>
       <actuator name="l_shoulder_scapula_motor">
+        <hardwareInterface>EffortJointInterface</hardwareInterface>
         <mechanicalReduction>1</mechanicalReduction>
       </actuator>
@@ -17,7 +18,8 @@
       <type>transmission_interface/SimpleTransmission</type>
       <joint name="l_shoulder_flection_joint">
-        <hardwareInterface>VelocityJointInterface</hardwareInterface>
+        <hardwareInterface>PositionJointInterface</hardwareInterface>
       </joint>
       <actuator name="l_shoulder_flection_motor">
+        <hardwareInterface>EffortJointInterface</hardwareInterface>
         <mechanicalReduction>1</mechanicalReduction>
       </actuator>
@@ -26,7 +28,8 @@
       <type>transmission_interface/SimpleTransmission</type>
       <joint name="l_shoulder_abduction_joint">
-        <hardwareInterface>VelocityJointInterface</hardwareInterface>
+        <hardwareInterface>PositionJointInterface</hardwareInterface>
       </joint>
       <actuator name="l_shoulder_abduction_motor">
+        <hardwareInterface>EffortJointInterface</hardwareInterface>
         <mechanicalReduction>1</mechanicalReduction>
       </actuator>
@@ -35,7 +38,8 @@
       <type>transmission_interface/SimpleTransmission</type>
       <joint name="l_shoulder_rotation_joint">
-        <hardwareInterface>VelocityJointInterface</hardwareInterface>
+        <hardwareInterface>PositionJointInterface</hardwareInterface>
       </joint>
       <actuator name="l_shoulder_rotation_motor">
+        <hardwareInterface>EffortJointInterface</hardwareInterface>
         <mechanicalReduction>1</mechanicalReduction>
       </actuator>
@@ -44,7 +48,8 @@
       <type>transmission_interface/SimpleTransmission</type>
       <joint name="l_elbow_flection_joint">
-        <hardwareInterface>VelocityJointInterface</hardwareInterface>
+        <hardwareInterface>PositionJointInterface</hardwareInterface>
       </joint>
       <actuator name="l_elbow_flection_motor">
+        <hardwareInterface>EffortJointInterface</hardwareInterface>
         <mechanicalReduction>1</mechanicalReduction>
       </actuator>
@@ -53,7 +58,8 @@
       <type>transmission_interface/SimpleTransmission</type>
       <joint name="l_forearm_pronation_joint">
-        <hardwareInterface>VelocityJointInterface</hardwareInterface>
+        <hardwareInterface>PositionJointInterface</hardwareInterface>
       </joint>
       <actuator name="l_forearm_pronation_motor">
+        <hardwareInterface>EffortJointInterface</hardwareInterface>
         <mechanicalReduction>1</mechanicalReduction>
       </actuator>
@@ -62,7 +68,8 @@
       <type>transmission_interface/SimpleTransmission</type>
       <joint name="l_wrist_abduction_joint">
-        <hardwareInterface>VelocityJointInterface</hardwareInterface>
+        <hardwareInterface>PositionJointInterface</hardwareInterface>
       </joint>
       <actuator name="l_wrist_abduction_motor">
+        <hardwareInterface>EffortJointInterface</hardwareInterface>
         <mechanicalReduction>1</mechanicalReduction>
       </actuator>
@@ -71,7 +78,8 @@
       <type>transmission_interface/SimpleTransmission</type>
       <joint name="l_wrist_abduction_virtual_joint">
-        <hardwareInterface>VelocityJointInterface</hardwareInterface>
+        <hardwareInterface>PositionJointInterface</hardwareInterface>
       </joint>
       <actuator name="l_wrist_abduction_virtual_motor">
+        <hardwareInterface>EffortJointInterface</hardwareInterface>
         <mechanicalReduction>1</mechanicalReduction>
       </actuator>
@@ -80,7 +88,8 @@
       <type>transmission_interface/SimpleTransmission</type>
       <joint name="l_wrist_flection_joint">
-        <hardwareInterface>VelocityJointInterface</hardwareInterface>
+        <hardwareInterface>PositionJointInterface</hardwareInterface>
       </joint>
       <actuator name="l_wrist_flection_motor">
+        <hardwareInterface>EffortJointInterface</hardwareInterface>
         <mechanicalReduction>1</mechanicalReduction>
       </actuator>

File: vizzy_description/urdf/arm/right_arm.gazebo.xacro (robot description, xacro)
@@ -50,5 +50,5 @@
 				<multiplier>1.0</multiplier>
 			</plugin>
-		</gazebo>
+    </gazebo>
   </xacro:macro>
 </robot>

File: vizzy_description/urdf/head/head.yarp.urdf.xacro (robot description, xacro)
@@ -8,5 +8,5 @@
  <xacro:include filename="$(find vizzy_description)/urdf/head/head.yarp.gazebo.xacro" />
  <xacro:include filename="$(find vizzy_description)/urdf/head/head.yarp.transmission.xacro" />
-  <xacro:macro name="head_yarp" params="name">
+  <xacro:macro name="head" params="name">
    <link name="neck_pan_link">
     <inertial>
@@ -60,5 +60,6 @@
     <axis
       xyz="0 0 1" />
-    <limit lower="-0.925024504" upper="0.925024504" effort="10" velocity="3" />
+    <!--<limit lower="-0.925024504" upper="0.925024504" effort="10.0" velocity="5.0" />-->
+    <limit lower="-2.025024504" upper="2.025024504" effort="10.0" velocity="5.0" />
   </joint>
   <link
@@ -114,5 +115,6 @@
     <axis
       xyz="0 0 1" />
-    <limit lower="-0.314159265" upper="0.645771823" effort="10" velocity="3" />
+    <!--<limit lower="-0.314159265" upper="0.645771823" effort="100.0" velocity="5.0" />-->
+    <limit lower="-2.014159265" upper="2.45771823" effort="100.0" velocity="5.0" />
   </joint>
   <link
@@ -168,8 +170,126 @@
     <axis
       xyz="0 0 1" />
-    <limit lower="-0.663225116" upper="0.663225116" effort="10" velocity="3" />
-  </joint>
-  <link
-    name="r_eye_pan_link">
+    <limit lower="-0.663225116" upper="0.663225116" effort="10.0" velocity="5.0" />
+  </joint>
+  <!-- eyes center virtual link and joint -->
+  <link name="eyes_center_link">
+		<inertial>
+			<origin xyz="0 0 0"
+      rpy="0.0 0.0 0" />
+			<mass value="0.1"/>
+			<inertia
+				ixx="0.001" ixy="0.0" ixz="0.0"
+				iyy="0.001" iyz="0.0" izz="0.001"/>
+		</inertial>
+  </link>
+  <joint name="eyes_center_vision_joint" type="fixed">
+    <origin xyz="0 0 0"       rpy="${-M_PI/2} 0.0 ${-M_PI/2}" />
+    <parent link="eyes_center_link" />
+    <child link="eyes_center_vision_link" />
+  </joint>
+  <link name="eyes_center_vision_link">
+		<inertial>
+			<origin xyz="0 0 0"
+      rpy="0.0 0.0 0" />
+			<mass value="0.1"/>
+			<inertia
+				ixx="0.001" ixy="0.0" ixz="0.0"
+				iyy="0.001" iyz="0.0" izz="0.001"/>
+		</inertial>
+  </link>
+  <joint name="eyes_center_joint" type="fixed">
+    <origin xyz="0 0 0"       rpy="${M_PI/2.0} 0.0 0.369599135716446" />
+    <parent link="eyes_tilt_link" />
+    <child link="eyes_center_link" />
+  </joint>
+  <!-- version virtual link and joint -->
+  <link name="version_link">
+		<inertial>
+			<origin xyz="0 0 0"
+      rpy="0.0 0.0 0" />
+			<mass value="0.01"/>
+			<inertia
+				ixx="0.001" ixy="0.0" ixz="0.0"
+				iyy="0.001" iyz="0.0" izz="0.001"/>
+		</inertial>
+  </link>
+  <joint name="version_joint" type="revolute">
+    <origin xyz="0 0 0"       rpy="0 0 0" />
+    <parent link="eyes_center_link" />
+    <child link="version_link" />
+    <axis  xyz="0 0 1" />
+    <limit lower="-0.698131" upper="0.698131" effort="10.0" velocity="5.0" />
+  </joint>
+  <link name="l_eye_version_link">
+ 		<inertial>
+			<origin xyz="0 0 0" rpy="0 0 0"/>
+			<mass value="0.01"/>
+			<inertia
+				ixx="0.001" ixy="0.0" ixz="0.0"
+				iyy="0.001" iyz="0.0" izz="0.001"/>
+		</inertial>
+  </link>
+  <joint
+    name="l_eye_version_joint"
+    type="revolute">
+    <origin
+      xyz="0.0 0.102 0.0"
+      rpy="0 0 0" />
+    <parent
+      link="eyes_center_link" />
+    <child
+      link="l_eye_version_link" />
+    <axis
+      xyz="0 0 1" />
+    <limit
+			lower="-1.0"
+			upper="1.0"
+      effort="1000.0"
+      velocity="5.0" />
+  </joint>
+  <link name="r_eye_version_link">
+ 		<inertial>
+			<origin xyz="0 0 0" rpy="0 0 0"/>
+			<mass value="0.01"/>
+			<inertia
+				ixx="0.001" ixy="0.0" ixz="0.0"
+				iyy="0.001" iyz="0.0" izz="0.001"/>
+		</inertial>
+  </link>
+  <joint
+    name="r_eye_version_joint"
+    type="revolute">
+    <origin
+      xyz="0.0 -0.102 0.0"
+      rpy="0 0.0 0" />
+    <parent
+      link="eyes_center_link" />
+    <child
+      link="r_eye_version_link" />
+    <axis
+      xyz="0 0 1" />
+    <limit
+			lower="-1.0"
+			upper="1.0"
+      effort="1000.0"
+      velocity="5.0"/>
+  </joint>
+  <link name="vergence_link">
+ 		<inertial>
+			<origin xyz="0 0 0" rpy="0 0 0"/>
+			<mass value="0.01"/>
+			<inertia
+				ixx="0.001" ixy="0.0" ixz="0.0"
+				iyy="0.001" iyz="0.0" izz="0.001"/>
+		</inertial>
+  </link>
+  <joint name="vergence_joint" type="revolute">
+    <origin xyz="0.0 0.0 0.0" rpy="0 0.0 0" />
+    <parent link="eyes_center_link" />
+    <child link="vergence_link" />
+    <axis  xyz="0 0 1" />
+    <limit lower="0.0" upper="0.698131" effort="10.0" velocity="5.0" />
+  </joint>
+  <link name="r_eye_vergence_link">
     <inertial>
       <origin
@@ -211,16 +331,20 @@
   </link>
   <joint
-    name="r_eye_pan_joint"
-    type="revolute">
-    <origin
-      xyz="0.0 0.0 -0.102"
-      rpy="${M_PI/2.0} 0.0 0.369599135716446" />
-    <parent
-      link="eyes_tilt_link" />
-    <child
-      link="r_eye_pan_link" />
-    <axis
-      xyz="0 0 1" />
-    <limit lower="-0.698131" upper="0.698131" effort="10" velocity="3" />
+    name="r_eye_vergence_joint"
+    type="revolute">
+    <origin
+      xyz="0.0 0.0 0.0"
+      rpy="0.0 0.0 0.0" />
+    <parent
+      link="r_eye_version_link" />
+    <child
+      link="r_eye_vergence_link" />
+    <axis
+      xyz="0 0 1" />
+		<limit
+			lower="-1.0"
+			upper="1.0"
+      effort="1000.0"
+      velocity="5.0"/>
   </joint>
   <link name="r_camera_link">
@@ -234,9 +358,22 @@
   <joint name="r_camera_joint" type="fixed">
     <origin xyz="0.0575 0.0 0.0" rpy="0.0 0.0 0.0" />
-    <parent link="r_eye_pan_link"/>
+    <parent link="r_eye_vergence_link"/>
     <child link="r_camera_link" />
   </joint>
-  <link name="l_eye_pan_link">
-    <inertial>
+  <link name="r_camera_vision_link">
+   <visual>
+      <origin xyz="0 0 0" rpy="0 0 0" />
+      <geometry>
+        <box size="0.001 0.001 0.001" />
+      </geometry>
+    </visual>
+  </link>
+  <joint name="r_camera_vision_joint" type="fixed">
+    <origin xyz="0.0 0.0 0.0" rpy="${-M_PI/2} 0.0 ${-M_PI/2}" />
+    <parent link="r_camera_link"/>
+    <child link="r_camera_vision_link" />
+  </joint>
+  <link name="l_eye_vergence_link">
+   <inertial>
       <origin
         xyz="0 0 -0.0200000000000069"
@@ -267,7 +404,7 @@
     </visual>
     <collision>
-      <origin
-        xyz="0 0 -0.0200000000000069"
-        rpy="0 0 1.5708" />
+ 	<origin
+        xyz="0.010 0.0 0.003"
+        rpy="0.0 ${M_PI} ${-M_PI/2}" />
       <geometry>
         <mesh
@@ -277,16 +414,20 @@
   </link>
   <joint
-    name="l_eye_pan_joint"
-    type="revolute">
-    <origin
-      xyz="0.0 0.0 0.102"
-      rpy="${M_PI/2.0} 0.0 0.369599135716446" />
-    <parent
-      link="eyes_tilt_link" />
-    <child
-      link="l_eye_pan_link" />
-    <axis
-      xyz="0 0 1" />
-    <limit lower="-0.698131" upper="0.698131" effort="10" velocity="3" />
+    name="l_eye_vergence_joint"
+    type="revolute">
+    <origin
+      xyz="0 0 0"
+      rpy="0 0 0" />
+    <parent
+      link="l_eye_version_link" />
+    <child
+      link="l_eye_vergence_link" />
+    <axis
+      xyz="0 0 1" />
+    <limit
+			lower="-1.0"
+			upper="1.0"
+      effort="1000.0"
+      velocity="5.0" />
   </joint>
   <link name="l_camera_link">
@@ -298,8 +439,7 @@
     </visual>
   </link>
-  <!-- Camera (Opencv convention) frames -->
   <joint name="l_camera_joint" type="fixed">
     <origin xyz="0.0575 0.0 0.0" rpy="0.0 0.0 0.0" />
-    <parent link="l_eye_pan_link"/>
+    <parent link="l_eye_vergence_link"/>
     <child link="l_camera_link" />
   </joint>
@@ -317,18 +457,5 @@
     <child link="l_camera_vision_link" />
   </joint>
-  <link name="r_camera_vision_link">
-   <visual>
-      <origin xyz="0 0 0" rpy="0 0 0" />
-      <geometry>
-        <box size="0.001 0.001 0.001" />
-      </geometry>
-    </visual>
-  </link>
-  <joint name="r_camera_vision_joint" type="fixed">
-    <origin xyz="0.0 0.0 0.0" rpy="${-M_PI/2} 0.0 ${-M_PI/2}" />
-    <parent link="r_camera_link"/>
-    <child link="r_camera_vision_link" />
-  </joint>
-  <!-- eyes center and ego virtual link and joint -->
+  <!-- eyes center virtual link and joint -->
   <link name="ego_frame">
     <inertial>
