Commit message: moveit is now working properly for both arms. Yeiii

File: vizzy_description/urdf/arm/left_arm.gazebo.xacro (robot description, xacro)
@@ -31,9 +31,4 @@
       <material>Gazebo/Orange</material>
     </gazebo>
-    <gazebo reference="l_wrist_abduction_virtual_link">
-      <!--<mu1>0.2</mu1>
-      <mu2>0.2</mu2>-->
-      <material>Gazebo/Orange</material>
-    </gazebo>
     <gazebo reference="l_wrist_flection_link">
       <!--<mu1>0.2</mu1>
@@ -41,13 +36,4 @@
     </gazebo>
     <gazebo reference="l_palm_link">
-      <!--<mu1>0.2</mu1>
-      <mu2>0.2</mu2>-->
-    </gazebo>
-    <gazebo>
-			<plugin name="mimic_plugin" filename="libgazebo_mimic_plugin.so">
-				<joint>l_wrist_abduction_joint</joint>
-				<mimicJoint>l_wrist_abduction_virtual_joint</mimicJoint>
-				<multiplier>1.0</multiplier>
-			</plugin>
     </gazebo>
   </xacro:macro>

File: vizzy_description/urdf/arm/left_arm.transmission.xacro (robot description, xacro)
@@ -75,14 +75,4 @@
       </actuator>
     </transmission>
-    <transmission name="l_wrist_abduction_virtual_transmission">
-      <type>transmission_interface/SimpleTransmission</type>
-      <joint name="l_wrist_abduction_virtual_joint">
-        <hardwareInterface>PositionJointInterface</hardwareInterface>
-      </joint>
-      <actuator name="l_wrist_abduction_virtual_motor">
-        <hardwareInterface>EffortJointInterface</hardwareInterface>
-        <mechanicalReduction>1</mechanicalReduction>
-      </actuator>
-    </transmission>
     <transmission name="l_wrist_flection_transmission">
       <type>transmission_interface/SimpleTransmission</type>

File: vizzy_description/urdf/arm/left_arm.urdf.xacro (robot description, xacro)
@@ -336,12 +336,27 @@
 		    xyz="0 0 1" />
 		  <limit lower="-1.48352986" upper="1.48352986" effort="10" velocity="3" />
-		  <dynamics damping="0.0" friction="0.1"/>
-		</joint>
-		<link
-		  name="l_wrist_abduction_virtual_link">
-		  <inertial>
-		    <origin
-		      xyz="0.0 0.0 0.005"
-		      rpy="${M_PI/2} 0.0 0.0" />
+		  <dynamics damping="0.0" friction="5.0"/>
+		</joint>
+		<joint
+		  name="l_wrist_abduction_joint"
+		  type="revolute">
+		  <origin
+		    xyz="0.0 0.0 0.18925"
+		    rpy="${M_PI/2.0} 0.0 0.0" />
+		  <parent
+		    link="l_forearm_pronation_link" />
+		  <child
+		    link="l_wrist_abduction_link" />
+		  <axis
+		    xyz="0 0 1" />
+		  <limit lower="-0.610865238" upper="0.610865238" effort="10" velocity="3" />
+		  <dynamics damping="0.0" friction="5.0"/>
+		</joint>
+		<link
+		  name="l_wrist_abduction_link">
+		  <inertial>
+		    <origin
+		      xyz="-0.0047 -0.028 0.003"
+		      rpy="0.0 0.0 0.0" />
 		    <mass
 		      value="0.151302636921624" />
@@ -356,61 +371,6 @@
 		  <visual>
 		    <origin
-		      xyz="0.0 0.0 0.005"
-		      rpy="${M_PI/2} 0.0 0.0" />
-		    <geometry>
-		      <mesh
-		        filename="package://vizzy_description/meshes/M6L_back.dae" />
-		    </geometry>
-		    <material
-		      name="">
-		      <color
-		        rgba="0.898039215686275 0.917647058823529 0.929411764705882 1" />
-		    </material>
-		  </visual>
-		  <collision>
-		    <origin
-		      xyz="0.0 0.0 0.005"
-		      rpy="${M_PI/2} 0.0 0.0" />
-		    <geometry>
-		      <mesh
-		        filename="package://vizzy_description/meshes/M6L_back.dae" />
-		    </geometry>
-		  </collision>
-		</link>
-		<joint
-		  name="l_wrist_abduction_joint"
-		  type="revolute">
-		  <origin
-		    xyz="0.0 0.0 0.11925"
-		    rpy="${M_PI/2.0} 0.0 0.0" />
-		  <parent
-		    link="l_forearm_pronation_link" />
-		  <child
-		    link="l_wrist_abduction_virtual_link" />
-		  <axis
-		    xyz="0 0 1" />
-		  <limit lower="-0.610865238" upper="0.610865238" effort="10" velocity="3" />
-		  <dynamics damping="0.0" friction="0.1"/>
-		</joint>
-		<link
-		  name="l_wrist_abduction_link">
-		  <inertial>
-		    <origin
-		      xyz="-0.0047 -0.028 0.003"
-		      rpy="${M_PI/2} 0.0 ${-M_PI/4}" />
-		    <mass
-		      value="0.151302636921624" />
-		    <inertia
-		      ixx="0.000116373512947626"
-		      ixy="1.31009871908069E-05"
-		      ixz="6.69703789973942E-05"
-		      iyy="0.00020031628400595"
-		      iyz="1.00268924727662E-05"
-		      izz="0.000162164313365602" />
-		  </inertial>
-		  <visual>
-		    <origin
-		      xyz="-0.0047 -0.028 0.003"
-		      rpy="${M_PI/2} 0.0 ${-M_PI/4}" />
+		      xyz="-0.0047 -0.028 -0.003"
+		      rpy="0.0 0.0 0.0" />
 		    <geometry>
 		      <mesh
@@ -425,6 +385,6 @@
 		  <collision>
 		    <origin
-		      xyz="-0.0047 -0.028 0.003"
-		      rpy="${M_PI/2} 0.0 ${-M_PI/4}" />
+		      xyz="-0.0047 -0.028 -0.003"
+		      rpy="0.0 0.0 0.0" />
 		    <geometry>
 		      <mesh
@@ -433,25 +393,9 @@
 		  </collision>
 		</link>
-		<joint
-		  name="l_wrist_abduction_virtual_joint"
-		  type="revolute">
-		  <origin
-		    xyz="0.0 0.0 0.18925"
-		    rpy="${M_PI/2.0} 0.0 0.0" />
-		  <parent
-		    link="l_forearm_pronation_link" />
-		  <child
-		    link="l_wrist_abduction_link" />
-		  <axis
-		    xyz="0 0 1" />
-		  <limit lower="-0.610865238" upper="0.610865238" effort="10" velocity="3" />
-    		  <mimic joint="l_wrist_abduction_joint" multiplier="1.0" offset="0"/>
-		  <dynamics damping="0.0" friction="0.1"/>
-		</joint>
 		<link
 		  name="l_wrist_flection_link">
 		  <inertial>
 		    <origin
-		      xyz="-0.106 -0.0077 -0.015"
+		      xyz="-0.106 -0.0077 -0.017"
 		      rpy="0.0 0.0 ${M_PI/2.0}" />
 		    <mass
@@ -467,6 +411,6 @@
 		  <visual>
 		    <origin
-		      xyz="-0.106 -0.0077 -0.015"
-		      rpy="0.0 0.0 ${M_PI/2.0}" />
+		      xyz="-0.106 -0.0077 -0.017"
+		      rpy="0.0 0.0 ${M_PI/2}" />
 		    <geometry>
 		      <mesh
@@ -481,5 +425,5 @@
 		  <collision>
 		    <origin
-		      xyz="-0.106 -0.0077 -0.015"
+		      xyz="-0.106 -0.0077 -0.017"
 		      rpy="0.0 0.0 ${M_PI/2.0}" />
 		    <geometry>
@@ -502,19 +446,33 @@
 		    xyz="0 0 1" />
 		  <limit lower="-0.610865238" upper="0.610865238" effort="10" velocity="3" />
-		  <dynamics damping="0.0" friction="0.1"/>
-		</joint>
-		<!--<link name="l_palm_link">
-		 <visual>
-		    <origin xyz="0.0 0.0 0.0" rpy="0.0 0.0 0.0" />
-		    <geometry>
-		      <box size="0.001 0.001 0.001" />
-		    </geometry>
-		  </visual>
-		</link>
+		  <dynamics damping="0.0" friction="1.0"/>
+		</joint>
+		<link name="l_palm_link">
+                    <inertial>
+                        <origin xyz="0 0 0" rpy="0 0 0" />
+                        <mass value="0.1" />
+                        <inertia
+                            ixx="1.0" ixy="0.0" ixz="0.0"
+                            iyy="1.0" iyz="0.0"
+                            izz="1.0" />
+                   </inertial>
+		   <visual>
+		       <origin xyz="0 0 0" rpy="0 0 0" />
+		       <geometry>
+		          <box size="0.001 0.001 0.001" />
+		       </geometry>
+		   </visual>
+                   <collision>
+                       <origin xyz="0 0 0" rpy="0 0 0" />
+                       <geometry>
+                           <cylinder length="0.001" radius="0.001" />
+                       </geometry>
+                   </collision>
+	        </link>
 		<joint name="l_palm_joint" type="fixed">
 		  <origin xyz="-0.1 0.0 0.0" rpy="${-M_PI/2} ${M_PI} 0.0" />
 		  <parent link="l_wrist_flection_link"/>
 		  <child link="l_palm_link" />
-		</joint>-->
+		</joint>
 		<!-- gazebo extensions -->
 		<xacro:left_arm_gazebo/>

File: vizzy_description/urdf/arm/right_arm.gazebo.xacro (robot description, xacro)
@@ -31,9 +31,4 @@
       <material>Gazebo/Orange</material>
     </gazebo>
-    <!--<gazebo reference="r_wrist_abduction_virtual_link">
-      <mu1>0.2</mu1>
-      <mu2>0.2</mu2>
-      <material>Gazebo/Orange</material>
-    </gazebo>-->
     <gazebo reference="r_wrist_flection_link">
       <!--<mu1>0.2</mu1>
@@ -42,11 +37,4 @@
     <gazebo reference="r_palm_link">
     </gazebo>
-    <!--<gazebo>
-			<plugin name="mimic_plugin" filename="libgazebo_mimic_plugin.so">
-				<joint>r_wrist_abduction_joint</joint>
-				<mimicJoint>r_wrist_abduction_virtual_joint</mimicJoint>
-				<multiplier>1.0</multiplier>
-			</plugin>
-    </gazebo>-->
   </xacro:macro>
 </robot>

File: vizzy_description/urdf/arm/right_arm.transmission.xacro (robot description, xacro)
@@ -75,14 +75,4 @@
       </actuator>
     </transmission>
-    <!--<transmission name="r_wrist_abduction_virtual_transmission">
-      <type>transmission_interface/SimpleTransmission</type>
-      <joint name="r_wrist_abduction_virtual_joint">
-        <hardwareInterface>PositionJointInterface</hardwareInterface>
-      </joint>
-      <actuator name="r_wrist_abduction_virtual_motor">
-        <hardwareInterface>EffortJointInterface</hardwareInterface>
-        <mechanicalReduction>1</mechanicalReduction>
-      </actuator>
-    </transmission>-->
     <transmission name="r_wrist_flection_transmission">
       <type>transmission_interface/SimpleTransmission</type>
@@ -95,14 +85,4 @@
       </actuator>
     </transmission>
-    <!--<transmission name="r_palm_transmission">
-      <type>transmission_interface/SimpleTransmission</type>
-      <joint name="r_palm_joint">
-        <hardwareInterface>PositionJointInterface</hardwareInterface>
-      </joint>
-      <actuator name="r_palm_motor">
-        <hardwareInterface>EffortJointInterface</hardwareInterface>
-        <mechanicalReduction>1</mechanicalReduction>
-      </actuator>
-    </transmission>-->
   </xacro:macro>
 </robot>

File: vizzy_description/urdf/arm/right_arm.urdf.xacro (robot description, xacro)
@@ -338,44 +338,4 @@
 		  <dynamics damping="0.0" friction="5.0"/>
 		</joint>
-		<!--<link
-		  name="r_wrist_abduction_virtual_link">
-		  <inertial>
-		    <origin
-		      xyz="0.0 0.0 -0.005"
-		      rpy="${-M_PI/2.0} 0 ${M_PI}" />
-		    <mass
-		      value="0.151302636921624" />
-		    <inertia
-		      ixx="0.000116373512947626"
-		      ixy="1.31009871908069E-05"
-		      ixz="6.69703789973942E-05"
-		      iyy="0.00020031628400595"
-		      iyz="1.00268924727662E-05"
-		      izz="0.000162164313365602" />
-		  </inertial>
-		  <visual>
-		    <origin
-		      xyz="0.0 0.0 -0.005"
-		      rpy="${-M_PI/2.0} 0 ${M_PI}" />
-		    <geometry>
-		      <mesh
-		        filename="package://vizzy_description/meshes/M6R_back.dae" />
-		    </geometry>
-		    <material
-		      name="">
-		      <color
-		        rgba="0.898039215686275 0.917647058823529 0.929411764705882 1" />
-		    </material>
-		  </visual>
-		  <collision>
-		    <origin
-		      xyz="0.0 0.0 -0.005"
-		      rpy="${-M_PI/2.0} 0 ${M_PI}" />
-		    <geometry>
-		      <mesh
-		        filename="package://vizzy_description/meshes/M6R_back.dae" />
-		    </geometry>
-		  </collision>
-		</link>-->
 		<joint
 		  name="r_wrist_abduction_joint"
@@ -433,19 +393,4 @@
 		  </collision>
 		</link>
-		<!--<joint
-		  name="r_wrist_abduction_virtual_joint"
-		  type="revolute">
-		  <origin
-		    xyz="0.0 0.0 -0.18925"
-		    rpy="${M_PI/2.0} 0.0 0.0" />
-		  <parent
-		    link="r_forearm_pronation_link" />
-		  <child
-		    link="r_wrist_abduction_link" />
-		  <axis
-		    xyz="0 0 1" />
-		  <limit lower="-0.610865238" upper="0.610865238" effort="10" velocity="3" />
-    		  <mimic joint="r_wrist_abduction_joint" multiplier="1.0" offset="0"/>
-		</joint>-->
 		<link
 		  name="r_wrist_flection_link">
@@ -481,5 +426,5 @@
 		    <origin
 		      xyz="0.106 0.0077 0.017"
-		      rpy="0.0 ${M_PI} ${-M_PI/2}" />
+		      rpy="0.0 ${M_PI} ${-M_PI/2.0}" />
 		    <geometry>
 		      <mesh
@@ -526,8 +471,7 @@
 	        </link>
 		<joint name="r_palm_joint" type="fixed">
-		  <origin xyz="0.1 0 0.0" rpy="${M_PI/2.0} 0 ${M_PI}" />
+		  <origin xyz="0.1 0 0.0" rpy="${M_PI/2.0} 0.0 ${M_PI}" />
 		  <parent link="r_wrist_flection_link"/>
 		  <child link="r_palm_link" />
-		  <!--<limit lower="0.0" upper="0.0" effort="10" velocity="3" />-->
 		</joint>
     <!-- gazebo extensions -->
