Commit message: fix thumb; add hand controllers
Fixed thumb link names
Added hand position controllers
Controllers not responding to commands yet

File: vizzy_description/urdf/arm/arm.gazebo.xacro (robot description, xacro)
@@ -312,10 +312,9 @@
       </xacro:if>
       <xacro:unless value="$(arg use_full_gazebo_model)">
-        <!-- TODO -->
-        <origin
-          xyz="0 0 0"
-          rpy="0 0 0" />
-        <geometry>
-          <cylinder length="0.01" radius="0.001"/>
+        <origin
+          xyz="-0.035 0 0"
+          rpy="0 ${M_PI/2} 0" />
+        <geometry>
+          <cylinder length="0.004" radius="0.020"/>
         </geometry>
       </xacro:unless>

File: vizzy_description/urdf/arm/arm.urdf.xacro (robot description, xacro)
@@ -311,5 +311,5 @@
           xyz="0 0 1"/>
         <limit lower="-0.610865238" upper="0.610865238" effort="10" velocity="3" />
-        <dynamics damping="0.0" friction="0.1"/>
+        <dynamics damping="0.0" friction="1.0"/>
       </joint>
       <xacro:right_hand parent="r_wrist_flection_link"/>

File: vizzy_description/urdf/hand/right_hand.gazebo.xacro (robot description, xacro)
@@ -1,3 +1,66 @@
 <?xml version="1.0"?>
 <robot xmlns:xacro="http://ros.org/wiki/xacro">
+  <!-- Instance mimic plugins for underactuated finger control -->
+  <xacro:macro name="right_hand_gazebo">
+    <!-- Min underactuated finger -->
+    <gazebo>
+      <plugin name="mimic_plugin" filename="libgazebo_mimic_plugin.so">
+        <joint>r_min_phal_1_joint</joint>
+        <mimicJoint>r_min_phal_2_joint</mimicJoint>
+        <multiplier>0.5</multiplier>
+      </plugin>
+    </gazebo>
+    <gazebo>
+      <plugin name="mimic_plugin" filename="libgazebo_mimic_plugin.so">
+        <joint>r_min_phal_1_joint</joint>
+        <mimicJoint>r_min_phal_3_joint</mimicJoint>
+        <multiplier>0.5</multiplier>
+      </plugin>
+    </gazebo>
+    <!-- Med underactuated finger -->
+    <gazebo>
+      <plugin name="mimic_plugin" filename="libgazebo_mimic_plugin.so">
+        <joint>r_med_phal_1_joint</joint>
+        <mimicJoint>r_med_phal_2_joint</mimicJoint>
+        <multiplier>0.5</multiplier>
+      </plugin>
+    </gazebo>
+    <gazebo>
+      <plugin name="mimic_plugin" filename="libgazebo_mimic_plugin.so">
+        <joint>r_med_phal_1_joint</joint>
+        <mimicJoint>r_med_phal_3_joint</mimicJoint>
+        <multiplier>0.5</multiplier>
+      </plugin>
+    </gazebo>
+    <!-- Ind underactuated finger -->
+    <gazebo>
+      <plugin name="mimic_plugin" filename="libgazebo_mimic_plugin.so">
+        <joint>r_ind_phal_1_joint</joint>
+        <mimicJoint>r_ind_phal_2_joint</mimicJoint>
+        <multiplier>0.5</multiplier>
+      </plugin>
+    </gazebo>
+    <gazebo>
+      <plugin name="mimic_plugin" filename="libgazebo_mimic_plugin.so">
+        <joint>r_ind_phal_1_joint</joint>
+        <mimicJoint>r_ind_phal_3_joint</mimicJoint>
+        <multiplier>0.5</multiplier>
+      </plugin>
+    </gazebo>
+    <!-- Thumb underactuated finger -->
+    <gazebo>
+      <plugin name="mimic_plugin" filename="libgazebo_mimic_plugin.so">
+        <joint>r_thumb_phal_2_joint</joint>
+        <mimicJoint>r_thumb_phal_3_joint</mimicJoint>
+        <multiplier>0.5</multiplier>
+      </plugin>
+    </gazebo>
+    <gazebo>
+      <plugin name="mimic_plugin" filename="libgazebo_mimic_plugin.so">
+        <joint>r_thumb_phal_2_joint</joint>
+        <mimicJoint>r_thumb_phal_4_joint</mimicJoint>
+        <multiplier>0.5</multiplier>
+      </plugin>
+    </gazebo>
+  </xacro:macro>
 </robot>

File: vizzy_description/urdf/hand/right_hand.transmission.xacro (robot description, xacro)
@@ -5,4 +5,94 @@
        xmlns:xacro="http://ros.org/wiki/xacro">
   <xacro:macro name="right_hand_transmissions">
+  	<transmission name="r_min_phal_1_transmission">
+      <type>transmission_interface/SimpleTransmission</type>
+      <joint name="r_min_phal_1_joint">
+        <hardwareInterface>hardware_interface/VelocityJointInterface</hardwareInterface>
+      </joint>
+      <actuator name="r_min_phal_1_motor">
+        <mechanicalReduction>1</mechanicalReduction>
+      </actuator>
+    </transmission>
+    <transmission name="r_med_phal_1_transmission">
+      <type>transmission_interface/SimpleTransmission</type>
+      <joint name="r_med_phal_1_joint">
+        <hardwareInterface>hardware_interface/VelocityJointInterface</hardwareInterface>
+      </joint>
+      <actuator name="r_med_phal_1_motor">
+        <mechanicalReduction>1</mechanicalReduction>
+      </actuator>
+    </transmission>
+    <transmission name="r_med_phal_2_transmission">
+      <type>transmission_interface/SimpleTransmission</type>
+      <joint name="r_med_phal_2_joint">
+        <hardwareInterface>hardware_interface/VelocityJointInterface</hardwareInterface>
+      </joint>
+      <actuator name="r_med_phal_2_motor">
+        <mechanicalReduction>1</mechanicalReduction>
+      </actuator>
+    </transmission>
+    <transmission name="r_med_phal_3_transmission">
+      <type>transmission_interface/SimpleTransmission</type>
+      <joint name="r_med_phal_3_joint">
+        <hardwareInterface>hardware_interface/VelocityJointInterface</hardwareInterface>
+      </joint>
+      <actuator name="r_med_phal_3_motor">
+        <mechanicalReduction>1</mechanicalReduction>
+      </actuator>
+    </transmission>
+    <transmission name="r_ind_phal_1_transmission">
+      <type>transmission_interface/SimpleTransmission</type>
+      <joint name="r_ind_phal_1_joint">
+        <hardwareInterface>hardware_interface/VelocityJointInterface</hardwareInterface>
+      </joint>
+      <actuator name="r_ind_phal_1_motor">
+        <mechanicalReduction>1</mechanicalReduction>
+      </actuator>
+    </transmission>
+    <transmission name="r_ind_phal_2_transmission">
+      <type>transmission_interface/SimpleTransmission</type>
+      <joint name="r_ind_phal_2_joint">
+        <hardwareInterface>hardware_interface/VelocityJointInterface</hardwareInterface>
+      </joint>
+      <actuator name="r_ind_phal_2_motor">
+        <mechanicalReduction>1</mechanicalReduction>
+      </actuator>
+    </transmission>
+    <transmission name="r_ind_phal_3_transmission">
+      <type>transmission_interface/SimpleTransmission</type>
+      <joint name="r_ind_phal_3_joint">
+        <hardwareInterface>hardware_interface/VelocityJointInterface</hardwareInterface>
+      </joint>
+      <actuator name="r_ind_phal_3_motor">
+        <mechanicalReduction>1</mechanicalReduction>
+      </actuator>
+    </transmission>
+    <transmission name="r_thumb_phal_1_transmission">
+      <type>transmission_interface/SimpleTransmission</type>
+      <joint name="r_thumb_phal_1_joint">
+        <hardwareInterface>hardware_interface/VelocityJointInterface</hardwareInterface>
+      </joint>
+      <actuator name="r_thumb_phal_1_motor">
+        <mechanicalReduction>1</mechanicalReduction>
+      </actuator>
+    </transmission>
+    <transmission name="r_thumb_phal_2_transmission">
+      <type>transmission_interface/SimpleTransmission</type>
+      <joint name="r_thumb_phal_2_joint">
+        <hardwareInterface>hardware_interface/VelocityJointInterface</hardwareInterface>
+      </joint>
+      <actuator name="r_thumb_phal_2_motor">
+        <mechanicalReduction>1</mechanicalReduction>
+      </actuator>
+    </transmission>
+    <transmission name="r_thumb_phal_3_transmission">
+      <type>transmission_interface/SimpleTransmission</type>
+      <joint name="r_thumb_phal_3_joint">
+        <hardwareInterface>hardware_interface/VelocityJointInterface</hardwareInterface>
+      </joint>
+      <actuator name="r_thumb_phal_3_motor">
+        <mechanicalReduction>1</mechanicalReduction>
+      </actuator>
+    </transmission>
   </xacro:macro>
 </robot>

File: vizzy_description/urdf/hand/right_hand.urdf.xacro (robot description, xacro)
@@ -35,9 +35,4 @@
             filename="package://vizzy_description/meshes/hand/r_hand_base_link.STL" />
         </geometry>
-        <material
-          name="">
-          <color
-            rgba="0.796078431372549 0.823529411764706 0.937254901960784 1" />
-        </material>
       </visual>
       <collision>
@@ -88,9 +83,4 @@
             filename="package://vizzy_description/meshes/hand/r_min_phal_1_link.STL" />
         </geometry>
-        <material
-          name="">
-          <color
-            rgba="0.898039215686275 0.917647058823529 0.929411764705882 1" />
-        </material>
       </visual>
       <collision>
@@ -199,9 +189,4 @@
             filename="package://vizzy_description/meshes/hand/r_min_phal_2_link.STL" />
         </geometry>
-        <material
-          name="">
-          <color
-            rgba="0.898039215686275 0.917647058823529 0.929411764705882 1" />
-        </material>
       </visual>
       <collision>
@@ -310,9 +295,4 @@
             filename="package://vizzy_description/meshes/hand/r_min_phal_3_link.STL" />
         </geometry>
-        <material
-          name="">
-          <color
-            rgba="0.898039215686275 0.917647058823529 0.929411764705882 1" />
-        </material>
       </visual>
       <collision>
@@ -421,9 +401,4 @@
             filename="package://vizzy_description/meshes/hand/r_med_phal_1_link.STL" />
         </geometry>
-        <material
-          name="">
-          <color
-            rgba="0.898039215686275 0.917647058823529 0.929411764705882 1" />
-        </material>
       </visual>
       <collision>
@@ -532,9 +507,4 @@
             filename="package://vizzy_description/meshes/hand/r_med_phal_2_link.STL" />
         </geometry>
-        <material
-          name="">
-          <color
-            rgba="0.898039215686275 0.917647058823529 0.929411764705882 1" />
-        </material>
       </visual>
       <collision>
@@ -643,9 +613,4 @@
             filename="package://vizzy_description/meshes/hand/r_med_phal_3_link.STL" />
         </geometry>
-        <material
-          name="">
-          <color
-            rgba="0.898039215686275 0.917647058823529 0.929411764705882 1" />
-        </material>
       </visual>
       <collision>
@@ -754,9 +719,4 @@
             filename="package://vizzy_description/meshes/hand/r_ind_phal_1_link.STL" />
         </geometry>
-        <material
-          name="">
-          <color
-            rgba="0.898039215686275 0.917647058823529 0.929411764705882 1" />
-        </material>
       </visual>
       <collision>
@@ -865,9 +825,4 @@
             filename="package://vizzy_description/meshes/hand/r_ind_phal_2_link.STL" />
         </geometry>
-        <material
-          name="">
-          <color
-            rgba="0.898039215686275 0.917647058823529 0.929411764705882 1" />
-        </material>
       </visual>
       <collision>
@@ -976,9 +931,4 @@
             filename="package://vizzy_description/meshes/hand/r_ind_phal_3_link.STL" />
         </geometry>
-        <material
-          name="">
-          <color
-            rgba="0.898039215686275 0.917647058823529 0.929411764705882 1" />
-        </material>
       </visual>
       <collision>
@@ -1087,9 +1037,4 @@
             filename="package://vizzy_description/meshes/hand/r_thumb_phal_1_link.STL" />
         </geometry>
-        <material
-          name="">
-          <color
-            rgba="0.898039215686275 0.917647058823529 0.929411764705882 1" />
-        </material>
       </visual>
       <collision>
@@ -1145,9 +1090,4 @@
             filename="package://vizzy_description/meshes/hand/r_thumb_phal_1_link_fix.STL" />
         </geometry>
-        <material
-          name="">
-          <color
-            rgba="0.898039215686275 0.917647058823529 0.929411764705882 1" />
-        </material>
       </visual>
       <collision>
@@ -1198,9 +1138,4 @@
             filename="package://vizzy_description/meshes/hand/r_thumb_phal_2_link.STL" />
         </geometry>
-        <material
-          name="">
-          <color
-            rgba="0.898039215686275 0.917647058823529 0.929411764705882 1" />
-        </material>
       </visual>
       <collision>
@@ -1285,20 +1220,19 @@
         xyz="0 0 0" />
     </joint>
-    <!--
     <link
       name="r_thumb_phal_3_link">
       <inertial>
         <origin
-          xyz="-0.0146795008539003 0.000321779082924474 -1.60568615682546E-05"
-          rpy="0 0 0" />
-        <mass
-          value="0.0093590453864441" />
-        <inertia
-          ixx="3.25448933286868E-07"
-          ixy="-7.67923909556657E-09"
-          ixz="-2.9182709100671E-10"
-          iyy="7.82460440615413E-07"
-          iyz="5.74839171195636E-10"
-          izz="7.70225558928889E-07" />
+          xyz="-0.0125548640176916 0.00056252197857469 -1.90460476551368E-05"
+          rpy="0 0 0" />
+        <mass
+          value="0.00838713518345204" />
+        <inertia
+          ixx="2.60505570751336E-07"
+          ixy="-2.79008349627709E-08"
+          ixz="1.74829416361065E-10"
+          iyy="4.40992619187728E-07"
+          iyz="6.2543048992729E-10"
+          izz="4.45479141195201E-07" />
       </inertial>
       <visual>
@@ -1310,9 +1244,4 @@
             filename="package://vizzy_description/meshes/hand/r_thumb_phal_3_link.STL" />
         </geometry>
-        <material
-          name="">
-          <color
-            rgba="0.898039215686275 0.917647058823529 0.929411764705882 1" />
-        </material>
       </visual>
       <collision>
@@ -1330,8 +1259,8 @@
       type="revolute">
       <origin
-        xyz="-0.01625 -0.007 0"
-        rpy="-3.1416 7.494E-16 -5.6162E-17" />
-      <parent
-        link="r_thumb_phal_2_link_fix" />
+        xyz="-0.0332692 0 0"
+        rpy="0 0 0" />
+      <parent
+        link="r_thumb_phal_2_link" />
       <child
         link="r_thumb_phal_3_link" />
@@ -1348,116 +1277,4 @@
       <inertial>
         <origin
-          xyz="-0.0118618974128648 -0.00596650611581801 -5.37425902391586E-11"
-          rpy="0 0 0" />
-        <mass
-          value="0.00257761324342116" />
-        <inertia
-          ixx="9.21932604321348E-08"
-          ixy="3.10961295113261E-08"
-          ixz="-1.64616534423459E-15"
-          iyy="1.23080606212339E-07"
-          iyz="-8.32014412402861E-16"
-          izz="9.04321801244888E-08" />
-      </inertial>
-      <visual>
-        <origin
-          xyz="0 0 0"
-          rpy="0 0 0" />
-        <geometry>
-          <mesh
-            filename="package://vizzy_description/meshes/hand/r_thumb_phal_3_link_fix.STL" />
-        </geometry>
-        <material
-          name="">
-          <color
-            rgba="1 1 1 1" />
-        </material>
-      </visual>
-      <collision>
-        <origin
-          xyz="0 0 0"
-          rpy="0 0 0" />
-        <geometry>
-          <mesh
-            filename="package://vizzy_description/meshes/hand/r_thumb_phal_3_link_fix.STL" />
-        </geometry>
-      </collision>
-    </link>
-    <joint
-      name="r_thumb_phal_3_joint_fix"
-      type="fixed">
-      <origin
-        xyz="-0.013 -0.007 0"
-        rpy="3.1416 -2.7756E-17 -1.8946E-16" />
-      <parent
-        link="r_thumb_phal_3_link" />
-      <child
-        link="r_thumb_phal_3_link_fix" />
-      <axis
-        xyz="0 0 0" />
-    </joint>
-    -->
-    <link
-      name="r_thumb_phal_4_link">
-      <inertial>
-        <origin
-          xyz="-0.0125548640176916 0.00056252197857469 -1.90460476551368E-05"
-          rpy="0 0 0" />
-        <mass
-          value="0.00838713518345204" />
-        <inertia
-          ixx="2.60505570751336E-07"
-          ixy="-2.79008349627709E-08"
-          ixz="1.74829416361065E-10"
-          iyy="4.40992619187728E-07"
-          iyz="6.2543048992729E-10"
-          izz="4.45479141195201E-07" />
-      </inertial>
-      <visual>
-        <origin
-          xyz="0 0 0"
-          rpy="0 0 0" />
-        <geometry>
-          <mesh
-            filename="package://vizzy_description/meshes/hand/r_thumb_phal_4_link.STL" />
-        </geometry>
-        <material
-          name="">
-          <color
-            rgba="0.898039215686275 0.917647058823529 0.929411764705882 1" />
-        </material>
-      </visual>
-      <collision>
-        <origin
-          xyz="0 0 0"
-          rpy="0 0 0" />
-        <geometry>
-          <mesh
-            filename="package://vizzy_description/meshes/hand/r_thumb_phal_4_link.STL" />
-        </geometry>
-      </collision>
-    </link>
-    <joint
-      name="r_thumb_phal_4_joint"
-      type="revolute">
-      <origin
-        xyz="-0.0332692 0 0"
-        rpy="0 0 0" />
-      <parent
-        link="r_thumb_phal_2_link" />
-      <child
-        link="r_thumb_phal_4_link" />
-      <axis
-        xyz="0 0 1" />
-      <limit
-        lower="0"
-        upper="1.57"
-        effort="0"
-        velocity="0" />
-    </joint>
-    <link
-      name="r_thumb_phal_4_link_fix">
-      <inertial>
-        <origin
           xyz="0.00766697409984854 -0.00206053700829757 1.96358397597241E-09"
           rpy="0 0 0" />
@@ -1478,5 +1295,5 @@
         <geometry>
           <mesh
-            filename="package://vizzy_description/meshes/hand/r_thumb_phal_4_link_fix.STL" />
+            filename="package://vizzy_description/meshes/hand/r_thumb_phal_3_link_fix.STL" />
         </geometry>
         <material
@@ -1492,10 +1309,10 @@
         <geometry>
           <mesh
-            filename="package://vizzy_description/meshes/hand/r_thumb_phal_4_link_fix.STL" />
-        </geometry>
-      </collision>
-    </link>
-    <joint
-      name="r_thumb_phal_4_joint_fix"
+            filename="package://vizzy_description/meshes/hand/r_thumb_phal_3_link_fix.STL" />
+        </geometry>
+      </collision>
+    </link>
+    <joint
+      name="r_thumb_phal_3_joint_fix"
       type="fixed">
       <origin
@@ -1503,10 +1320,13 @@
         rpy="-5.7918E-16 -5.8287E-16 -3.1416" />
       <parent
-        link="r_thumb_phal_4_link" />
-      <child
-        link="r_thumb_phal_4_link_fix" />
+        link="r_thumb_phal_3_link" />
+      <child
+        link="r_thumb_phal_3_link_fix" />
       <axis
         xyz="0 0 0" />
     </joint>
   </xacro:macro>
+  <!-- Gazebo extensions -->
+  <xacro:right_hand_transmissions/>
+  <xacro:right_hand_gazebo/>
 </robot>
