Commit message: fix typo and tabs

File: vizzy_description/urdf/arm/arm.urdf.xacro (robot description, xacro)
@@ -58,5 +58,5 @@
     </xacro:if>
     <xacro:unless value="$(arg use_full_hand_model)">
-      <xacro:property name="detailed_hand" value="true"/>
+      <xacro:property name="detailed_hand" value="false"/>
     </xacro:unless>
     <!-- Shoulder scapula -->
