Commit message: using mimic plugin for the hand

File: vizzy_description/urdf/hand/right_hand.transmission.xacro (robot description, xacro)
@@ -11,22 +11,4 @@
       </joint>
       <actuator name="r_min_phal_1_motor">
-        <mechanicalReduction>1</mechanicalReduction>
-      </actuator>
-    </transmission>
-    <transmission name="r_min_phal_2_transmission">
-      <type>transmission_interface/SimpleTransmission</type>
-      <joint name="r_min_phal_2_joint">
-        <hardwareInterface>VelocityJointInterface</hardwareInterface>
-      </joint>
-      <actuator name="r_min_phal_2_motor">
-        <mechanicalReduction>1</mechanicalReduction>
-      </actuator>
-    </transmission>
-    <transmission name="r_min_phal_3_transmission">
-      <type>transmission_interface/SimpleTransmission</type>
-      <joint name="r_min_phal_3_joint">
-        <hardwareInterface>VelocityJointInterface</hardwareInterface>
-      </joint>
-      <actuator name="r_min_phal_3_motor">
         <mechanicalReduction>1</mechanicalReduction>
       </actuator>

File: vizzy_description/urdf/hand/right_hand.urdf.xacro (robot description, xacro)
@@ -164,4 +164,5 @@
       effort="10"
       velocity="10" />
+    <mimic joint="r_min_phal_1_joint" multiplier="1.0" offset="0.0" />
   </joint>
   <link
@@ -222,4 +223,5 @@
       effort="10"
       velocity="10" />
+    <mimic joint="r_min_phal_1_joint" multiplier="1.0" offset="0.0" />
   </joint>
   <link
