Commit message: remove phal from thumb; add launcher
Remove extra phalanx from thumb in right hand.
Added an rviz launcher specifically for the right hand.

File: vizzy_description/urdf/hand/right_hand.urdf.xacro (robot description, xacro)
@@ -1285,4 +1285,5 @@
         xyz="0 0 0" />
     </joint>
+    <!--
     <link
       name="r_thumb_phal_3_link">
@@ -1396,4 +1397,5 @@
         xyz="0 0 0" />
     </joint>
+    -->
     <link
       name="r_thumb_phal_4_link">
@@ -1440,8 +1442,8 @@
       type="revolute">
       <origin
-        xyz="-0.0135 -0.007 0"
-        rpy="-3.1416 -8.3267E-17 -1.4545E-16" />
-      <parent
-        link="r_thumb_phal_3_link_fix" />
+        xyz="-0.0332692 0 0"
+        rpy="0 0 0" />
+      <parent
+        link="r_thumb_phal_2_link" />
       <child
         link="r_thumb_phal_4_link" />

Commit message: add simplified hand collision model
Contact sensors not yet simplified.

File: vizzy_description/urdf/hand/right_hand.urdf.xacro (robot description, xacro)
@@ -37,11 +37,17 @@
       </visual>
       <collision>
-        <origin
-          xyz="0 0 0"
-          rpy="0 0 0" />
-        <geometry>
-          <mesh
-            filename="package://vizzy_description/meshes/hand/r_hand_base_link.STL" />
-        </geometry>
+        <xacro:if value="$(arg use_full_gazebo_model)">
+          <origin xyz="0 0 0" rpy="0 0 0" />
+          <geometry>
+            <mesh
+              filename="package://vizzy_description/meshes/hand/r_hand_base_link.STL" />
+          </geometry>
+        </xacro:if>
+        <xacro:unless value="$(arg use_full_gazebo_model)">
+          <origin xyz="0 -0.0134 0" rpy="0 0 0" />
+          <geometry>
+            <box size="0.090 0.030 0.085"/>
+          </geometry>
+        </xacro:unless>
       </collision>
     </link>
@@ -85,11 +91,19 @@
       </visual>
       <collision>
-        <origin
-          xyz="0 0 0"
-          rpy="0 0 0" />
-        <geometry>
-          <mesh
-            filename="package://vizzy_description/meshes/hand/r_min_phal_1_link.STL" />
-        </geometry>
+        <xacro:if value="$(arg use_full_gazebo_model)">
+          <origin
+            xyz="0 0 0"
+            rpy="0 0 0" />
+          <geometry>
+            <mesh
+              filename="package://vizzy_description/meshes/hand/r_min_phal_1_link.STL" />
+          </geometry>
+        </xacro:if>
+        <xacro:unless value="$(arg use_full_gazebo_model)">
+          <origin xyz="-0.0176 0 0" rpy="0 0 0" />
+          <geometry>
+            <box size="0.0445 0.014 0.014"/>
+          </geometry>
+        </xacro:unless>
       </collision>
     </link>
@@ -191,11 +205,19 @@
       </visual>
       <collision>
-        <origin
-          xyz="0 0 0"
-          rpy="0 0 0" />
-        <geometry>
-          <mesh
-            filename="package://vizzy_description/meshes/hand/r_min_phal_2_link.STL" />
-        </geometry>
+        <xacro:if value="$(arg use_full_gazebo_model)">
+          <origin
+            xyz="0 0 0"
+            rpy="0 0 0" />
+          <geometry>
+            <mesh
+              filename="package://vizzy_description/meshes/hand/r_min_phal_2_link.STL" />
+          </geometry>
+        </xacro:if>
+        <xacro:unless value="$(arg use_full_gazebo_model)">
+          <origin xyz="-0.0145 0 0" rpy="0 0 0" />
+          <geometry>
+            <box size="0.0380 0.014 0.014"/>
+          </geometry>
+        </xacro:unless>
       </collision>
     </link>
@@ -297,11 +319,19 @@
       </visual>
       <collision>
-        <origin
-          xyz="0 0 0"
-          rpy="0 0 0" />
-        <geometry>
-          <mesh
-            filename="package://vizzy_description/meshes/hand/r_min_phal_3_link.STL" />
-        </geometry>
+        <xacro:if value="$(arg use_full_gazebo_model)">
+          <origin
+            xyz="0 0 0"
+            rpy="0 0 0" />
+          <geometry>
+            <mesh
+              filename="package://vizzy_description/meshes/hand/r_min_phal_3_link.STL" />
+          </geometry>
+        </xacro:if>
+        <xacro:unless value="$(arg use_full_gazebo_model)">
+          <origin xyz="-0.010 0 0" rpy="0 0 0" />
+          <geometry>
+            <box size="0.029 0.014 0.014"/>
+          </geometry>
+        </xacro:unless>
       </collision>
     </link>
@@ -403,11 +433,19 @@
       </visual>
       <collision>
-        <origin
-          xyz="0 0 0"
-          rpy="0 0 0" />
-        <geometry>
-          <mesh
-            filename="package://vizzy_description/meshes/hand/r_med_phal_1_link.STL" />
-        </geometry>
+        <xacro:if value="$(arg use_full_gazebo_model)">
+          <origin
+            xyz="0 0 0"
+            rpy="0 0 0" />
+          <geometry>
+            <mesh
+              filename="package://vizzy_description/meshes/hand/r_med_phal_1_link.STL" />
+          </geometry>
+        </xacro:if>
+        <xacro:unless value="$(arg use_full_gazebo_model)">
+          <origin xyz="-0.0176 0 0" rpy="0 0 0" />
+          <geometry>
+            <box size="0.0445 0.014 0.014"/>
+          </geometry>
+        </xacro:unless>
       </collision>
     </link>
@@ -509,11 +547,19 @@
       </visual>
       <collision>
-        <origin
-          xyz="0 0 0"
-          rpy="0 0 0" />
-        <geometry>
-          <mesh
-            filename="package://vizzy_description/meshes/hand/r_med_phal_2_link.STL" />
-        </geometry>
+        <xacro:if value="$(arg use_full_gazebo_model)">
+          <origin
+            xyz="0 0 0"
+            rpy="0 0 0" />
+          <geometry>
+            <mesh
+              filename="package://vizzy_description/meshes/hand/r_med_phal_2_link.STL" />
+          </geometry>
+        </xacro:if>
+        <xacro:unless value="$(arg use_full_gazebo_model)">
+          <origin xyz="-0.0145 0 0" rpy="0 0 0" />
+          <geometry>
+            <box size="0.0380 0.014 0.014"/>
+          </geometry>
+        </xacro:unless>
       </collision>
     </link>
@@ -615,11 +661,19 @@
       </visual>
       <collision>
-        <origin
-          xyz="0 0 0"
-          rpy="0 0 0" />
-        <geometry>
-          <mesh
-            filename="package://vizzy_description/meshes/hand/r_med_phal_3_link.STL" />
-        </geometry>
+        <xacro:if value="$(arg use_full_gazebo_model)">
+          <origin
+            xyz="0 0 0"
+            rpy="0 0 0" />
+          <geometry>
+            <mesh
+              filename="package://vizzy_description/meshes/hand/r_med_phal_3_link.STL" />
+          </geometry>
+        </xacro:if>
+        <xacro:unless value="$(arg use_full_gazebo_model)">
+          <origin xyz="-0.010 0 0" rpy="0 0 0" />
+          <geometry>
+            <box size="0.029 0.014 0.014"/>
+          </geometry>
+        </xacro:unless>
       </collision>
     </link>
@@ -721,11 +775,19 @@
       </visual>
       <collision>
-        <origin
-          xyz="0 0 0"
-          rpy="0 0 0" />
-        <geometry>
-          <mesh
-            filename="package://vizzy_description/meshes/hand/r_ind_phal_1_link.STL" />
-        </geometry>
+        <xacro:if value="$(arg use_full_gazebo_model)">
+          <origin
+            xyz="0 0 0"
+            rpy="0 0 0" />
+          <geometry>
+            <mesh
+              filename="package://vizzy_description/meshes/hand/r_ind_phal_1_link.STL" />
+          </geometry>
+        </xacro:if>
+        <xacro:unless value="$(arg use_full_gazebo_model)">
+          <origin xyz="-0.0176 0 0" rpy="0 0 0" />
+          <geometry>
+            <box size="0.0445 0.014 0.014"/>
+          </geometry>
+        </xacro:unless>
       </collision>
     </link>
@@ -827,11 +889,19 @@
       </visual>
       <collision>
-        <origin
-          xyz="0 0 0"
-          rpy="0 0 0" />
-        <geometry>
-          <mesh
-            filename="package://vizzy_description/meshes/hand/r_ind_phal_2_link.STL" />
-        </geometry>
+        <xacro:if value="$(arg use_full_gazebo_model)">
+          <origin
+            xyz="0 0 0"
+            rpy="0 0 0" />
+          <geometry>
+            <mesh
+              filename="package://vizzy_description/meshes/hand/r_ind_phal_2_link.STL" />
+          </geometry>
+        </xacro:if>
+        <xacro:unless value="$(arg use_full_gazebo_model)">
+          <origin xyz="-0.0145 0 0" rpy="0 0 0" />
+          <geometry>
+            <box size="0.0380 0.014 0.014"/>
+          </geometry>
+        </xacro:unless>
       </collision>
     </link>
@@ -933,11 +1003,19 @@
       </visual>
       <collision>
-        <origin
-          xyz="0 0 0"
-          rpy="0 0 0" />
-        <geometry>
-          <mesh
-            filename="package://vizzy_description/meshes/hand/r_ind_phal_3_link.STL" />
-        </geometry>
+        <xacro:if value="$(arg use_full_gazebo_model)">
+          <origin
+            xyz="0 0 0"
+            rpy="0 0 0" />
+          <geometry>
+            <mesh
+              filename="package://vizzy_description/meshes/hand/r_ind_phal_3_link.STL" />
+          </geometry>
+        </xacro:if>
+        <xacro:unless value="$(arg use_full_gazebo_model)">
+          <origin xyz="-0.010 0 0" rpy="0 0 0" />
+          <geometry>
+            <box size="0.029 0.014 0.014"/>
+          </geometry>
+        </xacro:unless>
       </collision>
     </link>
@@ -1039,11 +1117,19 @@
       </visual>
       <collision>
-        <origin
-          xyz="0 0 0"
-          rpy="0 0 0" />
-        <geometry>
-          <mesh
-            filename="package://vizzy_description/meshes/hand/r_thumb_phal_1_link.STL" />
-        </geometry>
+        <xacro:if value="$(arg use_full_gazebo_model)">
+          <origin
+            xyz="0 0 0"
+            rpy="0 0 0" />
+          <geometry>
+            <mesh
+              filename="package://vizzy_description/meshes/hand/r_thumb_phal_1_link.STL" />
+          </geometry>
+        </xacro:if>
+        <xacro:unless value="$(arg use_full_gazebo_model)">
+          <origin xyz="-0.00326 0 0" rpy="0 0 0" />
+          <geometry>
+            <box size="0.01551 0.014 0.014"/>
+          </geometry>
+        </xacro:unless>
       </collision>
     </link>
@@ -1092,11 +1178,20 @@
       </visual>
       <collision>
-        <origin
-          xyz="0 0 0"
-          rpy="0 0 0" />
-        <geometry>
-          <mesh
-            filename="package://vizzy_description/meshes/hand/r_thumb_phal_1_link_fix.STL" />
-        </geometry>
+        <xacro:if value="$(arg use_full_gazebo_model)">
+          <origin
+            xyz="0 0 0"
+            rpy="0 0 0" />
+          <geometry>
+            <mesh
+              filename="package://vizzy_description/meshes/hand/r_thumb_phal_1_link_fix.STL" />
+          </geometry>
+        </xacro:if>
+        <xacro:unless value="$(arg use_full_gazebo_model)">
+          <!-- TODO -->
+          <origin xyz="0 0 0.003" rpy="0 ${M_PI/2} 0" />
+          <geometry>
+            <box size="0.01852 0.014 0.014"/>
+          </geometry>
+        </xacro:unless>
       </collision>
     </link>
@@ -1140,11 +1235,19 @@
       </visual>
       <collision>
-        <origin
-          xyz="0 0 0"
-          rpy="0 0 0" />
-        <geometry>
-          <mesh
-            filename="package://vizzy_description/meshes/hand/r_thumb_phal_2_link.STL" />
-        </geometry>
+        <xacro:if value="$(arg use_full_gazebo_model)">
+          <origin
+            xyz="0 0 0"
+            rpy="0 0 0" />
+          <geometry>
+            <mesh
+              filename="package://vizzy_description/meshes/hand/r_thumb_phal_2_link.STL" />
+          </geometry>
+        </xacro:if>
+        <xacro:unless value="$(arg use_full_gazebo_model)">
+          <origin xyz="-0.01775 0 0" rpy="0 0 0" />
+          <geometry>
+            <box size="0.0445 0.014 0.014"/>
+          </geometry>
+        </xacro:unless>
       </collision>
     </link>
@@ -1246,11 +1349,19 @@
       </visual>
       <collision>
-        <origin
-          xyz="0 0 0"
-          rpy="0 0 0" />
-        <geometry>
-          <mesh
-            filename="package://vizzy_description/meshes/hand/r_thumb_phal_3_link.STL" />
-        </geometry>
+        <xacro:if value="$(arg use_full_gazebo_model)">
+          <origin
+            xyz="0 0 0"
+            rpy="0 0 0" />
+          <geometry>
+            <mesh
+              filename="package://vizzy_description/meshes/hand/r_thumb_phal_3_link.STL" />
+          </geometry>
+        </xacro:if>
+        <xacro:unless value="$(arg use_full_gazebo_model)">
+          <origin xyz="-0.010 0 0" rpy="0 0 0" />
+          <geometry>
+            <box size="0.029 0.014 0.014"/>
+          </geometry>
+        </xacro:unless>
       </collision>
     </link>
@@ -1259,5 +1370,5 @@
       type="revolute">
       <origin
-        xyz="-0.0332692 0 0"
+        xyz="-0.03300 0 0"
         rpy="0 0 0" />
       <parent
