Commit message: finish simplified hand meshes
Finished simplifying meshes for collision.
Also fixed hand model hierarchy: auxiliary *_fix links are now correctly specified as childless nodes.

File: vizzy_description/urdf/hand/right_hand.urdf.xacro (robot description, xacro)
@@ -6,50 +6,6 @@
   <!-- Load full inertial and collision model or a simplified model -->
   <xacro:arg name="use_full_gazebo_model" default="false"/>
-  <!-- Things that are needed only for Gazebo (not the physical robot).  These include
-       sensor and controller plugin specifications -->
-  <xacro:include filename="$(find vizzy_description)/urdf/hand/right_hand.gazebo.xacro"/>
-  <xacro:include filename="$(find vizzy_description)/urdf/hand/right_hand.transmission.xacro"/>
+  <!-- Define xacro macro -->
   <xacro:macro name="right_hand" params="parent">
-    <link
-      name="r_hand_base_link">
-      <inertial>
-        <origin
-          xyz="-0.00674439077967622 -0.00586648543041128 0.00390957138640023"
-          rpy="0 0 0" />
-        <mass
-          value="0.151046673988997" />
-        <inertia
-          ixx="0.000146470772741843"
-          ixy="1.43292089666054E-06"
-          ixz="2.07342201265105E-05"
-          iyy="0.00022421320055357"
-          iyz="2.70250923997076E-06"
-          izz="9.93519010859762E-05" />
-      </inertial>
-      <visual>
-        <origin
-          xyz="0 0 0"
-          rpy="0 0 0" />
-        <geometry>
-          <mesh
-            filename="package://vizzy_description/meshes/hand/r_hand_base_link.STL" />
-        </geometry>
-      </visual>
-      <collision>
-        <xacro:if value="$(arg use_full_gazebo_model)">
-          <origin xyz="0 0 0" rpy="0 0 0" />
-          <geometry>
-            <mesh
-              filename="package://vizzy_description/meshes/hand/r_hand_base_link.STL" />
-          </geometry>
-        </xacro:if>
-        <xacro:unless value="$(arg use_full_gazebo_model)">
-          <origin xyz="0 -0.0134 0" rpy="0 0 0" />
-          <geometry>
-            <box size="0.090 0.030 0.085"/>
-          </geometry>
-        </xacro:unless>
-      </collision>
-    </link>
     <joint
       name="r_hand_base_joint_fix"
@@ -57,5 +13,5 @@
       <origin
         xyz="0.007 -0.076 0.009"
-        rpy="${M_PI / 2} 0 0" />
+        rpy="1.570796 0 0" />
       <parent
         link="${parent}" />
@@ -66,18 +22,64 @@
     </joint>
     <link
+      name="r_hand_base_link">
+      <inertial>
+        <origin
+          xyz="-0.00674438981790416 -0.0058664849056831 0.00390957326685741"
+          rpy="0 0 0" />
+        <mass
+          value="0.151046667629674" />
+        <inertia
+          ixx="0.000146470764076254"
+          ixy="-1.43291885346107E-06"
+          ixz="-2.07342162004204E-05"
+          iyy="0.000224213192446366"
+          iyz="-2.70250573740841E-06"
+          izz="9.93519001771392E-05" />
+      </inertial>
+      <visual>
+        <origin
+          xyz="0 0 0"
+          rpy="0 0 0" />
+        <geometry>
+          <mesh
+            filename="package://vizzy_description/meshes/hand/r_hand_base_link.STL" />
+        </geometry>
+        <material
+          name="">
+          <color
+            rgba="0.796078431372549 0.823529411764706 0.937254901960784 1" />
+        </material>
+      </visual>
+      <collision>
+        <xacro:if value="$(arg use_full_gazebo_model)">
+          <origin xyz="0 0 0" rpy="0 0 0" />
+          <geometry>
+            <mesh
+              filename="package://vizzy_description/meshes/hand/r_hand_base_link.STL" />
+          </geometry>
+        </xacro:if>
+        <xacro:unless value="$(arg use_full_gazebo_model)">
+          <origin xyz="-0.008 -0.0134 0" rpy="0 0 0" />
+          <geometry>
+            <box size="0.090 0.030 0.0900"/>
+          </geometry>
+        </xacro:unless>
+      </collision>
+    </link>
+    <link
       name="r_min_phal_1_link">
       <inertial>
         <origin
-          xyz="-0.0178212692703573 0.000338633799509282 -8.48495256814547E-06"
+          xyz="-0.0065863332980695 0.000338633799509286 0.0178212692703573"
           rpy="0 0 0" />
         <mass
           value="0.0123116066856987" />
         <inertia
-          ixx="4.19810828425124E-07"
-          ixy="-8.28056937395445E-09"
-          ixz="-1.27867316658423E-10"
+          ixx="1.31758404800717E-06"
+          ixy="-3.84070099097907E-10"
+          ixz="-1.27867316658086E-10"
           iyy="1.33241779844217E-06"
-          iyz="3.84070099097823E-10"
-          izz="1.31758404800717E-06" />
+          iyz="-8.28056937395449E-09"
+          izz="4.19810828425124E-07" />
       </inertial>
       <visual>
@@ -89,19 +91,24 @@
             filename="package://vizzy_description/meshes/hand/r_min_phal_1_link.STL" />
         </geometry>
-      </visual>
-      <collision>
-        <xacro:if value="$(arg use_full_gazebo_model)">
-          <origin
-            xyz="0 0 0"
-            rpy="0 0 0" />
-          <geometry>
-            <mesh
-              filename="package://vizzy_description/meshes/hand/r_min_phal_1_link.STL" />
-          </geometry>
-        </xacro:if>
-        <xacro:unless value="$(arg use_full_gazebo_model)">
-          <origin xyz="-0.0176 0 0" rpy="0 0 0" />
-          <geometry>
-            <box size="0.0445 0.014 0.014"/>
+        <material
+          name="">
+          <color
+            rgba="0.898039215686275 0.917647058823529 0.929411764705882 1" />
+        </material>
+      </visual>
+      <collision>
+        <xacro:if value="$(arg use_full_gazebo_model)">
+          <origin
+            xyz="0 0 0"
+            rpy="0 0 0" />
+          <geometry>
+            <mesh
+              filename="package://vizzy_description/meshes/hand/r_hand/min_phal_1_link.STL" />
+          </geometry>
+        </xacro:if>
+        <xacro:unless value="$(arg use_full_gazebo_model)">
+          <origin xyz="-0.0068 0 0.0177" rpy="0 0 0" />
+          <geometry>
+            <box size="0.0136 0.0136 0.0445"/>
           </geometry>
         </xacro:unless>
@@ -112,10 +119,138 @@
       type="revolute">
       <origin
-        xyz="0.02708 -0.005836 0.043291"
-        rpy="5.9237E-16 1.3963 -3.1416" />
+        xyz="0.0206022740439909 -0.00583604310721738 0.0444337137891329"
+        rpy="6.21748940377807E-17 -0.174532925199439 3.14159265358979" />
       <parent
         link="r_hand_base_link" />
       <child
         link="r_min_phal_1_link" />
+      <axis
+        xyz="1 0 0" />
+      <limit
+        lower="0"
+        upper="1.57"
+        effort="0"
+        velocity="0" />
+    </joint>
+    <link
+      name="r_min_phal_1_link_fix">
+      <inertial>
+        <origin
+          xyz="-0.00172879723518117 0.00767822711194731 0.00062912481037776"
+          rpy="0 0 0" />
+        <mass
+          value="0.00282550462257503" />
+        <inertia
+          ixx="2.01497129990919E-07"
+          ixy="2.16240614332509E-08"
+          ixz="5.94116205047544E-08"
+          iyy="1.72890117193847E-07"
+          iyz="-2.30807929346575E-08"
+          izz="1.17876895053349E-07" />
+      </inertial>
+      <visual>
+        <origin
+          xyz="0 0 0"
+          rpy="0 0 0" />
+        <geometry>
+          <mesh
+            filename="package://vizzy_description/meshes/hand/r_min_phal_1_link_fix.STL" />
+        </geometry>
+        <material
+          name="">
+          <color
+            rgba="0.776470588235294 0.756862745098039 0.737254901960784 1" />
+        </material>
+      </visual>
+      <collision>
+        <xacro:if value="$(arg use_full_gazebo_model)">
+          <origin
+            xyz="0 0 0"
+            rpy="0 0 0" />
+          <geometry>
+            <mesh
+              filename="package://vizzy_description/meshes/hand/r_hand/r_min_phal_1_link_fix.STL" />
+          </geometry>
+        </xacro:if>
+        <xacro:unless value="$(arg use_full_gazebo_model)">
+          <origin xyz="-0.009 0.01200 0.01300"
+            rpy="-3.1416 -1.2217 1.5708" />
+          <geometry>
+            <box size="0.015 0.0045 0.011"/>
+          </geometry>
+        </xacro:unless>
+      </collision>
+    </link>
+    <joint
+      name="r_min_phal_1_joint_fix"
+      type="fixed">
+      <origin
+        xyz="-0.0135778483455014 0 0.033"
+        rpy="-2.79252680319092 -2.96655185942005E-17 1.5707963267949" />
+      <parent
+        link="r_min_phal_1_link" />
+      <child
+        link="r_min_phal_1_link_fix" />
+      <axis
+        xyz="0 0 0" />
+    </joint>
+    <link
+      name="r_min_phal_2_link">
+      <inertial>
+        <origin
+          xyz="-0.0146794976295984 0.000321778454853602 -1.60585011899778E-05"
+          rpy="0 0 0" />
+        <mass
+          value="0.00935905263397591" />
+        <inertia
+          ixx="3.25448973931958E-07"
+          ixy="7.6792767696661E-09"
+          ixz="2.91914436315786E-10"
+          iyy="7.82460629612251E-07"
+          iyz="-5.74854295945315E-10"
+          izz="7.70225783044348E-07" />
+      </inertial>
+      <visual>
+        <origin
+          xyz="0 0 0"
+          rpy="0 0 0" />
+        <geometry>
+          <mesh
+            filename="package://vizzy_description/meshes/hand/r_min_phal_2_link.STL" />
+        </geometry>
+        <material
+          name="">
+          <color
+            rgba="0.898039215686275 0.917647058823529 0.929411764705882 1" />
+        </material>
+      </visual>
+      <collision>
+        <xacro:if value="$(arg use_full_gazebo_model)">
+          <origin
+            xyz="0 0 0"
+            rpy="0 0 0" />
+          <geometry>
+            <mesh
+              filename="package://vizzy_right_hand/min_phal_2_link.STL" />
+          </geometry>
+        </xacro:if>
+        <xacro:unless value="$(arg use_full_gazebo_model)">
+          <origin xyz="-0.0145 0 0" rpy="0 0 0" />
+          <geometry>
+            <box size="0.0380 0.0136 0.0136"/>
+          </geometry>
+        </xacro:unless>
+      </collision>
+    </link>
+    <joint
+      name="r_min_phal_2_joint"
+      type="revolute">
+      <origin
+        xyz="-0.00657784834550136 0 0.0330000000000001"
+        rpy="0.390965355013273 1.57079631189374 0.404891786285083" />
+      <parent
+        link="r_min_phal_1_link" />
+      <child
+        link="r_min_phal_2_link" />
       <axis
         xyz="0 0 1" />
@@ -127,26 +262,26 @@
     </joint>
     <link
-      name="r_min_phal_1_link_fix">
-      <inertial>
-        <origin
-          xyz="-0.00172879723518149 0.00767822711194729 0.000629124810377732"
-          rpy="0 0 0" />
-        <mass
-          value="0.00282550462257503" />
-        <inertia
-          ixx="2.01497129990919E-07"
-          ixy="-2.16240614332529E-08"
-          ixz="-5.9411620504755E-08"
-          iyy="1.72890117193849E-07"
-          iyz="2.30807929346573E-08"
-          izz="1.1787689505335E-07" />
-      </inertial>
-      <visual>
-        <origin
-          xyz="0 0 0"
-          rpy="0 0 0" />
-        <geometry>
-          <mesh
-            filename="package://vizzy_description/meshes/hand/r_min_phal_1_link_fix.STL" />
+      name="r_min_phal_2_link_fix">
+      <inertial>
+        <origin
+          xyz="0.00103349935688929 0.00697346811741156 -0.0017476111791478"
+          rpy="0 0 0" />
+        <mass
+          value="0.00257761474790775" />
+        <inertia
+          ixx="1.23080849742913E-07"
+          ixy="4.8733648423492E-10"
+          ixz="3.10924773578245E-08"
+          iyy="9.04329465453797E-08"
+          iyz="2.75926783373023E-11"
+          izz="9.21929606188827E-08" />
+      </inertial>
+      <visual>
+        <origin
+          xyz="0 0 0"
+          rpy="0 0 0" />
+        <geometry>
+          <mesh
+            filename="package://vizzy_description/meshes/hand/r_min_phal_2_link_fix.STL" />
         </geometry>
         <material
@@ -157,79 +292,93 @@
       </visual>
       <collision>
-        <origin
-          xyz="0 0 0"
-          rpy="0 0 0" />
-        <geometry>
-          <mesh
-            filename="package://vizzy_description/meshes/hand/r_min_phal_1_link_fix.STL" />
-        </geometry>
-      </collision>
-    </link>
-    <joint
-      name="r_min_phal_1_joint_fix"
+        <xacro:if value="$(arg use_full_gazebo_model)">
+          <origin
+            xyz="0 0 0"
+            rpy="0 0 0" />
+          <geometry>
+            <mesh
+              filename="package://vizzy_description/meshes/hand/r_hand/r_min_phal_2_link_fix.STL" />
+          </geometry>
+        </xacro:if>
+        <xacro:unless value="$(arg use_full_gazebo_model)">
+          <origin xyz="0.009 0.0067 -0.0136"
+            rpy="3.1416 1.5551 -1.5708" />
+          <geometry>
+            <box size="0.008 0.0045 0.011"/>
+          </geometry>
+        </xacro:unless>
+      </collision>
+    </link>
+    <joint
+      name="r_min_phal_2_joint_fix"
       type="fixed">
       <origin
-        xyz="-0.033 0 -0.007"
-        rpy="1.9199 2.6299E-16 1.5708" />
-      <parent
-        link="r_min_phal_1_link" />
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