Commit message: setting up right hand in simulation

File: vizzy_description/urdf/hand/right_hand.gazebo.xacro (robot description, xacro)
@@ -30,4 +30,60 @@
    <gazebo reference="r_thumb_phal_4_link">
    </gazebo>
+		<gazebo>
+			<plugin name="mimic_plugin" filename="libgazebo_mimic_plugin.so">
+				<joint>r_min_phal_1_joint</joint>
+				<mimicJoint>r_min_phal_2_joint</mimicJoint>
+				<multiplier>0.5</multiplier>
+			</plugin>
+		</gazebo>
+		<gazebo>
+			<plugin name="mimic_plugin" filename="libgazebo_mimic_plugin.so">
+				<joint>r_min_phal_1_joint</joint>
+				<mimicJoint>r_min_phal_3_joint</mimicJoint>
+				<multiplier>0.5</multiplier>
+			</plugin>
+		</gazebo>
+		<gazebo>
+			<plugin name="mimic_plugin" filename="libgazebo_mimic_plugin.so">
+				<joint>r_med_phal_1_joint</joint>
+				<mimicJoint>r_med_phal_2_joint</mimicJoint>
+				<multiplier>0.5</multiplier>
+			</plugin>
+		</gazebo>
+		<gazebo>
+			<plugin name="mimic_plugin" filename="libgazebo_mimic_plugin.so">
+				<joint>r_med_phal_1_joint</joint>
+				<mimicJoint>r_med_phal_3_joint</mimicJoint>
+				<multiplier>0.5</multiplier>
+			</plugin>
+		</gazebo>
+		<gazebo>
+			<plugin name="mimic_plugin" filename="libgazebo_mimic_plugin.so">
+				<joint>r_ind_phal_1_joint</joint>
+				<mimicJoint>r_ind_phal_2_joint</mimicJoint>
+				<multiplier>0.5</multiplier>
+			</plugin>
+		</gazebo>
+		<gazebo>
+			<plugin name="mimic_plugin" filename="libgazebo_mimic_plugin.so">
+				<joint>r_ind_phal_1_joint</joint>
+				<mimicJoint>r_ind_phal_3_joint</mimicJoint>
+				<multiplier>0.5</multiplier>
+			</plugin>
+		</gazebo>
+		<gazebo>
+			<plugin name="mimic_plugin" filename="libgazebo_mimic_plugin.so">
+				<joint>r_thumb_phal_2_joint</joint>
+				<mimicJoint>r_thumb_phal_3_joint</mimicJoint>
+				<multiplier>0.5</multiplier>
+			</plugin>
+		</gazebo>
+		<gazebo>
+			<plugin name="mimic_plugin" filename="libgazebo_mimic_plugin.so">
+				<joint>r_thumb_phal_2_joint</joint>
+				<mimicJoint>r_thumb_phal_4_joint</mimicJoint>
+				<multiplier>0.5</multiplier>
+			</plugin>
+		</gazebo>
   </xacro:macro>
 </robot>

Commit message: remove unused/outdated mimic plugin references

File: vizzy_description/urdf/hand/right_hand.gazebo.xacro (robot description, xacro)
@@ -3,64 +3,4 @@
   <!-- Instance mimic plugins for underactuated finger control -->
   <xacro:macro name="right_hand_gazebo">
-    <!-- Min underactuated finger -->
-    <gazebo>
-      <plugin name="mimic_plugin" filename="libgazebo_mimic_plugin.so">
-        <joint>r_min_phal_1_joint</joint>
-        <mimicJoint>r_min_phal_2_joint</mimicJoint>
-        <multiplier>0.5</multiplier>
-      </plugin>
-    </gazebo>
-    <gazebo>
-      <plugin name="mimic_plugin" filename="libgazebo_mimic_plugin.so">
-        <joint>r_min_phal_1_joint</joint>
-        <mimicJoint>r_min_phal_3_joint</mimicJoint>
-        <multiplier>0.5</multiplier>
-      </plugin>
-    </gazebo>
-    <!-- Med underactuated finger -->
-    <gazebo>
-      <plugin name="mimic_plugin" filename="libgazebo_mimic_plugin.so">
-        <joint>r_med_phal_1_joint</joint>
-        <mimicJoint>r_med_phal_2_joint</mimicJoint>
-        <multiplier>0.5</multiplier>
-      </plugin>
-    </gazebo>
-    <gazebo>
-      <plugin name="mimic_plugin" filename="libgazebo_mimic_plugin.so">
-        <joint>r_med_phal_1_joint</joint>
-        <mimicJoint>r_med_phal_3_joint</mimicJoint>
-        <multiplier>0.5</multiplier>
-      </plugin>
-    </gazebo>
-    <!-- Ind underactuated finger -->
-    <gazebo>
-      <plugin name="mimic_plugin" filename="libgazebo_mimic_plugin.so">
-        <joint>r_ind_phal_1_joint</joint>
-        <mimicJoint>r_ind_phal_2_joint</mimicJoint>
-        <multiplier>0.5</multiplier>
-      </plugin>
-    </gazebo>
-    <gazebo>
-      <plugin name="mimic_plugin" filename="libgazebo_mimic_plugin.so">
-        <joint>r_ind_phal_1_joint</joint>
-        <mimicJoint>r_ind_phal_3_joint</mimicJoint>
-        <multiplier>0.5</multiplier>
-      </plugin>
-    </gazebo>
-    <!-- Thumb underactuated finger -->
-    <gazebo>
-      <plugin name="mimic_plugin" filename="libgazebo_mimic_plugin.so">
-        <joint>r_thumb_phal_2_joint</joint>
-        <mimicJoint>r_thumb_phal_3_joint</mimicJoint>
-        <multiplier>0.5</multiplier>
-      </plugin>
-    </gazebo>
-    <gazebo>
-      <plugin name="mimic_plugin" filename="libgazebo_mimic_plugin.so">
-        <joint>r_thumb_phal_2_joint</joint>
-        <mimicJoint>r_thumb_phal_4_joint</mimicJoint>
-        <multiplier>0.5</multiplier>
-      </plugin>
-    </gazebo>
   </xacro:macro>
 </robot>

Commit message: add right hand position controllers
Parameters still need to be fine-tuned, but everything seems to be working.
Each finger joint has dedicated motor.

File: vizzy_description/urdf/hand/right_hand.gazebo.xacro (robot description, xacro)
@@ -1,5 +1,6 @@
 <?xml version="1.0"?>
 <robot xmlns:xacro="http://ros.org/wiki/xacro">
-  <!-- Instance mimic plugins for underactuated finger control -->
+  <!-- TODO: Model underactuated fingers
+  	e.g. by instancing mimic joint plugin -->
   <xacro:macro name="right_hand_gazebo">
   </xacro:macro>

File: vizzy_description/urdf/hand/right_hand.transmission.xacro (robot description, xacro)
@@ -5,5 +5,5 @@
        xmlns:xacro="http://ros.org/wiki/xacro">
   <xacro:macro name="right_hand_transmissions">
-  	<transmission name="r_min_phal_1_transmission">
+    <transmission name="r_min_phal_1_transmission">
       <type>transmission_interface/SimpleTransmission</type>
       <joint name="r_min_phal_1_joint">
@@ -11,4 +11,22 @@
       </joint>
       <actuator name="r_min_phal_1_motor">
+        <mechanicalReduction>1</mechanicalReduction>
+      </actuator>
+    </transmission>
+    <transmission name="r_min_phal_2_transmission">
+      <type>transmission_interface/SimpleTransmission</type>
+      <joint name="r_min_phal_2_joint">
+        <hardwareInterface>hardware_interface/VelocityJointInterface</hardwareInterface>
+      </joint>
+      <actuator name="r_min_phal_2_motor">
+        <mechanicalReduction>1</mechanicalReduction>
+      </actuator>
+    </transmission>
+    <transmission name="r_min_phal_3_transmission">
+      <type>transmission_interface/SimpleTransmission</type>
+      <joint name="r_min_phal_3_joint">
+        <hardwareInterface>hardware_interface/VelocityJointInterface</hardwareInterface>
+      </joint>
+      <actuator name="r_min_phal_3_motor">
         <mechanicalReduction>1</mechanicalReduction>
       </actuator>

File: vizzy_description/urdf/hand/right_hand.urdf.xacro (robot description, xacro)
@@ -6,4 +6,5 @@
   <!-- Load full inertial and collision model or a simplified model -->
   <xacro:arg name="use_full_gazebo_model" default="false"/>
+  <xacro:include filename="$(find vizzy_description)/urdf/hand/right_hand.transmission.xacro" />
   <!-- Define xacro macro -->
   <xacro:macro name="right_hand" params="parent">
@@ -130,6 +131,6 @@
         lower="0"
         upper="1.57"
-        effort="0"
-        velocity="0" />
+        effort="10.6"
+        velocity="1.6" />
     </joint>
     <link
@@ -258,6 +259,6 @@
         lower="0"
         upper="1.57"
-        effort="0"
-        velocity="0" />
+        effort="10.6"
+        velocity="1.6" />
     </joint>
     <link
@@ -386,6 +387,6 @@
         lower="0"
         upper="1.57"
-        effort="0"
-        velocity="0" />
+        effort="10.6"
+        velocity="1.6" />
     </joint>
     <link
@@ -514,6 +515,6 @@
         lower="0"
         upper="1.57"
-        effort="0"
-        velocity="0" />
+        effort="10.6"
+        velocity="1.6" />
     </joint>
     <link
@@ -642,6 +643,6 @@
         lower="0"
         upper="1.57"
-        effort="0"
-        velocity="0" />
+        effort="10.6"
+        velocity="1.6" />
     </joint>
     <link
@@ -770,6 +771,6 @@
         lower="0"
         upper="1.57"
-        effort="0"
-        velocity="0" />
+        effort="10.6"
+        velocity="1.6" />
     </joint>
     <link
@@ -898,6 +899,6 @@
         lower="0"
         upper="1.57"
-        effort="0"
-        velocity="0" />
+        effort="10.6"
+        velocity="1.6" />
     </joint>
     <link
@@ -1026,6 +1027,6 @@
         lower="0"
         upper="1.57"
-        effort="0"
-        velocity="0" />
+        effort="10.6"
+        velocity="1.6" />
     </joint>
     <link
@@ -1154,6 +1155,6 @@
         lower="0"
         upper="1.57"
-        effort="0"
-        velocity="0" />
+        effort="10.6"
+        velocity="1.6" />
     </joint>
     <link
@@ -1282,6 +1283,6 @@
         lower="0"
         upper="1.57"
-        effort="0"
-        velocity="0" />
+        effort="10.6"
+        velocity="1.6" />
     </joint>
     <link
@@ -1409,6 +1410,6 @@
         lower="0"
         upper="1.57"
-        effort="0"
-        velocity="0" />
+        effort="10.6"
+        velocity="1.6" />
     </joint>
     <link
@@ -1489,6 +1490,6 @@
         lower="0"
         upper="1.57"
-        effort="0"
-        velocity="0" />
+        effort="10.6"
+        velocity="1.6" />
     </joint>
     <link
@@ -1602,4 +1603,6 @@
         xyz="0 0 0" />
     </joint>
+    <!-- Gazebo extensions -->
+    <xacro:right_hand_transmissions/>
   </xacro:macro>
 </robot>
