Commit message: Solving more kinetic stuff..

File: vizzy_description/urdf/common.urdf.xacro (robot description, xacro)
@@ -14,18 +14,18 @@
   <xacro:property name="SENSOR_BEAM_LENGTH" value="10.75" /> <!-- inches -->
 	<!-- Motor transmissions -->
-  <xacro:property name="2232U024SR_motor_transmission_reduction" value="100" /> <!--small-->
-  <xacro:property name="3242G024CR_motor_transmission_reduction" value="100" /> <!--medium-->
-  <xacro:property name="3257G024CR_motor_transmission_reduction" value="371" /> <!-- large -->
-  <xacro:property name="3863H024C_motor_transmission_reduction" value="700" /> <!-- huge -->
+  <xacro:property name="A2232U024SR_motor_transmission_reduction" value="100" /> <!--small-->
+  <xacro:property name="A3242G024CR_motor_transmission_reduction" value="100" /> <!--medium-->
+  <xacro:property name="A3257G024CR_motor_transmission_reduction" value="371" /> <!-- large -->
+  <xacro:property name="A3863H024C_motor_transmission_reduction" value="700" /> <!-- huge -->
 	<!-- Motor max efforts (N.m)-->
-  <xacro:property name="2232U024SR_motor_max_effort" value="2.8" />
-  <xacro:property name="3242G024CR_motor_max_effort" value="11.3" />
-  <xacro:property name="3257G024CR_motor_max_effort" value="105.6" />
-  <xacro:property name="3863H024C_motor_max_effort" value="525" />
+  <xacro:property name="A2232U024SR_motor_max_effort" value="2.8" />
+  <xacro:property name="A3242G024CR_motor_max_effort" value="11.3" />
+  <xacro:property name="A3257G024CR_motor_max_effort" value="105.6" />
+  <xacro:property name="A3863H024C_motor_max_effort" value="525" />
 	<!-- Motor max velocities degrees per second-->
-  <xacro:property name="2232U024SR_motor_max_velocitiy" value="426" />
-  <xacro:property name="3242G024CR_motor_max_velocitiy" value="300" />
-  <xacro:property name="3257G024CR_motor_max_velocitiy" value="300" />
-  <xacro:property name="3863H024C_motor_max_velocitiy" value="34" />
+  <xacro:property name="A2232U024SR_motor_max_velocitiy" value="426" />
+  <xacro:property name="A3242G024CR_motor_max_velocitiy" value="300" />
+  <xacro:property name="A3257G024CR_motor_max_velocitiy" value="300" />
+  <xacro:property name="A3863H024C_motor_max_velocitiy" value="34" />
   <!-- colors -->
   <material name="light_grey">

File: vizzy_description/urdf/torso/torso.transmission.xacro (robot description, xacro)
@@ -11,5 +11,5 @@
       </joint>
       <actuator name="waist_motor">
-        <mechanicalReduction>${3863H024C_motor_transmission_reduction}</mechanicalReduction>
+        <mechanicalReduction>${A3863H024C_motor_transmission_reduction}</mechanicalReduction>
       </actuator>
     </transmission>

File: vizzy_description/urdf/torso/torso.urdf.xacro (robot description, xacro)
@@ -61,5 +61,5 @@
     <axis
       xyz="0 0 1" />
-    <limit lower="-0.34906585" upper="0.34906585" effort="${3863H024C_motor_max_effort}" velocity="${3863H024C_motor_max_velocitiy*DEG_TO_RAD}" />
+    <limit lower="-0.34906585" upper="0.34906585" effort="${A3863H024C_motor_max_effort}" velocity="${A3863H024C_motor_max_velocitiy*DEG_TO_RAD}" />
   </joint>
   <link name="waist_fixed_virtual_link">
@@ -84,5 +84,5 @@
     <axis
       xyz="0 0 1" />
-    <limit lower="-0.34906585" upper="0.34906585" effort="${3863H024C_motor_max_effort}" velocity="${3863H024C_motor_max_velocitiy*DEG_TO_RAD}" />
+    <limit lower="-0.34906585" upper="0.34906585" effort="${A3863H024C_motor_max_effort}" velocity="${A3863H024C_motor_max_velocitiy*DEG_TO_RAD}" />
   </joint>
   <!-- gazebo extensions -->
