Commit message: minor changes

File: vizzy_description/plugins/ros.gazebo.xacro (robot description, xacro)
@@ -34,8 +34,8 @@
         <camera name="head">
           <!--<horizontal_fov>1.4912</horizontal_fov>-->
-          <horizontal_fov>1.4912</horizontal_fov>
+          <horizontal_fov>1.57079632679</horizontal_fov>
           <image>
-            <width>100</width>
-            <height>100</height>
+            <width>200</width>
+            <height>200</height>
 	    <!--<width>640</width>
             <height>480</height>-->

File: vizzy_description/urdf/head/head.ros.urdf.xacro (robot description, xacro)
@@ -60,5 +60,6 @@
     <axis
       xyz="0 0 1" />
-    <limit lower="-0.925024504" upper="0.925024504" effort="10.0" velocity="5.0" />
+    <!--<limit lower="-0.925024504" upper="0.925024504" effort="10.0" velocity="5.0" />-->
+    <limit lower="-2.025024504" upper="2.025024504" effort="10.0" velocity="5.0" />
   </joint>
   <link
@@ -115,5 +116,5 @@
       xyz="0 0 1" />
     <!--<limit lower="-0.314159265" upper="0.645771823" effort="100.0" velocity="5.0" />-->
-    <limit lower="-0.614159265" upper="0.645771823" effort="100.0" velocity="5.0" />
+    <limit lower="-2.014159265" upper="2.45771823" effort="100.0" velocity="5.0" />
   </joint>
   <link

Commit message: Revert "Merge branch 'master' of https://github.com/vislab-tecnico-lisboa/vizzy"
This reverts commit 2bcb53630b2c998dc2cb55be83fabcd4c9588693, reversing
changes made to 74adfcb3dac4797df8528e8c484abf1425be7f07.

File: vizzy_description/plugins/ros.gazebo.xacro (robot description, xacro)
@@ -34,8 +34,8 @@
         <camera name="head">
           <!--<horizontal_fov>1.4912</horizontal_fov>-->
-          <horizontal_fov>1.57079632679</horizontal_fov>
+          <horizontal_fov>1.4912</horizontal_fov>
           <image>
-            <width>200</width>
-            <height>200</height>
+            <width>100</width>
+            <height>100</height>
 	    <!--<width>640</width>
             <height>480</height>-->

File: vizzy_description/robots/vizzy.urdf.xacro (robot description, xacro)
@@ -1,4 +1,5 @@
 <?xml version="1.0"?>
 <robot  name="vizzy" xmlns:xacro="http://ros.org/wiki/xacro" >
+	<xacro:arg name="use_yarp" default="false"/>
   <!-- The following include files set up definitions of parts of the robot body  -->
   <!-- misc common stuff -->
@@ -11,10 +12,15 @@
   <xacro:include filename="$(find vizzy_description)/urdf/torso/torso.urdf.xacro" />
   <!-- head -->
-  <xacro:include filename="$(find vizzy_description)/urdf/head/head.ros.urdf.xacro" />
+  <xacro:if value="$(arg use_yarp)">
+  	<xacro:include filename="$(find vizzy_description)/urdf/head/head.yarp.urdf.xacro" />
+  </xacro:if>
+  <xacro:unless value="$(arg use_yarp)">
+  	<xacro:include filename="$(find vizzy_description)/urdf/head/head.ros.urdf.xacro" />
+  </xacro:unless>
   <!-- left arm -->
   <xacro:include filename="$(find vizzy_description)/urdf/arm/left_arm.urdf.xacro" />
   <!-- right arm -->
   <xacro:include filename="$(find vizzy_description)/urdf/arm/right_arm.urdf.xacro" />
-  <!-- The following include files contain gazebo plugins -->
+	<!-- The following include files contain gazebo plugins -->
   <!-- ROS -->
   <xacro:include filename="$(find vizzy_description)/plugins/ros.gazebo.xacro" />
@@ -43,5 +49,14 @@
   <xacro:camera_plugin name="l_camera" prefix="l"/>
   <xacro:camera_plugin name="r_camera" prefix="r"/>
+  <!-- instantiate Yarp plugins -->
+  <xacro:if value="$(arg use_yarp)">
+		<xacro:torso_gazebo_control/>
+		<xacro:head_gazebo_control/>
+		<xacro:left_arm_gazebo_control/>
+		<xacro:right_arm_gazebo_control/>
+  </xacro:if>
   <!-- instantiate ROS plugins -->
-  <xacro:ros_control_gazebo/>
+  <xacro:unless value="$(arg use_yarp)">
+		<xacro:ros_control_gazebo/>
+  </xacro:unless>
 </robot>

File: vizzy_description/urdf/head/head.ros.urdf.xacro (robot description, xacro)
@@ -60,6 +60,5 @@
     <axis
       xyz="0 0 1" />
-    <!--<limit lower="-0.925024504" upper="0.925024504" effort="10.0" velocity="5.0" />-->
-    <limit lower="-2.025024504" upper="2.025024504" effort="10.0" velocity="5.0" />
+    <limit lower="-0.925024504" upper="0.925024504" effort="10.0" velocity="5.0" />
   </joint>
   <link
@@ -116,5 +115,5 @@
       xyz="0 0 1" />
     <!--<limit lower="-0.314159265" upper="0.645771823" effort="100.0" velocity="5.0" />-->
-    <limit lower="-2.014159265" upper="2.45771823" effort="100.0" velocity="5.0" />
+    <limit lower="-0.614159265" upper="0.645771823" effort="100.0" velocity="5.0" />
   </joint>
   <link

File: vizzy_description/urdf/head/head.yarp.gazebo.xacro (robot description, xacro)
@@ -3,27 +3,15 @@
   <xacro:macro name="head_gazebo">
     <gazebo reference="neck_pan_link">
+      <mu1>0.2</mu1>
+      <mu2>0.2</mu2>
     </gazebo>
     <gazebo reference="neck_tilt_link">
+      <mu1>0.2</mu1>
+      <mu2>0.2</mu2>
     </gazebo>
     <gazebo reference="eyes_tilt_link">
+      <mu1>0.2</mu1>
+      <mu2>0.2</mu2>
     </gazebo>
-    <gazebo reference="version_link">
-    </gazebo>
-    <gazebo reference="r_eye_version_link">
-    </gazebo>
-    <gazebo reference="l_eye_version_link">
-    </gazebo>
-    <gazebo reference="vergence_link">
-    </gazebo>
-  <gazebo reference="r_eye_vergence_link">
-    </gazebo>
-    <gazebo reference="l_eye_vergence_link">
-    </gazebo>
- 		<gazebo reference="neck_pan_joint">
-		</gazebo>
- 		<gazebo reference="neck_tilt_joint">
-		</gazebo>
- 		<gazebo reference="eyes_tilt_joint">
-		</gazebo>
     <gazebo reference="r_eye_pan_link">
       <mu1>0.2</mu1>

File: vizzy_description/urdf/head/head.yarp.urdf.xacro (robot description, xacro)
@@ -237,5 +237,6 @@
     <child link="r_camera_link" />
   </joint>
-  <link name="l_eye_pan_link">
+  <link
+    name="l_eye_pan_link">
     <inertial>
       <origin
@@ -298,68 +299,8 @@
     </visual>
   </link>
-  <!-- Camera (Opencv convention) frames -->
   <joint name="l_camera_joint" type="fixed">
     <origin xyz="0.0575 0.0 0.0" rpy="0.0 0.0 0.0" />
     <parent link="l_eye_pan_link"/>
     <child link="l_camera_link" />
-  </joint>
-  <link name="l_camera_vision_link">
-   <visual>
-      <origin xyz="0 0 0" rpy="0 0 0" />
-      <geometry>
-        <box size="0.001 0.001 0.001" />
-      </geometry>
-    </visual>
-  </link>
-  <joint name="l_camera_vision_joint" type="fixed">
-    <origin xyz="0.0 0.0 0.0" rpy="${-M_PI/2} 0.0 ${-M_PI/2}" />
-    <parent link="l_camera_link"/>
-    <child link="l_camera_vision_link" />
-  </joint>
-  <link name="r_camera_vision_link">
-   <visual>
-      <origin xyz="0 0 0" rpy="0 0 0" />
-      <geometry>
-        <box size="0.001 0.001 0.001" />
-      </geometry>
-    </visual>
-  </link>
-  <joint name="r_camera_vision_joint" type="fixed">
-    <origin xyz="0.0 0.0 0.0" rpy="${-M_PI/2} 0.0 ${-M_PI/2}" />
-    <parent link="r_camera_link"/>
-    <child link="r_camera_vision_link" />
-  </joint>
-  <!-- eyes center and ego virtual link and joint -->
-  <link name="ego_frame">
-    <inertial>
-      <origin xyz="0 0 0" rpy="0.0 0.0 0" />
-      <mass value="0.001"/>
-      <inertia
-        ixx="0.001" ixy="0.0" ixz="0.0"
-        iyy="0.001" iyz="0.0" izz="0.001"/>
-    </inertial>
-  </link>
-  <joint name="ego_joint" type="fixed">
-    <origin
-      xyz="0.0 0.370 0.0"
-      rpy="0.0 ${M_PI/2.0} ${M_PI}" />
-    <parent link="waist_link"/>
-    <child link="ego_frame" />
-  </joint>
-  <link name="head_origin_frame">
-    <inertial>
-      <origin xyz="0 0 0" rpy="0.0 0.0 0" />
-      <mass value="0.001"/>
-      <inertia
-        ixx="0.001" ixy="0.0" ixz="0.0"
-        iyy="0.001" iyz="0.0" izz="0.001"/>
-    </inertial>
-  </link>
-  <joint name="head_origin_joint" type="fixed">
-    <origin
-      xyz="0.0 -0.04755 0.0"
-      rpy="0.0 -${M_PI/2.0} 0.0" />
-    <parent link="neck_tilt_link"/>
-    <child link="head_origin_frame" />
   </joint>
     <!-- gazebo extensions -->
