Commit message: removed virtual vergence and version joints from ros urdfs. Merged ros and yarp head urdfs.

File: vizzy_description/plugins/ros.gazebo.xacro (robot description, xacro)
@@ -19,9 +19,16 @@
         <wheelDiameter>0.2410</wheelDiameter>
         <torque>20</torque>
+        <updateRate>100</updateRate>
         <commandTopic>vizzy/cmd_vel</commandTopic>
         <odometryTopic>odom</odometryTopic>
         <odometryFrame>odom</odometryFrame>
         <robotBaseFrame>base_footprint</robotBaseFrame>
-        <updateRate>100.0</updateRate>
+        <odometrySource>0</odometrySource>
+        <wheelTorque>5</wheelTorque>
+        <wheelAcceleration>0</wheelAcceleration>
+        <publishWheelJointState>true</publishWheelJointState>
+        <publishTF>1</publishTF>
+        <publishWheelTF>true</publishWheelTF>
+        <rosDebugLevel>na</rosDebugLevel>
       </plugin>
     </gazebo>

File: vizzy_description/robots/vizzy.urdf.xacro (robot description, xacro)
@@ -14,6 +14,5 @@
   <xacro:include filename="$(find vizzy_description)/urdf/torso/torso.urdf.xacro" />
   <!-- head -->
- <xacro:include filename="$(find vizzy_description)/urdf/head/head.yarp.urdf.xacro"/>
- <xacro:include filename="$(find vizzy_description)/urdf/head/head.ros.urdf.xacro"/>
+ <xacro:include filename="$(find vizzy_description)/urdf/head/head.urdf.xacro"/>
   <!-- left arm -->
   <xacro:include filename="$(find vizzy_description)/urdf/arm/left_arm.urdf.xacro" />
@@ -32,10 +31,5 @@
   <xacro:torso name="torso"/>
   <!-- instantiate head -->
-  <xacro:if value="$(arg use_yarp)">
-  	<xacro:head_yarp name="head"/>
-  </xacro:if>
-  <xacro:unless value="$(arg use_yarp)">
-  	<xacro:head name="head"/>
-  </xacro:unless>
+  <xacro:head name="head"/>
   <!-- instantiate left arm -->
   <xacro:left_arm name="left_arm" parent="waist_link" sufix="l" reflect="1">

File: vizzy_description/urdf/head/head.transmission.xacro (robot description, xacro)
@@ -8,5 +8,5 @@
       <type>transmission_interface/SimpleTransmission</type>
       <joint name="neck_pan_joint">
-        <hardwareInterface>EffortJointInterface</hardwareInterface>
+        <hardwareInterface>VelocityJointInterface</hardwareInterface>
       </joint>
       <actuator name="neck_pan_motor">
@@ -17,5 +17,5 @@
       <type>transmission_interface/SimpleTransmission</type>
       <joint name="neck_tilt_joint">
-        <hardwareInterface>EffortJointInterface</hardwareInterface>
+        <hardwareInterface>VelocityJointInterface</hardwareInterface>
       </joint>
       <actuator name="neck_tilt_motor">
@@ -26,5 +26,5 @@
       <type>transmission_interface/SimpleTransmission</type>
       <joint name="eyes_tilt_joint">
-        <hardwareInterface>EffortJointInterface</hardwareInterface>
+        <hardwareInterface>VelocityJointInterface</hardwareInterface>
       </joint>
       <actuator name="eyes_tilt_motor">
@@ -32,55 +32,19 @@
       </actuator>
     </transmission>
-    <transmission name="version_transmission">
+    <transmission name="l_eye_transmission">
       <type>transmission_interface/SimpleTransmission</type>
-      <joint name="version_joint">
-        <hardwareInterface>EffortJointInterface</hardwareInterface>
+      <joint name="l_eye_joint">
+        <hardwareInterface>VelocityJointInterface</hardwareInterface>
       </joint>
-      <actuator name="version_motor">
-        <mechanicalReduction>100</mechanicalReduction>
-      </actuator>
-    </transmission>
-    <transmission name="l_eye_version_transmission">
-      <type>transmission_interface/SimpleTransmission</type>
-      <joint name="l_eye_version_joint">
-        <hardwareInterface>EffortJointInterface</hardwareInterface>
-      </joint>
-      <actuator name="l_eye_version_motor">
+      <actuator name="l_eye_motor">
         <mechanicalReduction>1</mechanicalReduction>
       </actuator>
     </transmission>
-    <transmission name="r_eye_version_transmission">
+    <transmission name="r_eye_transmission">
       <type>transmission_interface/SimpleTransmission</type>
-      <joint name="r_eye_version_joint">
-        <hardwareInterface>EffortJointInterface</hardwareInterface>
+      <joint name="r_eye_joint">
+        <hardwareInterface>VelocityJointInterface</hardwareInterface>
       </joint>
-      <actuator name="r_eye_version_motor">
-        <mechanicalReduction>1</mechanicalReduction>
-      </actuator>
-    </transmission>
-    <transmission name="vergence_transmission">
-      <type>transmission_interface/SimpleTransmission</type>
-      <joint name="vergence_joint">
-        <hardwareInterface>EffortJointInterface</hardwareInterface>
-      </joint>
-      <actuator name="vergence_motor">
-        <mechanicalReduction>100</mechanicalReduction>
-      </actuator>
-    </transmission>
-    <transmission name="l_eye_vergence_transmission">
-      <type>transmission_interface/SimpleTransmission</type>
-      <joint name="l_eye_vergence_joint">
-        <hardwareInterface>EffortJointInterface</hardwareInterface>
-      </joint>
-      <actuator name="l_eye_vergence_motor">
-        <mechanicalReduction>1</mechanicalReduction>
-      </actuator>
-    </transmission>
-    <transmission name="r_eye_vergence_transmission">
-      <type>transmission_interface/SimpleTransmission</type>
-      <joint name="r_eye_vergence_joint">
-        <hardwareInterface>EffortJointInterface</hardwareInterface>
-      </joint>
-      <actuator name="r_eye_vergence_motor">
+      <actuator name="r_eye_motor">
         <mechanicalReduction>1</mechanicalReduction>
       </actuator>

File: vizzy_description/urdf/head/head.urdf.xacro (robot description, xacro)
@@ -60,5 +60,7 @@
     <axis
       xyz="0 0 1" />
-    <limit lower="-0.925024504" upper="0.925024504" effort="10.0" velocity="3" />
+    <!--<limit lower="-0.925024504" upper="0.925024504" effort="10.0" velocity="5.0" />-->
+    <limit lower="-2.025024504" upper="2.025024504" effort="100.0" velocity="5.0" />
+    <dynamics damping="5.0" friction="10.0"/>
   </joint>
   <link
@@ -114,5 +116,7 @@
     <axis
       xyz="0 0 1" />
-    <limit lower="-0.314159265" upper="0.645771823" effort="100.0" velocity="1.0" />
+    <!--<limit lower="-0.314159265" upper="0.645771823" effort="100.0" velocity="5.0" />-->
+    <dynamics damping="0.0" friction="5.0"/>
+    <limit lower="-2.014159265" upper="2.45771823" effort="100.0" velocity="5.0" />
   </joint>
   <link
@@ -168,8 +172,9 @@
     <axis
       xyz="0 0 1" />
-    <limit lower="-0.663225116" upper="0.663225116" effort="10.0" velocity="3" />
-  </joint>
-  <!-- version virtual link and joint -->
-  <link name="version_link">
+    <limit lower="-0.663225116" upper="0.663225116" effort="10.0" velocity="5.0" />
+    <dynamics damping="0.0" friction="5.0"/>
+  </joint>
+  <!-- eyes center virtual link and joint -->
+  <link name="eyes_center_link">
 		<inertial>
 			<origin xyz="0 0 0"
@@ -181,15 +186,17 @@
 		</inertial>
   </link>
-  <joint name="version_joint" type="revolute">
+  <joint name="eyes_center_joint" type="fixed">
     <origin xyz="0 0 0"       rpy="${M_PI/2.0} 0.0 0.369599135716446" />
     <parent link="eyes_tilt_link" />
-    <child link="version_link" />
+    <child link="eyes_center_link" />
     <axis  xyz="0 0 1" />
-    <limit lower="-0.698131" upper="0.698131" effort="10.0" velocity="0.2" />
-  </joint>
-  <link name="l_eye_version_link">
- 		<inertial>
-			<origin xyz="0 0 0" rpy="0 0 0"/>
-			<mass value="0.01"/>
+    <limit lower="-0.698131" upper="0.698131" effort="10.0" velocity="5.0" />
+  </joint>
+  <!-- eyes center visual virtual link and joint -->
+  <link name="eyes_center_vision_link">
+		<inertial>
+			<origin xyz="0 0 0"
+      rpy="0.0 0.0 0" />
+			<mass value="0.1"/>
 			<inertia
 				ixx="0.001" ixy="0.0" ixz="0.0"
@@ -197,14 +204,59 @@
 		</inertial>
   </link>
+  <joint name="eyes_center_vision_joint" type="fixed">
+    <origin xyz="0 0 0"       rpy="${-M_PI/2} 0.0 ${-M_PI/2}" />
+    <parent link="eyes_center_link" />
+    <child link="eyes_center_vision_link" />
+  </joint>
+  <!-- eyes -->
+  <link name="l_eye_link">
+  <inertial>
+      <origin
+        xyz="0.0 0.0 0.0"
+        rpy="0 0 ${M_PI/2}" />
+      <mass
+        value="0.158520637460366" />
+      <inertia
+        ixx="0.000147614970454271"
+        ixy="-1.56210652664748E-09"
+        ixz="8.85544640354075E-10"
+        iyy="0.000177840459249179"
+        iyz="8.21234366300574E-06"
+        izz="0.000144884726537935" />
+    </inertial>
+    <visual>
+      <origin
+        xyz="0.0 0.0 0.0"
+        rpy="0.0 0.0 ${M_PI/2}" />
+      <geometry>
+        <mesh
+          filename="package://vizzy_description/meshes/M4.dae" />
+      </geometry>
+      <material
+        name="">
+        <color
+          rgba="0 0 0 1" />
+      </material>
+    </visual>
+    <collision>
+ 	<origin
+        xyz="0.0 0 0.0"
+        rpy="0 0 ${M_PI/2}" />
+      <geometry>
+        <mesh
+          filename="package://vizzy_description/meshes/M4.dae" />
+      </geometry>
+    </collision>
+  </link>
   <joint
-    name="l_eye_version_joint"
+    name="l_eye_joint"
     type="revolute">
     <origin
-      xyz="0.0 0.0 0.102"
-      rpy="${M_PI/2.0} 0.0 0.369599135716446" />
+      xyz="0.0 0.102 0.0"
+      rpy="0 ${M_PI} 0" />
     <parent
-      link="eyes_tilt_link" />
+      link="eyes_center_link" />
     <child
-      link="l_eye_version_link" />
+      link="l_eye_link" />
     <axis
       xyz="0 0 1" />
@@ -213,26 +265,56 @@
 			upper="1.0"
       effort="1000.0"
-      velocity="0.2" />
-    <mimic joint="version_joint" multiplier="1" offset="0"/>
-  </joint>
-  <link name="r_eye_version_link">
- 		<inertial>
-			<origin xyz="0 0 0" rpy="0 0 0"/>
-			<mass value="0.01"/>
-			<inertia
-				ixx="0.001" ixy="0.0" ixz="0.0"
-				iyy="0.001" iyz="0.0" izz="0.001"/>
-		</inertial>
+      velocity="5.0" />
+    <dynamics damping="0.0" friction="5.0"/>
+  </joint>
+  <link name="r_eye_link">
+  <inertial>
+      <origin
+        xyz="0.0 0.0 0.0"
+        rpy="0.0 0.0 ${M_PI/2}" />
+      <mass
+        value="0.158520637460366" />
+      <inertia
+        ixx="0.000147614970454271"
+        ixy="-1.56210652664748E-09"
+        ixz="8.85544640354075E-10"
+        iyy="0.000177840459249179"
+        iyz="8.21234366300574E-06"
+        izz="0.000144884726537935" />
+    </inertial>
+    <visual>
+      <origin
+        xyz="0.0 0.0 0.0"
+        rpy="0.0 0.0 ${M_PI/2}" />
+      <geometry>
+        <mesh
+          filename="package://vizzy_description/meshes/M4.dae" />
+      </geometry>
+      <material
+        name="">
+        <color
+          rgba="0 0 0 1" />
+      </material>
+    </visual>
+    <collision>
+      <origin
+        xyz="0.0 0.0 0.0"
+        rpy="0.0 0.0 ${M_PI/2}" />
+      <geometry>
+        <mesh
+          filename="package://vizzy_description/meshes/M4.dae" />
+      </geometry>
+    </collision>
   </link>
   <joint
-    name="r_eye_version_joint"
+    name="r_eye_joint"
     type="revolute">
     <origin
-      xyz="0.0 0.0 -0.102"
-      rpy="${M_PI/2.0} 0.0 0.369599135716446" />
+      xyz="0.0 -0.102 0.0"
+      rpy="0 ${M_PI} 0" />
     <parent
-      link="eyes_tilt_link" />
+      link="eyes_center_link" />
     <child
-      link="r_eye_version_link" />
+      link="r_eye_link" />
     <axis
       xyz="0 0 1" />
@@ -241,81 +323,8 @@
 			upper="1.0"
       effort="1000.0"
-      velocity="0.2"/>
-    <mimic joint="version_joint" multiplier="1" offset="0"/>
-  </joint>
-  <link name="vergence_link">
- 		<inertial>
-			<origin xyz="0 0 0" rpy="0 0 0"/>
-			<mass value="0.1"/>
-			<inertia
-				ixx="0.001" ixy="0.0" ixz="0.0"
-				iyy="0.001" iyz="0.0" izz="0.001"/>
-		</inertial>
-  </link>
-  <joint name="vergence_joint" type="revolute">
-    <origin xyz="0.0 0.0 0.0" rpy="${M_PI/2.0} 0.0 0.369599135716446" />
-    <parent link="eyes_tilt_link" />
-    <child link="vergence_link" />
-    <axis  xyz="0 0 1" />
-    <limit lower="0.0" upper="0.698131" effort="10.0" velocity="0.2" />
-  </joint>
-  <link name="r_eye_vergence_link">
-    <inertial>
-      <origin
-        xyz="0.010 0.0 0.003"
-        rpy="0.0 ${M_PI} ${-M_PI/2}" />
-      <mass
-        value="0.158520637460366" />
-      <inertia
-        ixx="0.000147614970454271"
-        ixy="-1.56210652664748E-09"
-        ixz="8.85544640354075E-10"
-        iyy="0.000177840459249179"
-        iyz="8.21234366300574E-06"
-        izz="0.000144884726537935" />
-    </inertial>
-    <visual>
-      <origin
-        xyz="0.010 0.0 0.003"
-        rpy="0.0 ${M_PI} ${-M_PI/2}" />
-      <geometry>
-        <mesh
-          filename="package://vizzy_description/meshes/M4.dae" />
-      </geometry>
-      <material
-        name="">
-        <color
-          rgba="0 0 0 1" />
-      </material>
-    </visual>
-    <collision>
-      <origin
-        xyz="0.010 0.0 0.003"
-        rpy="0.0 ${M_PI} ${-M_PI/2}" />
-      <geometry>
-        <mesh
-          filename="package://vizzy_description/meshes/M4.dae" />
-      </geometry>
-    </collision>
-  </link>
-  <joint
-    name="r_eye_vergence_joint"
-    type="revolute">
-    <origin
-      xyz="0.0 0.0 0.0"
-      rpy="0.0 0.0 0.0" />
-    <parent
-      link="r_eye_version_link" />
-    <child
-      link="r_eye_vergence_link" />
-    <axis
-      xyz="0 0 1" />
-		<limit
-			lower="-1.0"
-			upper="1.0"
-      effort="1000.0"
-      velocity="0.2"/>
-    <mimic joint="vergence_joint" multiplier="0.5" offset="0"/>
-  </joint>
+      velocity="5.0"/>
+    <dynamics damping="0.0" friction="5.0"/>
+  </joint>
+  <!-- cameras -->
   <link name="r_camera_link">
    <visual>
@@ -327,6 +336,6 @@
   </link>
   <joint name="r_camera_joint" type="fixed">
-    <origin xyz="0.0575 0.0 0.0" rpy="0.0 0.0 0.0" />
-    <parent link="r_eye_vergence_link"/>
+    <origin xyz="-0.0275 0.0 0.0" rpy="${M_PI/2} 0.0 ${-M_PI/2}" />
+    <parent link="r_eye_link"/>
     <child link="r_camera_link" />
   </joint>
@@ -340,65 +349,7 @@
   </link>
   <joint name="r_camera_vision_joint" type="fixed">
-    <origin xyz="0.0 0.0 0.0" rpy="0.0 ${M_PI/2} 0.0" />
+    <origin xyz="0.0 0.0 0.0" rpy="0.0 0.0 0.0" />
     <parent link="r_camera_link"/>
     <child link="r_camera_vision_link" />
-  </joint>
-  <link name="l_eye_vergence_link">
-   <inertial>
-      <origin
-        xyz="0 0 -0.0200000000000069"
-        rpy="0 0 1.5708" />
-      <mass
-        value="0.158520637460366" />
-      <inertia
-        ixx="0.000147614970454271"
-        ixy="-1.56210652664748E-09"
-        ixz="8.85544640354075E-10"
-        iyy="0.000177840459249179"
-        iyz="8.21234366300574E-06"
-        izz="0.000144884726537935" />
-    </inertial>
-    <visual>
-      <origin
-        xyz="0.010 0.0 0.003"
-        rpy="0.0 ${M_PI} ${-M_PI/2}" />
-      <geometry>
-        <mesh
-          filename="package://vizzy_description/meshes/M4.dae" />
-      </geometry>
-      <material
-        name="">
-        <color
-          rgba="0 0 0 1" />
-      </material>
-    </visual>
-    <collision>
-      <origin
-        xyz="0 0 -0.0200000000000069"
-        rpy="0 0 1.5708" />
-      <geometry>
-        <mesh
-          filename="package://vizzy_description/meshes/M4.dae" />
-      </geometry>
-    </collision>
-  </link>
-  <joint
-    name="l_eye_vergence_joint"
-    type="revolute">
-    <origin
-      xyz="0 0 0"
-      rpy="0 0 0" />
-    <parent
-      link="l_eye_version_link" />
-    <child
-      link="l_eye_vergence_link" />
-    <axis
-      xyz="0 0 1" />
-    <limit
-			lower="-1.0"
-			upper="1.0"
-      effort="1000.0"
-      velocity="0.2" />
-    <mimic joint="vergence_joint" multiplier="-0.5" offset="0"/>
   </joint>
   <link name="l_camera_link">
@@ -411,6 +362,6 @@
   </link>
   <joint name="l_camera_joint" type="fixed">
-    <origin xyz="0.0575 0.0 0.0" rpy="0.0 0.0 0.0" />
-    <parent link="l_eye_vergence_link"/>
+    <origin xyz="-0.0275 0.0 0.0" rpy="${M_PI/2} 0.0 ${-M_PI/2}" />
+    <parent link="l_eye_link"/>
     <child link="l_camera_link" />
   </joint>
@@ -424,7 +375,40 @@
   </link>
   <joint name="l_camera_vision_joint" type="fixed">
-    <origin xyz="0.0 0.0 0.0" rpy="0.0 ${M_PI/2} 0.0" />
+    <origin xyz="0.0 0.0 0.0" rpy="0.0 0.0 0.0" />
     <parent link="l_camera_link"/>
     <child link="l_camera_vision_link" />
+  </joint>
+  <!-- ego frame -->
+  <link name="ego_frame">
+    <inertial>
+      <origin xyz="0 0 0" rpy="0.0 0.0 0" />
+      <mass value="0.001"/>
+      <inertia
+        ixx="0.001" ixy="0.0" ixz="0.0"
+        iyy="0.001" iyz="0.0" izz="0.001"/>
+    </inertial>
+  </link>
+  <joint name="ego_joint" type="fixed">
+    <origin
+      xyz="0.0 0.370 0.0"
+      rpy="0.0 ${M_PI/2.0} ${M_PI}" />
+    <parent link="waist_link"/>
+    <child link="ego_frame" />
+  </joint>
+  <link name="head_origin_frame">
+    <inertial>
+      <origin xyz="0 0 0" rpy="0.0 0.0 0" />
+      <mass value="0.001"/>
+      <inertia
+        ixx="0.001" ixy="0.0" ixz="0.0"
+        iyy="0.001" iyz="0.0" izz="0.001"/>
+    </inertial>
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