Commit message: temporary changes for foveal stereo results generations

File: vizzy_description/plugins/ros.gazebo.xacro (robot description, xacro)
@@ -41,8 +41,9 @@
         <camera name="head">
           <!--<horizontal_fov>1.4912</horizontal_fov>-->
-          <horizontal_fov>1.4912</horizontal_fov>
+          <horizontal_fov>2.3561</horizontal_fov>
+          <!--<horizontal_fov>1.5708</horizontal_fov>-->
           <image>
-            <width>640</width>
-            <height>480</height>
+            <width>320</width>
+            <height>240</height>
 	    <!--<width>640</width>
             <height>480</height>-->

File: vizzy_description/robots/vizzy.urdf.xacro (robot description, xacro)
@@ -1,5 +1,5 @@
 <?xml version="1.0"?>
 <robot  name="vizzy" xmlns:xacro="http://ros.org/wiki/xacro" >
-	<xacro:arg name="use_yarp" default="false"/>
+  <xacro:arg name="use_yarp" default="false"/>
   <!-- The following include files set up definitions of parts of the robot body  -->
   <!-- misc common stuff -->

File: vizzy_description/robots/vizzy_head_only.urdf.xacro (robot description, xacro)
@@ -1,5 +1,5 @@
 <?xml version="1.0"?>
 <robot  name="vizzy" xmlns:xacro="http://ros.org/wiki/xacro" >
-<xacro:arg name="use_yarp" default="false"/>
+  <xacro:arg name="use_yarp" default="false"/>
   <!-- The following include files set up definitions of parts of the robot body  -->
   <!-- misc common stuff -->
@@ -8,10 +8,5 @@
   <xacro:include filename="$(find vizzy_description)/urdf/simple_base/base.urdf.xacro" />
   <!-- head -->
-  <xacro:if value="$(arg use_yarp)">
-  	<xacro:include filename="$(find vizzy_description)/urdf/head/head.yarp.urdf.xacro" />
-  </xacro:if>-->
-  <xacro:unless value="$(arg use_yarp)">
-  	<xacro:include filename="$(find vizzy_description)/urdf/head/head.ros.urdf.xacro" />
-  </xacro:unless>
+  <xacro:include filename="$(find vizzy_description)/urdf/head/head.urdf.xacro" />
   <!-- The following include files contain gazebo plugins -->
   <!-- ROS -->

File: vizzy_description/urdf/hand/right_hand.urdf.xacro (robot description, xacro)
@@ -9,121 +9,177 @@
   <xacro:include filename="$(find vizzy_description)/urdf/arm/right_arm.transmission.xacro"/>
   <xacro:macro name="right_hand" params="name parent sufix reflect *origin">
-    <joint name="r_palm_joint" type="fixed">
-		  <origin xyz="0.1 0 0.0" rpy="0 ${M_PI/2.0} 0" />
-		  <parent link="r_wrist_flection_link"/>
-		  <child link="r_palm_link" />
-		</joint>
-  <link
-    name="r_palm_link">
-    <inertial>
-      <origin
-        xyz="-0.006637 0.0034589 0.0058703"
-        rpy="0 0 0" />
-      <mass
-        value="0.14841" />
-      <inertia
-        ixx="0.00014253"
-        ixy="1.9852E-05"
-        ixz="-1.4353E-06"
-        iyy="9.7254E-05"
-        iyz="-2.6916E-06"
-        izz="0.0002182" />
-    </inertial>
-    <visual>
-      <origin
-        xyz="0 0 0"
-        rpy="0 0 0" />
-      <geometry>
-        <mesh
-          filename="package://vizzy_description/meshes/right_hand/r_palm_link.STL" />
-      </geometry>
-      <material
-        name="">
-        <color
-          rgba="0.79608 0.82353 0.93725 1" />
-      </material>
-    </visual>
-    <collision>
-      <origin
-        xyz="0 0 0"
-        rpy="0 0 0" />
-      <geometry>
-        <mesh
-          filename="package://vizzy_description/meshes/right_hand/r_palm_link.STL" />
-      </geometry>
-    </collision>
-  </link>
-  <link
-    name="min_phal_1_link">
-    <inertial>
-      <origin
-        xyz="-0.0065851 -4.2258E-05 0.019478"
-        rpy="0 0 0" />
-      <mass
-        value="0.014476" />
-      <inertia
-        ixx="1.7219E-06"
-        ixy="3.4428E-10"
-        ixz="3.009E-10"
-        iyy="1.7445E-06"
-        iyz="1.5436E-08"
-        izz="5.3067E-07" />
-    </inertial>
-    <visual>
-      <origin
-        xyz="0 0 0"
-        rpy="0 0 0" />
-      <geometry>
-        <mesh
-          filename="package://vizzy_description/meshes/right_hand/min_phal_1_link.STL" />
-      </geometry>
-      <material
-        name="">
-        <color
-          rgba="0.89804 0.91765 0.92941 1" />
-      </material>
-    </visual>
-    <collision>
-      <origin
-        xyz="0 0 0"
-        rpy="0 0 0" />
-      <geometry>
-        <mesh
-          filename="package://vizzy_description/meshes/right_hand/min_phal_1_link.STL" />
-      </geometry>
-    </collision>
-  </link>
-  <joint
-    name="min_phal_1_joint"
-    type="revolute">
-    <origin
-      xyz="0.020602 -0.005836 0.044434"
-      rpy="6.2175E-17 -0.17453 3.1416" />
-    <parent
-      link="r_palm_link" />
-    <child
-      link="min_phal_1_link" />
-    <axis
-      xyz="1 0 0" />
-    <limit
-      lower="0"
-      upper="1.7453"
-      effort="0"
-      velocity="0" />
-  </joint>
-  <link
-    name="min_phal_2_link">
-    <inertial>
-      <origin
-        xyz="-0.0065912 3.9323E-05 0.016339"
+  <link
+    name="r_hand_link">
+    <inertial>
+      <origin
+        xyz="0.0038463 -0.25763 0.60534"
+        rpy="0 0 0" />
+      <mass
+        value="0.14447" />
+      <inertia
+        ixx="0.00014079"
+        ixy="1.5176E-05"
+        ixz="1.0157E-05"
+        iyy="0.00013841"
+        iyz="5.8477E-05"
+        izz="0.00016255" />
+    </inertial>
+    <visual>
+      <origin
+        xyz="0 0 0"
+        rpy="0 0 0" />
+      <geometry>
+        <mesh
+          filename="package://vizzy_test/meshes/r_hand_link.STL" />
+      </geometry>
+      <material
+        name="">
+        <color
+          rgba="0.89804 0.91765 0.92941 1" />
+      </material>
+    </visual>
+    <collision>
+      <origin
+        xyz="0 0 0"
+        rpy="0 0 0" />
+      <geometry>
+        <mesh
+          filename="package://vizzy_test/meshes/r_hand_link.STL" />
+      </geometry>
+    </collision>
+  </link>
+  <joint
+    name="r_hand_joint"
+    type="fixed">
+    <origin
+      xyz="0.631985243056887 -0.118428097845849 -0.0023641314603528"
+      rpy="-2.73631640958448 -1.55026793601452 2.02896379866596" />
+    <parent
+      link="r_wrist_flection_link" />
+    <child
+      link="r_hand_link" />
+    <axis
+      xyz="0 0 0" />
+  </joint>
+  <link
+    name="r_thumb_1_link">
+    <inertial>
+      <origin
+        xyz="-0.00032032 0.0070152 0.0070409"
+        rpy="0 0 0" />
+      <mass
+        value="0.0081407" />
+      <inertia
+        ixx="6.5008E-07"
+        ixy="7.3119E-10"
+        ixz="2.5546E-09"
+        iyy="5.6171E-07"
+        iyz="2.5969E-09"
+        izz="2.906E-07" />
+    </inertial>
+    <visual>
+      <origin
+        xyz="0 0 0"
+        rpy="0 0 0" />
+      <geometry>
+        <mesh
+          filename="package://vizzy_test/meshes/r_thumb_1_link.STL" />
+      </geometry>
+      <material
+        name="">
+        <color
+          rgba="0.77647 0.75686 0.73725 1" />
+      </material>
+    </visual>
+    <collision>
+      <origin
+        xyz="0 0 0"
+        rpy="0 0 0" />
+      <geometry>
+        <mesh
+          filename="package://vizzy_test/meshes/r_thumb_1_link.STL" />
+      </geometry>
+    </collision>
+  </link>
+  <joint
+    name="r_thumb_1_joint"
+    type="fixed">
+    <origin
+      xyz="-0.051602659641749 -0.261993975608549 0.585670716685399"
+      rpy="1.58918253820798 -0.658618217290863 1.14526673964582" />
+    <parent
+      link="r_hand_link" />
+    <child
+      link="r_thumb_1_link" />
+    <axis
+      xyz="0 0 0" />
+  </joint>
+  <link
+    name="r_thumb_2_link">
+    <inertial>
+      <origin
+        xyz="4.3028E-05 0.0070072 0.013515"
+        rpy="0 0 0" />
+      <mass
+        value="0.014478" />
+      <inertia
+        ixx="1.7439E-06"
+        ixy="3.4418E-10"
+        ixz="1.4451E-08"
+        iyy="1.7213E-06"
+        iyz="3.0158E-10"
+        izz="5.3077E-07" />
+    </inertial>
+    <visual>
+      <origin
+        xyz="0 0 0"
+        rpy="0 0 0" />
+      <geometry>
+        <mesh
+          filename="package://vizzy_test/meshes/r_thumb_2_link.STL" />
+      </geometry>
+      <material
+        name="">
+        <color
+          rgba="0.77647 0.75686 0.73725 1" />
+      </material>
+    </visual>
+    <collision>
+      <origin
+        xyz="0 0 0"
+        rpy="0 0 0" />
+      <geometry>
+        <mesh
+          filename="package://vizzy_test/meshes/r_thumb_2_link.STL" />
+      </geometry>
+    </collision>
+  </link>
+  <joint
+    name="r_thumb_2_joint"
+    type="fixed">
+    <origin
+      xyz="-0.000155193715695168 0 -0.0329996350723843"
+      rpy="2.77558825516292E-17 0.00470285720488725 -5.55117651032584E-17" />
+    <parent
+      link="r_thumb_1_link" />
+    <child
+      link="r_thumb_2_link" />
+    <axis
+      xyz="0 0 0" />
+  </joint>
+  <link
+    name="r_thumb_3_link">
+    <inertial>
+      <origin
+        xyz="-3.9325E-05 0.0070133 0.01016"
         rpy="0 0 0" />
       <mass
         value="0.011277" />
       <inertia
-        ixx="1.007E-06"
+        ixx="1.0456E-06"
         ixy="5.324E-10"
-        ixz="5.414E-10"
-        iyy="1.0456E-06"
-        iyz="1.1256E-08"
+        ixz="1.1256E-08"
+        iyy="1.007E-06"
+        iyz="5.4133E-10"
         izz="4.1298E-07" />
     </inertial>
@@ -134,45 +190,40 @@
       <geometry>
         <mesh
-          filename="package://vizzy_description/meshes/right_hand/min_phal_2_link.STL" />
-      </geometry>
-      <material
-        name="">
-        <color
-          rgba="0.89804 0.91765 0.92941 1" />
-      </material>
-    </visual>
-    <collision>
-      <origin
-        xyz="0 0 0"
-        rpy="0 0 0" />
-      <geometry>
-        <mesh
-          filename="package://vizzy_description/meshes/right_hand/min_phal_2_link.STL" />
-      </geometry>
-    </collision>
-  </link>
-  <joint
-    name="min_phal_2_joint"
-    type="revolute">
-    <origin
-      xyz="0 0 0.033"
-      rpy="0 -7.2164E-16 0" />
-    <parent
-      link="min_phal_1_link" />
-    <child
-      link="min_phal_2_link" />
-    <axis
-      xyz="1 0 0" />
-    <limit
-      lower="0"
-      upper="1.5708"
-      effort="0"
-      velocity="0" />
-  </joint>
-  <link
-    name="min_phal_3_link">
-    <inertial>
-      <origin
-        xyz="-0.0065949 -2.2728E-05 0.013411"
+          filename="package://vizzy_test/meshes/r_thumb_3_link.STL" />
+      </geometry>
+      <material
+        name="">
+        <color
+          rgba="0.77647 0.75686 0.73725 1" />
+      </material>
+    </visual>
+    <collision>
+      <origin
+        xyz="0 0 0"
+        rpy="0 0 0" />
+      <geometry>
+        <mesh
+          filename="package://vizzy_test/meshes/r_thumb_3_link.STL" />
+      </geometry>
+    </collision>
+  </link>
+  <joint
+    name="r_thumb_3_joint"
+    type="fixed">
+    <origin
+      xyz="0 0 -0.0265000000000002"
+      rpy="2.08166817117217E-15 -7.63278329429795E-17 4.94049245958195E-15" />
+    <parent
+      link="r_thumb_2_link" />
+    <child
+      link="r_thumb_3_link" />
+    <axis
+      xyz="0 0 0" />
+  </joint>
+  <link
+    name="r_thumb_4_link">
+    <inertial>
+      <origin
+        xyz="-1.702E-05 -2.2727E-05 0.0049109"
         rpy="0 0 0" />
       <mass
@@ -180,115 +231,264 @@
       <inertia
         ixx="5.7614E-07"
-        ixy="5.3191E-10"
-        ixz="-3.8097E-11"
-        iyy="5.3414E-07"
+        ixy="5.3189E-10"
+        ixz="-3.8147E-11"
+        iyy="5.3439E-07"
         iyz="3.9566E-09"
-        izz="3.158E-07" />
-    </inertial>
-    <visual>
-      <origin
-        xyz="0 0 0"
-        rpy="0 0 0" />
-      <geometry>
-        <mesh
-          filename="package://vizzy_description/meshes/right_hand/min_phal_3_link.STL" />
-      </geometry>
-      <material
-        name="">
-        <color
-          rgba="0.89804 0.91765 0.92941 1" />
-      </material>
-    </visual>
-    <collision>
-      <origin
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
Commit message: Added low-level motor interface between yarp and ros for the left arm PID parameters set for the left arm Added friction in the joints of the URDF left and right arms Commented out mu1 and mu2 on all the links of the left and right arms

File: vizzy_description/plugins/ros.gazebo.xacro (robot description, xacro)
@@ -25,5 +25,5 @@
         <robotBaseFrame>base_footprint</robotBaseFrame>
         <odometrySource>0</odometrySource>
-        <wheelTorque>5</wheelTorque>
+        <wheelTorque>10</wheelTorque>
         <wheelAcceleration>0</wheelAcceleration>
         <publishWheelJointState>true</publishWheelJointState>

File: vizzy_description/urdf/arm/left_arm.gazebo.xacro (robot description, xacro)
@@ -3,44 +3,44 @@
   <xacro:macro name="left_arm_gazebo">
     <gazebo reference="l_shoulder_scapula_link">
-      <mu1>0.2</mu1>
-      <mu2>0.2</mu2>
+      <!--<mu1>0.2</mu1>
+      <mu2>0.2</mu2>-->
     </gazebo>
     <gazebo reference="l_shoulder_flection_link">
-      <mu1>0.2</mu1>
-      <mu2>0.2</mu2>
+      <!--<mu1>0.2</mu1>
+      <mu2>0.2</mu2>-->
     </gazebo>
     <gazebo reference="l_shoulder_abduction_link">
-      <mu1>0.2</mu1>
-      <mu2>0.2</mu2>
+      <!--<mu1>0.2</mu1>
+      <mu2>0.2</mu2>-->
     </gazebo>
     <gazebo reference="l_shoulder_rotation_link">
-      <mu1>0.2</mu1>
-      <mu2>0.2</mu2>
+      <!--<mu1>0.2</mu1>
+      <mu2>0.2</mu2>-->
     </gazebo>
     <gazebo reference="l_elbow_flection_link">
-      <mu1>0.2</mu1>
-      <mu2>0.2</mu2>
+      <!--<mu1>0.2</mu1>
+      <mu2>0.2</mu2>-->
     </gazebo>
     <gazebo reference="l_forearm_pronation_link">
-      <mu1>0.2</mu1>
-      <mu2>0.2</mu2>
+      <!--<mu1>0.2</mu1>
+      <mu2>0.2</mu2>-->
     </gazebo>
     <gazebo reference="l_wrist_abduction_link">
-      <mu1>0.2</mu1>
-      <mu2>0.2</mu2>
+      <!--<mu1>0.2</mu1>
+      <mu2>0.2</mu2>-->
       <material>Gazebo/Orange</material>
     </gazebo>
     <gazebo reference="l_wrist_abduction_virtual_link">
-      <mu1>0.2</mu1>
-      <mu2>0.2</mu2>
+      <!--<mu1>0.2</mu1>
+      <mu2>0.2</mu2>-->
       <material>Gazebo/Orange</material>
     </gazebo>
     <gazebo reference="l_wrist_flection_link">
-      <mu1>0.2</mu1>
-      <mu2>0.2</mu2>
+      <!--<mu1>0.2</mu1>
+      <mu2>0.2</mu2>-->
     </gazebo>
     <gazebo reference="l_palm_link">
-      <mu1>0.2</mu1>
-      <mu2>0.2</mu2>
+      <!--<mu1>0.2</mu1>
+      <mu2>0.2</mu2>-->
     </gazebo>
     <gazebo>

File: vizzy_description/urdf/arm/left_arm.urdf.xacro (robot description, xacro)
@@ -61,4 +61,5 @@
 		    xyz="0 0 1" />
 		  <limit lower="-0.314159265" upper="0.314159265" effort="10" velocity="3" />
+		  <dynamics damping="0.0" friction="0.6"/>
 		</joint>
 		<link
@@ -115,4 +116,5 @@
 		    xyz="0 0 1" />
 		  <limit lower="-1.30899694" upper="2.35619449" effort="10" velocity="3" />
+		  <dynamics damping="0.0" friction="0.6"/>
 		</joint>
 		<link
@@ -169,4 +171,5 @@
 		    xyz="0 0 1" />
 		  <limit lower="0" upper="1.30899694" effort="10" velocity="3" />
+		  <dynamics damping="0.0" friction="0.6"/>
 		</joint>
 		<link
@@ -223,4 +226,5 @@
 		    xyz="0 0 1" />
 		  <limit lower="-1.48352986" upper="1.48352986" effort="10" velocity="3" />
+		  <dynamics damping="0.0" friction="0.6"/>
 		</joint>
 		<link
@@ -277,4 +281,5 @@
 		    xyz="0 0 1" />
 		  <limit lower="0" upper="1.91986218" effort="10" velocity="3" />
+		  <dynamics damping="0.0" friction="0.6"/>
 		</joint>
 		<link
@@ -331,4 +336,5 @@
 		    xyz="0 0 1" />
 		  <limit lower="-1.48352986" upper="1.48352986" effort="10" velocity="3" />
+		  <dynamics damping="0.0" friction="0.6"/>
 		</joint>
 		<link
@@ -385,4 +391,5 @@
 		    xyz="0 0 1" />
 		  <limit lower="-0.610865238" upper="0.610865238" effort="10" velocity="3" />
+		  <dynamics damping="0.0" friction="0.6"/>
 		</joint>
 		<link
@@ -440,4 +447,5 @@
 		  <limit lower="-0.610865238" upper="0.610865238" effort="10" velocity="3" />
     		  <mimic joint="l_wrist_abduction_joint" multiplier="1.0" offset="0"/>
+		  <dynamics damping="0.0" friction="0.6"/>
 		</joint>
 		<link
@@ -494,4 +502,5 @@
 		    xyz="0 0 1" />
 		  <limit lower="-0.610865238" upper="0.610865238" effort="10" velocity="3" />
+		  <dynamics damping="0.0" friction="0.6"/>
 		</joint>
 		<!--<link name="l_palm_link">

File: vizzy_description/urdf/arm/right_arm.gazebo.xacro (robot description, xacro)
@@ -3,44 +3,44 @@
   <xacro:macro name="right_arm_gazebo">
     <gazebo reference="r_shoulder_scapula_link">
-      <mu1>0.2</mu1>
-      <mu2>0.2</mu2>
+      <!--<mu1>0.2</mu1>
+      <mu2>0.2</mu2>-->
     </gazebo>
     <gazebo reference="r_shoulder_flection_link">
-      <mu1>0.2</mu1>
-      <mu2>0.2</mu2>
+      <!--<mu1>0.2</mu1>
+      <mu2>0.2</mu2>-->
     </gazebo>
     <gazebo reference="r_shoulder_abduction_link">
-      <mu1>0.2</mu1>
-      <mu2>0.2</mu2>
+      <!--<mu1>0.2</mu1>
+      <mu2>0.2</mu2>-->
     </gazebo>
     <gazebo reference="r_shoulder_rotation_link">
-      <mu1>0.2</mu1>
-      <mu2>0.2</mu2>
+      <!--<mu1>0.2</mu1>
+      <mu2>0.2</mu2>-->
     </gazebo>
     <gazebo reference="r_elbow_flection_link">
-      <mu1>0.2</mu1>
-      <mu2>0.2</mu2>
+      <!--<mu1>0.2</mu1>
+      <mu2>0.2</mu2>-->
     </gazebo>
     <gazebo reference="r_forearm_pronation_link">
-      <mu1>0.2</mu1>
-      <mu2>0.2</mu2>
+      <!--<mu1>0.2</mu1>
+      <mu2>0.2</mu2>-->
     </gazebo>
     <gazebo reference="r_wrist_abduction_link">
-      <mu1>0.2</mu1>
-      <mu2>0.2</mu2>
+      <!--<mu1>0.2</mu1>
+      <mu2>0.2</mu2>-->
       <material>Gazebo/Orange</material>
     </gazebo>
     <gazebo reference="r_wrist_abduction_virtual_link">
-      <mu1>0.2</mu1>
-      <mu2>0.2</mu2>
+      <!--<mu1>0.2</mu1>
+      <mu2>0.2</mu2>-->
       <material>Gazebo/Orange</material>
     </gazebo>
     <gazebo reference="r_wrist_flection_link">
-      <mu1>0.2</mu1>
-      <mu2>0.2</mu2>
+      <!--<mu1>0.2</mu1>
+      <mu2>0.2</mu2>-->
     </gazebo>
     <gazebo reference="r_palm_link">
-      <mu1>0.2</mu1>
-      <mu2>0.2</mu2>
+      <!--<mu1>0.2</mu1>
+      <mu2>0.2</mu2>-->
     </gazebo>
     <gazebo>

File: vizzy_description/urdf/arm/right_arm.urdf.xacro (robot description, xacro)
@@ -61,4 +61,5 @@
 		    xyz="0 0 1" />
 		  <limit lower="-0.314159265" upper="0.314159265" effort="10" velocity="3" />
+		  <dynamics damping="0.0" friction="5.0"/>
 		</joint>
 		<link
@@ -115,4 +116,5 @@
 		    xyz="0 0 1" />
 		  <limit lower="-1.30899694" upper="2.35619449" effort="10" velocity="3" />
+		  <dynamics damping="0.0" friction="5.0"/>
 		</joint>
 		<link
@@ -169,4 +171,5 @@
 		    xyz="0 0 1" />
 		  <limit lower="0" upper="1.30899694" effort="10" velocity="3" />
+		  <dynamics damping="0.0" friction="5.0"/>
 		</joint>
 		<link
@@ -223,4 +226,5 @@
 		    xyz="0 0 1" />
 		  <limit lower="-1.48352986" upper="1.48352986" effort="10" velocity="3" />
+		  <dynamics damping="0.0" friction="5.0"/>
 		</joint>
 		<link
@@ -277,4 +281,5 @@
 		    xyz="0 0 1" />
 		  <limit lower="0" upper="1.91986218" effort="10" velocity="3" />
+		  <dynamics damping="0.0" friction="5.0"/>
 		</joint>
 		<link
@@ -331,4 +336,5 @@
 		    xyz="0 0 1" />
 		  <limit lower="-1.48352986" upper="1.48352986" effort="10" velocity="3" />
+		  <dynamics damping="0.0" friction="5.0"/>
 		</joint>
 		<link
@@ -385,4 +391,5 @@
 		    xyz="0 0 1" />
 		  <limit lower="-0.610865238" upper="0.610865238" effort="10" velocity="3" />
+		  <dynamics damping="0.0" friction="5.0"/>
 		</joint>
 		<link
@@ -494,4 +501,5 @@
 		    xyz="0 0 1" />
 		  <limit lower="-0.610865238" upper="0.610865238" effort="10" velocity="3" />
+		  <dynamics damping="0.0" friction="5.0"/>
 		</joint>
 		<!--<link name="r_palm_link">

File: vizzy_description/urdf/base/base.urdf.xacro (robot description, xacro)
@@ -321,4 +321,5 @@
     <axis
       xyz="0 0 1" />
+        <dynamics damping="0.0" friction="100.0"/>
   </joint>
   <link
@@ -374,4 +375,5 @@
     <axis
       xyz="0 0 1" />
+    <dynamics damping="0.0" friction="100.0"/>
   </joint>
   <!-- gazebo extensions -->
