Commit message: fix base description files
Simplified and structured the base urdf
Fixes #59
Reorganized meshes and removed redundant files

File: vizzy_description/plugins/ros.gazebo.xacro (robot description, xacro)
@@ -9,26 +9,27 @@
     </gazebo>
   </xacro:macro>
-  <!-- base controller plugin -->
+  <!-- Base controller (differential drive) plugin -->
   <xacro:macro name="ros_differential_drive_gazebo">
     <gazebo>
-      <plugin name="differential_drive_controller" filename="libgazebo_ros_diff_drive.so">
-        <!-- hack -->
-        <leftJoint>r_wheel_joint</leftJoint>
-	<legacyMode>true</legacyMode>
-        <rightJoint>l_wheel_joint</rightJoint>
+      <plugin
+        name="differential_drive_controller"
+        filename="libgazebo_ros_diff_drive.so">
+        <leftJoint>l_wheel_joint</leftJoint>
+        <rightJoint>r_wheel_joint</rightJoint>
         <wheelSeparation>0.4580</wheelSeparation>
-        <wheelDiameter>0.2410</wheelDiameter>
+        <wheelDiameter>0.39628</wheelDiameter>
         <torque>20</torque>
+        <legacyMode>true</legacyMode>
         <updateRate>100</updateRate>
         <commandTopic>vizzy/cmd_vel</commandTopic>
         <odometryTopic>odom</odometryTopic>
         <odometryFrame>odom</odometryFrame>
-        <robotBaseFrame>base_link</robotBaseFrame>
-        <odometrySource>0</odometrySource>
+        <robotBaseFrame>base_footprint</robotBaseFrame>
+        <odometrySource>encoder</odometrySource>
         <wheelTorque>10</wheelTorque>
         <wheelAcceleration>0</wheelAcceleration>
+        <publishTf>1</publishTf>
+        <publishWheelTF>true</publishWheelTF>
         <publishWheelJointState>true</publishWheelJointState>
-        <publishTF>1</publishTF>
-        <publishWheelTF>true</publishWheelTF>
         <rosDebugLevel>na</rosDebugLevel>
       </plugin>
@@ -47,8 +48,8 @@
             <width>320</width>
             <height>240</height>
-	    <!--<width>640</width>
-            <height>480</height>-->
-            <!--<width>320</width>
-            <height>240</height>-->
+	          <!--
+            <width>640</width>
+            <height>480</height>
+            -->
             <format>R8G8B8</format>
           </image>
@@ -73,12 +74,14 @@
           <cameraInfoTopicName>camera_info</cameraInfoTopicName>
           <frameName>${prefix}_camera_link</frameName>
-          <!--<distortion>
-            <k1>-0.4738</k1>
-            <k2>0.190309</k2>
-            <k3>0.0</k3>
-            <p1>-0.000375676</p1>
-            <p2>-0.000663688</p2>
-            <center> 0.4809  0.4887</center>
-          </distortion>-->
+          <!--
+          <distortion>
+          <k1>-0.4738</k1>
+          <k2>0.190309</k2>
+          <k3>0.0</k3>
+          <p1>-0.000375676</p1>
+          <p2>-0.000663688</p2>
+          <center> 0.4809  0.4887</center>
+          </distortion>
+          -->
         </plugin>
       </sensor>

File: vizzy_description/urdf/base/base.gazebo.xacro (robot description, xacro)
@@ -1,52 +1,149 @@
 <?xml version="1.0"?>
 <robot xmlns:xacro="http://ros.org/wiki/xacro">
-  <xacro:macro name="base_gazebo">
+  <!-- Load full inertial and collision model or a simplified model -->
+  <xacro:arg name="use_full_gazebo_model" default="false"/>
+  <!-- Base link -->
+  <xacro:macro name="vizzy_base_link_inertial">
+    <xacro:if value="$(arg use_full_gazebo_model)">
+      <inertial>
+        <mass value="60" />
+        <origin xyz="0.18986 0 0.2" />
+        <inertia
+          ixx="3000.0" ixy="0.0" ixz="0.0"
+          iyy="3000.0" iyz="0.0"
+          izz="30.0" />
+      </inertial>
+    </xacro:if>
+    <xacro:unless value="$(arg use_full_gazebo_model)">
+      <inertial>
+        <mass value="60" />
+        <origin xyz="0.18986 0 0.2" />
+        <inertia
+          ixx="3000.0" ixy="0.0" ixz="0.0"
+          iyy="3000.0" iyz="0.0"
+          izz="30.0" />
+      </inertial>
+    </xacro:unless>
+  </xacro:macro>
+  <xacro:macro name="vizzy_base_link_collision" >
+    <xacro:if value="$(arg use_full_gazebo_model)">
+      <collision>
+        <origin
+          xyz="0.188 0.001 0.197"
+          rpy="0 0 0" />
+        <geometry>
+          <mesh filename="package://vizzy_description/meshes/base/segway.dae"/>
+        </geometry>
+      </collision>
+    </xacro:if>
+    <xacro:unless value="$(arg use_full_gazebo_model)">
+      <collision>
+        <origin
+          xyz="0.188 0.001 0.25"
+          rpy="0 0 0" />
+        <geometry>
+          <!-- TODO: refine geometry? -->
+          <box size=".08 .35 .45" />
+        </geometry>
+      </collision>
+    </xacro:unless>
+  </xacro:macro>
+  <xacro:macro name="gazebo_vizzy_base_link_surface">
     <gazebo reference="base_link">
-      <mu1>0.2</mu1>
-      <mu2>0.2</mu2>
+      <mu1 value="1.0" />
+      <mu2 value="1.0" />
+      <kp  value="1000000.0" />
+      <kd  value="1.0" />
     </gazebo>
-    <gazebo reference="base_footprint">
-      <mu1>0.2</mu1>
-      <mu2>0.2</mu2>
+  </xacro:macro>
+  <!-- Caster wheels -->
+  <xacro:macro name="vizzy_caster_wheel_base_link_inertial">
+    <inertial>
+      <origin
+        xyz="-0.0118 0.0084 0.083"
+        rpy="0 0 0" />
+      <mass
+        value="0.4" />
+      <inertia
+        ixx="0.00375" ixy="0.0" ixz="0.0"
+        iyy="0.00375" iyz="0.0"
+        izz="0.00375" />
+    </inertial>
+  </xacro:macro>
+  <xacro:macro name="vizzy_caster_wheel_base_link_collision">
+    <collision>
+      <origin
+        xyz="0 0 0.05"
+        rpy="0 0 0" />
+      <geometry>
+         <cylinder length="0.02" radius="0.01"/>
+      </geometry>
+    </collision>
+  </xacro:macro>
+  <xacro:macro name="vizzy_caster_wheel_link_inertial">
+    <inertial>
+      <origin
+        xyz="0 0 0"
+        rpy="0 0 0" />
+      <mass
+        value="0.5" />
+      <xacro:cylinder_inertia
+        m="0.5"
+        r="0.0491365"
+        h="0.02"/>
+    </inertial>
+  </xacro:macro>
+  <xacro:macro name="vizzy_caster_wheel_link_collision">
+    <collision>
+      <origin
+        xyz="0 0 0"
+        rpy="0 0 0"/>
+      <geometry>
+        <cylinder length="0.02" radius="0.0491365"/>
+      </geometry>
+    </collision>
+  </xacro:macro>
+  <xacro:macro name="gazebo_vizzy_caster_wheel_link_surface"
+    params="prefix">
+    <gazebo reference="${prefix}_wheel_link">
+      <mu1 value="1.0" />
+      <mu2 value="1.0" />
+      <kp  value="1000000.0" />
+      <kd  value="1.0" />
     </gazebo>
-    <gazebo reference="b_wheel_base_link">
-      <!-- <mu1 value="100.0" />
-      <mu2 value="100.0" />
+  </xacro:macro>
+  <!-- Active wheels -->
+  <xacro:macro name="vizzy_wheel_link_inertial"
+    params="rpy">
+    <inertial>
+      <origin
+        xyz="0 0 0"
+        rpy="${rpy}" />
+      <mass
+        value="5" />
+      <xacro:cylinder_inertia
+        m="5"
+        r="0.19814"
+        h="0.06"/>
+    </inertial>
+  </xacro:macro>
+  <xacro:macro name="vizzy_wheel_link_collision"
+    params="rpy">
+    <collision>
+      <origin
+        xyz="0 0 0"
+        rpy="${rpy}" />
+      <geometry>
+        <cylinder length="0.06" radius="0.19814"/>
+      </geometry>
+   </collision>
+  </xacro:macro>
+  <xacro:macro name="gazebo_vizzy_wheel_link_surface"
+    params="prefix">
+    <gazebo reference="${prefix}_wheel_link" >
+      <mu1 value="1.0" />
+      <mu2 value="1.0" />
       <kp  value="1000000.0" />
-      <kd  value="1.0" /> -->
-      <mu1>10000</mu1>
-      <mu2>10000</mu2>
-    </gazebo>
-    <gazebo reference="b_wheel_link">
-      <mu1>10000</mu1>
-      <mu2>10000</mu2>
-    </gazebo>
-    <gazebo reference="f_wheel_base_link">
-      <!-- <mu1 value="100.0" />
-      <mu2 value="100.0" />
-      <kp  value="1000000.0" />
-      <kd  value="1.0" /> -->
-      <mu1>10000</mu1>
-      <mu2>10000</mu2>
-    </gazebo>
-    <gazebo reference="f_wheel_link">
-      <mu1>10000</mu1>
-      <mu2>10000</mu2>
-    </gazebo>
-    <gazebo reference="l_wheel_base_link">
-      <mu1>10000</mu1>
-      <mu2>10000</mu2>
-    </gazebo>
-    <gazebo reference="l_wheel_link">
-      <mu1>10000</mu1>
-      <mu2>10000</mu2>
-    </gazebo>
-    <gazebo reference="r_wheel_base_link">
-      <mu1>10000</mu1>
-      <mu2>10000</mu2>
-    </gazebo>
-    <gazebo reference="r_wheel_link">
-      <mu1>10000</mu1>
-      <mu2>10000</mu2>
+      <kd  value="1.0" />
     </gazebo>
   </xacro:macro>

File: vizzy_description/urdf/base/base.urdf.xacro (robot description, xacro)
@@ -4,384 +4,208 @@
        xmlns:interface="http://playerstage.sourceforge.net/gazebo/xmlschema/#interface"
        xmlns:xacro="http://ros.org/wiki/xacro">
+  <!-- Load full inertial and collision model or a simplified model -->
+  <xacro:arg name="use_full_gazebo_model" default="false"/>
   <!-- Things that are needed only for Gazebo (not the physical robot).  These include
        sensor and controller plugin specifications -->
- <xacro:include filename="$(find vizzy_description)/urdf/base/base.gazebo.xacro" />
- <xacro:include filename="$(find vizzy_description)/urdf/base/base.transmission.xacro" />
- <xacro:macro name="base" params="name">
-  <!-- root link, on the ground just below the robot origin -->
-  <link name="base_footprint">
-  </link>
-  <joint name="base_footprint_joint" type="fixed">
-   <origin xyz="0.1934543 0.0 0.04" rpy="0.0 0.0 ${M_PI}" />
-   <parent link="base_footprint"/>
-   <child link="base_link" />
-  </joint>
-  <link
-    name="base_link">
-    <inertial>
-      <origin
-        xyz="0.19 0 0.2"
-        rpy="0 0 0" />
-      <mass
-        value="11.7973473742999" />
-      <inertia
-        ixx="0.438925207385402"
-        ixy="0.000141568676799447"
-        ixz="7.95805262167885E-07"
-        iyy="0.326554522375815"
-        iyz="0.00194386671838748"
-        izz="0.296176192213331" />
-    </inertial>
-    <visual>
-      <origin
-        xyz="0.188 0.001 0.197"
-        rpy="0 0 0" />
-      <geometry>
-        <mesh
-          filename="package://vizzy_description/meshes/Segway.dae" />
-      </geometry>
-      <material
-        name="">
-        <color
-          rgba="0.866666666666667 0.866666666666667 0.890196078431373 1" />
-      </material>
-    </visual>
-    <collision>
-      <origin
-        xyz="0.188 0.001 0.197"
-        rpy="0 0 0" />
-      <geometry>
-        <mesh
-          filename="package://vizzy_description/meshes/Segway.dae" />
-      </geometry>
-    </collision>
-  </link>
-  <link
-    name="f_wheel_base_link">
-    <inertial>
-      <origin
-        xyz="-0.0118 0.0084 0.083"
-        rpy="0 0 0" />
-      <mass
-        value="0.0522202580480446" />
-      <inertia
-        ixx="0.000109063640814005"
-        ixy="1.29634203029402E-06"
-        ixz="-2.56834920297101E-05"
-        iyy="0.000107815897797672"
-        iyz="1.74895161672912E-05"
-        izz="3.21409232257602E-05" />
-    </inertial>
-    <visual>
-      <origin
-        xyz="-0.0118 0.0084 0.083"
-        rpy="0 0 0" />
-      <geometry>
-        <mesh
-          filename="package://vizzy_description/meshes/Front.dae" />
-      </geometry>
-      <material
-        name="">
-        <color
-          rgba="0.796078431372549 0.823529411764706 0.937254901960784 1" />
-      </material>
-    </visual>
-    <collision>
-      <origin
-        xyz="-0.0118 0.0084 0.083"
-        rpy="0 0 0" />
-      <geometry>
-        <mesh
-          filename="package://vizzy_description/meshes/Front.dae" />
-      </geometry>
-    </collision>
-  </link>
-  <joint
-    name="f_wheel_base_joint"
-    type="continuous">
-    <origin
-      xyz="0.43986 0.001 0.14806"
-      rpy="${M_PI} 0.0 0.0" />
-    <parent
-      link="base_link" />
-    <child
-      link="f_wheel_base_link" />
-    <axis
-      xyz="0 0 1" />
-  </joint>
-  <link
-    name="f_wheel_link">
-    <inertial>
-      <origin
-        xyz="0 0 0"
-        rpy="0 0 0" />
-      <mass
-        value="0.146715525294139" />
-      <inertia
-        ixx="0.000105012932391273"
-        ixy="-1.06408513998821E-20"
-        ixz="-6.7762635780344E-21"
-        iyy="0.000105012932391273"
-        iyz="4.99749438880037E-20"
-        izz="0.00019960379578771" />
-    </inertial>
-    <visual>
-      <origin
-        xyz="0 0 0"
-        rpy="0 0 0" />
-      <geometry>
-        <mesh
-          filename="package://vizzy_description/meshes/F_W.dae" />
-      </geometry>
-      <material
-        name="">
-        <color
-          rgba="0.796078431372549 0.823529411764706 0.937254901960784 1" />
-      </material>
-    </visual>
-    <collision>
-      <origin
-        xyz="0 0 0"
-        rpy="0 0 0" />
-      <geometry>
-        <!-- <mesh
-          filename="package://vizzy_description/meshes/F_W.dae" />  -->
-        <cylinder length="0.02" radius="0.05"/>
-      </geometry>
-    </collision>
-  </link>
-  <joint
-    name="f_wheel_joint"
-    type="continuous">
-    <origin
-      xyz="-0.030027 0.020142 0.138923486"
-      rpy="-1.5708 0.83904 2.5507" />
-    <parent
-      link="f_wheel_base_link" />
-    <child
-      link="f_wheel_link" />
-    <axis
-      xyz="0 0 1" />
-  </joint>
-  <link
-    name="b_wheel_base_link">
-    <inertial>
-      <origin
-        xyz="-0.0118 0.0084 0.083"
-        rpy="0 0 0" />
-      <mass
-        value="0.0522202580480446" />
-      <inertia
-        ixx="0.000109063640814005"
-        ixy="1.29634203029405E-06"
-        ixz="-2.568349202971E-05"
-        iyy="0.000107815897797672"
-        iyz="1.74895161672911E-05"
-        izz="3.21409232257601E-05" />
-    </inertial>
-    <visual>
-      <origin
-        xyz="-0.0118 0.0084 0.083"
-        rpy="0 0 0" />
-      <geometry>
-        <mesh
-          filename="package://vizzy_description/meshes/Back.dae" />
-      </geometry>
-      <material
-        name="">
-        <color
-          rgba="0.796078431372549 0.823529411764706 0.937254901960784 1" />
-      </material>
-    </visual>
-    <collision>
-      <origin
-        xyz="-0.0118 0.0084 0.083"
-        rpy="0 0 0" />
-      <geometry>
-        <mesh
-          filename="package://vizzy_description/meshes/Back.dae" />
-      </geometry>
-    </collision>
-  </link>
-  <joint
-    name="b_wheel_base_joint"
-    type="continuous">
-    <origin
-      xyz="-0.060139 0.001 0.14806"
-      rpy="${M_PI} 0.0 0.0" />
-    <parent
-      link="base_link" />
-    <child
-      link="b_wheel_base_link" />
-    <axis
-      xyz="0 0 1" />
-  </joint>
-  <link
-    name="b_wheel_link">
-    <inertial>
-      <origin
-        xyz="0 0 0"
-        rpy="0 0 0" />
-      <mass
-        value="0.146715525294139" />
-      <inertia
-        ixx="0.000105012932391273"
-        ixy="1.07996700774923E-20"
-        ixz="-1.6940658945086E-21"
-        iyy="0.000105012932391273"
-        iyz="-1.18584612615602E-20"
-        izz="0.00019960379578771" />
-    </inertial>
-    <visual>
-      <origin
-        xyz="0 0 0"
-        rpy="0 0 0" />
-      <geometry>
-        <mesh
-          filename="package://vizzy_description/meshes/B_W.dae" />
-      </geometry>
-      <material
-        name="">
-        <color
-          rgba="0.796078431372549 0.823529411764706 0.937254901960784 1" />
-      </material>
-    </visual>
-    <collision>
-      <origin
-        xyz="0 0 0"
-        rpy="0 0 0" />
-      <geometry>
-        <!-- <mesh
-          filename="package://vizzy_description/meshes/B_W.dae" /> -->
-        <cylinder length="0.02" radius="0.05"/>
-      </geometry>
-    </collision>
-  </link>
-  <joint
-    name="b_wheel_joint"
-    type="continuous">
-    <origin
-      xyz="-0.0300271872634975 0.0201420335543447 0.138923486"
-      rpy="-1.5707963267949 0.83904346430428 2.5507386456365" />
-    <parent
-      link="b_wheel_base_link" />
-    <child
-      link="b_wheel_link" />
-    <axis
-      xyz="0 0 1" />
-  </joint>
-  <link
-    name="r_wheel_link">
-    <inertial>
-      <origin
-        xyz="0 0 0"
-        rpy="0 0 0" />
-      <mass
-        value="150.22861917507719" />
-      <inertia
-        ixx="0.0106873251772162"
-        ixy="4.79944507056635E-17"
-        ixz="3.53158602954754E-16"
-        iyy="0.0106873821917694"
-        iyz="1.38940097207607E-06"
-        izz="0.0205152843016012" />
-    </inertial>
-    <visual>
-      <origin
-        xyz="0 0 0"
-        rpy="0 0 0" />
-      <geometry>
-        <mesh
-          filename="package://vizzy_description/meshes/Left.dae" />
-      </geometry>
-      <material
-        name="">
-        <color
-          rgba="0.494117647058824 0.494117647058824 0.494117647058824 1" />
-      </material>
-    </visual>
-    <collision>
-      <origin
-        xyz="0 0 0"
-        rpy="0 0 0" />
-      <geometry>
-        <!-- <mesh
-          filename="package://vizzy_description/meshes/Left.dae" /> -->
-        <cylinder length="0.06" radius="0.198"/>
-      </geometry>
-    </collision>
-  </link>
-  <joint
-    name="r_wheel_joint"
-    type="continuous">
-    <origin
-      xyz="0.18986 0.246 0.15814"
-      rpy="1.5708 1.5708 0" />
-    <parent
-      link="base_link" />
-    <child
-      link="r_wheel_link" />
-    <axis
-      xyz="0 0 1" />
-        <dynamics damping="0.0" friction="100.0"/>
-  </joint>
-  <link
-    name="l_wheel_link">
-    <inertial>
-      <origin
-        xyz="0 0 0"
-        rpy="3.15 0 0" />
-      <mass
-        value="150.22861917507742" />
-      <inertia
-        ixx="0.0106873471854323"
-        ixy="7.49808591987845E-18"
-        ixz="-1.93571153328442E-16"
-        iyy="0.0106874041999854"
-        iyz="1.38940098137139E-06"
-        izz="0.0205152843016018" />
-    </inertial>
-    <visual>
-      <origin
-        xyz="0 0 0"
-        rpy="3.15 0 0" />
-      <geometry>
-        <mesh
-          filename="package://vizzy_description/meshes/Right.dae" />
-      </geometry>
-      <material
-        name="">
-        <color
-          rgba="0.494117647058824 0.494117647058824 0.494117647058824 1" />
-      </material>
-    </visual>
-    <collision>
-      <origin
-        xyz="0 0 0"
-        rpy="3.15 0 0" />
-      <geometry>
-        <!-- <mesh
-          filename="package://vizzy_description/meshes/Right.dae" />  -->
-        <cylinder length="0.06" radius="0.198"/>
-      </geometry>
-    </collision>
-  </link>
-  <joint
-    name="l_wheel_joint"
-    type="continuous">
-    <origin
-      xyz="0.18986 -0.244 0.15814"
-      rpy="1.5708 1.5708 0" />
-    <parent
-      link="base_link" />
-    <child
-      link="l_wheel_link" />
-    <axis
-      xyz="0 0 1" />
-    <dynamics damping="0.0" friction="100.0"/>
-  </joint>
-  <!-- gazebo extensions -->
-  <xacro:base_gazebo/>
-  <xacro:base_transmissions/>
+  <xacro:include filename="$(find vizzy_description)/urdf/base/base.gazebo.xacro">
+    <xacro:arg name="use_full_gazebo_model" value="$(arg use_full_gazebo_model)"/>
+  </xacro:include>
+  <xacro:include filename="$(find vizzy_description)/urdf/base/base.transmission.xacro"/>
+  <!-- Robot base macro -->
+  <xacro:macro name="base" params="name">
+    <!-- Root link, on the ground just below the robot origin -->
+    <link name="base_footprint">
+    </link>
+    <joint name="base_footprint_joint" type="fixed">
+      <origin
+        xyz="0.1934543 0.0 0.04"
+        rpy="0.0 0.0 ${M_PI}"/>
+      <parent link="base_footprint"/>
+      <child link="base_link"/>
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
File: vizzy_description/urdf/common.urdf.xacro (robot description, xacro)
@@ -13,20 +13,27 @@
   <xacro:property name="BASE_PLATE_Z_OFFSET" value="4.25" /> <!-- inches -->
   <xacro:property name="SENSOR_BEAM_LENGTH" value="10.75" /> <!-- inches -->
-	<!-- Motor transmissions -->
+  <!-- Motor transmissions -->
   <xacro:property name="A2232U024SR_motor_transmission_reduction" value="100" /> <!--small-->
   <xacro:property name="A3242G024CR_motor_transmission_reduction" value="100" /> <!--medium-->
   <xacro:property name="A3257G024CR_motor_transmission_reduction" value="371" /> <!-- large -->
   <xacro:property name="A3863H024C_motor_transmission_reduction" value="700" /> <!-- huge -->
-	<!-- Motor max efforts (N.m)-->
+  <!-- Motor max efforts (N.m) -->
   <xacro:property name="A2232U024SR_motor_max_effort" value="2.8" />
   <xacro:property name="A3242G024CR_motor_max_effort" value="11.3" />
   <xacro:property name="A3257G024CR_motor_max_effort" value="105.6" />
   <xacro:property name="A3863H024C_motor_max_effort" value="525" />
-	<!-- Motor max velocities degrees per second-->
+  <!-- Motor max velocities degrees per second -->
   <xacro:property name="A2232U024SR_motor_max_velocitiy" value="426" />
   <xacro:property name="A3242G024CR_motor_max_velocitiy" value="300" />
   <xacro:property name="A3257G024CR_motor_max_velocitiy" value="300" />
   <xacro:property name="A3863H024C_motor_max_velocitiy" value="34" />
-  <!-- colors -->
+  <!-- Inertia calculation macros -->
+  <xacro:macro name="cylinder_inertia" params="m r h">
+    <inertia
+      ixx="${m*(3*r*r+h*h)/12}" ixy = "0" ixz = "0"
+      iyy="${m*(3*r*r+h*h)/12}" iyz = "0"
+      izz="${m*r*r/2}"/>
+  </xacro:macro>
+  <!-- Colors -->
   <material name="light_grey">
     <color rgba="0.7 0.7 0.7 1" />
@@ -42,5 +49,21 @@
   </material>
   <material name="orange">
-    <color rgba="${255/255} ${108/255} ${10/255} 1.0"/>
+    <color rgba="${255/255} ${108/255} ${10/255} 1"/>
+  </material>
+  <!-- #E5EAED: Light gray 1-->
+  <material name="light_gray_1">
+    <color rgba="${229/255} ${234/255} ${237/255} 1"/>
+  </material>
+  <!-- #DDDDE3: Light gray 2 -->
+  <material name="ligh_gray_2">
+    <color rgba="${221/255} ${221/255} ${227/255} 1"/>
+  </material>
+  <!-- #CBD2EF: Light gray 3 -->
+  <material name="light_gray_3">
+    <color rgba="${203/255} ${210/255} ${239/255} 1"/>
+  </material>
+  <!-- #7E7E7E: Gray 1 -->
+  <material name="gray_1">
+    <color rgba="${126/255} ${126/255} ${126/255} 1"/>
   </material>
 </root>
