Commit message: fix incorrect diff drive args

File: vizzy_description/plugins/ros.gazebo.xacro (robot description, xacro)
@@ -15,6 +15,6 @@
         name="differential_drive_controller"
         filename="libgazebo_ros_diff_drive.so">
-        <leftJoint>l_wheel_joint</leftJoint>
-        <rightJoint>r_wheel_joint</rightJoint>
+        <leftJoint>r_wheel_joint</leftJoint> <!-- SWITCHED ON PURPOSE - TODO: FIND WHY right and left wheels have to be switch for the plugin to work properly-->
+        <rightJoint>l_wheel_joint</rightJoint>
         <wheelSeparation>0.4580</wheelSeparation>
         <wheelDiameter>0.39628</wheelDiameter>

File: vizzy_description/robots/vizzy.urdf.xacro (robot description, xacro)
@@ -48,4 +48,6 @@
       ros_topic="scan"
       update_rate="40"
+      visualize="false"
+      resolution="0.03"
       min_angle="${-(5 * M_PI)/12}"
       max_angle="${(5 * M_PI)/12}"
@@ -59,4 +61,6 @@
       ros_topic="scan_rear"
       update_rate="10"
+      visualize="false"
+      resolution="0.03"
       min_angle="${-(5 * M_PI)/12}"
       max_angle="${(5 * M_PI)/12}"

File: vizzy_description/urdf/sensors/hokuyo_04lx_laser.gazebo.xacro (robot description, xacro)
@@ -1,5 +1,5 @@
 <?xml version="1.0"?>
 <root xmlns:xacro="http://ros.org/wiki/xacro">
-  <xacro:macro name="hokuyo_04lx_laser_gazebo" params="name ros_topic update_rate min_angle max_angle max_range">
+  <xacro:macro name="hokuyo_04lx_laser_gazebo" params="name ros_topic update_rate min_angle max_angle max_range resolution visualize">
     <gazebo reference="${name}_link">
       <sensor type="ray" name="${name}">
@@ -7,5 +7,5 @@
         <update_rate>${update_rate}</update_rate>
         <pose>0 0 0 0 0 0</pose>
-        <visualize>true</visualize>
+        <visualize>${visualize}</visualize>
         <ray>
           <scan>
@@ -20,5 +20,5 @@
             <min>0.02</min>
             <max>${max_range}</max>
-            <resolution>0.03</resolution>
+            <resolution>${resolution}</resolution>
           </range>
           <noise>

File: vizzy_description/urdf/sensors/hokuyo_04lx_laser.urdf.xacro (robot description, xacro)
@@ -1,42 +1,50 @@
 <?xml version="1.0"?>
 <root xmlns:sensor="http://playerstage.sourceforge.net/gazebo/xmlschema/#sensor"
-      xmlns:controller="http://playerstage.sourceforge.net/gazebo/xmlschema/#controller"
-      xmlns:interface="http://playerstage.sourceforge.net/gazebo/xmlschema/#interface"
-      xmlns:xacro="http://ros.org/wiki/xacro">
+    xmlns:controller="http://playerstage.sourceforge.net/gazebo/xmlschema/#controller"
+    xmlns:interface="http://playerstage.sourceforge.net/gazebo/xmlschema/#interface"
+    xmlns:xacro="http://ros.org/wiki/xacro">
   <xacro:include filename="$(find vizzy_description)/urdf/sensors/hokuyo_04lx_laser.gazebo.xacro" />
-  <xacro:macro name="hokuyo_04lx_laser" params="name parent *origin mesh_file scale ros_topic update_rate min_angle max_angle max_range">
-    <joint name="${name}_joint" type="fixed">
-      <xacro:insert_block name="origin" />
-      <parent link="${parent}_link"/>
-      <child link="${name}_link"/>
-    </joint>
-    <link name="${name}_link">
-      <inertial>
-        <mass value="0.001" />
-        <xacro:insert_block name="origin" />
-        <inertia ixx="0.0001" ixy="0" ixz="0" iyy="0.000001" iyz="0" izz="0.0001" />
-      </inertial>
-      <visual>
-        <origin xyz="0 0 0.058" rpy="0 0 0" />
-        <geometry>
-          <mesh filename="${mesh_file}" scale="${scale}" />
-        </geometry>
-      </visual>
-    </link>
-    <!-- go from the base of the laser to the actual sensor location -->
-    <joint name="${name}_laser_joint" type="fixed">
-      <origin xyz="0 0 0.058" />
-      <parent link="${name}_link"/>
-      <child link="${name}_laser_link"/>
-    </joint>
-    <link name="${name}_laser_link" type="laser">
-      <inertial>
-        <mass value="0.001" />
-        <origin xyz="0 0 0" rpy="0 0 0" />
-        <inertia ixx="0.0001" ixy="0" ixz="0" iyy="0.000001" iyz="0" izz="0.0001" />
-      </inertial>
-    </link>
-    <!-- gazebo extensions -->
-    <xacro:hokuyo_04lx_laser_gazebo name="${name}_laser" ros_topic="${ros_topic}" update_rate="${update_rate}" min_angle="${min_angle}" max_angle="${max_angle}" max_range="${max_range}"/>
+  <xacro:macro name="hokuyo_04lx_laser" params="name parent *origin mesh_file scale ros_topic update_rate min_angle max_angle max_range resolution visualize">
+  <joint name="${name}_joint" type="fixed">
+    <xacro:insert_block name="origin" />
+    <parent link="${parent}_link"/>
+    <child link="${name}_link"/>
+  </joint>
+  <link name="${name}_link">
+    <inertial>
+    <mass value="0.001" />
+    <xacro:insert_block name="origin" />
+    <inertia ixx="0.0001" ixy="0" ixz="0" iyy="0.000001" iyz="0" izz="0.0001" />
+    </inertial>
+    <visual>
+    <origin xyz="0 0 0.058" rpy="0 0 0" />
+    <geometry>
+      <mesh filename="${mesh_file}" scale="${scale}" />
+    </geometry>
+    </visual>
+  </link>
+  <!-- go from the base of the laser to the actual sensor location -->
+  <joint name="${name}_laser_joint" type="fixed">
+    <origin xyz="0 0 0.058" />
+    <parent link="${name}_link"/>
+    <child link="${name}_laser_link"/>
+  </joint>
+  <link name="${name}_laser_link" type="laser">
+    <inertial>
+    <mass value="0.001" />
+    <origin xyz="0 0 0" rpy="0 0 0" />
+    <inertia ixx="0.0001" ixy="0" ixz="0" iyy="0.000001" iyz="0" izz="0.0001" />
+    </inertial>
+  </link>
+  <!-- gazebo extensions -->
+  <xacro:hokuyo_04lx_laser_gazebo
+    name="${name}_laser"
+    ros_topic="${ros_topic}"
+    update_rate="${update_rate}"
+    min_angle="${min_angle}"
+    max_angle="${max_angle}"
+    max_range="${max_range}"
+    resolution="${resolution}"
+    visualize="${visualize}"/>
   </xacro:macro>
 </root>

Commit message: add mimic plugin to right hand
Added a gazebo plugin to model underactuated finger behaviour

File: vizzy_description/plugins/ros.gazebo.xacro (robot description, xacro)
@@ -33,4 +33,28 @@
         <publishWheelJointState>true</publishWheelJointState>
         <rosDebugLevel>na</rosDebugLevel>
+      </plugin>
+    </gazebo>
+  </xacro:macro>
+  <!-- Mimic plugin to model underactuated joints -->
+  <xacro:macro name="gazebo_mimic_plugin">
+    <gazebo>
+      <plugin name="hand_mimic_plugin" filename="libgazebo_mimic_plugin.so">
+        <!-- Fingers -->
+        <actuatedJoint name="r_thumb_phal_1_joint">
+          <mimicJoint name="r_thumb_phal_2_joint" multiplier="0.5" />
+          <mimicJoint name="r_thumb_phal_3_joint" multiplier="0.5" />
+        </actuatedJoint>
+        <actuatedJoint name="r_ind_phal_1_joint">
+          <mimicJoint name="r_ind_phal_2_joint" multiplier="0.5" />
+          <mimicJoint name="r_ind_phal_3_joint" multiplier="0.5" />
+        </actuatedJoint>
+        <!-- Vizzy's med and min fingers are coupled and act as one -->
+        <actuatedJoint name="r_med_phal_1_joint">
+          <mimicJoint name="r_med_phal_2_joint" multiplier="0.5" />
+          <mimicJoint name="r_med_phal_3_joint" multiplier="0.5" />
+          <mimicJoint name="r_min_phal_1_joint" multiplier="0.5" />
+          <mimicJoint name="r_min_phal_3_joint" multiplier="0.5" />
+          <mimicJoint name="r_min_phal_2_joint" multiplier="0.5" />
+        </actuatedJoint>
       </plugin>
     </gazebo>

File: vizzy_description/robots/vizzy.urdf.xacro (robot description, xacro)
@@ -104,3 +104,6 @@
     <xacro:ros_control_gazebo/>
   </xacro:unless>
+  <xacro:if value="$(arg use_full_hand_model)">
+    <xacro:gazebo_mimic_plugin/>
+  </xacro:if>
 </robot>

File: vizzy_description/urdf/hand/right_hand.gazebo.xacro (robot description, xacro)
@@ -1,7 +1,27 @@
 <?xml version="1.0"?>
 <robot xmlns:xacro="http://ros.org/wiki/xacro">
-  <!-- TODO: Model underactuated fingers
-  	e.g. by instancing mimic joint plugin -->
   <xacro:macro name="right_hand_gazebo">
+    <!-- Mimic plugin to model underactuated joints -->
+    <gazebo>
+      <plugin name="hand_mimic_plugin" filename="libMimicPlugin.so">
+        <!-- Fingers -->
+        <actuatedJoint name="r_thumb_phal_1_joint">
+          <mimicJoint name="r_thumb_phal_2_joint" multiplier="0.5" />
+          <mimicJoint name="r_thumb_phal_3_joint" multiplier="0.5" />
+        </actuatedJoint>
+        <actuatedJoint name="r_ind_phal_1_joint">
+          <mimicJoint name="r_ind_phal_2_joint" multiplier="0.5" />
+          <mimicJoint name="r_ind_phal_3_joint" multiplier="0.5" />
+        </actuatedJoint>
+        <!-- Vizzy's med and min fingers are coupled and act as one -->
+        <actuatedJoint name="r_med_phal_1_joint">
+          <mimicJoint name="r_med_phal_2_joint" multiplier="0.5" />
+          <mimicJoint name="r_med_phal_3_joint" multiplier="0.5" />
+          <mimicJoint name="r_min_phal_1_joint" multiplier="0.5" />
+          <mimicJoint name="r_min_phal_3_joint" multiplier="0.5" />
+          <mimicJoint name="r_min_phal_2_joint" multiplier="0.5" />
+        </actuatedJoint>
+      </plugin>
+    </gazebo>
   </xacro:macro>
 </robot>
